File: hardware/CONEPROJ.kicad_sch (KiCad schematic)
At the start: 223 parts, among them U1 OSD3358-512M-BAS

Commit message: Schematic Progress
Almost done. Need to add the PWM signals and do the packet radio and GPS
Parts:
- removed BAL?: BQ29209, symbol bq29209:BQ29209
- removed C?: 1uF, symbol Device:C_Small
- removed C?: 10uF, symbol Device:C_Small
- removed C? (x2): 0.22uF, symbol Device:C_Small
- removed C?: 0.1uF, symbol Device:C_Small
- removed J?: Barrel_Jack_Switch, symbol Connector:Barrel_Jack_Switch
- removed L? (x2): 120, symbol Device:L_Small
- removed LIPO: JST_XH, symbol bq29209:JST_XH
- removed PROT?: S-8261, symbol bq29209:S-8261
- removed R? (x2): 0 DNP, symbol Device:R_Small
- removed R? (x3): 0, symbol Device:R_Small
- removed R?: 100k, symbol Device:R_Small
- removed U?: TPS2105DBVR, SOT95P280X145-5N, symbol TPS2105DBVR:TPS2105DBVR
- removed U?: TXS0108ERGYR, symbol bq29209:TXS0108ERGYR
- added C2: 10uF, Very_Footprints:C_0805_2012Metric, symbol elias-rescue:C_Small-Very_Capacitor
- added C3, C?: 0.1uF, Very_Footprints:C_0402_1005Metric, symbol elias-rescue:C_Small-Very_Capacitor
- added C4: 0.1uF, symbol Device:C_Small
- added J1: LIPO, Connector_JST:JST_PH_S3B-PH-SM4-TB_1x03-1MP_P2.00mm_Horizontal, symbol Connector_Generic:Conn_01x03
- added J2: PWR-CAN, Connector_JST:JST_PH_S4B-PH-SM4-TB_1x04-1MP_P2.00mm_Horizontal, symbol Connector_Generic:Conn_02x02_Top_Bottom
- added J? (x2): U.FL-R-SMT-1(10), U.FL-R-SMT-1_10_:HRS_U.FL-R-SMT-1(10), symbol U.FL-R-SMT-1_10_:U.FL-R-SMT-1(10)
- added Q2, Q3, Q4: BSS138, SOT95P240X111-3N:SOT95P240X111-3N, symbol elias-rescue:BSS138-Very_Transistor
- added R3, R5, R7: 100k, Very_Footprints:R_0402_1005Metric, symbol elias-rescue:US_R0402-Very_Resistor
- added U13: TXS0108ERGYR, IC_TXS0108ERGYR:IC_TXS0108ERGYR, symbol TXS0108ERGYR:TXS0108ERGYR
- added U16: NEO-M8N-0, XCVR_NEO-M8N-0:XCVR_NEO-M8N-0, symbol NEO-M8N-0:NEO-M8N-0
- added U18: RFM69HCW, XCVR_RFM69HW:XCVR_RFM69HW, symbol RFM69HW:COM-13909
- added U2: ATECC608A-MAHDA-T, SON50P200X300X60-9N:SON50P200X300X60-9N, symbol ATECC608A-MAHDA-T:ATECC608A-MAHDA-T
- added U4: S-8261AAJMD-G2JT2G, SOT95P275X135-6:SOT95P275X135-6, symbol S-8261AAJMD-G2JT2G:S-8261AAJMD-G2JT2G
- added U5: BQ29209DRBR, BQ29209DRBR:IC_DRV8601DRBT, symbol BQ29209DRBR:BQ29209DRBR
- J3, J4: renamed from J?; footprint HRS_U.FL-R-SMT-1(10) -> U.FL-R-SMT-1_10_:HRS_U.FL-R-SMT-1(10)
- OSC1: renamed from OSC?; footprint (none) -> OSCDFN250X200X89-4N:OSCDFN250X200X89-4N
- Q1: renamed from Q?; footprint (none) -> Package_SO:SO-8_3.9x4.9mm_P1.27mm; PN (none) -> SI4778DY-T1-GE3
- R1: renamed from R?; value 0.1, 0805 -> 0.1; footprint (none) -> Resistor_SMD:R_0805_2012Metric_Pad1.20x1.40mm_HandSolder; symbol Device:R_US -> Device:R_Small
- R10, R11, R12, R13, R14, R15, R38, R39, R40, R53, R58, R59, R6, R60, R61, R62, R63, R64, R65, R66, R67, R68: renamed from R?; symbol Device:R_US -> Device:R_Small
- R57: renamed from R?; value 33 -> 0
- U10: renamed from U?; footprint (none) -> IC_TXS0108ERGYR:IC_TXS0108ERGYR; symbol bq29209:TXS0108ERGYR -> TXS0108ERGYR:TXS0108ERGYR; MANUFACTURER (none) -> Texas Instruments; MAXIMUM_PACKAGE_HEIGHT (none) -> 1 mm; PARTREV (none) -> H; STANDARD (none) -> Manufacturer Recommendations
- U11: renamed from U?; footprint XCVR_WL1835MODGBMOCT -> WL1835MODGBMOCT:XCVR_WL1835MODGBMOCT
- U12: renamed from U?; footprint (none) -> SOT95P280X145-5N:SOT95P280X145-5N; symbol bq29209:SN74LV1T126DBVR -> SN74LV1T126DBVR:SN74LV1T126DBVR
- U14, U8: renamed from U?; footprint PSON50P145X100X60-6N -> PSON50P145X100X60-6N:PSON50P145X100X60-6N
- U19: renamed from U?; footprint (none) -> SOIC127P599X175-8N:SOIC127P599X175-8N
- U3: renamed from U?; footprint (none) -> Package_TO_SOT_SMD:SOT-23-5_HandSoldering
- U6: renamed from U?; footprint (none) -> AP1509-50SG-13:SO08; symbol bq29209:AP1509 -> AP1509-50SG-13:AP1509-50SG-13
- U7: renamed from U?; footprint (none) -> SOT65P210X110-5N:SOT65P210X110-5N; symbol SN74LVC1G07:SN74LVC1G07 -> SN74LVC1G07DCKR:SN74LVC1G07DCKR
- U9: renamed from U?; footprint (none) -> MP2615GQ-Z:MP2615GQ-Z
- X1: renamed from X?; footprint (none) -> ALPS_SCHA5B0200:ALPS_SCHA5B0200; symbol bq29209:SCHA5B0200 -> SCHA5B0200:SCHA5B0200; DESCRIPTION (none) -> Conn Micro SD Card RCP 8 POS Solder RA SMD Reel; MP (none) -> SCHA5B0200
- gave numbers to parts that had none: 146
- renumbered CAN to CAN1, GPS to GPS1, I2C to I2C1, MOD to MOD1, PAU to PAU1, POW to POW1, PWR to PWR1, RST to RST1, SD to SD1
Connections:
- net USB1_VBUS is gone; now on net USB0_VBUS: C43.1, R57.2, U14.6 (VBUS)
- net USB_DC is gone; now on net USB0_VBUS: U1.Y8 (VIN_USB_1), U1.Y9 (VIN_USB_2)
- net +3V3: now also C23.2, C36.2, U10.19 (VCCB), C4.1, U13.19 (VCCB), U2.8 (VCC); no longer C1.1, R2.2, U3.4 (VCC), X1.6 (VSS)
- net 5.0V: now also U6.2 (VOUT); no longer U6.3 (FB)
- net BATT_MID: now also R14.1, R15.1, J1.2 (Pin_2); no longer R14.2, R15.2
- net BT_EN: now also U13.18 (B2)
- net BT_EN_1V8: now also U13.3 (A2)
- net CANH: now also J2.3 (Pin_3)
- net CANL: now also J2.4 (Pin_4)
- net CHG_EN: now also R11.1, R12.2; no longer R11.2, R12.1
- net DO: now also U4.1 (DO)
- net GND: now also C18.1, C43.2, C5.1, C6.2, C7.2, C9.2, Q1.1 (S), R12.1, U14.4 (GND), X1.6 (VSS), X1.CMN (COMMON), C4.2, J1.3 (Pin_3), J2.2 (Pin_2), J?.1, J?.3, U2.4 (GND), U4.2 (VM), U4.6 (VSS), U5.5 (GND), U5.6 (~{CB_EN}); no longer C18.2, R12.2, U10.11 (GND), U10.TP, X1. (GND)
- net GNDPWR: now also X1.S1 (SHIELD), X1.S2 (SHIELD), X1.S3 (SHIELD), X1.S4 (SHIELD), X1.S5 (SHIELD), X1.S6 (SHIELD); no longer X1. (GND)
- net I2C0_SCL: now also U2.6 (SCL)
- net I2C0_SDA: now also U2.5 (SDA)
- net MMC2_CLK: now also U13.13 (B7)
- net MMC2_CMD: now also U13.12 (B8)
- net MMC2_DAT0: now also U13.14 (B6)
- net MMC2_DAT1: now also U13.15 (B5)
- net MMC2_DAT2: now also U13.16 (B4)
- net MMC2_DAT3: now also U13.17 (B3)
- net RESET: now also C18.2; no longer C18.1
- net USB1_ID: now also U14.3 (ID)
- net VCC: now also J2.1 (Pin_1)
- net VDD_1V8: now also C34.1, C41.1, U10.2 (VCCA), U13.2 (VCCA)
- net V_BATT: now also R13.1, J1.1 (Pin_1); no longer R13.2
- net WL_EN: now also U13.20 (B1)
- net WL_EN_1V8: now also U13.1 (A1)
- net WL_SDIO_CLK: now also U13.8 (A7)
- net WL_SDIO_CMD: now also U13.9 (A8)
- net WL_SDIO_D0: now also U13.7 (A6)
- net WL_SDIO_D1: now also U13.6 (A5)
- net WL_SDIO_D2: now also U13.5 (A4)
- net WL_SDIO_D3: now also U13.4 (A3)
- net at C8.1: now also R13.2, U5.1 (VC2); no longer R13.1
- net at R54.1, R55.1, U10.10 (OE)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: now also U13.10 (OE)
- net at D4.1 (K), L1.1: now also U6.3 (FB); no longer U6.2 (OUT)
- net at C8.2, C9.1: now also R14.2, U5.2 (VC1); no longer R14.1
- net at C7.1: now also U5.4 (CD)
- net at U1.F18 (MMC0_DAT2), X1.1 (DAT2): now also R90.1; no longer R87.1
- net at U1.F17 (MMC0_DAT3), X1.2 (DAT3/CD): now also R91.1; no longer R86.1
- net at U1.G18 (MMC0_CMD), X1.3 (CMD): now also R87.1; no longer R90.1
- net at U1.G17 (MMC0_CLK), X1.5 (CLK): now also R86.1; no longer R91.1
- net at U1.G16 (MMC0_DAT0), X1.7 (DAT0): now also R88.1; no longer R89.1
- net at U1.G15 (MMC0_DAT1), X1.8 (DAT1): now also R89.1; no longer R88.1
- net at U1.C15 (SPI0_CS1): now also X1.DT (DETECH); no longer X1.CD (CD#)
- net at C5.2, R6.2: now also U4.5 (VDD)
- net at C6.1, R10.2: now also U5.7 (VDD)
- removed net BATT_MINUS: C5.1, C6.2, C7.2, C9.2, Q1.1 (S), R15.1
- net MDIR_1A: no longer names the net of U1.T13 (GPMC_CSN3)
- net MDIR_1B: no longer names the net of U1.U17 (GPMC_WPN)
- new net: J?.1, J?.3
- new net: C1.1, R2.2, U3.4 (VCC)
- new net: R15.2, U5.3 (VC1_CB)
- new net: U16.10 (GND), U16.12 (GND), U16.13 (GND), U16.24 (GND)
- new net: R11.2, U5.8 (OUT)
- new net: J?.2, U18.9 (ANT)
- new net: U18.1 (GND), U18.10 (GND), U18.8 (GND)
- new net +10V: C2.1, C3.1
- new net B_OUT: Q4.3 (D)
- new net B_PWM: Q4.1 (G), R7.1
- new net G_OUT: Q2.3 (D)
- new net G_PWM: Q2.1 (G), R3.1
- new net R_OUT: Q3.3 (D)
- new net R_PWM: Q3.1 (G), R5.1
- new net VSS: C2.2, C3.2, Q2.2 (S), Q3.2 (S), Q4.2 (S), R3.2, R5.2, R7.2
- no-connect marks 184 -> 187
Other:
- note added: "0.1 Ohm resistor for 1A charge"
- note added: "CELL pin left open: 2S SEL pin left open, 4.2V per cell"
- note added: "I_chg = 1kV / R6 * R4 = 1000mA"
- note added: "LIPO CONNECTOR"
- note added: "Overcharge Protection at 4.3V Overcharge timeout td = C19 * 9.0s/uF = 0.9 seconds Discharge Protection at 2.5V CHG_EN goes HIGH to disable charge"
- note added: "RGB LED CONTROL"
- note added: "SIP D BOOTSEL PWM"
- note removed: "SIP D BOOTSEL"
- moved on the sheet: C1, C10, C12, C13, C14, C15, C16, C17, C18, C19, C20, C21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

Commit message: Layout almost done...
Parts:
- removed C46: 10uF, symbol Device:C_Small
- removed CAN1, I2C1, PWR1, UT0, UT1, UT5: JST-SH, symbol bq29209:JST-SH
- removed DSM2: JST-ZH, symbol bq29209:JST-ZH
- removed GP0, GP1, GPS1, S1.1, S1.2: JST-SH1, symbol bq29209:JST-SH1
- removed J?: U.FL-R-SMT-1(10), U.FL-R-SMT-1_10_:HRS_U.FL-R-SMT-1(10), symbol U.FL-R-SMT-1_10_:U.FL-R-SMT-1(10)
- removed U16: NEO-M8N-0, XCVR_NEO-M8N-0:XCVR_NEO-M8N-0, symbol NEO-M8N-0:NEO-M8N-0
- added C305, C56: 0.1uF, Capacitor_SMD:C_0603_1608Metric_Pad1.08x0.95mm_HandSolder, symbol Device:C_Small
- added C53, C59: 10uF, Capacitor_SMD:C_0805_2012Metric_Pad1.18x1.45mm_HandSolder, symbol Device:C_Small
- added D314: GRN, LED_SMD:LED_0603_1608Metric_Pad1.05x0.95mm_HandSolder, symbol Device:LED
- added D315: RED, LED_SMD:LED_0603_1608Metric_Pad1.05x0.95mm_HandSolder, symbol Device:LED
- added D316: BLU, LED_SMD:LED_0603_1608Metric_Pad1.05x0.95mm_HandSolder, symbol Device:LED
- added H301, H302, H303, H304: MountingHole_Pad, MountingHole:MountingHole_3.2mm_M3_DIN965_Pad, symbol Mechanical:MountingHole_Pad
- added J305: GPS_MAG, Connector_JST:JST_XH_S6B-XH-A_1x06_P2.50mm_Horizontal, symbol Connector_Generic:Conn_01x06
- added J306: RGB OUT, Connector_JST:JST_XH_S4B-XH-A_1x04_P2.50mm_Horizontal, symbol Connector_Generic:Conn_01x04
- added J309: USB_B, Connector_USB:USB_B_TE_5787834_Vertical, symbol Connector:USB_B
- added J310: USB_C_Receptacle_USB2.0, Connector_USB:USB_C_Receptacle_HRO_TYPE-C-31-M-12, symbol Connector:USB_C_Receptacle_USB2.0
- added J311: TC2030-IDC, TDC-2030-IDC:TC2030-IDC, symbol elias-rescue:TC2030-IDC-Very_Connector
- added R305, R306: 5.1k, Resistor_SMD:R_0603_1608Metric_Pad0.98x0.95mm_HandSolder, symbol Device:R_Small
- added R307: 10k, Resistor_SMD:R_0603_1608Metric_Pad0.98x0.95mm_HandSolder, symbol Device:R_Small
- added R308, R309: 240, Resistor_SMD:R_0603_1608Metric_Pad0.98x0.95mm_HandSolder, symbol Device:R_Small
- added R310: 1k, Resistor_SMD:R_0603_1608Metric_Pad0.98x0.95mm_HandSolder, symbol Device:R_Small
- added TP315: TP_U0_RX, TestPoint:TestPoint_Pad_D1.0mm, symbol Connector:TestPoint_Small
- added TP316: TP_U0_TX, TestPoint:TestPoint_Pad_D1.0mm, symbol Connector:TestPoint_Small
- added U311: NC7WZ126, SOP50P310X90-8N:SOP50P310X90-8N, symbol elias-rescue:NC7WZ126-Very_Buffer
- C1: renamed from C6; footprint (none) -> Capacitor_SMD:C_0603_1608Metric_Pad1.08x0.95mm_HandSolder
- C10: renamed from C32; footprint (none) -> Capacitor_SMD:C_0603_1608Metric_Pad1.08x0.95mm_HandSolder
- C12: renamed from C28; footprint (none) -> Capacitor_SMD:C_0805_2012Metric_Pad1.18x1.45mm_HandSolder
- C13: renamed from C47; footprint (none) -> Capacitor_SMD:C_0603_1608Metric_Pad1.08x0.95mm_HandSolder
- C14: renamed from C31; footprint (none) -> Capacitor_SMD:C_0603_1608Metric_Pad1.08x0.95mm_HandSolder
- C15: renamed from C5; footprint (none) -> Capacitor_SMD:C_0603_1608Metric_Pad1.08x0.95mm_HandSolder
- C17: renamed from C8; footprint (none) -> Capacitor_SMD:C_0603_1608Metric_Pad1.08x0.95mm_HandSolder
- C18: renamed from C9; footprint (none) -> Capacitor_SMD:C_0603_1608Metric_Pad1.08x0.95mm_HandSolder
- C19: renamed from C7; footprint (none) -> Capacitor_SMD:C_0603_1608Metric_Pad1.08x0.95mm_HandSolder
- C25: renamed from C33; footprint (none) -> Capacitor_SMD:C_0805_2012Metric_Pad1.18x1.45mm_HandSolder
- C26: renamed from C35; footprint (none) -> Capacitor_SMD:C_0805_2012Metric_Pad1.18x1.45mm_HandSolder
- C27: renamed from C12; footprint (none) -> Capacitor_SMD:C_0603_1608Metric_Pad1.08x0.95mm_HandSolder
- C28: renamed from C1; footprint (none) -> Capacitor_SMD:C_0603_1608Metric_Pad1.08x0.95mm_HandSolder
- C29: renamed from C24; footprint (none) -> Capacitor_SMD:C_0603_1608Metric_Pad1.08x0.95mm_HandSolder
- C3: renamed from C11; footprint (none) -> Capacitor_SMD:C_0805_2012Metric_Pad1.18x1.45mm_HandSolder
- C30: renamed from C29; footprint (none) -> Capacitor_SMD:C_0603_1608Metric_Pad1.08x0.95mm_HandSolder
- C301: renamed from C4; footprint (none) -> Capacitor_SMD:C_0603_1608Metric_Pad1.08x0.95mm_HandSolder
- C302: renamed from C?; value 0.1uF -> 10uF; footprint Very_Footprints:C_0402_1005Metric -> Capacitor_SMD:C_0805_2012Metric_Pad1.18x1.45mm_HandSolder
- C303: renamed from C3; footprint Very_Footprints:C_0402_1005Metric -> Capacitor_SMD:C_0603_1608Metric_Pad1.08x0.95mm_HandSolder
- C304: renamed from C2; footprint Very_Footprints:C_0805_2012Metric -> Capacitor_SMD:C_0805_2012Metric_Pad1.18x1.45mm_HandSolder
- C31: renamed from C30; footprint (none) -> Capacitor_SMD:C_0603_1608Metric_Pad1.08x0.95mm_HandSolder
- C32: renamed from C25; footprint (none) -> Capacitor_SMD:C_0603_1608Metric_Pad1.08x0.95mm_HandSolder
- C33: renamed from C18; footprint (none) -> Capacitor_SMD:C_0603_1608Metric_Pad1.08x0.95mm_HandSolder
- C34: renamed from C50; footprint (none) -> Capacitor_SMD:C_0805_2012Metric_Pad1.18x1.45mm_HandSolder
- C35: renamed from C49; footprint (none) -> Capacitor_SMD:C_0603_1608Metric_Pad1.08x0.95mm_HandSolder
- C37: renamed from C13; footprint (none) -> Capacitor_SMD:C_0603_1608Metric_Pad1.08x0.95mm_HandSolder
- C38: renamed from C10; footprint (none) -> Capacitor_SMD:C_0805_2012Metric_Pad1.18x1.45mm_HandSolder
- C39: renamed from C14; footprint (none) -> Capacitor_SMD:C_0603_1608Metric_Pad1.08x0.95mm_HandSolder
- C4: renamed from C20; footprint (none) -> Capacitor_SMD:C_0603_1608Metric_Pad1.08x0.95mm_HandSolder
- C40: renamed from C15; footprint (none) -> Capacitor_SMD:C_0603_1608Metric_Pad1.08x0.95mm_HandSolder
- C41: renamed from C16; footprint (none) -> Capacitor_SMD:C_0603_1608Metric_Pad1.08x0.95mm_HandSolder
- C42: renamed from C38; footprint (none) -> Capacitor_SMD:C_0603_1608Metric_Pad1.08x0.95mm_HandSolder
- C43: renamed from C37; footprint (none) -> Capacitor_SMD:C_0603_1608Metric_Pad1.08x0.95mm_HandSolder
- C44: renamed from C40; footprint (none) -> Capacitor_SMD:C_0603_1608Metric_Pad1.08x0.95mm_HandSolder
- C47: renamed from C19; value 0.1uf -> 0.1uF; footprint (none) -> Capacitor_SMD:C_0603_1608Metric_Pad1.08x0.95mm_HandSolder
- C48: renamed from C21; footprint (none) -> Capacitor_SMD:C_0603_1608Metric_Pad1.08x0.95mm_HandSolder
- C49: renamed from C36; footprint (none) -> Capacitor_SMD:C_0603_1608Metric_Pad1.08x0.95mm_HandSolder
- C5: renamed from C17; footprint (none) -> Capacitor_SMD:C_0805_2012Metric_Pad1.18x1.45mm_HandSolder
- C50: renamed from C41; footprint (none) -> Capacitor_SMD:C_0603_1608Metric_Pad1.08x0.95mm_HandSolder
- C51: renamed from C23; footprint (none) -> Capacitor_SMD:C_0603_1608Metric_Pad1.08x0.95mm_HandSolder
- C52: renamed from C34; footprint (none) -> Capacitor_SMD:C_0603_1608Metric_Pad1.08x0.95mm_HandSolder
- C54: renamed from C22; footprint (none) -> Capacitor_SMD:C_0603_1608Metric_Pad1.08x0.95mm_HandSolder
- C55: renamed from C43; footprint (none) -> Capacitor_SMD:C_0603_1608Metric_Pad1.08x0.95mm_HandSolder
- C57: renamed from C39; footprint (none) -> Capacitor_SMD:C_0603_1608Metric_Pad1.08x0.95mm_HandSolder
- C58: renamed from C26; footprint (none) -> Capacitor_SMD:C_0603_1608Metric_Pad1.08x0.95mm_HandSolder
- C6: renamed from C44; footprint (none) -> Capacitor_SMD:C_0603_1608Metric_Pad1.08x0.95mm_HandSolder
- C60: renamed from C42; footprint (none) -> Capacitor_SMD:C_0805_2012Metric_Pad1.18x1.45mm_HandSolder
- C7: renamed from C27; footprint (none) -> Capacitor_SMD:C_0805_2012Metric_Pad1.18x1.45mm_HandSolder
- C8: renamed from C48; footprint (none) -> Capacitor_SMD:C_0603_1608Metric_Pad1.08x0.95mm_HandSolder
- C9: renamed from C45; footprint (none) -> Capacitor_SMD:C_0603_1608Metric_Pad1.08x0.95mm_HandSolder
- D1: renamed from D4; footprint (none) -> LED_SMD:LED_0603_1608Metric_Pad1.05x0.95mm_HandSolder
- D2: footprint (none) -> LED_SMD:LED_0603_1608Metric_Pad1.05x0.95mm_HandSolder
- D3: renamed from D1; footprint (none) -> LED_SMD:LED_0603_1608Metric_Pad1.05x0.95mm_HandSolder
- D301: renamed from D6; footprint (none) -> LED_SMD:LED_0603_1608Metric_Pad1.05x0.95mm_HandSolder
- D302: renamed from D7; footprint (none) -> LED_SMD:LED_0603_1608Metric_Pad1.05x0.95mm_HandSolder
- D303: renamed from D8; footprint (none) -> LED_SMD:LED_0603_1608Metric_Pad1.05x0.95mm_HandSolder
- D304: renamed from D9; footprint (none) -> LED_SMD:LED_0603_1608Metric_Pad1.05x0.95mm_HandSolder
- D305: renamed from D5; footprint (none) -> LED_SMD:LED_0603_1608Metric_Pad1.05x0.95mm_HandSolder
- D306: renamed from D10; footprint (none) -> LED_SMD:LED_0603_1608Metric_Pad1.05x0.95mm_HandSolder
- D307: renamed from D11; footprint (none) -> LED_SMD:LED_0603_1608Metric_Pad1.05x0.95mm_HandSolder
- D308: renamed from D12; footprint (none) -> LED_SMD:LED_0603_1608Metric_Pad1.05x0.95mm_HandSolder
- D309: renamed from D13; footprint (none) -> LED_SMD:LED_0603_1608Metric_Pad1.05x0.95mm_HandSolder
- D310: renamed from D14; footprint (none) -> LED_SMD:LED_0603_1608Metric_Pad1.05x0.95mm_HandSolder
- D311: renamed from D15; footprint (none) -> LED_SMD:LED_0603_1608Metric_Pad1.05x0.95mm_HandSolder
- D312: renamed from D16; footprint (none) -> LED_SMD:LED_0603_1608Metric_Pad1.05x0.95mm_HandSolder
- D313: renamed from D3; footprint (none) -> LED_SMD:LED_0603_1608Metric_Pad1.05x0.95mm_HandSolder
- J301: renamed from J2; footprint Connector_JST:JST_PH_S4B-PH-SM4-TB_1x04-1MP_P2.00mm_Horizontal -> Connector_PinSocket_1.27mm:PinSocket_2x02_P1.27mm_Vertical
- L1, L2: footprint (none) -> Inductor_SMD:L_Bourns_SRN6045TA
- MOD301: renamed from MOD1; footprint (none) -> SW_RS-032G05A3-SMRT:SW_RS-032G05A3-SMRT
- PAU301: renamed from PAU1; footprint (none) -> SW_RS-032G05A3-SMRT:SW_RS-032G05A3-SMRT
- POW301: renamed from POW1; footprint (none) -> SW_RS-032G05A3-SMRT:SW_RS-032G05A3-SMRT
- R100: renamed from R74; footprint (none) -> Resistor_SMD:R_0603_1608Metric_Pad0.98x0.95mm_HandSolder
- R101: renamed from R80; footprint (none) -> Resistor_SMD:R_0603_1608Metric_Pad0.98x0.95mm_HandSolder
- R102: renamed from R79; footprint (none) -> Resistor_SMD:R_0603_1608Metric_Pad0.98x0.95mm_HandSolder
- R103: renamed from R83; footprint (none) -> Resistor_SMD:R_0603_1608Metric_Pad0.98x0.95mm_HandSolder
- R104: renamed from R85; footprint (none) -> Resistor_SMD:R_0603_1608Metric_Pad0.98x0.95mm_HandSolder
- R105: renamed from R84; footprint (none) -> Resistor_SMD:R_0603_1608Metric_Pad0.98x0.95mm_HandSolder
- R106: renamed from R55; footprint (none) -> Resistor_SMD:R_0603_1608Metric_Pad0.98x0.95mm_HandSolder
- R108: renamed from R36; footprint (none) -> Resistor_SMD:R_0603_1608Metric_Pad0.98x0.95mm_HandSolder
- R111: renamed from R56; footprint (none) -> Resistor_SMD:R_0603_1608Metric_Pad0.98x0.95mm_HandSolder
- R113: renamed from R16; footprint (none) -> Resistor_SMD:R_0603_1608Metric_Pad0.98x0.95mm_HandSolder
- R115: renamed from R17; footprint (none) -> Resistor_SMD:R_0603_1608Metric_Pad0.98x0.95mm_HandSolder
- R116: renamed from R18; footprint (none) -> Resistor_SMD:R_0603_1608Metric_Pad0.98x0.95mm_HandSolder
- R118: renamed from R20; footprint (none) -> Resistor_SMD:R_0603_1608Metric_Pad0.98x0.95mm_HandSolder
- R120: renamed from R22; footprint (none) -> Resistor_SMD:R_0603_1608Metric_Pad0.98x0.95mm_HandSolder
- R122: renamed from R24; footprint (none) -> Resistor_SMD:R_0603_1608Metric_Pad0.98x0.95mm_HandSolder
- R123: renamed from R76; footprint (none) -> Resistor_SMD:R_0603_1608Metric_Pad0.98x0.95mm_HandSolder
- R124: renamed from R75; footprint (none) -> Resistor_SMD:R_0603_1608Metric_Pad0.98x0.95mm_HandSolder
- R125: renamed from R19; footprint (none) -> Resistor_SMD:R_0603_1608Metric_Pad0.98x0.95mm_HandSolder
- R127: renamed from R21; footprint (none) -> Resistor_SMD:R_0603_1608Metric_Pad0.98x0.95mm_HandSolder
- R129: renamed from R23; footprint (none) -> Resistor_SMD:R_0603_1608Metric_Pad0.98x0.95mm_HandSolder
- R131: renamed from R25; footprint (none) -> Resistor_SMD:R_0603_1608Metric_Pad0.98x0.95mm_HandSolder
- R135: renamed from R27; footprint (none) -> Resistor_SMD:R_0603_1608Metric_Pad0.98x0.95mm_HandSolder
- R140: renamed from R31; footprint (none) -> Resistor_SMD:R_0603_1608Metric_Pad0.98x0.95mm_HandSolder
- R143: renamed from R30; footprint (none) -> Resistor_SMD:R_0603_1608Metric_Pad0.98x0.95mm_HandSolder
- R149: renamed from R45; footprint (none) -> Resistor_SMD:R_0603_1608Metric_Pad0.98x0.95mm_HandSolder
- R158: renamed from R26; footprint (none) -> Resistor_SMD:R_0603_1608Metric_Pad0.98x0.95mm_HandSolder
- R16: renamed from R28; footprint (none) -> Resistor_SMD:R_0603_1608Metric_Pad0.98x0.95mm_HandSolder
- R17: renamed from R29; footprint (none) -> Resistor_SMD:R_0603_1608Metric_Pad0.98x0.95mm_HandSolder
- R18: renamed from R43; footprint (none) -> Resistor_SMD:R_0603_1608Metric_Pad0.98x0.95mm_HandSolder
- R190: renamed from R37; footprint (none) -> Resistor_SMD:R_0603_1608Metric_Pad0.98x0.95mm_HandSolder
- R2: renamed from R9; footprint (none) -> Resistor_SMD:R_0603_1608Metric_Pad0.98x0.95mm_HandSolder
- R20: renamed from R42; footprint (none) -> Resistor_SMD:R_0603_1608Metric_Pad0.98x0.95mm_HandSolder
- R21: renamed from R59; footprint (none) -> Resistor_SMD:R_0603_1608Metric_Pad0.98x0.95mm_HandSolder
- R22: renamed from R58; footprint (none) -> Resistor_SMD:R_0603_1608Metric_Pad0.98x0.95mm_HandSolder
- R23: renamed from R8; footprint (none) -> Resistor_SMD:R_0603_1608Metric_Pad0.98x0.95mm_HandSolder
- R24: renamed from R33; footprint (none) -> Resistor_SMD:R_0603_1608Metric_Pad0.98x0.95mm_HandSolder
- R26: renamed from R91; footprint (none) -> Resistor_SMD:R_0603_1608Metric_Pad0.98x0.95mm_HandSolder
- R27: renamed from R15; footprint (none) -> Resistor_SMD:R_0603_1608Metric_Pad0.98x0.95mm_HandSolder
- R28: renamed from R13; footprint (none) -> Resistor_SMD:R_0603_1608Metric_Pad0.98x0.95mm_HandSolder
- R29: renamed from R66; footprint (none) -> Resistor_SMD:R_0603_1608Metric_Pad0.98x0.95mm_HandSolder
- R3: renamed from R40; footprint (none) -> Resistor_SMD:R_0603_1608Metric_Pad0.98x0.95mm_HandSolder
- R30: renamed from R14; footprint (none) -> Resistor_SMD:R_0603_1608Metric_Pad0.98x0.95mm_HandSolder
- R301: renamed from R57; footprint (none) -> Resistor_SMD:R_0603_1608Metric_Pad0.98x0.95mm_HandSolder
- R302: renamed from R3; footprint Very_Footprints:R_0402_1005Metric -> Resistor_SMD:R_0603_1608Metric_Pad0.98x0.95mm_HandSolder
- R303: renamed from R5; footprint Very_Footprints:R_0402_1005Metric -> Resistor_SMD:R_0603_1608Metric_Pad0.98x0.95mm_HandSolder
- R304: renamed from R7; footprint Very_Footprints:R_0402_1005Metric -> Resistor_SMD:R_0603_1608Metric_Pad0.98x0.95mm_HandSolder
- R31: renamed from R65; footprint (none) -> Resistor_SMD:R_0603_1608Metric_Pad0.98x0.95mm_HandSolder
- R32: renamed from R68; footprint (none) -> Resistor_SMD:R_0603_1608Metric_Pad0.98x0.95mm_HandSolder
- R33: renamed from R67; footprint (none) -> Resistor_SMD:R_0603_1608Metric_Pad0.98x0.95mm_HandSolder
- R34: renamed from R10; footprint (none) -> Resistor_SMD:R_0603_1608Metric_Pad0.98x0.95mm_HandSolder
- R35: renamed from R90; footprint (none) -> Resistor_SMD:R_0603_1608Metric_Pad0.98x0.95mm_HandSolder
- R4: renamed from R53; footprint (none) -> Resistor_SMD:R_0603_1608Metric_Pad0.98x0.95mm_HandSolder
- R44: renamed from R6; footprint (none) -> Resistor_SMD:R_0603_1608Metric_Pad0.98x0.95mm_HandSolder
- R5: renamed from R38; footprint (none) -> Resistor_SMD:R_0603_1608Metric_Pad0.98x0.95mm_HandSolder
- R54: renamed from R89; footprint (none) -> Resistor_SMD:R_0603_1608Metric_Pad0.98x0.95mm_HandSolder
- R55: renamed from R88; footprint (none) -> Resistor_SMD:R_0603_1608Metric_Pad0.98x0.95mm_HandSolder
- R56: renamed from R87; footprint (none) -> Resistor_SMD:R_0603_1608Metric_Pad0.98x0.95mm_HandSolder
- R57: renamed from R86; footprint (none) -> Resistor_SMD:R_0603_1608Metric_Pad0.98x0.95mm_HandSolder
- R58: renamed from R2; footprint (none) -> Resistor_SMD:R_0603_1608Metric_Pad0.98x0.95mm_HandSolder
- R59: renamed from R41; footprint (none) -> Resistor_SMD:R_0603_1608Metric_Pad0.98x0.95mm_HandSolder
- R6: renamed from R39; footprint (none) -> Resistor_SMD:R_0603_1608Metric_Pad0.98x0.95mm_HandSolder
- R60: renamed from R34; footprint (none) -> Resistor_SMD:R_0603_1608Metric_Pad0.98x0.95mm_HandSolder
- R61: renamed from R60; footprint (none) -> Resistor_SMD:R_0603_1608Metric_Pad0.98x0.95mm_HandSolder
- R62: renamed from R61; footprint (none) -> Resistor_SMD:R_0603_1608Metric_Pad0.98x0.95mm_HandSolder
- R63: renamed from R62; footprint (none) -> Resistor_SMD:R_0603_1608Metric_Pad0.98x0.95mm_HandSolder
- R64: renamed from R63; footprint (none) -> Resistor_SMD:R_0603_1608Metric_Pad0.98x0.95mm_HandSolder
- R7: renamed from R11; footprint (none) -> Resistor_SMD:R_0603_1608Metric_Pad0.98x0.95mm_HandSolder
- R76: renamed from R4; footprint (none) -> Resistor_SMD:R_0603_1608Metric_Pad0.98x0.95mm_HandSolder
- R77: renamed from R32; footprint (none) -> Resistor_SMD:R_0603_1608Metric_Pad0.98x0.95mm_HandSolder
- R78: renamed from R46; footprint (none) -> Resistor_SMD:R_0603_1608Metric_Pad0.98x0.95mm_HandSolder
- R79: renamed from R47; footprint (none) -> Resistor_SMD:R_0603_1608Metric_Pad0.98x0.95mm_HandSolder
- R8: renamed from R12; footprint (none) -> Resistor_SMD:R_0603_1608Metric_Pad0.98x0.95mm_HandSolder
- R80: renamed from R48; footprint (none) -> Resistor_SMD:R_0603_1608Metric_Pad0.98x0.95mm_HandSolder
- R81: renamed from R49; footprint (none) -> Resistor_SMD:R_0603_1608Metric_Pad0.98x0.95mm_HandSolder
- R82: renamed from R50; footprint (none) -> Resistor_SMD:R_0603_1608Metric_Pad0.98x0.95mm_HandSolder
- R83: renamed from R51; footprint (none) -> Resistor_SMD:R_0603_1608Metric_Pad0.98x0.95mm_HandSolder
- R84: renamed from R44; footprint (none) -> Resistor_SMD:R_0603_1608Metric_Pad0.98x0.95mm_HandSolder
- R85: renamed from R69; footprint (none) -> Resistor_SMD:R_0603_1608Metric_Pad0.98x0.95mm_HandSolder
- R86: renamed from R70; footprint (none) -> Resistor_SMD:R_0603_1608Metric_Pad0.98x0.95mm_HandSolder
- R87: renamed from R77; footprint (none) -> Resistor_SMD:R_0603_1608Metric_Pad0.98x0.95mm_HandSolder
- R88: renamed from R78; footprint (none) -> Resistor_SMD:R_0603_1608Metric_Pad0.98x0.95mm_HandSolder
- R89: renamed from R35; footprint (none) -> Resistor_SMD:R_0603_1608Metric_Pad0.98x0.95mm_HandSolder
- R9: renamed from R52; footprint (none) -> Resistor_SMD:R_0603_1608Metric_Pad0.98x0.95mm_HandSolder
- R91: renamed from R64; footprint (none) -> Resistor_SMD:R_0603_1608Metric_Pad0.98x0.95mm_HandSolder
- R92: renamed from R71; footprint (none) -> Resistor_SMD:R_0603_1608Metric_Pad0.98x0.95mm_HandSolder
- R93: renamed from R54; footprint (none) -> Resistor_SMD:R_0603_1608Metric_Pad0.98x0.95mm_HandSolder
- R96: renamed from R72; footprint (none) -> Resistor_SMD:R_0603_1608Metric_Pad0.98x0.95mm_HandSolder
- R97: renamed from R73; footprint (none) -> Resistor_SMD:R_0603_1608Metric_Pad0.98x0.95mm_HandSolder
- R98: renamed from R82; footprint (none) -> Resistor_SMD:R_0603_1608Metric_Pad0.98x0.95mm_HandSolder
- R99: renamed from R81; footprint (none) -> Resistor_SMD:R_0603_1608Metric_Pad0.98x0.95mm_HandSolder
- RST301: renamed from RST1; footprint (none) -> SW_RS-032G05A3-SMRT:SW_RS-032G05A3-SMRT
- SD301: renamed from SD1; footprint (none) -> SW_RS-032G05A3-SMRT:SW_RS-032G05A3-SMRT
- TP301: renamed from TP4; footprint (none) -> TestPoint:TestPoint_Pad_D1.0mm
- TP302: renamed from TP6; footprint (none) -> TestPoint:TestPoint_Pad_D1.0mm
- TP303: renamed from TP7; footprint (none) -> TestPoint:TestPoint_Pad_D1.0mm
- TP304: renamed from TP5; footprint (none) -> TestPoint:TestPoint_Pad_D1.0mm
- TP305: renamed from TP1; footprint (none) -> TestPoint:TestPoint_Pad_D1.0mm
- TP306: renamed from TP2; footprint (none) -> TestPoint:TestPoint_Pad_D1.0mm
- TP307: renamed from TP3; footprint (none) -> TestPoint:TestPoint_Pad_D1.0mm
- TP308: renamed from TP8; footprint (none) -> TestPoint:TestPoint_Pad_D1.0mm
- TP309: renamed from TP9; footprint (none) -> TestPoint:TestPoint_Pad_D1.0mm
- TP310: renamed from TP10; footprint (none) -> TestPoint:TestPoint_Pad_D1.0mm
- TP311: renamed from TP11; footprint (none) -> TestPoint:TestPoint_Pad_D1.0mm
- TP312: renamed from TP12; footprint (none) -> TestPoint:TestPoint_Pad_D1.0mm
- TP313: renamed from TP13; footprint (none) -> TestPoint:TestPoint_Pad_D1.0mm
- TP314: renamed from TP14; footprint (none) -> TestPoint:TestPoint_Pad_D1.0mm
- Y1: footprint (none) -> Crystal:Crystal_SMD_Qantek_QC5CB-2Pin_5x3.2mm
- Y2: footprint (none) -> Crystal:Crystal_SMD_3215-2Pin_3.2x1.5mm
- gave numbers to parts that had none: 1
- renumbered J1 to J302, X1 to J303, J3 to J307, J4 to J308, OSC1 to OSC301, Q2 to Q301, Q3 to Q302, Q4 to Q303, R1 to R107, U12 to U2, U14 to U3, U4 to U301, U9 to U302, U5 to U303, U6 to U304, U19 to U305, U15 to U306, U2 to U307, U17 to U308, U1 to U309, U18 to U310, U8 to U4, U3 to U5, U7 to U6, U11 to U7, U13 to U9
Connections:
- net +10V is gone; now on net VCC: C303.1, C304.1
- net B_PWM is gone; now on net PWM_2A: Q303.1 (G), R304.1
- net G_PWM is gone; now on net PWM_1B: Q301.1 (G), R302.1
- net R_PWM is gone; now on net PWM_1A: Q302.1 (G), R303.1
- net SPI1_MOSI is gone; now on net RF69_MOSI: U309.D12 (MCASP0_AXR0)
- net SPI1_SCK is gone; now on net RF69_SCK: U309.A13 (MCASP0_ACLKX)
- net SPI1_SS1 is gone; now on net RF69_NSS: U309.H18 (RMII1_REF_CLK)
- net +3V3: now also C302.2, U310.13 (3.3V), C305.2, C53.1, C56.1, C59.1, R307.1, U311.1 (OE1), U311.7 (OE2), U311.8 (VCC)
- net 5.0V: now also J305.1 (Pin_1)
- net B_OUT: now also J306.4 (Pin_4)
- net GND: now also C302.1, U10.11 (GND), U303.9 (EPAD), U310.1 (GND), U310.10 (GND), U310.8 (GND), U9.11 (GND), C305.1, C53.2, C56.2, C59.2, H301.1, H302.1, H303.1, H304.1, J305.2 (Pin_2), J309.4 (GND), J310.A1 (GND), J310.A12 (GND), J310.B1 (GND), J310.B12 (GND), J311.5 (GND), R305.2, R306.2, R307.2, U311.4 (GND)
- net GNDPWR: now also J309.5 (Shield), J310.S1 (SHIELD)
- net GPIO1_17: now also U310.14 (DIO0)
- net GPIO1_25: now also U310.6 (RESET)
- net G_OUT: now also J306.2 (Pin_2)
- net I2C2_SCL: now also J305.5 (Pin_5)
- net I2C2_SDA: now also J305.6 (Pin_6)
- net PWM_1A: now also D315.2 (A)
- net PWM_1B: now also D314.2 (A)
- net PWM_2A: now also D316.2 (A)
- net R_OUT: now also J306.3 (Pin_3)
- net UART0_RX: now also TP315.1, U311.6 (Y1)
- net UART0_TX: now also TP316.1, U311.5 (A2)
- net UART5_RX: now also J305.3 (Pin_3)
- net UART5_TX: now also J305.4 (Pin_4)
- net USB0_D_N: now also J309.2 (D-)
- net USB0_D_P: now also J309.3 (D+)
- net USB0_VBUS: now also J309.1 (VBUS), J310.A4 (VBUS), J310.A9 (VBUS), J310.B4 (VBUS), J310.B9 (VBUS)
- net USB1_D_N: now also J310.A7 (D-), J310.B7 (D-)
- net USB1_D_P: now also J310.A6 (D+), J310.B6 (D+)
- net VCC: now also J306.1 (Pin_1)
- net VSS: now also R308.2, R309.2, R310.2
- net RF69_MISO: now reaches U310.2 (MISO)
- net RF69_MOSI: now reaches U310.3 (MOSI)
- net RF69_SCK: now reaches U310.4 (SCK)
- net RF69_NSS: now reaches U310.5 (NSS)
- new net: J311.3 (RXD), U311.3 (Y2)
- new net: J311.4 (TXD), U311.2 (A1)
- new net: J310.A5 (CC1), R306.1
- new net: D316.1 (K), R310.1
- new net: D314.1 (K), R308.1
- new net: J310.B5 (CC2), R305.1
- new net: D315.1 (K), R309.1
- no-connect marks 187 -> 196
Other:
- note added: "GPS NEO-M8N BDS Compass Receiver Module"
- note added: "RF69 PACKET RADIO"
- note removed: "GPIO CONNECTORS"
- moved on the sheet: C14, C17, C27, C302, C303, C304, C33, C42, C43, C44, C47, C48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

Commit message: Start layout
Parts:
- removed D1, D2, D3: LED, LED_SMD:LED_0603_1608Metric_Pad1.05x0.95mm_HandSolder, symbol Device:LED
- added D1, D2, D3: D_Small, Diode_SMD:D_SOD-123, symbol Device:D_Small
- J301: footprint Connector_PinSocket_1.27mm:PinSocket_2x02_P1.27mm_Vertical -> DT:DTM-13
- J309: footprint Connector_USB:USB_B_TE_5787834_Vertical -> Connector_USB:USB_B_OST_USB-B1HSxx_Horizontal
Connections:
- net BT_OE is gone; now on net WL_BT_OE: U309.L18 (MII1_RX_CLK)
- net GNDPWR is gone; now on net GND: J303.S1 (SHIELD), J303.S2 (SHIELD), J303.S3 (SHIELD), J303.S4 (SHIELD), J303.S5 (SHIELD), J303.S6 (SHIELD), J309.5 (Shield), J310.S1 (SHIELD), R107.2
- net VSS is gone; now on net GND: C303.2, C304.2, Q301.2 (S), Q302.2 (S), Q303.2 (S), R302.2, R303.2, R304.2, R308.2, R309.2, R310.2
- net GND: now also D1.2 (A)
- net VCC: now also D2.2 (A)
- net V_BATT: now also D3.2 (A)
- net at L1.1, U304.3 (FB): now also D1.1 (K)
- net at C3.1, U304.1 (VIN): now also D2.1 (K), D3.1 (K)
Other:
- moved on the sheet: R27

Commit message: fanout is hard
Parts:
- added J312: Conn_01x04, Connector_Molex:Molex_PicoBlade_53261-0471_1x04-1MP_P1.25mm_Horizontal, symbol Connector_Generic:Conn_01x04
- J305: footprint Connector_JST:JST_XH_S6B-XH-A_1x06_P2.50mm_Horizontal -> Connector_Molex:Molex_PicoBlade_53261-0671_1x06-1MP_P1.25mm_Horizontal
Connections:
- net GND: now also J305.6 (Pin_6); no longer J305.2 (Pin_2)
- net I2C2_SCL: now also J312.2 (Pin_2); no longer J305.5 (Pin_5)
- net I2C2_SDA: now also J312.3 (Pin_3); no longer J305.6 (Pin_6)
- net UART5_RX: now also J305.2 (Pin_2); no longer J305.3 (Pin_3)
- net UART5_TX: now also J305.3 (Pin_3); no longer J305.4 (Pin_4)
- net USB0_ID: no longer names the net of U4.3 (ID)
- net USB0_ID: no longer U309.P16 (USB0_ID)
- net USB1_ID: no longer names the net of U3.3 (ID)
- net USB1_ID: no longer U309.P17 (USB1_ID)
- no-connect marks 196 -> 203

Commit message: Nearly done!
Parts:
- removed D303, D304, D306, D307: BLU, LED_SMD:LED_0603_1608Metric_Pad1.05x0.95mm_HandSolder, symbol Device:LED
- removed D309: RED, LED_SMD:LED_0603_1608Metric_Pad1.05x0.95mm_HandSolder, symbol Device:LED
- removed D310, D311, D312: GRN, LED_SMD:LED_0603_1608Metric_Pad1.05x0.95mm_HandSolder, symbol Device:LED
- removed R29, R31, R32, R33: 240, Resistor_SMD:R_0603_1608Metric_Pad0.98x0.95mm_HandSolder, symbol Device:R_Small
- removed R61, R62, R63, R64: 1k, Resistor_SMD:R_0603_1608Metric_Pad0.98x0.95mm_HandSolder, symbol Device:R_Small
- removed TP315: TP_U0_RX, TestPoint:TestPoint_Pad_D1.0mm, symbol Connector:TestPoint_Small
- removed TP316: TP_U0_TX, TestPoint:TestPoint_Pad_D1.0mm, symbol Connector:TestPoint_Small
- J311: footprint TDC-2030-IDC:TC2030-IDC -> Connector:Tag-Connect_TC2030-IDC-FP_2x03_P1.27mm_Vertical
Connections:
- net 5.0V: no longer J305.1 (Pin_1)
- net SYS_5V: now also J305.1 (Pin_1)
- net USB0_VBUS: no longer C55.1, J310.A4 (VBUS), J310.A9 (VBUS), J310.B4 (VBUS), J310.B9 (VBUS), R301.2, U3.6 (VBUS), U309.Y9 (VIN_USB_2)
- net 0 renamed USR_LED0
- net 1 renamed USR_LED1
- net 2 renamed USR_LED2
- net 3 renamed USR_LED3
- net B0 renamed BATT_LED_1
- net B1 renamed BATT_LED_2
- net B2 renamed BATT_LED_3
- net B3 renamed BATT_LED_4
- new net USB1_VBUS: C55.1, J310.A4 (VBUS), J310.A9 (VBUS), J310.B4 (VBUS), J310.B9 (VBUS), R301.2, U3.6 (VBUS), U309.Y9 (VIN_USB_2)
- no-connect marks 203 -> 204
Other:
- moved on the sheet: D301, D302, D308, R21, R22, R91
