File: hardware/CONEPROJ.kicad_sch (KiCad schematic)
At the start: 103 parts, among them J2 693071020811, J304 U.FL-R-SMT-1(10), J306 RGB OUT, J311 TC2030-IDC, J4 DTM1312PA12PBR008, J5 TC2030-IDC, J6 UC-31PFFP-QS8001, Q2 Q_Dual_NMOS_S1G1S2G2D2D2D1D1, Q3 Q_Dual_NMOS_S1G1S2G2D2D2D1D1, Q4 Q_Dual_NMOS_S1G1S2G2D2D2D1D1, Q5 Q_Dual_NMOS_S1G1S2G2D2D2D1D1, Q6 Q_Dual_NMOS_S1G1S2G2D2D2D1D1, Q7 Q_Dual_NMOS_S1G1S2G2D2D2D1D1, U10 RP2040, U2 SN65HVD230, U304 AP1509, U310 RFM69HCW, U311 SN74LVC2G126DCUR, U5 MCP2515-xST, U6 RT9742GGJ5, U7 W25Q128JVS, U8 MCP2515-xSO, U9 WS2815B, Y2 16mhz, Y3 12mhz

Commit message: almost done
Parts:
- removed C303: 0.1uF, Capacitor_SMD:C_0603_1608Metric_Pad1.08x0.95mm_HandSolder, symbol elias-rescue:C_Small-Very_Capacitor
- removed C304: 10uF, Capacitor_SMD:C_0805_2012Metric_Pad1.18x1.45mm_HandSolder, symbol elias-rescue:C_Small-Very_Capacitor
- removed J306: RGB OUT, Connector_JST:JST_XH_S5B-XH-A-1_1x05_P2.50mm_Horizontal, symbol Connector_Generic:Conn_01x05
- added C?: 0.1uF, Capacitor_SMD:C_0603_1608Metric_Pad1.08x0.95mm_HandSolder, symbol elias-rescue:C_Small-Very_Capacitor
- added C?: 10uF, Capacitor_SMD:C_0805_2012Metric_Pad1.18x1.45mm_HandSolder, symbol elias-rescue:C_Small-Very_Capacitor
Connections:
- net GND: now also C?.2, C?.2
- net VCC: now also C?.1, C?.1

Commit message: Can't change it now!
Parts:
- gave numbers to parts that had none: 2
Connections:
- net VCC: no longer J4.B6
- net VIN: now also J4.B6
Changed lines of the file:
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@@
     (effects (font (size 1.27 1.27)) (justify right bottom))
   )
-  (label "VCC" (at 415.29 281.94 180)
+  (label "VIN" (at 415.29 281.94 180)
     (effects (font (size 1.27 1.27)) (justify right bottom))
   )
@@
   (symbol (lib_id "elias-rescue:C_Small-Very_Capacitor") (at 456.565 271.78 0) (mirror y) (unit 1)
     (in_bom yes) (on_board yes)
-    (property "Reference" "C?" (id 0) (at 454.2282 270.6116 0)
+    (property "Reference" "C20" (id 0) (at 454.2282 270.6116 0)
       (effects (font (size 1.27 1.27)) (justify left))
     )
@@
   (symbol (lib_id "elias-rescue:C_Small-Very_Capacitor") (at 441.325 271.78 0) (unit 1)
     (in_bom yes) (on_board yes)
-    (property "Reference" "C?" (id 0) (at 443.6618 270.6116 0)
+    (property "Reference" "C2" (id 0) (at 443.6618 270.6116 0)
       (effects (font (size 1.27 1.27)) (justify left))
     )
@@
   (symbol (lib_id "power:GND") (at 456.565 275.59 0) (unit 1)
     (in_bom yes) (on_board yes) (fields_autoplaced)
-    (property "Reference" "#PWR?" (id 0) (at 456.565 281.94 0)
+    (property "Reference" "#PWR0113" (id 0) (at 456.565 281.94 0)
       (effects (font (size 1.27 1.27)) hide)
     )
@@
   (symbol (lib_id "power:GND") (at 441.325 275.59 0) (unit 1)
     (in_bom yes) (on_board yes) (fields_autoplaced)
-    (property "Reference" "#PWR?" (id 0) (at 441.325 281.94 0)
+    (property "Reference" "#PWR0115" (id 0) (at 441.325 281.94 0)
       (effects (font (size 1.27 1.27)) hide)
     )
@@
       (reference "#PWR0112") (unit 1) (value "GND") (footprint "")
     )
+    (path "/c448a753-7209-4de5-aa84-164df3948945"
+      (reference "#PWR0113") (unit 1) (value "GND") (footprint "")
+    )
     (path "/54ba24e3-2912-4331-8e77-cbac8dc39d0a"
       (reference "#PWR0114") (unit 1) (value "GND") (footprint "")
     )
+    (path "/df884e43-58fc-48a1-a545-d30a3cb1db71"
+      (reference "#PWR0115") (unit 1) (value "GND") (footprint "")
+    )
     (path "/8bc84bb2-3518-4e6b-ba0e-3a08acb752c0"
       (reference "#PWR0116") (unit 1) (value "GND") (footprint "")
@@
       (reference "#PWR0180") (unit 1) (value "GND") (footprint "")
     )
-    (path "/c448a753-7209-4de5-aa84-164df3948945"
-      (reference "#PWR?") (unit 1) (value "GND") (footprint "")
-    )
-    (path "/df884e43-58fc-48a1-a545-d30a3cb1db71"
-      (reference "#PWR?") (unit 1) (value "GND") (footprint "")
+    (path "/809b8cf6-aa34-4885-969a-ea9d7d5bb7d3"
+      (reference "C2") (unit 1) (value "10uF") (footprint "Capacitor_SMD:C_0805_2012Metric_Pad1.18x1.45mm_HandSolder")
     )
     (path "/f303bae3-07e1-45ad-b2a2-06dc904ca6c2"
@@
       (reference "C19") (unit 1) (value "0.1uF") (footprint "Capacitor_SMD:C_0603_1608Metric_Pad1.08x0.95mm_HandSolder")
     )
+    (path "/7a37ca2b-03f8-42b8-84e4-5a722be13d07"
+      (reference "C20") (unit 1) (value "0.1uF") (footprint "Capacitor_SMD:C_0603_1608Metric_Pad1.08x0.95mm_HandSolder")
+    )
     (path "/fdd639c9-9c8e-4e1a-bb96-783aa436a358"
       (reference "C21") (unit 1) (value "22pf") (footprint "Capacitor_SMD:C_0603_1608Metric_Pad1.08x0.95mm_HandSolder")
@@
       (reference "C305") (unit 1) (value "0.1uF") (footprint "Capacitor_SMD:C_0603_1608Metric_Pad1.08x0.95mm_HandSolder")
     )
-    (path "/7a37ca2b-03f8-42b8-84e4-5a722be13d07"
-      (reference "C?") (unit 1) (value "0.1uF") (footprint "Capacitor_SMD:C_0603_1608Metric_Pad1.08x0.95mm_HandSolder")
-    )
-    (path "/809b8cf6-aa34-4885-969a-ea9d7d5bb7d3"
-      (reference "C?") (unit 1) (value "10uF") (footprint "Capacitor_SMD:C_0805_2012Metric_Pad1.18x1.45mm_HandSolder")
-    )
     (path "/1e616cea-39e5-4f60-9cfc-b30728e65923"

Commit message: Schematic cleanup
Parts:
- added R11, R12: 1k, Resistor_SMD:R_0603_1608Metric_Pad0.98x0.95mm_HandSolder, symbol Device:R_Small
- C11, C16, C2, C20, C302: symbol elias-rescue:C_Small-Very_Capacitor -> Device:C_Small
- C12, C6, C9: DESCRIPTION CAP CER 1UF 50V X7R 0603 -> CAP CER 1UF 16V X7R 0603; MPN (none) -> CL10B105MO8NNWC
- C21, C22: value 22pf -> 10pF; DESCRIPTION CAP CER 22PF 100V X7R 0603 -> CAP CER 10PF 50V X7R 0603; MPN C0603C220K1RACAUTO -> C0603C100K5RACAUTO
- C7, C8: MPN (none) -> C0603C100K5RACAUTO
- CM4A2, CM4B2: MPN2 (none) -> 501531-3410
- J311: symbol elias-rescue:TC2030-IDC-Very_Connector -> TDC-2030-IDC:TC2030-IDC; MPN (none) -> TC2030-FTDI-C232HD-DDHSP-0
- J4: Comment DTM1312PA12PBR008 -> (none); DESCRIPTION (none) -> CONN HEADER R/A 24POS; EU_RoHS_Compliance Compliant -> (none); MPN (none) -> DTM1312PA12PBR008
- J5: symbol elias-rescue:TC2030-IDC-Very_Connector -> TDC-2030-IDC:TC2030-IDC; MPN (none) -> TC2030-USB
- J6: DESCRIPTION (none) -> CONN RCP USB3.1 TYPC 24P PNL MNT; MPN (none) -> UC-31PFFP-QS8001
- Module2: DESCRIPTION (none) -> COMPUTE 4 1GB RAM 0GB LITE WIFI; MPN (none) -> SC0691
- Module2: DESCRIPTION (none) -> COMPUTE 4 1GB RAM 0GB LITE WIFI
- Q2, Q3, Q4, Q5, Q6, Q7: MPN SI4778DY-T1-GE3 -> STS8DNF3LL
- R10, R13, R14, R23, R24, R27, R29, R302, R303, R304, R31, R9: symbol elias-rescue:US_R0402-Very_Resistor -> Device:R_Small
- R104: value 120, DNP -> 120,DNF; DESCRIPTION (none) -> RES 120 OHM 1% 1/10W 0603; MPN (none) -> RMCF0603FT120R
- R18: value 12K 1% -> 12k; DESCRIPTION (none) -> RES 12K OHM 1% 1/10W 0603; MPN (none) -> RMCF0603FT12K0
- R2, R8: value R_Small -> 5.1k; DESCRIPTION (none) -> RES 5.1K OHM 1% 1/10W 0603; MPN (none) -> RMCF0603FT5K10
- R6, R7: DESCRIPTION RES 27.4 OHM 5% 1/10W 0603 -> RES 27.4 OHM 1% 1/10W 0603; MPN (none) -> RMCF0603FT27R4
- TP2: DESCRIPTION (none) -> +3.3V rail test point
- TP3: DESCRIPTION (none) -> +1.8V rail test point
- U10: DESCRIPTION (none) -> RP2040TR13; MPN (none) -> SC0914(13)
- U2: DESCRIPTION (none) -> IC TRANSCEIVER HALF 1/1 8SOIC
- U311: symbol elias-rescue:NC7WZ126-Very_Buffer -> NC7WZ126K8X:NC7WZ126K8X; OC_FARNELL (none) -> 1417647; OC_NEWARK (none) -> 34C1587; PACKAGE (none) -> SO-8; SUPPLIER (none) -> FAIRCHILD SEMICONDUCTOR
- U5: DESCRIPTION (none) -> IC CAN CONTROLLER W/SPI 20TSSOP
- U7: DESCRIPTION (none) -> IC FLASH 128MBIT SPI/QUAD 8SOIC; MPN (none) -> W25Q128JVS
- U8: DESCRIPTION (none) -> IC CAN CONTROLLER W/SPI 18SOIC
- U9: DESCRIPTION 12mA RGB SMD,5.4x5x1.65mm Light Emitting Diodes (LED) ROHS -> 12mA RGB SMD,5.4x5x1.65mm Light Emitting Diodes (LED) ROHS
- Y2: DESCRIPTION CRYSTAL 16.0000MHZ 22PF SMD -> CRYSTAL 16.0000MHZ 8PF SMD; MPN SXT22422AA27-16.000MT -> FA-20H 16.0000MF10Z-AJ5
Connections:
- net +3V3: now also R11.2, R12.2
- net GND: now also C21.1, C22.2; no longer C21.2, C22.1, R10.2, R13.2, R14.2, R23.2, R24.2, R27.2, R29.2, R302.2, R303.2, R304.2, R31.2, R9.2
- net GPO_1: no longer R303.1
- net GPO_2: no longer R31.1
- net GPO_3: no longer R304.1
- net GPO_4: no longer R29.1
- net GPO_5: no longer R23.1
- net GPO_6: no longer R302.1
- net GPO_7: no longer R14.1
- net GPO_8: no longer R10.1
- net GPO_9: no longer R13.1
- net I2C1_SCL: now also R12.1
- net I2C1_SDA: now also R11.1
- net LEDB: no longer R27.1
- net LEDG: no longer R24.1
- net LEDR: no longer R9.1
- net MCP_OSC1: now also C22.1; no longer C22.2
- net MCP_OSC2: now also C21.2; no longer C21.1
- net PICO_USB_DM: now also J5.2 (SWDIO); no longer J5.3 (RXD)
- net TXD0: now also U311.3 (Y2); no longer U311.5 (A2)
- net at J311.2 (SWDIO): now also U311.5 (A2)
- net at J311.3 (NRESET): no longer U311.3 (Y2)
Other:
- note added: "CAN"
- note added: "CONNECTOR"
- note added: "I2C Pullups not sure if required"
- note added: "RP2040 RPROC"
- note removed: "GPS NEO-M8N BDS Compass Receiver Module"
- note removed: "PICO RPROC"
- note removed: "POWER INPUT"
- moved on the sheet: C10, C11, C12, C13, C14, C15, C16, C17, C18, C19, C2, C20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
