File: hardware/CONEPROJ.kicad_pcb (KiCad board)
At the start: 4 copper layers, 86 x 100 mm, 102 parts, among them J2 693071020811, J304 U.FL-R-SMT-1(10), J306 RGB OUT, J311 TC2030-IDC, J4 DTM1312PA12PBR008, J5 TC2030-IDC, J6 UC-31PFFP-QS8001, Q2 Q_Dual_NMOS_S1G1S2G2D2D2D1D1, Q3 Q_Dual_NMOS_S1G1S2G2D2D2D1D1, Q4 Q_Dual_NMOS_S1G1S2G2D2D2D1D1, Q5 Q_Dual_NMOS_S1G1S2G2D2D2D1D1, Q6 Q_Dual_NMOS_S1G1S2G2D2D2D1D1, Q7 Q_Dual_NMOS_S1G1S2G2D2D2D1D1, U10 RP2040, U2 SN65HVD230, U304 AP1509, U310 RFM69HCW, U311 SN74LVC2G126DCUR, U5 MCP2515-xST, U6 RT9742GGJ5, U7 W25Q128JVS, U8 MCP2515-xSO, U9 WS2815B, Y2 16mhz, Y3 12mhz

Commit message: almost done
Parts:
- removed C303: 0.1uF, Capacitor_SMD:C_0603_1608Metric_Pad1.08x0.95mm_HandSolder
- removed C304: 10uF, Capacitor_SMD:C_0805_2012Metric_Pad1.18x1.45mm_HandSolder
- removed J306: RGB OUT, Connector_JST:JST_XH_S5B-XH-A-1_1x05_P2.50mm_Horizontal
- added C2: 10uF, Capacitor_SMD:C_0805_2012Metric_Pad1.18x1.45mm_HandSolder, F.Cu at (33.5, 55.4)
- added C20: 0.1uF, Capacitor_SMD:C_0603_1608Metric_Pad1.08x0.95mm_HandSolder, F.Cu at (35.4, 55.2)
- moved D1 3.33 mm to (25.4, 59.5), turned to 90 degrees
Connections:
- J4 pad B6: VCC -> /VIN
Routing:
- net /LEDA_OUT: track 0.00 -> 48.7 mm, vias 0 -> 1
- net /I2C1_SDA: track 107.4 -> 152.7 mm, vias 3 -> 5
- net /I2C1_SCL: track 107.6 -> 147.2 mm, vias 3 -> 5
- net VCC: track 18.3 -> 53.0 mm, vias 0 -> 4
- net /RXD3: track 74.7 -> 89.4 mm
- net GND: track 234.6 -> 247.8 mm, vias 53 -> 61
- net /TXD3: track 76.8 -> 88.8 mm
- net /CANH: track 4.90 -> 14.4 mm
- net +5V: track 139.3 -> 131.4 mm, vias 1 -> 8
- net /CANL: track 5.13 -> 12.1 mm
- net /VIN: track 0.00 -> 6.04 mm
- net /GPO_8_OUT: track 0.00 -> 3.07 mm
- net /GPO_7_OUT: track 0.00 -> 2.99 mm
- net /G_OUT: track 6.46 -> 7.50 mm
- net /GPO_9_OUT: track 4.02 -> 5.02 mm
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
Commit message: Can't change it now!
Parts:
- moved TP3 0.90 mm to (77.6, 110.4)
- moved TP2 0.25 mm to (75.5, 110.2)
Routing:
- net GND: track 247.8 -> 246.0 mm
- net /SD_DAT1: track 33.2 -> 31.4 mm
- net /SD_CMD: track 41.4 -> 40.5 mm
- net /GPO_3: track 55.8 -> 56.5 mm
- net +5V: track 131.4 -> 130.7 mm
- net /SD_CLK: track 35.2 -> 34.6 mm
- net /LED_GRN: track 34.8 -> 35.4 mm
- net /SD_PWR_ON: track 35.8 -> 36.3 mm
