File: hardware/carrier/CONEPROJ.kicad_sch (KiCad schematic)
At the start: 85 parts, among them J2 Conn_02x15_Odd_Even_Shielded, J3 Conn_02x15_Odd_Even_Shielded, J304 U.FL-R-SMT-1(10), J4 DTM1312PA12PBR008, J5 TC2030-IDC, J6 UC-31PFFP-QS8001, J7 Conn_02x15_Odd_Even_Shielded, J8 Conn_02x15_Odd_Even_Shielded, Q2 Q_Dual_NMOS_S1G1S2G2D2D2D1D1, Q3 Q_Dual_NMOS_S1G1S2G2D2D2D1D1, Q4 Q_Dual_NMOS_S1G1S2G2D2D2D1D1, Q5 Q_Dual_NMOS_S1G1S2G2D2D2D1D1, Q6 Q_Dual_NMOS_S1G1S2G2D2D2D1D1, Q7 Q_Dual_NMOS_S1G1S2G2D2D2D1D1, U10 RP2040, U2 SN65HVD230, U304 AP1509, U310 RFM69HCW, U5 MCP2515-xST, U7 W25Q128JVS, U8 MCP2515-xSO, U9 WS2815B, Y2 16mhz, Y3 12mhz

Commit message: backup
Parts:
- removed J3, J7, J8: Conn_02x15_Odd_Even_Shielded, TE_DTM1312PA12PBR008:PinSocket_2x16_P1.27mm_Vertical_SMD, symbol Connector_Generic_Shielded:Conn_02x15_Odd_Even_Shielded
- removed J6: UC-31PFFP-QS8001, AMPHENOL_UC-31PFFP-QS8001:AMPHENOL_UC-31PFFP-QS8001, symbol AMPHENOL_UC-31PFFP-QS8001:UC-31PFFP-QS8001
- removed R2, R8: 5.1k, Resistor_SMD:R_0603_1608Metric_Pad0.98x0.95mm_HandSolder, symbol Device:R_Small
- added JP2, JP3: Jumper_2_Open, Jumper:SolderJumper-2_P1.3mm_Open_RoundedPad1.0x1.5mm, symbol Jumper:Jumper_2_Open
Connections:
- net MCP_INT is gone; now on net EXT_IO3: U5.13 (~{INT}), U8.12 (~{INT})
- net RF69_INT is gone; now on net EXT_IO1: U310.14 (DIO0)
- net RF69_MISO is gone; now on net EXT_SPI_MISO: U310.2 (MISO)
- net RF69_MOSI is gone; now on net EXT_SPI_MOSI: U310.3 (MOSI)
- net RF69_NSS is gone; now on net EXT_SPI_SS0: U310.5 (NSS)
- net RF69_RESET is gone; now on net EXT_IO2: U310.6 (RESET)
- net RF69_SCK is gone; now on net EXT_SPI_SCK: U310.4 (SCK)
- net RXD3 is gone; now on net EXT_UART_RX: J4.B12
- net SPI0_CE0_N is gone; now on net EXT_SPI_SS1: U5.18 (~{CS}), U8.16 (~{CS})
- net SPI0_MISO is gone; now on net EXT_SPI_MISO: U5.17 (SO), U8.15 (SO)
- net SPI0_MOSI is gone; now on net EXT_SPI_MOSI: U5.16 (SI), U8.14 (SI)
- net SPI0_SCLK is gone; now on net EXT_SPI_SCK: U5.14 (SCK), U8.13 (SCK)
- net TXD3 is gone; now on net EXT_UART_TX: J4.B11
- net VIN is gone; now on net EXT_12V: C3.1, D2.1 (K), J4.B6, U304.1 (VIN)
- net +3V3: now also J2.3 (Pin_3)
- net +5V: now also J2.4 (Pin_4)
- net GND: now also J2.1 (Pin_1)
- net GPO_1: no longer U10.16 (GPIO13)
- net GPO_2: no longer U10.15 (GPIO12)
- net GPO_3: no longer U10.14 (GPIO11)
- net GPO_4: no longer U10.11 (GPIO8)
- net GPO_5: no longer U10.12 (GPIO9)
- net GPO_6: no longer U10.13 (GPIO10)
- net GPO_7: no longer U10.2 (GPIO0)
- net GPO_8: no longer U10.3 (GPIO1)
- net GPO_9: no longer U10.4 (GPIO2)
- net LEDA: no longer U10.17 (GPIO14)
- net LEDB: no longer U10.9 (GPIO7)
- net LEDG: no longer U10.8 (GPIO6)
- net LEDR: no longer U10.5 (GPIO3)
- net EXT_IO1: now reaches J2.10 (Pin_10)
- net EXT_UART_TX: now reaches J2.11 (Pin_11)
- net EXT_IO2: now reaches J2.12 (Pin_12)
- net EXT_UART_RTS: now reaches J2.13 (Pin_13)
- net EXT_IO3: now reaches J2.14 (Pin_14)
- net EXT_UART_CTS: now reaches J2.15 (Pin_15)
- net EXT_IO4: now reaches J2.16 (Pin_16)
- net EXT_IO5: now reaches J2.18 (Pin_18)
- net EXT_12V: now reaches J2.2 (Pin_2)
- net EXT_SPI_MISO: now reaches J2.20 (Pin_20)
- net EXT_SPI_MOSI: now reaches J2.22 (Pin_22)
- net EXT_SPI_SCK: now reaches J2.24 (Pin_24)
- net EXT_SPI_SS0: now reaches J2.26 (Pin_26)
- net EXT_I2C_SCL: now reaches J2.27 (Pin_27)
- net EXT_I2C_SCL: now also J4.B10, R12.1, JP3.1 (A)
- net EXT_SPI_SS1: now reaches J2.28 (Pin_28)
- net EXT_I2C_SDA: now reaches J2.29 (Pin_29)
- net EXT_I2C_SDA: now also J4.B9, R11.1, JP2.1 (A)
- net EXT_SPI_SS2: now reaches J2.30 (Pin_30)
- net EXT_CAN_TX: now reaches J2.6 (Pin_6)
- net EXT_CAN_RX: now reaches J2.8 (Pin_8)
- net EXT_UART_RX: now reaches J2.9 (Pin_9)
- removed net I2C1_SCL: J4.B10, R12.1, U10.7 (GPIO5)
- removed net I2C1_SDA: J4.B9, R11.1, U10.6 (GPIO4)
- new net RP2040_I2C_SCL: JP3.2 (B), U10.8 (GPIO6)
- new net RP2040_I2C_SDA: JP2.2 (B), U10.7 (GPIO5)
- new net RP2040_SPI_CSn: U10.3 (GPIO1)
- new net RP2040_SPI_RX: U10.2 (GPIO0)
- new net RP2040_SPI_SCK: U10.4 (GPIO2)
- new net RP2040_SPI_TX: U10.5 (GPIO3)
- no-connect marks 38 -> 31
Other:
- note removed: "I2C Pullups not sure if required"
- moved on the sheet: C302, J304, U310

Commit message: asdf
Parts:
- removed JP2, JP3: Jumper_2_Open, Jumper:SolderJumper-2_P1.3mm_Open_RoundedPad1.0x1.5mm, symbol Jumper:Jumper_2_Open
- removed R10, R13, R14, R23, R24, R27, R29, R302, R303, R304, R31, R9: 100k, Resistor_SMD:R_0603_1608Metric_Pad0.98x0.95mm_HandSolder, symbol Device:R_Small
- J2: symbol Connector_Generic_Shielded:Conn_02x15_Odd_Even_Shielded -> Connector_Generic_Shielded:Conn_02x16_Odd_Even_Shielded
Connections:
- net EXT_IO4 is gone; now on net GND: J2.16 (Pin_16)
- net EXT_IO5 is gone; now on net GND: J2.18 (Pin_18)
- net EXT_SPI_SS2 is gone; now on net EXT_SPI_SS0: J2.30 (Pin_30)
- net EXT_UART_CTS is gone; now on net +3V3: J2.15 (Pin_15)
- net EXT_UART_RTS is gone; now on net +3V3: J2.13 (Pin_13)
- net RP2040_I2C_SCL is gone; now on net LEDG: U10.8 (GPIO6)
- net RP2040_I2C_SDA is gone; now on net EXT_I2C_SDA: U10.7 (GPIO5)
- net RP2040_SPI_CSn is gone; now on net GPO_8: U10.3 (GPIO1)
- net RP2040_SPI_SCK is gone; now on net GPO_9: U10.4 (GPIO2)
- net RP2040_SPI_TX is gone; now on net LEDR: U10.5 (GPIO3)
- net +3V3: now also J2.17 (Pin_17), J2.2 (Pin_2); no longer J2.3 (Pin_3)
- net +5V: now also J2.1 (Pin_1), J2.3 (Pin_3); no longer J2.4 (Pin_4)
- net CAN_RX: now also J2.11 (Pin_11)
- net CAN_TX: now also J2.9 (Pin_9)
- net EXT_12V: now also J2.27 (Pin_27), J2.29 (Pin_29); no longer J2.2 (Pin_2)
- net EXT_CAN_RX: no longer J2.8 (Pin_8)
- net EXT_CAN_TX: no longer J2.6 (Pin_6)
- net EXT_I2C_SCL: now also J2.12 (Pin_12), U10.6 (GPIO4); no longer J2.27 (Pin_27)
- net EXT_I2C_SDA: now also J2.10 (Pin_10); no longer J2.29 (Pin_29)
- net EXT_IO1: now also J2.31 (Pin_31); no longer J2.10 (Pin_10)
- net EXT_IO2: now also J2.32 (Pin_32); no longer J2.12 (Pin_12)
- net EXT_IO3: now also J2.20 (Pin_20); no longer J2.14 (Pin_14)
- net EXT_SPI_MISO: now also J2.24 (Pin_24), U10.27 (GPIO16); no longer J2.20 (Pin_20)
- net EXT_SPI_MOSI: now also J2.26 (Pin_26), U10.30 (GPIO19); no longer J2.22 (Pin_22)
- net EXT_SPI_SCK: now also J2.28 (Pin_28), U10.29 (GPIO18); no longer J2.24 (Pin_24)
- net EXT_SPI_SS0: no longer J2.26 (Pin_26)
- net EXT_SPI_SS1: now also J2.22 (Pin_22), U10.28 (GPIO17); no longer J2.28 (Pin_28)
- net EXT_UART_RX: now also J2.5 (Pin_5); no longer J2.9 (Pin_9)
- net EXT_UART_TX: now also J2.7 (Pin_7); no longer J2.11 (Pin_11)
- net GND: now also J2.14 (Pin_14); no longer J2.1 (Pin_1)
- net GPO_4: now also U10.11 (GPIO8)
- net LEDB: now also U10.9 (GPIO7)
- net LED_GRN: now also J2.4 (Pin_4)
- net LED_RED: now also J2.8 (Pin_8)
- net MODE_BTN: now also J2.19 (Pin_19)
- net PAUSE_BTN: now also J2.21 (Pin_21)
- net WIFI_LED: now also J2.6 (Pin_6)

Commit message: almost Finish carrier board
Connections:
- net RP2040_SPI_RX is gone; now on net GPO_7: U10.2 (GPIO0)
- net +5V: now also J4.B5
- net EXT_12V: now also J2.23 (Pin_23), J2.25 (Pin_25); no longer J2.27 (Pin_27), J2.29 (Pin_29)
- net EXT_IO1: now also J2.27 (Pin_27); no longer J2.31 (Pin_31)
- net EXT_IO3: now also U10.18 (GPIO15)
- net GPO_1: now also U10.16 (GPIO13)
- net GPO_2: now also U10.15 (GPIO12)
- net GPO_3: now also U10.14 (GPIO11)
- net GPO_6: now also U10.13 (GPIO10)
- net LEDA: now also U10.17 (GPIO14)
- net PICO_USB__P: now reaches R6.1, U10.47 (USB_DP)
- net GPO_12: now reaches U10.12 (GPIO9)
- net PICO_USB__N: now reaches R7.2, U10.46 (USB_DM)
- net EXT_IO4: now reaches J4.B4
- net EXT_IO4: now also J2.29 (Pin_29)
- net EXT_IO5: now reaches J4.B8
- net EXT_IO5: now also J2.31 (Pin_31)
- net PICO_USB_N: now reaches J5.3 (NRESET)
- net PICO_USB_N: now also R7.1
- net PICO_USB_DM: no longer names the net of J5.2 (SWDIO)
- net PICO_USB_DM: no longer R7.1
- net PICO_USB_DP renamed PICO_USB_P
- no-connect marks 31 -> 30
Other:
- moved on the sheet: R6, R7

Commit message: Add 3v3 regulator for carrier board
Parts:
- added C25, C26: 10uF, Capacitor_SMD:C_0805_2012Metric_Pad1.18x1.45mm_HandSolder, symbol Device:C_Small
- added D4: D_Small, Diode_SMD:D_SOD-123, symbol Device:D_Small
- added L2: 6.8uH, Inductor_SMD:L_Bourns_SRN6045TA, symbol Device:L_Small
- added R2, R8: 10k, Resistor_SMD:R_0603_1608Metric_Pad0.98x0.95mm_HandSolder, symbol Device:R_Small
- added TP2: vbat_sense, TestPoint:TestPoint_Pad_D1.0mm, symbol Connector:TestPoint
- added U3: AP1509, AP1509-50SG-13:SO08, symbol AP1509-50SG-13:AP1509-50SG-13
Connections:
- net GPO_12 is gone; now on net GPO_5: U10.12 (GPIO9)
- net +3V3: now also C26.1, L2.2, U3.2 (VOUT)
- net EXT_12V: now also C25.1, R2.1, U3.1 (VIN)
- net GND: now also C25.2, C26.2, D4.2 (A), R8.2, U3.4 (SD), U3.5 (GND5), U3.6 (GND6), U3.7 (GND7), U3.8 (GND8); no longer U304.4 (SD)
- net 5V_EN: now reaches U10.31 (GPIO20)
- net 5V_EN: now also U304.4 (SD)
- net VBAT_SENSE: now reaches U10.32 (GPIO21)
- net VBAT_SENSE: now also U10.38 (GPIO26_ADC0), R2.2, R8.1, TP2.1
- new net: D4.1 (K), L2.1, U3.3 (FB)
- no-connect marks 30 -> 33
Other:
- moved on the sheet: C3, C5, D1, D2, L1, U304

Commit message: Add motor controller for popups or whatever
Parts:
- removed Q3, Q4: Q_Dual_NMOS_S1G1S2G2D2D2D1D1, Package_SO:SO-8_3.9x4.9mm_P1.27mm, symbol Device:Q_Dual_NMOS_S1G1S2G2D2D2D1D1
- added C27: 470nf, Capacitor_SMD:C_0805_2012Metric_Pad1.18x1.45mm_HandSolder, symbol Device:C_Small
- added C28: 10nf, Capacitor_SMD:C_0805_2012Metric_Pad1.18x1.45mm_HandSolder, symbol Device:C_Small
- added C29, C30: 100nf, Capacitor_SMD:C_0805_2012Metric_Pad1.18x1.45mm_HandSolder, symbol Device:C_Small
- added C31: 10uf, Capacitor_SMD:CP_Elec_5x5.9, symbol Device:C_Polarized_Small
- added U4: DRV8844PWP, IC_TPS61196PWPRQ1, symbol DRV8844PWP:DRV8844PWP
Connections:
- net GND: now also C27.2, C30.2, C31.2, U4.14 (VNEG-2), U4.19 (LGND), U4.2 (VNEG-1), U4.29 (VNEG)
- net GPO_1: now also U4.26 (EN1)
- net GPO_1_OUT: now also U4.5 (OUTPUT1)
- net GPO_2_OUT: now also U4.7 (OUTPUT2)
- net GPO_3_OUT: now also U4.8 (OUTPUT3)
- net GPO_6_OUT: now also U4.10 (OUTPUT4)
- new net: C29.1, U4.3 (VCP)
- new net: C29.2, C30.1, C31.1, U4.11 (VM), U4.4 (VM-1)
- new net: C28.1, U4.1 (CP1)
- new net: C28.2, U4.2 (VNEG-1)
- new net: C27.1, U4.15 (V3P3OUT)
- no-connect marks 33 -> 35

Commit message: Finish motor driver
Parts:
- removed Q6: Q_Dual_NMOS_S1G1S2G2D2D2D1D1, Package_SO:SO-8_3.9x4.9mm_P1.27mm, symbol Device:Q_Dual_NMOS_S1G1S2G2D2D2D1D1
- C28: value 10nf -> 0.01uf
- C29: value 100nf -> 0.1uf
- C30: value 100nf -> 10uf
Connections:
- net GPO_2 is gone; now on net EN2: U10.15 (GPIO12)
- net GPO_3 is gone; now on net EN3: U10.14 (GPIO11)
- net GPO_4 is gone; now on net EN4: U10.11 (GPIO8)
- net GND: now also U4.28 (VNEG), U4.30 (GND), U4.31 (GND), U4.32 (GND), U4.33 (GND), U4.34 (GND), U4.35 (GND), U4.36 (GND), U4.37 (GND), U4.38 (GND), U4.39 (GND), U4.40 (GND), U4.41 (GND), U4.42 (GND), U4.43 (GND), U4.44 (GND), U4.45 (GND), U4.46 (GND), U4.47 (GND), U4.48 (GND), U4.49 (GND), U4.50 (GND), U4.6 (SRC12), U4.9 (SRC34)
- net GPO_5: now also U4.27 (IN1)
- net GPO_6: now also U4.25 (IN2)
- net GPO_6_OUT: no longer U4.10 (OUTPUT4)
- net MCP_RESET: now also U10.37 (GPIO25)
- net CP1: now reaches C28.1, U4.1 (CP1)
- net CP2: now reaches C28.2, U4.2 (VNEG-1)
- net GPO_11: now reaches U10.34 (GPIO22)
- net GPO_11: now also U4.21 (IN4)
- net GPO_10: now reaches U10.35 (GPIO23)
- net GPO_10: now also U4.23 (IN3)
- net DRV_SLEEP: now reaches U10.36 (GPIO24)
- net DRV_SLEEP: now also U4.17 (NSLEEP)
- net EN4: now reaches U4.20 (EN4)
- net EN3: now reaches U4.22 (EN3)
- net EN2: now reaches U4.24 (EN2)
- net GPO_1 renamed EN1
- net GPO_1_OUT renamed MOTOR1_OUT1
- net GPO_2_OUT renamed MOTOR1_OUT2
- net GPO_3_OUT renamed MOTOR2_OUT1
- net GPO_4_OUT renamed MOTOR2_OUT2
- net MOTOR2_OUT2: now also U4.10 (OUTPUT4)
- no-connect marks 35 -> 32
Other:
- moved on the sheet: C28

Commit message: ughhhhhhhhhhhhhhhhhhhhhhh
Parts:
- removed C2: 10uF, Capacitor_SMD:C_0805_2012Metric_Pad1.18x1.45mm_HandSolder, symbol Device:C_Small
- removed C20: 0.1uF, Capacitor_SMD:C_0603_1608Metric_Pad1.08x0.95mm_HandSolder, symbol Device:C_Small
- removed D1, D4: D_Small, Diode_SMD:D_SOD-123, symbol Device:D_Small
- removed L1: 6.8uH, Inductor_SMD:L_Bourns_SRN6045TA, symbol Device:L_Small
- removed U3, U304: AP1509, AP1509-50SG-13:SO08, symbol AP1509-50SG-13:AP1509-50SG-13
- added C32, C33: 5.6nf, Capacitor_SMD:C_0805_2012Metric_Pad1.18x1.45mm_HandSolder, symbol Device:C_Small
- added C34, C35: 0.1uf, Capacitor_SMD:C_0805_2012Metric_Pad1.18x1.45mm_HandSolder, symbol Device:C_Small
- added C36, C37, C38, C39, C40, C41, C42, C43: DNP, Capacitor_SMD:C_0805_2012Metric_Pad1.18x1.45mm_HandSolder, symbol Device:C_Small
- added L3: 10uh, Inductor_SMD:L_Bourns-SRN6028, symbol Device:L_Small
- added R10, R13: 200k, Resistor_SMD:R_0603_1608Metric_Pad0.98x0.95mm_HandSolder, symbol Device:R_Small
- added R14, R17: 14k, Resistor_SMD:R_0603_1608Metric_Pad0.98x0.95mm_HandSolder, symbol Device:R_Small
- added R18, R20: 52.3k, Resistor_SMD:R_0603_1608Metric_Pad0.98x0.95mm_HandSolder, symbol Device:R_Small
- added R19, R23, R9: 10k, Resistor_SMD:R_0603_1608Metric_Pad0.98x0.95mm_HandSolder, symbol Device:R_Small
- added TP3, TP6: 5VOUT, TestPoint:TestPoint_Pad_D1.0mm, symbol Connector:TestPoint
- added TP4, TP7: 3V3OUT, TestPoint:TestPoint_Pad_D1.0mm, symbol Connector:TestPoint
- added TP5, TP8: 1V8OUT, TestPoint:TestPoint_Pad_D1.0mm, symbol Connector:TestPoint
- added U3, U6: AP64200Q, Package_SO:SOIC-8-1EP_3.9x4.9mm_P1.27mm_EP2.29x3mm_ThermalVias, symbol AP1509-50SG-13:AP64200Q
- C25, C26, C3, C5: value 10uF -> 10uf; DESCRIPTION CAP CER 10UF 16V X5R 0805 -> CAP CER 10UF 25V X5R 0805; MPN CL21A106KOQNNNE -> C0805C106M3PAC7800
- C27: value 470nf -> 0.47uf; DESCRIPTION (none) -> CAP CER 0.47UF 6.3V X7R 0805; MPN (none) -> CGJ4J2X7R0J474K125AA
- C28: DESCRIPTION (none) -> CAP CER SMD 0805 .01UF 100V X7R; MPN (none) -> C0805C103K1RAC7210
- C29: DESCRIPTION (none) -> CAP CER 0.1UF 16V X7R 0805; MPN (none) -> 0805 (2012 Metric) 0,94mm
- C30: DESCRIPTION (none) -> CAP CER 10UF 25V X5R 0805; MPN (none) -> C0805C106M3PAC7800
- C31: DESCRIPTION (none) -> CAP ALUM 10UF 20% 50V SMD; MPN (none) -> 50TZV10M5X6.1
- L2: value 6.8uH -> 10uh; footprint Inductor_SMD:L_Bourns_SRN6045TA -> Inductor_SMD:L_Bourns-SRN6028; DESCRIPTION FIXED IND 6.3UH 3A 46.8 MOHM SMD -> (none); MPN NRS6045T6R3MMGK -> (none)
- U4: DESCRIPTION (none) -> IC MTR DRV BIPOLR 8-60V 28HTSSOP; MPN (none) -> DRV8844PWP
Connections:
- net +1V1: now also TP5.1
- net +3V3: now also C39.1, C41.1, C43.1, L3.2, R20.1, R9.1, TP4.1; no longer C26.1, L2.2
- net +5V: now also L2.2, C38.1, C40.1, C42.1, R18.1, TP3.1; no longer C5.1
- net 5V_EN: now also U3.3 (EN)
- net CAN_RX: now also J2.9 (Pin_9); no longer J2.11 (Pin_11)
- net CAN_TX: now also J2.11 (Pin_11); no longer J2.9 (Pin_9)
- net EXT_12V: now also C25.2, C26.2, C29.2, C3.2, C30.1, C31.1, C5.2, U4.11 (VM), U4.4 (VM-1), U9.2 (VDD), U3.2 (VIN), U6.2 (VIN), U6.3 (EN); no longer C25.1, C3.1, J4.B6
- net GND: now also C25.1, C26.1, C3.1, C5.1, C32.2, C33.2, C36.2, C37.2, C40.2, C41.2, C42.2, C43.2, R10.2, R13.2, R19.2, R23.2, TP6.1, TP7.1, TP8.1, U3.7 (GND), U3.9 (GND), U6.7 (GND), U6.9 (GND); no longer C25.2, C26.2, C3.2, C5.2
- net VCC: now also J4.B6; no longer U9.2 (VDD)
- net at L2.1: now also C34.2, U3.8 (SW)
- net DRV_RESET: now reaches U4.16 (NRESET)
- net DRV_RESET: now also R9.2
- new net: C32.1, R14.2
- new net: C34.1, U3.1 (BST)
- new net: C35.1, U6.1 (BST)
- new net: C35.2, L3.1, U6.8 (SW)
- new net: C36.1, R14.1, U3.6 (COMP)
- new net: R10.1, U3.4 (RT)
- new net: C33.1, R17.2
- new net: C37.1, R17.1, U6.6 (COMP)
- new net: C39.2, R20.2, R23.1, U6.5 (FB)
- new net: C38.2, R18.2, R19.1, U3.5 (FB)
- new net: R13.1, U6.4 (RT)
Other:
- moved on the sheet: C302, D2, J304, U310

Commit message: Submitted for fab.
Future cone, could u squash the last few commits and tag this as a
release
Parts:
- added JP2: LED Voltage Select, Jumper:SolderJumper-3_P1.3mm_Bridged12_RoundedPad1.0x1.5mm_NumberLabels, symbol Jumper:SolderJumper_3_Bridged12
- C32, C33: footprint Capacitor_SMD:C_0805_2012Metric_Pad1.18x1.45mm_HandSolder -> Capacitor_SMD:C_1206_3216Metric; DESCRIPTION (none) -> CAP CER 1206 5.6NF 1000V X7R 10%; MPN (none) -> C1206C562KDRACAUTO
- J304: PACKAGE None -> (none)
- J5: MPN TC2030-USB -> (none)
- L2: DESCRIPTION (none) -> FIXED IND 10UH 1.9A 78 MOHM SMD; MPN (none) -> SRN6028-100M
- L3: value 10uh -> 6.8uh; DESCRIPTION (none) -> FIXED IND 6.8UH 2.2A 63 MOHM SMD; MPN (none) -> SRN6028-6R8M
- R10, R13: DESCRIPTION (none) -> RES 200K OHM 5% 1/10W 0603; MPN (none) -> RMCF0603JT200K
- R14, R17: DESCRIPTION (none) -> RES 14K OHM 1% 1/10W 0603; MPN (none) -> RMCF0603FT14K0
- R18, R20: DESCRIPTION (none) -> RES 52.3K OHM 1% 1/10W 0603; MPN (none) -> RMCF0603FT52K3
- R2: value 10k -> 36k; DESCRIPTION RES 240 OHM 5% 1/10W 0603 -> RES 36K OHM 5% 1/10W 0603; MPN RC0603JR-07240RL -> RMCF0603JT36K0
- TP2: value vbat_sense -> VBAT_SENSE
- U3, U6: DESCRIPTION (none) -> DCDC CONV HV BUCK SO-8EP T&R 4K; MPN (none) -> AP64200QSP-13
Connections:
- net EXT_12V: now also JP2.2 (C); no longer U9.2 (VDD)
- net WS2815B_VCC: now reaches C4.1, U9.1 (VCC)
- net WS2815B_VCC: now also JP2.3 (B)
- net VCC renamed VBAT
- new net WS2815B_VDD: JP2.1 (A), U9.2 (VDD)
Other:
- note added: "CONNECTORS"
- note added: "Internal PCB Edge connector"
- note added: "MOTOR DRIVER"
- note added: "Main outer connector"
- note added: "PCB Antenna would be nice here for use without an SMA connector"
- note added: "Pretty sure the resistor network here needs to be recalculated for 3.3V. Consult Datasheet"
- note added: "Unsure if supply voltage should go to VCC or VDD. Datasheet says VDD but that doesn't make a ton of sense to me. If this part doesn't work, bridge the other half"
- note removed: "CONNECTOR"
- moved on the sheet: C10, C12, C13, C14, C15, C17, C18, C19, C23, C24, C27, C28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
