File: hardware/carrier/CONEPROJ.kicad_pcb (KiCad board)
At the start: 4 copper layers, 86 x 50.5 mm, 103 parts, among them J2 Conn_02x15_Odd_Even_Shielded, J304 U.FL-R-SMT-1(10), J4 DTM1312PA12PBR008, J5 TC2030-IDC, Q2 Q_Dual_NMOS_S1G1S2G2D2D2D1D1, Q5 Q_Dual_NMOS_S1G1S2G2D2D2D1D1, Q7 Q_Dual_NMOS_S1G1S2G2D2D2D1D1, U10 RP2040, U2 SN65HVD230, U3 AP64200Q, U310 RFM69HCW, U4 DRV8844PWP, U5 MCP2515-xST, U6 AP64200Q, U7 W25Q128JVS, U8 MCP2515-xSO, U9 WS2815B, Y2 16mhz, Y3 12mhz

Commit message: :ha:
Parts:
- removed C24: 0.1uF, Capacitor_SMD:C_0603_1608Metric_Pad1.08x0.95mm_HandSolder
- removed C26: 10uf, Capacitor_SMD:C_0805_2012Metric_Pad1.18x1.45mm_HandSolder
- removed C29, C35: 0.1uf, Capacitor_SMD:C_0805_2012Metric_Pad1.18x1.45mm_HandSolder
- removed C302: 10uF, Capacitor_SMD:C_0805_2012Metric_Pad1.18x1.45mm_HandSolder
- removed C31: 10uf, Capacitor_SMD:CP_Elec_5x5.9
- removed C33: 5.6nf, Capacitor_SMD:C_1206_3216Metric
- removed C38, C40: DNP, Capacitor_SMD:C_0805_2012Metric_Pad1.18x1.45mm_HandSolder
- removed C9: 1uF, Capacitor_SMD:C_0603_1608Metric_Pad1.08x0.95mm_HandSolder
- removed D301, D308: GRN, LED_SMD:LED_0603_1608Metric_Pad1.05x0.95mm_HandSolder
- removed D302: RED, LED_SMD:LED_0603_1608Metric_Pad1.05x0.95mm_HandSolder
- removed H304: MountingHole_Pad, MountingHole:MountingHole_3.2mm_M3_DIN965_Pad
- removed J304: U.FL-R-SMT-1(10), U.FL-R-SMT-1_10_:HRS_U.FL-R-SMT-1(10)
- removed L2: 10uh, Inductor_SMD:L_Bourns-SRN6028
- removed MOD301, PAU301: SW_SPST, SW_RS-032G05A3-SMRT:SW_RS-032G05A3-SMRT
- removed Q5, Q7: Q_Dual_NMOS_S1G1S2G2D2D2D1D1, Package_SO:SO-8_3.9x4.9mm_P1.27mm
- removed R104: 120,DNF, Resistor_SMD:R_0603_1608Metric_Pad0.98x0.95mm_HandSolder
- removed R22, R91: 240, Resistor_SMD:R_0603_1608Metric_Pad0.98x0.95mm_HandSolder
- removed TP5, TP8: 1V8OUT, TestPoint:TestPoint_Pad_D1.0mm
- removed TP6: 5VOUT, TestPoint:TestPoint_Pad_D1.0mm
- removed U310: RFM69HCW, XCVR_RFM69HW:XCVR_RFM69HW
- removed U7: W25Q128JVS, Package_SO:SOIC-8_5.23x5.23mm_P1.27mm
- added AE2: Antenna_Shield, RF_Antenna:Texas_SWRA117D_2.4GHz_Left, F.Cu at (29.6, 65.3)
- added C2: 1uF, Capacitor_SMD:C_0402_1005Metric, F.Cu at (44.9, 85.1)
- added C20: C_Small, Capacitor_SMD:C_0402_1005Metric, F.Cu at (28.5, 79.8)
- added C44: 10uf, Capacitor_SMD:C_0805_2012Metric_Pad1.18x1.45mm_HandSolder, F.Cu at (94.8, 58.3)
- added C45: 10uF, Capacitor_SMD:C_0805_2012Metric_Pad1.18x1.45mm_HandSolder, F.Cu at (61.2, 96.3)
- added C46: 0.01uf, Capacitor_SMD:C_0805_2012Metric_Pad1.18x1.45mm_HandSolder, F.Cu at (106.2, 58.3)
- added C47: 10uf, Capacitor_SMD:CP_Elec_5x5.9, F.Cu at (89.5, 65.3)
- added D3: RED, LED_SMD:LED_0603_1608Metric_Pad1.05x0.95mm_HandSolder, F.Cu at (32.2, 102.4)
- added D4: GRN, LED_SMD:LED_0603_1608Metric_Pad1.05x0.95mm_HandSolder, F.Cu at (32.1, 101.0)
- added D5: D_Small, Diode_SMD:D_SOD-123, F.Cu at (89.9, 55.3)
- added J3: DM3AT-SF-PEJM5, Connector_Hirose_SD:HRS_DM3AT-SF-PEJM5, F.Cu at (93.2, 93.4)
- added J6: Conn_ARM_JTAG_SWD_10, Connector:Tag-Connect_TC2050-IDC-NL_2x05_P1.27mm_Vertical, F.Cu at (39.4, 70.5)
- added L4: L_Small, Inductor_SMD:L_0402_1005Metric, F.Cu at (26.4, 79.8)
- added L6: 6.8uh, Inductor_SMD:L_Bourns-SRN6028, F.Cu at (74.0, 72.8)
- added Q3: Q_Dual_NMOS_S1G1S2G2D2D2D1D1, Package_SO:SO-8_3.9x4.9mm_P1.27mm, F.Cu at (76.6, 52.3)
- added Q4: Q_Dual_NMOS_S1G1S2G2D2D2D1D1, Package_SO:SO-8_3.9x4.9mm_P1.27mm, F.Cu at (76.6, 57.6)
- added R24: 10k, Resistor_SMD:R_0402_1005Metric, F.Cu at (89.8, 98.3)
- added R25: 10k, Resistor_SMD:R_0402_1005Metric, F.Cu at (35.6, 107.9)
- added R26: 10k, Resistor_SMD:R_0402_1005Metric, F.Cu at (38.5, 77.0)
- added R27: 10k, Resistor_SMD:R_0402_1005Metric, F.Cu at (37.5, 77.0)
- added R29: 14k, Resistor_SMD:R_0603_1608Metric_Pad0.98x0.95mm_HandSolder, F.Cu at (70.5, 66.0)
- added R30: 36k, Resistor_SMD:R_0402_1005Metric, F.Cu at (85.8, 55.4)
- added R31: 10k, Resistor_SMD:R_0402_1005Metric, F.Cu at (83.8, 55.4)
- added R34: 52.3k, Resistor_SMD:R_0603_1608Metric_Pad0.98x0.95mm_HandSolder, F.Cu at (73.5, 62.3)
- added R35: 10k, Resistor_SMD:R_0603_1608Metric_Pad0.98x0.95mm_HandSolder, F.Cu at (77.2, 63.0)
- added R36: 1k, Resistor_SMD:R_0402_1005Metric, F.Cu at (25.8, 110.6)
- added R37: 1k, Resistor_SMD:R_0402_1005Metric, F.Cu at (26.0, 109.5)
- added R38: 51k, Resistor_SMD:R_0402_1005Metric, F.Cu at (78.0, 116.3)
- added R39: 10k, Resistor_SMD:R_0603_1608Metric_Pad0.98x0.95mm_HandSolder, F.Cu at (93.0, 71.6)
- added R40: 51k, Resistor_SMD:R_0402_1005Metric, F.Cu at (78.0, 117.5)
- added SW2: SW_Push, Connector_CK:PTS810SJG250SMTRLFS, F.Cu at (36.7, 110.8)
- added SW3: SW_Push, Connector_CK:PTS810SJG250SMTRLFS, F.Cu at (43.3, 110.9)
- C10, C14, C4: footprint Capacitor_SMD:C_0603_1608Metric_Pad1.08x0.95mm_HandSolder -> Capacitor_SMD:C_0402_1005Metric
- C11, C16: value 10uF -> 1uF; footprint Capacitor_SMD:C_0805_2012Metric_Pad1.18x1.45mm_HandSolder -> Capacitor_SMD:C_0402_1005Metric
- C12: value 1uF -> 10uF; footprint Capacitor_SMD:C_0603_1608Metric_Pad1.08x0.95mm_HandSolder -> Capacitor_SMD:C_0402_1005Metric
- C13: value 0.1uF -> 1uF; footprint Capacitor_SMD:C_0603_1608Metric_Pad1.08x0.95mm_HandSolder -> Capacitor_SMD:C_0402_1005Metric
- C15: value 0.1uF -> 10uF; footprint Capacitor_SMD:C_0603_1608Metric_Pad1.08x0.95mm_HandSolder -> Capacitor_SMD:C_0402_1005Metric
- C17, C18, C19, C23: value 0.1uF -> C_Small; footprint Capacitor_SMD:C_0603_1608Metric_Pad1.08x0.95mm_HandSolder -> Capacitor_SMD:C_0402_1005Metric
- C21, C22: value 10pF -> C_Small; footprint Capacitor_SMD:C_0603_1608Metric_Pad1.08x0.95mm_HandSolder -> Capacitor_SMD:C_0402_1005Metric
- C27: value 0.47uf -> 10uf
- C28: value 0.01uf -> 1uF; footprint Capacitor_SMD:C_0805_2012Metric_Pad1.18x1.45mm_HandSolder -> Capacitor_SMD:C_0402_1005Metric
- C3: value 10uf -> 0.1uF; footprint Capacitor_SMD:C_0805_2012Metric_Pad1.18x1.45mm_HandSolder -> Capacitor_SMD:C_0402_1005Metric
- C30: value 10uf -> 5.6nf; footprint Capacitor_SMD:C_0805_2012Metric_Pad1.18x1.45mm_HandSolder -> Capacitor_SMD:C_1206_3216Metric
- C32: value 5.6nf -> 0.1uf; footprint Capacitor_SMD:C_1206_3216Metric -> Capacitor_SMD:C_0805_2012Metric_Pad1.18x1.45mm_HandSolder
- C34: value 0.1uf -> DNP
- C37: value DNP -> 1uF; footprint Capacitor_SMD:C_0805_2012Metric_Pad1.18x1.45mm_HandSolder -> Capacitor_SMD:C_0402_1005Metric
- C42: value DNP -> 0.47uf
- C43: value DNP -> 0.1uf
- C5: value 10uf -> 10uF
- C6: value 1uF -> 0.1uF; footprint Capacitor_SMD:C_0603_1608Metric_Pad1.08x0.95mm_HandSolder -> Capacitor_SMD:C_0805_2012Metric_Pad1.18x1.45mm_HandSolder
- C7, C8: value 10pF -> 0.1uF; footprint Capacitor_SMD:C_0603_1608Metric_Pad1.08x0.95mm_HandSolder -> Capacitor_SMD:C_0402_1005Metric
- D2: value D_Small -> GRN; footprint Diode_SMD:D_SOD-123 -> LED_SMD:LED_0603_1608Metric_Pad1.05x0.95mm_HandSolder
- J2: value Conn_02x15_Odd_Even_Shielded -> U.FL-R-SMT-1(10); footprint TE_DTM1312PA12PBR008:PinSocket_2x16_P1.27mm_Vertical_SMD -> U.FL-R-SMT-1_10_:HRS_U.FL-R-SMT-1(10)
- J5: value TC2030-IDC -> USB4120-03-C_REVA; footprint Connector:Tag-Connect_TC2030-IDC-FP_2x03_P1.27mm_Vertical -> Connector_GCT_USB:GCT_USB4120-03-C_REVA
- L3: value 6.8uh -> L_Small; footprint Inductor_SMD:L_Bourns-SRN6028 -> Inductor_SMD:L_0402_1005Metric
- Q2: moved to F.Cu
- R10, R13: value 200k -> 0; footprint Resistor_SMD:R_0603_1608Metric_Pad0.98x0.95mm_HandSolder -> Resistor_SMD:R_0402_1005Metric
- R11, R12: value 1k -> 0; footprint Resistor_SMD:R_0603_1608Metric_Pad0.98x0.95mm_HandSolder -> Resistor_SMD:R_0402_1005Metric; moved to F.Cu
- R14: value 14k -> 1k; footprint Resistor_SMD:R_0603_1608Metric_Pad0.98x0.95mm_HandSolder -> Resistor_SMD:R_0402_1005Metric
- R15, R5: value 1k -> 100k; footprint Resistor_SMD:R_0603_1608Metric_Pad0.98x0.95mm_HandSolder -> Resistor_SMD:R_0402_1005Metric
- R16, R9: value 10k -> 0; footprint Resistor_SMD:R_0603_1608Metric_Pad0.98x0.95mm_HandSolder -> Resistor_SMD:R_0402_1005Metric
- R17: value 14k -> 0; footprint Resistor_SMD:R_0603_1608Metric_Pad0.98x0.95mm_HandSolder -> Resistor_SMD:R_0402_1005Metric
- R18, R20: value 52.3k -> 240
- R19: value 10k -> 240
- R2: value 36k -> 442k; footprint Resistor_SMD:R_0603_1608Metric_Pad0.98x0.95mm_HandSolder -> Resistor_SMD:R_0402_1005Metric; moved to F.Cu
- R21: value 240 -> DNP; footprint Resistor_SMD:R_0603_1608Metric_Pad0.98x0.95mm_HandSolder -> Resistor_SMD:R_0402_1005Metric
- R23: value 10k -> 200k
- R3: value 1k -> 120,DNF; footprint Resistor_SMD:R_0603_1608Metric_Pad0.98x0.95mm_HandSolder -> Resistor_SMD:R_0805_2012Metric
- R4: value 10k,DNF -> 10k; footprint Resistor_SMD:R_0603_1608Metric_Pad0.98x0.95mm_HandSolder -> Resistor_SMD:R_0402_1005Metric
- R6: value 27.4 -> 499; footprint Capacitor_SMD:C_0603_1608Metric_Pad1.08x0.95mm_HandSolder -> Resistor_SMD:R_0402_1005Metric
- R7: value 27.4 -> 0; footprint Capacitor_SMD:C_0603_1608Metric_Pad1.08x0.95mm_HandSolder -> Resistor_SMD:R_0402_1005Metric
- R8: value 10k -> 0; footprint Resistor_SMD:R_0603_1608Metric_Pad0.98x0.95mm_HandSolder -> Resistor_SMD:R_0402_1005Metric; moved to F.Cu
- TP2: value VBAT_SENSE -> CHIP_PU; moved to F.Cu
- TP3: value 5VOUT -> VBAT_SENSE
- U10: value RP2040 -> DRV8844PWP; footprint RP2040:RP2040-QFN-56 -> DRV8844PWP:IC_TPS61196PWPRQ1
- U2: value SN65HVD230 -> ESP-PSRAM32
- U3: value AP64200Q -> SN65HVD230; footprint Package_SO:SOIC-8-1EP_3.9x4.9mm_P1.27mm_EP2.29x3mm_ThermalVias -> Package_SO:SOIC-8_3.9x4.9mm_P1.27mm
- U4: value DRV8844PWP -> ESP32-S3R2; footprint DRV8844PWP:IC_TPS61196PWPRQ1 -> Package_DFN_QFN:QFN-56-1EP_7x7mm_P0.4mm_EP5.6x5.6mm; moved to F.Cu
- U5: value MCP2515-xST -> W25Q128JVS; footprint Package_SO:TSSOP-20_4.4x6.5mm_P0.65mm -> Package_SO:SOIC-8_5.23x5.23mm_P1.27mm
- U6: value AP64200Q -> WS2815B; footprint Package_SO:SOIC-8-1EP_3.9x4.9mm_P1.27mm_EP2.29x3mm_ThermalVias -> WS2815B:worldsemi-WS2815B-MFG
- U8: value MCP2515-xSO -> AP64200Q; footprint Package_SO:SOIC-18W_7.5x11.6mm_P1.27mm -> Package_SO:SOIC-8-1EP_3.9x4.9mm_P1.27mm_EP2.29x3mm_ThermalVias
- U9: value WS2815B -> RFM69HCW; footprint WS2815B:worldsemi-WS2815B-MFG -> XCVR_RFM69HW:XCVR_RFM69HW
- Y2: value 16mhz -> 40MHZ; footprint Crystal:Crystal_SMD_2520-4Pin_2.5x2.0mm -> Crystal:Crystal_SMD_2016-4Pin_2.0x1.6mm
- Y3: value 12mhz -> 32.7k; footprint Crystal:Crystal_SMD_3225-4Pin_3.2x2.5mm_HandSoldering -> Crystal:Crystal_SMD_MicroCrystal_CC7V-T1A-2Pin_3.2x1.5mm
- moved R4 70.2 mm to (44.7, 108.1), turned to 0 degrees
- moved C10 68.6 mm to (30.2, 83.4), turned to 90 degrees
- moved C6 67.2 mm to (37.9, 59.0), turned to 0 degrees
- moved C19 65.6 mm to (36.1, 93.8), turned to -90 degrees
- moved C12 65.4 mm to (29.2, 83.4), turned to 90 degrees
- moved C43 65.4 mm to (102.5, 58.3), turned to 180 degrees
- moved R6 64.1 mm to (39.8, 77.0)
- moved C17 62.2 mm to (28.5, 80.8), turned to 0 degrees
- moved C23 62.1 mm to (37.4, 93.8)
- moved R7 61.2 mm to (35.7, 80.1), turned to -90 degrees
- moved C18 60.0 mm to (35.7, 74.8), turned to 0 degrees
- moved C4 58.2 mm to (50.4, 105.4)
- moved C13 57.8 mm to (32.7, 80.1), turned to 90 degrees
- moved C25 55.2 mm to (83.7, 66.5), turned to 90 degrees
- moved U4 54.1 mm to (37.3, 85.9), turned to 0 degrees
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- renumbered H302 to H1
Connections:
- C10 pad 1: +1V1 -> /VDD3V3
- C11 pad 1: +3V3 -> /VDD3V3
- C12 pad 1: +1V1 -> /VDD3V3
- C13 pad 1: +3V3 -> /VDDA
- C14 pad 1: +3V3 -> /VDDSPI
- C15 pad 1: +3V3 -> /VDDA
- C16 pad 1: +3V3 -> /VDDSPI
- C17 pad 1: +3V3 -> GND
- C17 pad 2: GND -> /LNA_IN
- C18 pad 1: +3V3 -> /XTAL_P
- C19 pad 1: +3V3 -> /RTC_XTAL_P
- C21 pad 2: /MCP_OSC2 -> Net-(C21-Pad2)
- C22 pad 1: /MCP_OSC1 -> /XTAL_N
- C23 pad 1: +3V3 -> /RTC_XTAL_N
- C25 pad 2: /EXT_12V -> /VIN
- C27 pad 1: Net-(C27-Pad1) -> GND
- C27 pad 2: GND -> /VIN
- C28 pad 1: /CP1 -> /VDD3V3
- C28 pad 2: /CP2 -> GND
- C3 pad 1: GND -> /VDDSPI
- C3 pad 2: /EXT_12V -> GND
- C30 pad 1: /EXT_12V -> Net-(C30-Pad1)
- C32 pad 2: GND -> Net-(C32-Pad2)
- C34 pad 2: Net-(C34-Pad2) -> GND
- C36 pad 1: Net-(C36-Pad1) -> +3V3
- C36 pad 2: GND -> Net-(C36-Pad2)
- C39 pad 2: Net-(C39-Pad2) -> GND
- C4 pad 1: /WS2815B_VCC -> /VDDSPI
- C42 pad 1: +5V -> Net-(C42-Pad1)
- C43 pad 1: +3V3 -> Net-(C43-Pad1)
- C43 pad 2: GND -> /VIN
- C5 pad 1: GND -> +3V3
- C5 pad 2: /EXT_12V -> GND
- C6 pad 1: +3V3 -> /WS2815B_VCC
- C7 pad 1: Net-(C7-Pad1) -> /VDDRTC
- C8 pad 1: GND -> /VDDCPU
- C8 pad 2: Net-(C8-Pad2) -> GND
- D2 pad 1: /EXT_12V -> Net-(D2-Pad1)
- D2 pad 2: /VBAT -> +3V3
- J2 pad 1: +5V -> GND
- J2 pad 2: +3V3 -> Net-(J2-Pad2)
- J2 pad 3: +5V -> GND
- J4 pad A1: /MOTOR1_OUT1 -> /GPO1
- J4 pad A10: /R_OUT -> /MOTOR2_OUT2
- J4 pad A11: /G_OUT -> /VBAT
- J4 pad A12: /B_OUT -> GND
- J4 pad A2: /MOTOR1_OUT2 -> /GPO2
- J4 pad A3: /MOTOR2_OUT1 -> /GPO3
- J4 pad A4: /MOTOR2_OUT2 -> /GPO4
- J4 pad A5: /GPO_5_OUT -> /GPO6
- J4 pad A6: /GPO_6_OUT -> /GPO5
- J4 pad A7: /GPO_7_OUT -> /MOTOR1_OUT1
- J4 pad A8: /GPO_8_OUT -> /MOTOR1_OUT2
- J4 pad A9: /GPO_9_OUT -> /MOTOR2_OUT1
- J4 pad B1: /CANL -> unconnected-(J4-PadB1)
- J4 pad B10: /EXT_I2C_SCL -> unconnected-(J4-PadB10)
- J4 pad B11: /EXT_UART_TX -> unconnected-(J4-PadB11)
- J4 pad B12: /EXT_UART_RX -> unconnected-(J4-PadB12)
- J4 pad B2: /CANH -> unconnected-(J4-PadB2)
- J4 pad B3: /LEDA_OUT -> unconnected-(J4-PadB3)
- J4 pad B4: /EXT_IO4 -> unconnected-(J4-PadB4)
- J4 pad B5: +5V -> unconnected-(J4-PadB5)
- J4 pad B6: /VBAT -> unconnected-(J4-PadB6)
- J4 pad B7: GND -> unconnected-(J4-PadB7)
- J4 pad B8: /EXT_IO5 -> unconnected-(J4-PadB8)
- J4 pad B9: /EXT_I2C_SDA -> unconnected-(J4-PadB9)
- JP2 pad 2: /EXT_12V -> /VIN
- L3 pad 1: Net-(C35-Pad2) -> /LNA_IN
- L3 pad 2: +3V3 -> /RF_ANT
- Q2 pad 2: /GPO_9 -> /GPIO_GPO1
- Q2 pad 4: /LEDR -> /GPIO_GPO2
- Q2 pad 5: /R_OUT -> /GPO2
- Q2 pad 6: /R_OUT -> /GPO2
- Q2 pad 7: /GPO_9_OUT -> /GPO1
- Q2 pad 8: /GPO_9_OUT -> /GPO1
- R10 pad 1: Net-(R10-Pad1) -> /SPIWP
- R10 pad 2: GND -> Net-(R10-Pad2)
- R11 pad 1: /EXT_I2C_SDA -> /SPICLK
- R11 pad 2: +3V3 -> Net-(R11-Pad2)
- R12 pad 1: /EXT_I2C_SCL -> /SPIQ
- R12 pad 2: +3V3 -> Net-(R12-Pad2)
- R13 pad 1: Net-(R13-Pad1) -> /SPID
- R13 pad 2: GND -> Net-(R13-Pad2)
- R14 pad 1: Net-(C36-Pad1) -> /GPIO_CAN_EN
- R14 pad 2: Net-(C32-Pad1) -> GND
- R15 pad 1: Net-(R15-Pad1) -> /VDDSPI
- R15 pad 2: GND -> /SPICS0
- R16 pad 1: +3V3 -> /GPIO_USB_D_N
- R16 pad 2: /MCP_RESET -> /USB_D_N
- R17 pad 1: Net-(C37-Pad1) -> /GPIO_USB_D_P
- R17 pad 2: Net-(C33-Pad1) -> /USB_D_P
- R18 pad 1: +5V -> Net-(D2-Pad1)
- R18 pad 2: Net-(C38-Pad2) -> /LED_GRN
- R19 pad 1: Net-(C38-Pad2) -> Net-(D3-Pad1)
- R2 pad 1: /EXT_12V -> /SPICLK_P
- R2 pad 2: /VBAT_SENSE -> GND
- R20 pad 1: +3V3 -> Net-(D4-Pad1)
- R20 pad 2: Net-(C39-Pad2) -> GND
- R21 pad 1: Net-(D302-Pad1) -> /RTC_XTAL_P
- R21 pad 2: GND -> /RTC_XTAL_N
- R23 pad 1: Net-(C39-Pad2) -> Net-(R23-Pad1)
- R3 pad 1: /USB_BOOT -> /CAN_N
- R3 pad 2: /QSPI_SS -> /CAN_P
- R4 pad 1: /QSPI_SS -> /CHIP_PU
- R5 pad 1: Net-(R5-Pad1) -> /SPICS1
- R5 pad 2: Net-(C8-Pad2) -> /VDDSPI
- R6 pad 1: /PICO_USB__P -> /U0TXD
- R6 pad 2: /PICO_USB_P -> Net-(R6-Pad2)
- R7 pad 1: /PICO_USB_N -> /XTAL_N
- R7 pad 2: /PICO_USB__N -> Net-(R7-Pad2)
- R8 pad 1: /VBAT_SENSE -> /RTC_XTAL_N
- R8 pad 2: GND -> Net-(R8-Pad2)
- R9 pad 1: +3V3 -> /SPIHD
- R9 pad 2: /DRV_RESET -> Net-(R9-Pad2)
- TP2 pad 1: /VBAT_SENSE -> /CHIP_PU
- TP3 pad 1: +5V -> /GPIO2
- TP4 pad 1: +3V3 -> GND
- TP7 pad 1: GND -> +3V3
- U10 pad 1: +3V3 -> /CP1
- U10 pad 10: +3V3 -> /MOTOR2_OUT2
- U10 pad 11: /EN4 -> /VIN
- U10 pad 12: /GPO_5 -> unconnected-(U10-Pad12)
- U10 pad 13: /GPO_6 -> unconnected-(U10-Pad13)
- U10 pad 14: /EN3 -> GND
- U10 pad 15: /EN2 -> Net-(C42-Pad1)
- U10 pad 16: /EN1 -> /DRV_RESET
- U10 pad 17: /LEDA -> /DRV_SLEEP
- U10 pad 18: /EXT_IO3 -> unconnected-(U10-Pad18)
- U10 pad 2: /GPO_7 -> /CP2
- U10 pad 20: Net-(C7-Pad1) -> /EN4
- U10 pad 21: Net-(R5-Pad1) -> /GPO_11
- U10 pad 22: +3V3 -> /EN3
- U10 pad 23: +1V1 -> /GPO_10
- U10 pad 24: unconnected-(U10-Pad24) -> /EN2
- U10 pad 25: unconnected-(U10-Pad25) -> /GPO_6
- U10 pad 26: unconnected-(U10-Pad26) -> /EN1
- U10 pad 27: /EXT_SPI_MISO -> /GPO_5
- U10 pad 28: /EXT_SPI_SS1 -> GND
- U10 pad 29: /EXT_SPI_SCK -> GND
- U10 pad 3: /GPO_8 -> Net-(C43-Pad1)
- U10 pad 30: /EXT_SPI_MOSI -> GND
- U10 pad 31: /5V_EN -> GND
- U10 pad 32: /VBAT_SENSE -> GND
- U10 pad 33: +3V3 -> GND
- U10 pad 34: /GPO_11 -> GND
- U10 pad 35: /GPO_10 -> GND
- U10 pad 36: /DRV_SLEEP -> GND
- U10 pad 37: /MCP_RESET -> GND
- U10 pad 38: /VBAT_SENSE -> GND
- U10 pad 39: unconnected-(U10-Pad39) -> GND
- U10 pad 4: /GPO_9 -> /VIN
- U10 pad 40: unconnected-(U10-Pad40) -> GND
- U10 pad 41: unconnected-(U10-Pad41) -> GND
- U10 pad 42: +3V3 -> GND
- U10 pad 43: +3V3 -> GND
- U10 pad 44: +3V3 -> GND
- U10 pad 45: +1V1 -> GND
- U10 pad 46: /PICO_USB__N -> GND
- U10 pad 47: /PICO_USB__P -> GND
- U10 pad 48: +3V3 -> GND
- U10 pad 49: +3V3 -> GND
- U10 pad 5: /LEDR -> /MOTOR1_OUT1
- U10 pad 50: +1V1 -> GND
- U10 pad 6: /EXT_I2C_SCL -> GND
- U10 pad 7: /EXT_I2C_SDA -> /MOTOR1_OUT2
- U10 pad 8: /LEDG -> /MOTOR2_OUT1
- U10 pad 9: /LEDB -> GND
- U2 pad 1: /CAN_TX -> /SPICS1
- U2 pad 2: GND -> /SPID
- U2 pad 3: +3V3 -> /SPIWP
- U2 pad 4: /CAN_RX -> GND
- U2 pad 5: unconnected-(U2-Pad5) -> /SPIQ
- U2 pad 6: /CANL -> /SPICLK
- U2 pad 7: /CANH -> /SPIHD
- U2 pad 8: Net-(R15-Pad1) -> /VDDSPI
- U3 pad 1: Net-(C34-Pad1) -> /GPIO_CAN_P
- U3 pad 2: /EXT_12V -> GND
- U3 pad 3: /5V_EN -> +3V3
- U3 pad 4: Net-(R10-Pad1) -> /GPIO_CAN_N
- U3 pad 5: Net-(C38-Pad2) -> unconnected-(U3-Pad5)
- U3 pad 6: Net-(C36-Pad1) -> /CAN_N
- U3 pad 7: GND -> /CAN_P
- U3 pad 8: Net-(C34-Pad2) -> /GPIO_CAN_EN
- U4 pad 1: /CP1 -> /LNA_IN
- U4 pad 10: /MOTOR2_OUT2 -> /GPIO5
- U4 pad 11: /EXT_12V -> /GPIO6
- U4 pad 12: unconnected-(U4-Pad12) -> /DC
- U4 pad 13: unconnected-(U4-Pad13) -> /BL
- U4 pad 14: GND -> /FSPICS1
- U4 pad 15: Net-(C27-Pad1) -> /GPIO10
- U4 pad 16: /DRV_RESET -> /GPIO11
- U4 pad 17: /DRV_SLEEP -> /GPIO12
- U4 pad 18: unconnected-(U4-Pad18) -> /GPIO13
- U4 pad 19: GND -> /GPIO14
- U4 pad 2: /CP2 -> /VDD3V3
- U4 pad 20: /EN4 -> /VDDRTC
- U4 pad 21: /GPO_11 -> /RTC_XTAL_P
- U4 pad 22: /EN3 -> Net-(R8-Pad2)
- U4 pad 23: /GPO_10 -> /CAN_N
- U4 pad 24: /EN2 -> /CAN_P
- U4 pad 25: /GPO_6 -> /GPIO_USB_D_N
- U4 pad 26: /EN1 -> /GPIO_USB_D_P
- U4 pad 27: /GPO_5 -> /CAN_EN
- U4 pad 28: GND -> /SPICS1
- U4 pad 29: GND -> /VDDSPI
- U4 pad 3: Net-(C29-Pad1) -> /VDD3V3
- U4 pad 30: GND -> Net-(R9-Pad2)
- U4 pad 31: GND -> Net-(R10-Pad2)
- U4 pad 32: GND -> /SPICS0
- U4 pad 33: GND -> Net-(R11-Pad2)
- U4 pad 34: GND -> Net-(R12-Pad2)
- U4 pad 35: GND -> Net-(R13-Pad2)
- U4 pad 36: GND -> /SPICLK_N
- U4 pad 37: GND -> /SPICLK_P
- U4 pad 38: GND -> /FSPIHD
- U4 pad 39: GND -> /FSPICS0
- U4 pad 4: /EXT_12V -> /CHIP_PU
- U4 pad 40: GND -> /FSPID
- U4 pad 41: GND -> /FSPICLK
- U4 pad 42: GND -> /FSPIQ
- U4 pad 43: GND -> /GPIO38
- U4 pad 44: GND -> /MTCK
- U4 pad 45: GND -> /MTDO
- U4 pad 46: GND -> /VDDCPU
- U4 pad 47: GND -> /MTDI
- U4 pad 48: GND -> /MTMS
- U4 pad 49: GND -> Net-(R6-Pad2)
- U4 pad 5: /MOTOR1_OUT1 -> /GPIO0
- U4 pad 50: GND -> /U0RXD
- U4 pad 6: GND -> /GPIO1
- U4 pad 7: /MOTOR1_OUT2 -> /GPIO2
- U4 pad 8: /MOTOR2_OUT1 -> /GPIO3
- U4 pad 9: GND -> /GPIO4
- U5 pad 1: /CAN_TX -> /SPICS0
- U5 pad 2: /CAN_RX -> /SPIQ
- U5 pad 3: unconnected-(U5-Pad3) -> /SPIWP
- U5 pad 4: unconnected-(U5-Pad4) -> GND
- U5 pad 5: unconnected-(U5-Pad5) -> /SPID
- U5 pad 6: unconnected-(U5-Pad6) -> /SPICLK
- U5 pad 7: unconnected-(U5-Pad7) -> /SPIHD
- U5 pad 8: /MCP_OSC2 -> /VDDSPI
- U6 pad 1: Net-(C35-Pad1) -> /WS2815B_VCC
- U6 pad 2: /EXT_12V -> /WS2815B_VDD
- U6 pad 3: /EXT_12V -> /LEDA_OUT
- U6 pad 4: Net-(R13-Pad1) -> /LEDA
- U6 pad 5: Net-(C39-Pad2) -> GND
- U6 pad 6: Net-(C37-Pad1) -> /LEDA
- U8 pad 1: /CAN_TX -> Net-(C32-Pad1)
- U8 pad 2: /CAN_RX -> /VIN
- U8 pad 3: unconnected-(U8-Pad3) -> /VIN
- U8 pad 4: unconnected-(U8-Pad4) -> Net-(R23-Pad1)
- U8 pad 5: unconnected-(U8-Pad5) -> Net-(C36-Pad2)
- U8 pad 6: unconnected-(U8-Pad6) -> Net-(C34-Pad1)
- U8 pad 7: /MCP_OSC2 -> GND
- U8 pad 8: /MCP_OSC1 -> Net-(C32-Pad2)
- U9 pad 1: /WS2815B_VCC -> GND
- U9 pad 2: /WS2815B_VDD -> /FSPIQ
- U9 pad 3: /LEDA_OUT -> /FSPID
- U9 pad 4: /LEDA -> /FSPICLK
- U9 pad 5: GND -> /FSPICS1
- U9 pad 6: /LEDA -> /RF69_RESET
- Y2 pad 1: /MCP_OSC1 -> /XTAL_P
- Y2 pad 3: /MCP_OSC2 -> /XTAL_N
- Y3 pad 1: Net-(C8-Pad2) -> /RTC_XTAL_P
- Y3 pad 2: GND -> /RTC_XTAL_N
Routing:
- net /EXT_12V: track 140.8 -> 0.00 mm, vias 19 -> 0
- net /EXT_I2C_SDA: track 110.6 -> 0.00 mm, vias 4 -> 0
- net /EXT_I2C_SCL: track 106.1 -> 0.00 mm, vias 4 -> 0
- net /CAN_TX: track 90.7 -> 0.00 mm, vias 2 -> 0
- net /CAN_RX: track 89.7 -> 0.00 mm, vias 2 -> 0
- net GND: track 144.0 -> 60.0 mm, vias 46 -> 42
- net +3V3: track 94.7 -> 13.6 mm, vias 21 -> 15
- net /EXT_UART_RX: track 80.9 -> 0.00 mm, vias 2 -> 0
- net /EXT_UART_TX: track 78.6 -> 0.00 mm, vias 2 -> 0
- net /5V_EN: track 78.2 -> 0.00 mm, vias 6 -> 0
- net /FSPIQ: track 0.00 -> 72.3 mm, vias 0 -> 4
- net /VBAT_SENSE: track 71.3 -> 0.00 mm, vias 5 -> 0
- net /EXT_SPI_MOSI: track 70.4 -> 0.00 mm, vias 4 -> 0
- net /EXT_SPI_SCK: track 68.8 -> 0.00 mm, vias 4 -> 0
- net /EXT_SPI_MISO: track 67.9 -> 0.00 mm, vias 4 -> 0
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- added copper zone on F.Cu, net /MOTOR1_OUT1
- added copper zone on F.Cu, net /MOTOR1_OUT2
- added copper zone on F.Cu, net /MOTOR2_OUT1
- added copper zone on F.Cu, net /MOTOR2_OUT2
- added copper zone on F.Cu, net /VBAT
- added copper zone on B.Cu, net /VIN
- added copper zone on F.Cu, net /VIN
- added copper zone on In2.Cu, net /VIN
- added copper zone on F.Cu, net Net-(C30-Pad1)
- added copper zone on F.Cu, net Net-(C32-Pad2)
- added copper zone on F.Cu, net Net-(C36-Pad2)
- added copper zone on F.Cu, net Net-(R23-Pad1)
- removed copper zone on F.Cu, net (none)
- removed copper zone on B.Cu, net +3V3
- removed copper zone on F.Cu, net +5V
- removed copper zone on In2.Cu, net +5V
- removed copper zone on B.Cu, net /B_OUT
- removed copper zone on B.Cu, net /EXT_12V
- removed copper zone on F.Cu, net /EXT_12V
- removed copper zone on In1.Cu, net /EXT_12V
- removed copper zone on In2.Cu, net /EXT_12V
- removed copper zone on B.Cu, net /GPO_7_OUT
- removed copper zone on B.Cu, net /GPO_8_OUT
- removed copper zone on B.Cu, net /GPO_9_OUT
- removed copper zone on B.Cu, net /G_OUT
- removed copper zone on B.Cu, net /MOTOR1_OUT1
- removed copper zone on B.Cu, net /MOTOR1_OUT2
- removed copper zone on B.Cu, net /MOTOR2_OUT1
- removed copper zone on B.Cu, net /MOTOR2_OUT2
- removed copper zone on B.Cu, net /R_OUT
- removed copper zone on B.Cu, net GND
- removed copper zone on In2.Cu, net GND
- removed copper zone on F.Cu, net Net-(C33-Pad1)
- removed copper zone on F.Cu, net Net-(C34-Pad2)
- removed copper zone on F.Cu, net Net-(C35-Pad1)
- removed copper zone on F.Cu, net Net-(C35-Pad2)
- removed copper zone on F.Cu, net Net-(C36-Pad1)
- removed copper zone on F.Cu, net Net-(C37-Pad1)
- removed copper zone on F.Cu, net Net-(C38-Pad2)
- removed copper zone on F.Cu, net Net-(C39-Pad2)
- removed copper zone on F.Cu, net Net-(R10-Pad1)
- removed copper zone on F.Cu, net Net-(R13-Pad1)
Other:
- board size 86 x 50.5 mm -> 86 x 114.1 mm
- board text removed: "+1V8"
- board text removed: "+3V3"
- board text removed: "+5V"
- board text removed: "12V"
- board text removed: "12v"
- board text removed: "3v3"
- board text removed: "5V"
- board text removed: "5v"
- board text removed: "BLU"
- board text removed: "BTN 1"
- board text removed: "BTN 2"
- board text removed: "Button 1"
- board text removed: "Button 2"
- board text removed: "CAN"
- board text removed: "CAN RGB CONTROLLER V3 Designed by Connor Rigby 2022"
- board text removed: "CAN RX"
- board text removed: "CAN TX"
- board text removed: "CANH"
- board text removed: "CANL"
- board text removed: "EXT IO3"
- board text removed: "EXT IO4"
- board text removed: "GND"
- board text removed: "GPO7"
- board text removed: "GPO8"
- board text removed: "GPO9"
- board text removed: "GRN"
- board text removed: "IO4"
- board text removed: "IO5"
- board text removed: "JLCJLCJLCJLC"
- board text removed: "LED 1"
- board text removed: "LED 2"
- board text removed: "LED 3"
- board text removed: "LEDA"
- board text removed: "LOW SIDE DRIVERS"
- board text removed: "M1 1"
- board text removed: "M1 2"
- board text removed: "M2 1"
- board text removed: "M2 2"
- board text removed: "MCP CS"
- board text removed: "MCP INT"
- board text removed: "MISO"
- board text removed: "MOSI"
- board text removed: "MOTOR CONTROL"
- board text removed: "POWER I/O"
- board text removed: "Probably don't need to remove the soldermask"
- board text removed: "RADIO CS"
- board text removed: "RADIO INT"
- board text removed: "RADIO RST"
- board text removed: "RED"
- board text removed: "RP2040 DEBUG"
- board text removed: "RX"
- board text removed: "SCL"
- board text removed: "SCLK"
- board text removed: "SDA"
- board text removed: "TX"
- board text removed: "VBATT"
- board text removed: "VDD VBAT VCC"
- board text removed: "cap here"
- board text removed: "https://github.com/ConnorRigby"

Commit message: im cry
Parts:
- moved R2 1.13 mm to (43.8, 84.6)
- moved C2 1.06 mm to (43.9, 85.4)
- moved C10 1.01 mm to (29.4, 82.8)
- moved C11 1.01 mm to (27.4, 82.8)
- moved C12 1.01 mm to (28.4, 82.8)
Routing:
- net /FSPICS1: track 37.6 -> 64.5 mm
- net /GPIO0: track 6.39 -> 32.8 mm, vias 0 -> 1
- net /CHIP_PU: track 6.55 -> 32.8 mm, vias 0 -> 1
- net /BL: track 8.06 -> 34.2 mm
- net /GPIO5: track 10.5 -> 35.5 mm
- net /DC: track 9.01 -> 34.0 mm
- net /GPIO6: track 9.61 -> 33.8 mm
- net /GPIO10: track 27.3 -> 4.88 mm
- net /GPIO4: track 11.3 -> 33.4 mm
- net /GPIO11: track 26.5 -> 4.62 mm
- net /GPIO3: track 12.1 -> 33.2 mm
- net /GPIO12: track 25.6 -> 4.76 mm
- net /GPIO2: track 62.0 -> 82.1 mm
- net /GPIO1: track 13.7 -> 32.8 mm
- net GND: track 60.0 -> 63.1 mm
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
Commit message: asdf
Parts:
- moved G*** 49.1 mm to (-13.1, 75.0)
- moved U6 8.17 mm to (37.2, 58.2)
- moved C6 4.84 mm to (37.1, 63.8)
- moved JP2 4.84 mm to (37.0, 61.5)
- moved AE2 4.17 mm to (30.3, 61.2)
- moved R3 2.37 mm to (55.5, 47.8)
- moved C5 2.37 mm to (55.5, 58.8)
- moved R14 2.37 mm to (52.2, 49.9)
- moved U3 2.37 mm to (55.5, 52.6)
- moved J6 0.23 mm to (39.5, 70.3)
Routing:
- net /GPIO10: track 4.88 -> 39.6 mm
- net /GPIO12: track 4.76 -> 35.9 mm
- net /GPIO11: track 4.62 -> 35.4 mm
- net /GPIO13: track 25.3 -> 50.5 mm, vias 1 -> 2
- net /BL: track 34.2 -> 57.2 mm, vias 1 -> 2
- net /DC: track 34.0 -> 55.9 mm, vias 1 -> 2
- net /GPIO6: track 33.8 -> 55.3 mm, vias 1 -> 2
- net /GPIO4: track 33.4 -> 52.1 mm, vias 1 -> 2
- net /GPIO_GPO5: track 33.0 -> 14.4 mm
- net /GPIO5: track 35.5 -> 54.0 mm, vias 1 -> 2
- net /FSPICS1: track 64.5 -> 82.3 mm
- net /GPIO_GPO6: track 34.5 -> 17.4 mm
- net Net-(J3-PadSWA): track 53.3 -> 69.9 mm
- net /CAN_EN: track 4.41 -> 20.3 mm
- net /GPIO_GPO4: track 36.4 -> 20.6 mm
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
Commit message: im the worst
Parts:
- added AE3: Antenna_Shield, RF_Antenna:Texas_SWRA416_868MHz_915MHz, F.Cu at (79.7, 132.6)
- added C24: C_Small, Capacitor_SMD:C_0402_1005Metric, F.Cu at (39.7, 79.2)
- added C26: C_Small, Capacitor_SMD:C_0402_1005Metric, F.Cu at (37.8, 79.2)
- added C29: 0.1uF, Capacitor_SMD:C_0402_1005Metric, F.Cu at (38.8, 63.0)
- added C31: 0.1uF, Capacitor_SMD:C_0402_1005Metric, F.Cu at (41.4, 77.0)
- added C33: 1uF, Capacitor_SMD:C_0402_1005Metric, F.Cu at (42.3, 65.2)
- added C35: 0.1uF, Capacitor_SMD:C_0402_1005Metric, F.Cu at (45.4, 65.2)
- added C38: 1uF, Capacitor_SMD:C_0402_1005Metric, F.Cu at (44.4, 65.2)
- added C40: 0.1uF, Capacitor_SMD:C_0402_1005Metric, F.Cu at (46.7, 72.1)
- added C48: 0.1uF, Capacitor_SMD:C_0402_1005Metric, F.Cu at (40.3, 77.0)
- added C49: 0.1uF, Capacitor_SMD:C_0402_1005Metric, F.Cu at (34.6, 72.0)
- added C50: 0.1uF, Capacitor_SMD:C_0402_1005Metric, F.Cu at (34.6, 68.5)
- added C51: 0.1uF, Capacitor_SMD:C_0402_1005Metric, F.Cu at (40.6, 63.0)
- added C52: 0.1uF, Capacitor_SMD:C_0402_1005Metric, F.Cu at (46.7, 68.0)
- added C9: 0.1uF, Capacitor_SMD:C_0402_1005Metric, F.Cu at (38.8, 60.3)
- added J7: U.FL-R-SMT-1(10), U.FL-R-SMT-1_10_:HRS_U.FL-R-SMT-1(10), F.Cu at (54.3, 132.5)
- added R22: 0, Resistor_SMD:R_0402_1005Metric, F.Cu at (49.8, 133.5)
- added R28: 0, Resistor_SMD:R_0402_1005Metric, F.Cu at (50.3, 133.0)
- added R32: 0, Resistor_SMD:R_0402_1005Metric, F.Cu at (88.5, 123.8)
- added R33: 0, Resistor_SMD:R_0402_1005Metric, F.Cu at (88.5, 124.8)
- added R41: 27R4, Resistor_SMD:R_0402_1005Metric, F.Cu at (44.9, 62.5)
- added R42: 27R4, Resistor_SMD:R_0402_1005Metric, F.Cu at (44.9, 63.6)
- added SW4: SW_Push, SW_RS-032G05A3-SMRT:SW_RS-032G05A3-SMRT, F.Cu at (31.4, 71.5)
- added TC2: TC2030-IDC, Connector:Tag-Connect_TC2030-IDC-NL_2x03_P1.27mm_Vertical, F.Cu at (31.6, 129.1)
- added TC3: TC2030-IDC, Connector:Tag-Connect_TC2030-IDC-NL_2x03_P1.27mm_Vertical, F.Cu at (42.6, 81.2)
- added U11: RP2040, RP2040:RP2040-QFN-56, F.Cu at (40.5, 71.0)
- added U7: W25Q128JVS, Package_SO:SOIC-8_5.23x5.23mm_P1.27mm, F.Cu at (32.2, 61.7)
- added Y4: 40MHZ, Crystal:Crystal_SMD_3225-4Pin_3.2x2.5mm, F.Cu at (38.4, 81.4)
- AE2: footprint RF_Antenna:Texas_SWRA117D_2.4GHz_Left -> RF_Antenna:Texas_SWRA117D_2.4GHz_Right
- R37: value 1k -> 100k
- SW2, SW3: footprint Connector_CK:PTS810SJG250SMTRLFS -> SW_RS-032G05A3-SMRT:SW_RS-032G05A3-SMRT
- U4: footprint Package_DFN_QFN:QFN-56-1EP_7x7mm_P0.4mm_EP5.6x5.6mm -> Package_DFN_QFN:QFN-56-1EP_7x7mm_P0.4mm_EP5.6x5.6mm_ThermalVias
- Y2: footprint Crystal:Crystal_SMD_2016-4Pin_2.0x1.6mm -> Crystal:Crystal_SMD_3225-4Pin_3.2x2.5mm
- moved G*** 103.4 mm to (88.6, 94.1)
- moved AE2 75.4 mm to (49.8, 134.0), turned to 180 degrees
- moved C20 56.6 mm to (50.2, 132.0), turned to 180 degrees
- moved C21 56.2 mm to (47.3, 131.0)
- moved L4 56.0 mm to (49.3, 131.0), turned to 180 degrees
- moved L3 53.8 mm to (49.8, 129.4), turned to -90 degrees
- moved J6 53.1 mm to (31.5, 122.7)
- moved C18 52.4 mm to (46.9, 126.0), turned to -45 degrees
- moved C17 51.9 mm to (50.3, 128.0), turned to 180 degrees
- moved R40 51.9 mm to (34.2, 89.7), turned to -90 degrees
- moved Y2 51.3 mm to (44.7, 127.1), turned to 135 degrees
- moved R38 50.4 mm to (35.3, 89.7), turned to -90 degrees
- moved R37 50.2 mm to (27.0, 59.3), turned to -90 degrees
- moved C22 50.1 mm to (42.0, 128.2), turned to -135 degrees
- moved C11 48.7 mm to (52.4, 124.6), turned to -90 degrees
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Connections:
- AE2 pad 1: /RF_ANT -> Net-(AE2-Pad1)
- C10 pad 1: /VDD3V3 -> +3V3
- C11 pad 1: /VDD3V3 -> +3V3
- C12 pad 1: /VDD3V3 -> +3V3
- C13 pad 1: /VDDA -> +3V3
- C14 pad 1: /VDDSPI -> +3V3
- C15 pad 1: /VDDA -> +3V3
- C16 pad 1: /VDDSPI -> +3V3
- C28 pad 1: /VDD3V3 -> +3V3
- C3 pad 1: /VDDSPI -> +3V3
- C4 pad 1: /VDDSPI -> +3V3
- C7 pad 1: /VDDRTC -> +3V3
- C8 pad 1: /VDDCPU -> +3V3
- J3 pad 4: /VDD3V3 -> +3V3
- J4 pad B1: unconnected-(J4-PadB1) -> /CAN_P
- J4 pad B2: unconnected-(J4-PadB2) -> /CAN_N
- R14 pad 1: /GPIO_CAN_EN -> /GPIO21
- R15 pad 1: /VDDSPI -> +3V3
- R30 pad 2: /GPIO2 -> /VBAT_SENSE
- R31 pad 1: /GPIO2 -> /VBAT_SENSE
- R36 pad 1: /EXT_I2C_SDA -> /RP_SS
- R36 pad 2: +3V3 -> /USB_BOOT
- R37 pad 1: /EXT_I2C_SCL -> +3V3
- R37 pad 2: +3V3 -> /RP_SS
- R5 pad 2: /VDDSPI -> +3V3
- SW2 pad 1: /GPIO0_BOOTSTRAP -> /CHIP_PU
- SW2 pad 2: /GPIO0_BOOTSTRAP -> Net-(C37-Pad1)
- SW3 pad 1: /CHIP_PU -> /GPIO0_BOOTSTRAP
- SW3 pad 2: /CHIP_PU -> GND
- TP3 pad 1: /GPIO2 -> /VBAT_SENSE
- U10 pad 20: /EN4 -> /GPIO11
- U10 pad 21: /GPO_11 -> /GPIO10
- U10 pad 22: /EN3 -> /GPIO8
- U10 pad 23: /GPO_10 -> /GPIO7
- U10 pad 24: /EN2 -> /GPIO6
- U10 pad 25: /GPO_6 -> /GPIO5
- U10 pad 26: /EN1 -> /GPIO4
- U10 pad 27: /GPO_5 -> /GPIO3
- U2 pad 8: /VDDSPI -> +3V3
- U3 pad 1: /GPIO_CAN_P -> /GPIO18
- U3 pad 4: /GPIO_CAN_N -> /GPIO17
- U3 pad 8: /GPIO_CAN_EN -> /GPIO21
- U4 pad 12: /DC -> /GPIO7
- U4 pad 13: /BL -> /GPIO8
- U4 pad 17: /GPIO12 -> /DRV_SLEEP
- U4 pad 2: /VDD3V3 -> +3V3
- U4 pad 20: /VDDRTC -> +3V3
- U4 pad 23: /CAN_N -> /GPIO17
- U4 pad 24: /CAN_P -> /GPIO18
- U4 pad 27: /CAN_EN -> /GPIO21
- U4 pad 29: /VDDSPI -> +3V3
- U4 pad 3: /VDD3V3 -> +3V3
- U4 pad 43: /GPIO38 -> /VBAT_SENSE
- U4 pad 46: /VDDCPU -> +3V3
- U4 pad 55: /VDDA -> +3V3
- U4 pad 56: /VDDA -> +3V3
- U4 pad 7: /GPIO2 -> /RF69_RESET
- U5 pad 8: /VDDSPI -> +3V3
- U9 pad 14: /RF69_INT -> /GPIO1
- U9 pad 9: Net-(J2-Pad2) -> /RF69_RF_ANT
Routing:
- net +3V3: track 13.6 -> 407.8 mm, vias 15 -> 38
- net /VBAT_SENSE: track 0.00 -> 134.8 mm, vias 0 -> 2
- net /FSPID: track 52.9 -> 176.5 mm, vias 0 -> 4
- net /FSPICLK: track 53.1 -> 173.1 mm, vias 0 -> 2
- net /FSPIQ: track 62.9 -> 180.9 mm
- net /GPIO7: track 0.00 -> 91.9 mm
- net /GPIO8: track 0.00 -> 91.0 mm
- net /VIN: track 0.00 -> 80.4 mm, vias 12 -> 13
- net /FSPICS0: track 50.1 -> 130.2 mm, vias 0 -> 2
- net /GPIO17: track 0.00 -> 76.3 mm, vias 0 -> 2
- net /GPIO2: track 75.3 -> 0.00 mm, vias 2 -> 0
- net /GPIO21: track 0.00 -> 71.0 mm, vias 0 -> 2
- net Net-(J3-PadSWA): track 69.9 -> 1.17 mm
- net GND: track 67.2 -> 134.7 mm, vias 81 -> 80
- net /GPIO18: track 0.00 -> 67.3 mm, vias 0 -> 2
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- added copper zone on In2.Cu, net GND
- removed copper zone on In2.Cu, net +3V3
Other:
- board size 86 x 114.1 mm -> 86 x 97.7 mm

Commit message: asdf
Parts:
- removed R38, R40: 51k, Resistor_SMD:R_0402_1005Metric
- added TP10: CS1, TestPoint:TestPoint_Pad_D1.0mm, B.Cu at (63.4, 118.3)
- added TP11: CS2, TestPoint:TestPoint_Pad_D1.0mm, B.Cu at (47.6, 100.3)
- added TP5: MOSI, TestPoint:TestPoint_Pad_D1.0mm, B.Cu at (79.0, 98.3)
- added TP6: MISO, TestPoint:TestPoint_Pad_D1.0mm, B.Cu at (79.0, 94.9)
- added TP8: SCLK, TestPoint:TestPoint_Pad_D1.0mm, B.Cu at (79.0, 96.6)
- added TP9: CS0, TestPoint:TestPoint_Pad_D1.0mm, B.Cu at (79.0, 100.0)
- G***: moved to F.Cu
- J5: value USB4120-03-C_REVA -> Conn_01x10; footprint Connector_GCT_USB:GCT_USB4120-03-C_REVA -> Connector_PinHeader_2.54mm:PinHeader_1x10_P2.54mm_Vertical
- moved J5 61.8 mm to (104.4, 86.2)
- moved R18 55.6 mm to (72.5, 79.7)
- moved D2 55.6 mm to (76.0, 79.7)
- moved D3 51.2 mm to (76.0, 81.4)
- moved R19 51.2 mm to (72.5, 81.4)
- moved D4 50.9 mm to (76.0, 83.1)
- moved R20 50.9 mm to (72.5, 83.1)
- moved TP4 1.99 mm to (69.9, 79.6)
- moved TP7 0.33 mm to (72.1, 77.6)
- moved R36 0.28 mm to (33.4, 66.7)
- moved C47 0.26 mm to (89.7, 65.3)
- moved C2 0.11 mm to (42.5, 112.9)
- moved R2 0.11 mm to (42.5, 112.1)
- moved C26 0.09 mm to (37.8, 79.1)
- moved C24 0.08 mm to (39.7, 79.1)
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Connections:
- net /GPIO11 renamed /EN4
- net /GPIO17 renamed /GPIO_CAN_N
- net /GPIO18 renamed /GPIO_CAN_P
- net /GPIO4 renamed /EN1
- net /GPIO6 renamed /EN2
- net /GPIO8 renamed /EN3
- net /RF69_RESET renamed /GPIO2
- net /U0RXD renamed /TXD
- net /U0TXD renamed /RXD
- net /VBAT_SENSE renamed /GPIO38
- D3 pad 2: /LED_RED -> +3V3
- D4 pad 2: /WIFI_LED -> +3V3
- J3 pad P1: unconnected-(J3-PadP1) -> GND
- J4 pad B12: unconnected-(J4-PadB12) -> /CAN_N
- J4 pad B2: /CAN_N -> unconnected-(J4-PadB2)
- R18 pad 2: /LED_GRN -> GND
- R19 pad 2: GND -> /LED_RED
- R20 pad 2: GND -> /LED_GREEN
- R41 pad 1: unconnected-(R41-Pad1) -> /CONN_RP_USB_D_P
- R42 pad 1: unconnected-(R42-Pad1) -> /CONN_RP_USB_D_N
- U11 pad 26: /RP_RUN -> /GPIO14
- U11 pad 27: unconnected-(U11-Pad27) -> /LED_GREEN
- U11 pad 28: unconnected-(U11-Pad28) -> /LED_RED
- U11 pad 30: unconnected-(U11-Pad30) -> /GPIO13
Routing:
- net /CONN_RP_USB_D_N: track 0.00 -> 84.6 mm, vias 0 -> 3
- net /CONN_RP_USB_D_P: track 0.00 -> 84.6 mm, vias 0 -> 3
- net /USB_D_P: track 0.00 -> 68.2 mm, vias 0 -> 1
- net /USB_D_N: track 0.00 -> 66.4 mm, vias 0 -> 1
- net +3V3: track 407.8 -> 471.6 mm, vias 38 -> 25
- net /GPIO13: track 6.28 -> 57.5 mm, vias 0 -> 2
- net /GPIO14: track 5.81 -> 55.0 mm, vias 0 -> 2
- net /FSPICLK: track 173.1 -> 215.4 mm
- net /FSPID: track 176.5 -> 218.7 mm
- net /FSPIQ: track 180.9 -> 220.4 mm
- net /LED_GREEN: track 0.00 -> 34.8 mm, vias 0 -> 2
- net /LED_RED: track 0.00 -> 32.7 mm, vias 0 -> 2
- net GND: track 134.7 -> 146.6 mm
- net /GPIO_CAN_P: track 67.3 -> 79.1 mm
- net /CAN_N: track 8.70 -> 18.1 mm
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Other:
- outline, holes or cut-outs redrawn
- board text added: "3V3"
- board text added: "CS0"
- board text added: "CS1"
- board text added: "CS2"
- board text added: "ESP D+"
- board text added: "ESP D-"
- board text added: "GND"
- board text added: "GPIO0"
- board text added: "MISO"
- board text added: "MOSI"
- board text added: "RESET"
- board text added: "RFM69"
- board text added: "RP D+"
- board text added: "RP D-"
- board text added: "SCLK"
- board text added: "USB BOOT"
- board text added: "WIFI / BT"

Commit message: Compromises were made
Parts:
- added R38: 10k, Resistor_SMD:R_0402_1005Metric, F.Cu at (35.5, 99.8)
- added TP12: RP_RUN, TestPoint:TestPoint_Pad_D1.0mm, B.Cu at (43.5, 100.3)
- moved G*** 50.5 mm to (38.2, 90.9)
- moved C49 1.15 mm to (34.6, 73.2)
- moved C50 0.32 mm to (34.6, 68.1)
Connections:
- J4 pad B10: unconnected-(J4-PadB10) -> /CONN_B10
- J4 pad B11: unconnected-(J4-PadB11) -> /CONN_B11
- J4 pad B2: unconnected-(J4-PadB2) -> /CONN_B2
- J4 pad B3: unconnected-(J4-PadB3) -> /CONN_B3
- J4 pad B4: unconnected-(J4-PadB4) -> /CONN_RP_USB_D_P
- J4 pad B5: unconnected-(J4-PadB5) -> /USB_D_P
- J4 pad B6: unconnected-(J4-PadB6) -> GND
- J4 pad B7: unconnected-(J4-PadB7) -> +3V3
- J4 pad B8: unconnected-(J4-PadB8) -> /USB_D_N
- J4 pad B9: unconnected-(J4-PadB9) -> /CONN_RP_USB_D_N
- U11 pad 5: unconnected-(U11-Pad5) -> /CONN_B2
- U11 pad 6: unconnected-(U11-Pad6) -> /CONN_B11
- U11 pad 7: unconnected-(U11-Pad7) -> /CONN_B10
- U11 pad 8: unconnected-(U11-Pad8) -> /CONN_B3
Routing:
- net /USB_D_N: track 66.4 -> 135.8 mm
- net /CONN_RP_USB_D_P: track 84.6 -> 153.7 mm
- net /CONN_RP_USB_D_N: track 84.6 -> 152.7 mm
- net /USB_D_P: track 68.2 -> 132.7 mm
- net +3V3: track 471.6 -> 528.9 mm
- net /CONN_B10: track 0.00 -> 36.3 mm, vias 0 -> 1
- net /CONN_B11: track 0.00 -> 35.2 mm, vias 0 -> 1
- net /CONN_B3: track 0.00 -> 29.0 mm, vias 0 -> 1
- net /CONN_B2: track 0.00 -> 27.3 mm, vias 0 -> 1
- net /GPIO14: track 55.0 -> 73.7 mm
- net /VIN: track 80.4 -> 92.2 mm
- net GND: track 146.6 -> 147.2 mm
- added copper zone on F.Cu, net (none)
Other:
- board text added: "CAN H"
- board text added: "CAN L"
- board text added: "CAN RGB Controller V4 Rev A 05/2022"
- board text added: "GPO1"
- board text added: "GPO2"
- board text added: "GPO3"
- board text added: "GPO4"
- board text added: "GPO5"
- board text added: "GPO6"
- board text added: "MOTOR1 A"
- board text added: "MOTOR1 B"
- board text added: "MOTOR2 A"
- board text added: "MOTOR2 B"
- board text added: "RP2040 RUN"
- board text added: "RXD"
- board text added: "SCL"
- board text added: "SDA"
- board text added: "TTL 3V3"
- board text added: "TXD"
- board text added: "USB0 D+"
- board text added: "USB0 D-"
- board text added: "USB1 D+"
- board text added: "USB1 D-"
- board text added: "VBATT"
