File: hardware/platform-esp/platform-esp.kicad_sch (KiCad schematic)
At the start: 56 parts, among them J1 Conn_ARM_JTAG_SWD_10, J2 DM3AT-SF-PEJM5, J3 DEBUG, J4 USB_C_Receptacle_USB2.0, SW1 SW_Push, SW2 SW_Push, U1 W25Q128JVS, U2 ESP-PSRAM32, U3 ESP32-S3R2, Y1 40MHZ, Y2 32.7k

Commit message: ESP Multi Gauge prototype
Parts:
- removed C3, C7: C_Small, Capacitor_SMD:C_0402_1005Metric, symbol Device:C_Small
- removed J2: DM3AT-SF-PEJM5, Connector_Hirose_SD:HRS_DM3AT-SF-PEJM5, symbol Connector_Hirose_SD:DM3AT-SF-PEJM5
- removed J3: DEBUG, Connector:Tag-Connect_TC2030-IDC-FP_2x03_P1.27mm_Vertical, symbol Connector_Generic:Conn_01x05
- removed J4: USB_C_Receptacle_USB2.0, Connector_USB:USB_C_Receptacle_HRO_TYPE-C-31-M-12, symbol Connector:USB_C_Receptacle_USB2.0
- removed R2: DNP, Resistor_SMD:R_0402_1005Metric, symbol Device:R_Small
- removed R8: 0, Resistor_SMD:R_0402_1005Metric, symbol Device:R_Small
- removed Y2: 32.7k, Crystal:Crystal_SMD_MicroCrystal_CC7V-T1A-2Pin_3.2x1.5mm, symbol Device:Crystal_Small
- added C22, C23: 10uf, Capacitor_SMD:C_0805_2012Metric_Pad1.18x1.45mm_HandSolder, symbol Device:C_Small
- added C24: 5.6nf, Capacitor_SMD:C_1206_3216Metric, symbol Device:C_Small
- added C25: 0.1uf, Capacitor_SMD:C_0805_2012Metric_Pad1.18x1.45mm_HandSolder, symbol Device:C_Small
- added C26, C27, C28, C29: DNP, Capacitor_SMD:C_0805_2012Metric_Pad1.18x1.45mm_HandSolder, symbol Device:C_Small
- added C30: 0.1uF, Capacitor_SMD:C_0402_1005Metric, symbol Device:C_Small
- added C32: 10uF, Capacitor_SMD:C_0402_1005Metric, symbol Device:C_Small
- added C33, C34, C35, C36, C37, C38, C39, C40, C41, C42: 1uF, Capacitor_SMD:C_0402_1005Metric, symbol Device:C_Small
- added D1, D10, D11, D2, D3, D4, D5, D8, D9: WS2812B, LED_SMD:LED_WS2812B_PLCC4_5.0x5.0mm_P3.2mm, symbol LED:WS2812B
- added D6: D_Small, Diode_SMD:D_SOD-123F, symbol Device:D_Small
- added J3: PWR_CAN, Connector_JST:JST_GH_BM04B-GHS-TBT_1x04-1MP_P1.25mm_Vertical, symbol Connector:Conn_01x04_Male
- added J4: USB4120-03-C_REVA, Connector_GCT_USB:GCT_USB4120-03-C_REVA, symbol Connector_GCT_USB:USB4120-03-C_REVA
- added J6: TC2030-IDC, Connector:Tag-Connect_TC2030-IDC-NL_2x03_P1.27mm_Vertical, symbol Connector_TDC:TC2030-IDC
- added L4: 6.8uh, Inductor_SMD:L_Bourns-SRN6028, symbol Device:L_Small
- added R21: 200k, Resistor_SMD:R_0603_1608Metric_Pad0.98x0.95mm_HandSolder, symbol Device:R_Small
- added R22: 14k, Resistor_SMD:R_0603_1608Metric_Pad0.98x0.95mm_HandSolder, symbol Device:R_Small
- added R23: 52.3k, Resistor_SMD:R_0603_1608Metric_Pad0.98x0.95mm_HandSolder, symbol Device:R_Small
- added R24: 10k, Resistor_SMD:R_0603_1608Metric_Pad0.98x0.95mm_HandSolder, symbol Device:R_Small
- added R25: 36k, Resistor_SMD:R_0402_1005Metric, symbol Device:R_Small
- added R26, R27: 10k, Resistor_SMD:R_0402_1005Metric, symbol Device:R_Small
- added R29: 0, Resistor_SMD:R_0402_1005Metric, symbol Device:R_Small
- added TP1, TP2: 3V3OUT, TestPoint:TestPoint_Pad_D1.0mm, symbol Connector:TestPoint
- added TP10: DC, TestPoint:TestPoint_Pad_D1.0mm, symbol Connector:TestPoint
- added TP11: RST, TestPoint:TestPoint_Pad_D1.0mm, symbol Connector:TestPoint
- added TP12: BL, TestPoint:TestPoint_Pad_D1.0mm, symbol Connector:TestPoint
- added TP13: VDD3V3, TestPoint:TestPoint_Pad_D1.0mm, symbol Connector:TestPoint
- added TP14: GND, TestPoint:TestPoint_Pad_D1.0mm, symbol Connector:TestPoint
- added TP3: VBAT_SENSE, TestPoint:TestPoint_Pad_D1.0mm, symbol Connector:TestPoint
- added TP4: CHIP_PU, TestPoint:TestPoint_Pad_D1.0mm, symbol Connector:TestPoint
- added TP5: NEO_OUT, TestPoint:TestPoint_Pad_D1.0mm, symbol Connector:TestPoint
- added TP6: FSPID, TestPoint:TestPoint_Pad_D1.0mm, symbol Connector:TestPoint
- added TP7: FSPICS1, TestPoint:TestPoint_Pad_D1.0mm, symbol Connector:TestPoint
- added TP8: FSPIQ, TestPoint:TestPoint_Pad_D1.0mm, symbol Connector:TestPoint
- added TP9: FSPICLK, TestPoint:TestPoint_Pad_D1.0mm, symbol Connector:TestPoint
- added U4: AP64200Q, Package_SO:SOIC-8-1EP_3.9x4.9mm_P1.27mm_EP2.29x3mm_ThermalVias, symbol AP1509-50SG-13:AP64200Q
- added U5: LTC2875-DD, Package_DFN_QFN:DFN-8-1EP_3x3mm_P0.5mm_EP1.66x2.38mm, symbol Interface_CAN_LIN:LTC2875-DD
- AE1: footprint RF_Antenna:Texas_SWRA117D_2.4GHz_Right -> RF_Antenna:Johanson_2450AT18x100
Connections:
- net +3V3: now also C27.1, C28.1, C29.1, C30.1, C32.1, C33.1, C34.1, C35.1, C36.1, C37.1, C38.1, C39.1, C40.1, C41.1, C42.1, L4.2, R23.1, TP13.1, TP2.1, U5.3 (VCC)
- net CHIP_PU: now also TP4.1
- net GND: now also R19.2, R20.2, C22.1, C23.1, C24.2, C26.2, C28.2, C29.2, C30.2, C32.2, C42.2, D1.3 (VSS), D10.3 (VSS), D11.3 (VSS), D2.3 (VSS), D3.3 (VSS), D4.3 (VSS), D5.3 (VSS), D8.3 (VSS), D9.3 (VSS), J3.1 (Pin_1), J4.A1 (GND_A), J4.A12 (GND_A), J4.B1 (GND_B), J4.B12 (GND_B), J6.5 (GND), R21.2, R24.2, R26.2, R27.2, TP1.1, TP14.1, U4.7 (GND), U4.9 (GND), U5.2 (GND), U5.9 (GND)
- net GPIO14: now also R29.1, TP5.1
- net GPIO2: now also R25.2, R26.1, TP3.1
- net GPIO6: now also TP11.1
- net U0RXD: now also J6.4 (TXD)
- net U0TXD: now also J6.3 (RXD)
- net USB_D_N: now also J4.A7 (D1-), J4.B7 (D2-)
- net USB_D_P: now also J4.A6 (D1+), J4.B6 (D2+)
- net RF_ANT: now reaches AE1.1 (A), C5.2, L1.2, L2.1
- net CC2: now reaches R19.1
- net CC2: now also J4.B5 (CC2)
- net CC1: now reaches R20.1
- net CC1: now also J4.A5 (CC1)
- net GPIO17 renamed CAN_N
- net CAN_N: now also U5.4 (RXD)
- net GPIO18 renamed CAN_P
- net CAN_P: now also U5.1 (TXD)
- net GPIO19 renamed GPIO_USB_D_N
- net GPIO20 renamed GPIO_USB_D_P
- net GPIO21 renamed CAN_EN
- net CAN_EN: now also R27.1, U5.8 (RS)
- net GPIO33 renamed FSPIHD
- net GPIO34 renamed FSPICS0
- net GPIO35 renamed FSPID
- net FSPID: now also TP6.1
- net GPIO36 renamed FSPICLK
- net FSPICLK: now also TP9.1
- net GPIO37 renamed FSPIQ
- net FSPIQ: now also TP8.1
- net GPIO7 renamed DC
- net DC: now also TP10.1
- net GPIO8 renamed BL
- net BL: now also TP12.1
- net GPIO9 renamed FSPICS1
- net FSPICS1: now also TP7.1
- net RTC_XTAL_P: no longer names the net of U3.21 (XTAL_32K_P)
- new net: C35.2, D3.1 (VDD)
- new net: D3.2 (DOUT), D4.4 (DIN)
- new net: D2.2 (DOUT), D3.4 (DIN)
- new net: C38.2, D8.1 (VDD)
- new net: D8.2 (DOUT), D9.4 (DIN)
- new net: D5.2 (DOUT), D8.4 (DIN)
- new net: C37.2, D5.1 (VDD)
- new net: C25.1, U4.1 (BST)
- new net: R21.1, U4.4 (RT)
- new net: C27.2, R23.2, R24.1, U4.5 (FB)
- new net: C26.1, R22.1, U4.6 (COMP)
- new net: C25.2, L4.1, U4.8 (SW)
- new net: C40.2, D10.1 (VDD)
- new net: D10.2 (DOUT), D11.4 (DIN)
- new net: D10.4 (DIN), D9.2 (DOUT)
- new net: D4.2 (DOUT), D5.4 (DIN)
- new net: C34.2, D2.1 (VDD)
- new net: D1.2 (DOUT), D2.4 (DIN)
- new net: D1.4 (DIN), R29.2
- new net: C33.2, D1.1 (VDD)
- new net: C24.1, R22.2
- new net: C41.2, D11.1 (VDD)
- new net: C39.2, D9.1 (VDD)
- new net: C36.2, D4.1 (VDD)
- new net: J4.S1 (SHIELD), J4.S2 (SHIELD), J4.S3 (SHIELD), J4.S4 (SHIELD)
- new net CAN_DRV_N: J3.3 (Pin_3), U5.6 (CANL)
- new net CAN_DRV_P: J3.4 (Pin_4), U5.7 (CANH)
- new net EXT_VIN: D6.2 (A), J3.2 (Pin_2)
- new net USB_VBUS: J4.A4 (VBUS_A), J4.A9 (VBUS_A), J4.B4 (VBUS_B), J4.B9 (VBUS_B)
- new net VIN: C22.2, C23.2, D6.1 (K), R25.1, U4.2 (VIN), U4.3 (EN)
- no-connect marks 4 -> 24
Other:
- note added: "Pretty sure the resistor network here needs to be recalculated for 3.3V. Consult Datasheet"
- note added: "SCREEN"
- note removed: "ESP32-S3 SDMMC Host can be configured to use arbitrary GPIOs for each of the signals."
- moved on the sheet: AE1, C1, C10, C11, C12, C13, C14, C15, C16, C17, C18, C19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
