File: hardware/platform-esp/platform-esp.kicad_sch (KiCad schematic)
At the start: 56 parts, among them J1 Conn_ARM_JTAG_SWD_10, J2 DM3AT-SF-PEJM5, J3 DEBUG, J4 USB_C_Receptacle_USB2.0, SW1 SW_Push, SW2 SW_Push, U1 W25Q128JVS, U2 ESP-PSRAM32, U3 ESP32-S3R2, Y1 40MHZ, Y2 32.7k

Commit message: circle pcb go brrrr lmao
Changed lines of the file:
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@@
     (effects (font (size 1.27 1.27)) (justify right bottom))
   )
-  (label "VDDA" (at 184.785 25.4 0)
+  (label "VDDA" (at 253.365 25.4 0)
     (effects (font (size 1.27 1.27)) (justify left bottom))
   )
@@
       (effects (font (size 1.27 1.27)) (justify left bottom) hide)
     )
-    (property "MF" "Hirose" (id 6) (at 234.315 89.535 0)
+    (property "MF" "Hirose" (id 7) (at 234.315 89.535 0)
       (effects (font (size 1.27 1.27)) (justify left bottom) hide)
     )

Commit message: backup
Parts:
- removed J3: DEBUG, Connector:Tag-Connect_TC2030-IDC-FP_2x03_P1.27mm_Vertical, symbol Connector_Generic:Conn_01x05
- removed J4: USB_C_Receptacle_USB2.0, Connector_USB:USB_C_Receptacle_HRO_TYPE-C-31-M-12, symbol Connector:USB_C_Receptacle_USB2.0
- added C22, C23: 10uf, Capacitor_SMD:C_0805_2012Metric_Pad1.18x1.45mm_HandSolder, symbol Device:C_Small
- added C24: 5.6nf, Capacitor_SMD:C_1206_3216Metric, symbol Device:C_Small
- added C25: 0.1uf, Capacitor_SMD:C_0805_2012Metric_Pad1.18x1.45mm_HandSolder, symbol Device:C_Small
- added C26, C27, C28, C29: DNP, Capacitor_SMD:C_0805_2012Metric_Pad1.18x1.45mm_HandSolder, symbol Device:C_Small
- added C30: 0.1uF, Capacitor_SMD:C_0402_1005Metric, symbol Device:C_Small
- added D1, D10, D11, D2, D3, D4, D5, D8, D9: WS2812B, LED_SMD:LED_WS2812B_PLCC4_5.0x5.0mm_P3.2mm, symbol LED:WS2812B
- added J3: Conn_01x04_Male, Connector_JST:JST_GH_BM04B-GHS-TBT_1x04-1MP_P1.25mm_Vertical, symbol Connector:Conn_01x04_Male
- added J4: USB4120-03-C_REVA, Connector_GCT_USB:GCT_USB4120-03-C_REVA, symbol Connector_GCT_USB:USB4120-03-C_REVA
- added J5: DF52-8S-0.8H(21), Connector_Hirose_SD:HIROSE_DF52-8S-0.8H(21), symbol Connector_Hirose_SD:DF52-8S-0.8H(21)
- added J6: TC2030-IDC, Connector:Tag-Connect_TC2030-IDC-NL_2x03_P1.27mm_Vertical, symbol Connector_TDC:TC2030-IDC
- added L4: 6.8uh, Inductor_SMD:L_Bourns-SRN6028, symbol Device:L_Small
- added R21: 200k, Resistor_SMD:R_0603_1608Metric_Pad0.98x0.95mm_HandSolder, symbol Device:R_Small
- added R22: 14k, Resistor_SMD:R_0603_1608Metric_Pad0.98x0.95mm_HandSolder, symbol Device:R_Small
- added R23: 52.3k, Resistor_SMD:R_0603_1608Metric_Pad0.98x0.95mm_HandSolder, symbol Device:R_Small
- added R24: 10k, Resistor_SMD:R_0603_1608Metric_Pad0.98x0.95mm_HandSolder, symbol Device:R_Small
- added R25: 36k, Resistor_SMD:R_0402_1005Metric, symbol Device:R_Small
- added R26, R27: 10k, Resistor_SMD:R_0402_1005Metric, symbol Device:R_Small
- added TP1, TP2: 3V3OUT, TestPoint:TestPoint_Pad_D1.0mm, symbol Connector:TestPoint
- added TP3: VBAT_SENSE, TestPoint:TestPoint_Pad_D1.0mm, symbol Connector:TestPoint
- added U4: AP64200Q, Package_SO:SOIC-8-1EP_3.9x4.9mm_P1.27mm_EP2.29x3mm_ThermalVias, symbol AP1509-50SG-13:AP64200Q
- added U5: LTC2875-DD, Package_DFN_QFN:DFN-8-1EP_3x3mm_P0.5mm_EP1.66x2.38mm, symbol Interface_CAN_LIN:LTC2875-DD
- SW1, SW2: footprint SW_RS-032G05A3-SMRT:SW_RS-032G05A3-SMRT -> (none)
Connections:
- net +3V3: now also C27.1, C28.1, C29.1, C30.1, L4.2, R23.1, TP2.1, U5.3 (VCC)
- net GND: now also R19.2, R20.2, C22.1, C23.1, C24.2, C26.2, C28.2, C29.2, C30.2, J4.A1 (GND_A), J4.A12 (GND_A), J4.B1 (GND_B), J4.B12 (GND_B), J6.5 (GND), R21.2, R24.2, R26.2, R27.2, TP1.1, U4.7 (GND), U4.9 (GND), U5.2 (GND), U5.9 (GND)
- net U0RXD: now also J6.4 (TXD)
- net U0TXD: now also J6.3 (RXD)
- net USB_D_N: now also J4.A7 (D1-), J4.B7 (D2-)
- net USB_D_P: now also J4.A6 (D1+), J4.B6 (D2+)
- net CC2: now reaches R19.1
- net CC2: now also J4.B5 (CC2)
- net CC1: now reaches R20.1
- net CC1: now also J4.A5 (CC1)
- new net: C25.1, U4.1 (BST)
- new net: R21.1, U4.4 (RT)
- new net: C27.2, R23.2, R24.1, U4.5 (FB)
- new net: C26.1, R22.1, U4.6 (COMP)
- new net: C25.2, L4.1, U4.8 (SW)
- new net: C24.1, R22.2
- new net: J5.P1 (SHIELD), J5.P2 (SHIELD)
- new net: J4.A4 (VBUS_A), J4.A9 (VBUS_A)
- new net: J4.B4 (VBUS_B), J4.B9 (VBUS_B)
- new net: J4.S1 (SHIELD), J4.S2 (SHIELD), J4.S3 (SHIELD), J4.S4 (SHIELD)
- new net CAN_DRV_N: U5.6 (CANL)
- new net CAN_DRV_P: U5.7 (CANH)
- new net CAN_EN: R27.1, U5.8 (RS)
- new net CAN_N: U5.4 (RXD)
- new net CAN_P: U5.1 (TXD)
- new net VBAT_SENSE: R25.2, R26.1, TP3.1
- new net VIN: C22.2, C23.2, R25.1, U4.2 (VIN), U4.3 (EN)
- no-connect marks 4 -> 10
Other:
- note added: "Pretty sure the resistor network here needs to be recalculated for 3.3V. Consult Datasheet"
- moved on the sheet: R19

Commit message: ?remind 2 hours to route the screen next
Parts:
- removed J5: DF52-8S-0.8H(21), Connector_Hirose_SD:HIROSE_DF52-8S-0.8H(21), symbol Connector_Hirose_SD:DF52-8S-0.8H(21)
- added C31: 1uF, Capacitor_SMD:C_0402_1005Metric, symbol Device:C_Small
- added R28: 10k, Resistor_SMD:R_0402_1005Metric, symbol Device:R_Small
- J3: value Conn_01x04_Male -> PWR_CAN
Connections:
- net GPIO34 is gone; now on net FSPICS0: U3.39 (GPIO34)
- net GPIO35 is gone; now on net FSPID: U3.40 (GPIO35)
- net GPIO36 is gone; now on net FSPICLK: U3.41 (GPIO36)
- net GPIO37 is gone; now on net FSPIQ: U3.42 (GPIO37)
- net VDD3V3 is gone; now on net +3V3: C13.2, L3.1, U3.2 (VDD3P3), U3.3 (VDD3P3)
- net +3V3: now also J2.4 (VDD), C31.1, R28.1
- net GND: now also J2.6 (VSS), J2.SWB, C31.2
- net FSPICS0: now reaches J2.2 (CD/DAT3)
- net FSPIQ: now reaches J2.3 (CMD)
- net FSPICLK: now reaches J2.5 (CLK)
- net FSPID: now reaches J2.7 (DAT0)
- net at J2.SWA: now also R28.2
- net USB_VBUS: now reaches J4.A4 (VBUS_A), J4.A9 (VBUS_A)
- net USB_VBUS: now also J4.B4 (VBUS_B), J4.B9 (VBUS_B)
- net GPIO33 renamed FSPIHD
- no-connect marks 10 -> 11
Other:
- note added: "SPID = MOSI SPIQ = MISO"

Commit message: asdf
Parts:
- added C32: 10uF, Capacitor_SMD:C_0402_1005Metric, symbol Device:C_Small
- added C33, C34, C35, C36, C37, C38, C39, C40, C41: 1uF, Capacitor_SMD:C_0402_1005Metric, symbol Device:C_Small
- added R29: 0, Resistor_SMD:R_0402_1005Metric, symbol Device:R_Small
Connections:
- net +3V3: now also C32.1, C33.1, C34.1, C35.1, C36.1, C37.1, C38.1, C39.1, C40.1, C41.1
- net GND: now also D1.3 (VSS), D10.3 (VSS), D11.3 (VSS), D2.3 (VSS), D3.3 (VSS), D4.3 (VSS), D5.3 (VSS), D8.3 (VSS), D9.3 (VSS), J3.1 (Pin_1), C32.2
- net VIN: now also J3.2 (Pin_2)
- net at D3.1 (VDD): now also C35.2
- net at D3.2 (DOUT): now also D4.4 (DIN)
- net at D3.4 (DIN): now also D2.2 (DOUT)
- net at D8.1 (VDD): now also C38.2
- net at D8.2 (DOUT): now also D9.4 (DIN)
- net at D8.4 (DIN): now also D5.2 (DOUT)
- net at D10.1 (VDD): now also C40.2
- net at D10.2 (DOUT): now also D11.4 (DIN)
- net at D10.4 (DIN): now also D9.2 (DOUT)
- net at D5.1 (VDD): now also C37.2
- net at D5.4 (DIN): now also D4.2 (DOUT)
- net at D2.1 (VDD): now also C34.2
- net at D2.4 (DIN): now also D1.2 (DOUT)
- net at D1.1 (VDD): now also C33.2
- net at D1.4 (DIN): now also R29.2
- net at D4.1 (VDD): now also C36.2
- net at D9.1 (VDD): now also C39.2
- net at D11.1 (VDD): now also C41.2
Other:
- moved on the sheet: D1, D10, D11, D2, D3, D4, D5, D8, D9, J3

Commit message: fdsa
Parts:
- added C42: 1uF, Capacitor_SMD:C_0402_1005Metric, symbol Device:C_Small
- added TP10: DC, TestPoint:TestPoint_Pad_D1.0mm, symbol Connector:TestPoint
- added TP11: RST, TestPoint:TestPoint_Pad_D1.0mm, symbol Connector:TestPoint
- added TP12: BL, TestPoint:TestPoint_Pad_D1.0mm, symbol Connector:TestPoint
- added TP13: VDD3V3, TestPoint:TestPoint_Pad_D1.0mm, symbol Connector:TestPoint
- added TP14: GND, TestPoint:TestPoint_Pad_D1.0mm, symbol Connector:TestPoint
- added TP4: CHIP_PU, TestPoint:TestPoint_Pad_D1.0mm, symbol Connector:TestPoint
- added TP5: NEO_OUT, TestPoint:TestPoint_Pad_D1.0mm, symbol Connector:TestPoint
- added TP6: FSPID, TestPoint:TestPoint_Pad_D1.0mm, symbol Connector:TestPoint
- added TP7: FSPICS1, TestPoint:TestPoint_Pad_D1.0mm, symbol Connector:TestPoint
- added TP8: FSPIQ, TestPoint:TestPoint_Pad_D1.0mm, symbol Connector:TestPoint
- added TP9: FSPICLK, TestPoint:TestPoint_Pad_D1.0mm, symbol Connector:TestPoint
- AE1: footprint RF_Antenna:Texas_SWRA117D_2.4GHz_Right -> RF_Antenna:Texas_SWRA117D_2.4GHz_Left
Connections:
- net GPIO17 is gone; now on net CAN_N: U3.23 (GPIO17)
- net GPIO18 is gone; now on net CAN_P: U3.24 (GPIO18)
- net GPIO21 is gone; now on net CAN_EN: U3.27 (GPIO21)
- net VBAT_SENSE is gone; now on net GPIO2: R25.2, R26.1, TP3.1
- net +3V3: now also C42.1, TP13.1
- net CAN_DRV_N: now also J3.3 (Pin_3)
- net CAN_DRV_P: now also J3.4 (Pin_4)
- net CHIP_PU: now also TP4.1
- net FSPICLK: now also TP9.1
- net FSPID: now also TP6.1
- net FSPIQ: now also TP8.1
- net GND: now also C42.2, TP14.1
- net GPIO14: now also R29.1, TP5.1
- new net BL: TP12.1
- new net DC: TP10.1
- new net FSPICS1: TP7.1
- new net RST: TP11.1
- no-connect marks 11 -> 29
Other:
- note added: "SCREEN"

Commit message: route diff pairs or whatever idr
Connections:
- net RF_ANT: now reaches AE1.1 (A), C5.2, L1.2, L2.1
- net GPIO19 renamed GPIO_USB_D_N
- net GPIO20 renamed GPIO_USB_D_P
Other:
- moved on the sheet: R14, R15
Changed lines of the file:
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@@
     (stroke (width 0) (type default) (color 0 0 0 0))
   )
-  (wire (pts (xy 160.02 103.505) (xy 175.26 103.505))
+  (wire (pts (xy 160.02 103.505) (xy 182.245 103.505))
     (stroke (width 0) (type default) (color 0 0 0 0))
   )
@@
     (stroke (width 0) (type default) (color 0 0 0 0))
   )
-  (wire (pts (xy 180.34 106.045) (xy 190.5 106.045))
+  (wire (pts (xy 187.325 106.045) (xy 197.485 106.045))
     (stroke (width 0) (type default) (color 0 0 0 0))
   )
@@
     (stroke (width 0) (type default) (color 0 0 0 0))
   )
-  (wire (pts (xy 160.02 106.045) (xy 175.26 106.045))
+  (wire (pts (xy 160.02 106.045) (xy 182.245 106.045))
     (stroke (width 0) (type default) (color 0 0 0 0))
   )
@@
     (stroke (width 0) (type default) (color 0 0 0 0))
   )
-  (wire (pts (xy 180.34 103.505) (xy 190.5 103.505))
+  (wire (pts (xy 187.325 103.505) (xy 197.485 103.505))
     (stroke (width 0) (type default) (color 0 0 0 0))
   )
@@
     (effects (font (size 1.27 1.27)) (justify left bottom))
   )
-  (label "GPIO20" (at 168.91 106.045 180)
-    (effects (font (size 1.27 1.27)) (justify right bottom))
-  )
   (label "FSPICS1" (at 175.895 138.43 0)
     (effects (font (size 1.27 1.27)) (justify left bottom))
   )
-  (label "USB_D_P" (at 190.5 106.045 180)
+  (label "USB_D_P" (at 197.485 106.045 180)
     (effects (font (size 1.27 1.27)) (justify right bottom))
   )
@@
     (effects (font (size 1.27 1.27)) (justify left bottom))
   )
+  (label "GPIO_USB_D_N" (at 170.18 103.505 0)
+    (effects (font (size 1.27 1.27)) (justify left bottom))
+  )
   (label "CC1" (at 319.405 163.195 0)
     (effects (font (size 1.27 1.27)) (justify left bottom))
@@
     (effects (font (size 1.27 1.27)) (justify left bottom))
   )
+  (label "GPIO_USB_D_P" (at 170.18 106.045 0)
+    (effects (font (size 1.27 1.27)) (justify left bottom))
+  )
   (label "FSPICS0" (at 190.5 113.665 180)
     (effects (font (size 1.27 1.27)) (justify right bottom))
@@
     (effects (font (size 1.27 1.27)) (justify left bottom))
   )
+  (label "RF_ANT" (at 34.925 38.735 0)
+    (effects (font (size 1.27 1.27)) (justify left bottom))
+  )
   (label "CAN_DRV_N" (at 320.04 2.54 180)
     (effects (font (size 1.27 1.27)) (justify right bottom))
@@
     (effects (font (size 1.27 1.27)) (justify right bottom))
   )
-  (label "GPIO19" (at 168.91 103.505 180)
-    (effects (font (size 1.27 1.27)) (justify right bottom))
-  )
   (label "CC2" (at 378.46 170.815 180)
     (effects (font (size 1.27 1.27)) (justify right bottom))
@@
     (effects (font (size 1.27 1.27)) (justify left bottom))
   )
-  (label "USB_D_N" (at 190.5 103.505 180)
+  (label "USB_D_N" (at 197.485 103.505 180)
     (effects (font (size 1.27 1.27)) (justify right bottom))
   )
@@
     (pin "1")
   )
-  (symbol (lib_id "Device:R_Small") (at 177.8 106.045 90) (unit 1)
+  (symbol (lib_id "Device:R_Small") (at 184.785 106.045 90) (unit 1)
     (in_bom yes) (on_board yes)
-    (property "Reference" "R15" (id 0) (at 171.45 107.315 90))
-    (property "Value" "0" (id 1) (at 174.625 107.315 90))
-    (property "Footprint" "Resistor_SMD:R_0402_1005Metric" (id 2) (at 177.8 106.045 0)
+    (property "Reference" "R15" (id 0) (at 178.435 107.315 90))
+    (property "Value" "0" (id 1) (at 181.61 107.315 90))
+    (property "Footprint" "Resistor_SMD:R_0402_1005Metric" (id 2) (at 184.785 106.045 0)
       (effects (font (size 1.27 1.27)) hide)
     )
-    (property "Datasheet" "~" (id 3) (at 177.8 106.045 0)
+    (property "Datasheet" "~" (id 3) (at 184.785 106.045 0)
       (effects (font (size 1.27 1.27)) hide)
     )
@@
     (pin "2")
   )
-  (symbol (lib_id "Device:R_Small") (at 177.8 103.505 90) (unit 1)
+  (symbol (lib_id "Device:R_Small") (at 184.785 103.505 90) (unit 1)
     (in_bom yes) (on_board yes)
-    (property "Reference" "R14" (id 0) (at 171.45 104.775 90))
-    (property "Value" "0" (id 1) (at 174.625 104.775 90))
-    (property "Footprint" "Resistor_SMD:R_0402_1005Metric" (id 2) (at 177.8 103.505 0)
+    (property "Reference" "R14" (id 0) (at 178.435 104.775 90))
+    (property "Value" "0" (id 1) (at 181.61 104.775 90))
+    (property "Footprint" "Resistor_SMD:R_0402_1005Metric" (id 2) (at 184.785 103.505 0)
       (effects (font (size 1.27 1.27)) hide)
     )
-    (property "Datasheet" "~" (id 3) (at 177.8 103.505 0)
+    (property "Datasheet" "~" (id 3) (at 184.785 103.505 0)
       (effects (font (size 1.27 1.27)) hide)
     )

Commit message: Guess it's done
Parts:
- added D6: D_Small, Diode_SMD:D_SOD-123F, symbol Device:D_Small
- SW1, SW2: footprint (none) -> PTS810SJG250SMTRLFS; symbol Switch:SW_Push -> Connector_CK:PTS810SJK250SMTRLFS; DESCRIPTION (none) -> IP40 Black Button Tactile Switch, SPST-NO 50 mA 3mm Surface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; MPN (none) -> PTS810SJK250SMTRLFS
Connections:
- net GPIO7 is gone; now on net DC: U3.12 (GPIO7)
- net GPIO8 is gone; now on net BL: U3.13 (GPIO8)
- net GPIO9 is gone; now on net FSPICS1: U3.14 (GPIO9)
- net RST is gone; now on net GPIO6: TP11.1
- net CHIP_PU: now also SW2.1, SW2.2; no longer SW1.1
- net GND: now also SW1.3, SW1.4; no longer SW2.2
- net GPIO0_BOOTSTRAP: now also SW1.1, SW1.2; no longer SW2.1
- net VIN: now also D6.1 (K); no longer J3.2 (Pin_2)
- net at C21.1: now also SW2.3, SW2.4; no longer SW1.2
- new net EXT_VIN: D6.2 (A), J3.2 (Pin_2)
- no-connect marks 29 -> 25
Other:
- moved on the sheet: AE1, C1, C10, C11, C12, C13, C14, C15, C16, C17, C18, C19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

Commit message: restart esp gauge
Parts:
- removed C3, C7: C_Small, Capacitor_SMD:C_0402_1005Metric, symbol Device:C_Small
- removed C31: 1uF, Capacitor_SMD:C_0402_1005Metric, symbol Device:C_Small
- removed J2: DM3AT-SF-PEJM5, Connector_Hirose_SD:HRS_DM3AT-SF-PEJM5, symbol Connector_Hirose_SD:DM3AT-SF-PEJM5
- removed R2: DNP, Resistor_SMD:R_0402_1005Metric, symbol Device:R_Small
- removed R28: 10k, Resistor_SMD:R_0402_1005Metric, symbol Device:R_Small
- removed R8: 0, Resistor_SMD:R_0402_1005Metric, symbol Device:R_Small
- removed SW1, SW2: SW_Push, PTS810SJG250SMTRLFS, symbol Connector_CK:PTS810SJK250SMTRLFS
- removed Y2: 32.7k, Crystal:Crystal_SMD_MicroCrystal_CC7V-T1A-2Pin_3.2x1.5mm, symbol Device:Crystal_Small
- added SW1, SW2: SW_Push, SW_RS-032G05A3-SMRT:SW_RS-032G05A3-SMRT, symbol Switch:SW_Push
- AE1: footprint RF_Antenna:Texas_SWRA117D_2.4GHz_Left -> RF_Antenna:Johanson_2450AT18x100
Connections:
- net +3V3: no longer C13.2, L3.1, U3.2 (VDD3P3), U3.3 (VDD3P3)
- net CHIP_PU: now also SW1.1
- net GND: now also SW2.2
- net GPIO0_BOOTSTRAP: now also SW2.1
- net at C21.1: now also SW1.2
- net RTC_XTAL_P: no longer names the net of U3.21 (XTAL_32K_P)
- new net VDD3V3: C13.2, L3.1, U3.2 (VDD3P3), U3.3 (VDD3P3)
- no-connect marks 25 -> 24
Other:
- note removed: "ESP32-S3 SDMMC Host can be configured to use arbitrary GPIOs for each of the signals."
- note removed: "SPID = MOSI SPIQ = MISO"
- moved on the sheet: C42, TP10, TP11, TP12, TP13, TP14, TP6, TP7, TP8, TP9
