File: hardware/platform-esp/platform-esp.kicad_pcb (KiCad board)
At the start: 2 copper layers, 86 x 50.9 mm, 57 parts, among them J1 Conn_ARM_JTAG_SWD_10, J2 DM3AT-SF-PEJM5, J3 DEBUG, J4 USB_C_Receptacle_USB2.0, SW1 SW_Push, SW2 SW_Push, U1 W25Q128JVS, U2 ESP-PSRAM32, U3 ESP32-S3R2, Y1 40MHZ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

Commit message: circle pcb go brrrr lmao
Parts:
- removed CONN: Conn_02x15_Odd_Even_Shielded, TE_DTM1312PA12PBR008:PinSocket_2x16_P1.27mm_Vertical_SMD
- J1, J2: moved to B.Cu
- moved J3 67.8 mm to (25.5, 24.7)
- moved J1 63.3 mm to (31.8, 24.7), turned to 180 degrees
- moved C8 52.1 mm to (26.8, 43.0), turned to 90 degrees
- moved U1 49.5 mm to (63.8, 31.9), turned to 180 degrees
- moved U2 48.1 mm to (62.8, 24.7), turned to 180 degrees
- moved J2 47.5 mm to (36.6, 37.3)
- moved C12 45.0 mm to (41.7, 26.3), turned to 90 degrees
- moved Y1 44.2 mm to (33.6, 24.3), turned to 45 degrees
- moved C6 43.9 mm to (35.0, 22.8), turned to -45 degrees
- moved C2 43.6 mm to (32.2, 25.7), turned to 135 degrees
- moved R5 43.5 mm to (39.2, 38.0), turned to -90 degrees
- moved C5 43.1 mm to (35.0, 33.0), turned to -45 degrees
- moved L1 43.0 mm to (36.8, 34.0), turned to 180 degrees
- moved C14 42.9 mm to (35.9, 38.0), turned to -90 degrees
- moved J4 42.0 mm to (63.1, 51.8), turned to 45 degrees
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Routing:
- net GND: track 0.00 -> 74.8 mm, vias 0 -> 19
- net +3V3: track 0.00 -> 31.6 mm, vias 0 -> 6
- net /GPIO0_BOOTSTRAP: track 0.00 -> 22.1 mm
- net /MTMS: track 0.00 -> 19.2 mm
- net /CHIP_PU: track 0.00 -> 17.2 mm
- net /MTDI: track 0.00 -> 16.2 mm
- net /MTCK: track 0.00 -> 15.2 mm
- net Net-(AE1-Pad1): track 0.00 -> 14.8 mm
- net /MTDO: track 0.00 -> 14.0 mm
- net /U0RXD: track 0.00 -> 12.2 mm
- net /XTAL_P: track 0.00 -> 11.9 mm
- net /GPIO46: track 0.00 -> 11.7 mm
- net /GPIO17: track 0.00 -> 11.2 mm
- net Net-(C8-Pad2): track 0.00 -> 11.1 mm
- net /GPIO45: track 0.00 -> 11.0 mm
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Other:
- board size 86 x 50.9 mm -> 58.5 x 58.5 mm
- copper layers 2 -> 4
- board text added: "REMEMBER TO IMPEDIANCE MATCH THIS TRACE DUMMY"

Commit message: backup
Parts:
- removed SW1, SW2: SW_Push, SW_RS-032G05A3-SMRT:SW_RS-032G05A3-SMRT
- added C22: 10uf, Capacitor_SMD:C_0805_2012Metric_Pad1.18x1.45mm_HandSolder, F.Cu at (90.2, 68.0)
- added C23: 10uf, Capacitor_SMD:C_0805_2012Metric_Pad1.18x1.45mm_HandSolder, F.Cu at (88.4, 67.9)
- added C24: 5.6nf, Capacitor_SMD:C_1206_3216Metric, F.Cu at (86.6, 55.9)
- added C25: 0.1uf, Capacitor_SMD:C_0805_2012Metric_Pad1.18x1.45mm_HandSolder, F.Cu at (86.0, 57.9)
- added C26: DNP, Capacitor_SMD:C_0805_2012Metric_Pad1.18x1.45mm_HandSolder, F.Cu at (86.6, 53.8)
- added C27: DNP, Capacitor_SMD:C_0805_2012Metric_Pad1.18x1.45mm_HandSolder, F.Cu at (82.2, 66.6)
- added C28: DNP, Capacitor_SMD:C_0805_2012Metric_Pad1.18x1.45mm_HandSolder, F.Cu at (82.2, 57.9)
- added C29: DNP, Capacitor_SMD:C_0805_2012Metric_Pad1.18x1.45mm_HandSolder, F.Cu at (85.6, 66.6)
- added C30: 0.1uF, Capacitor_SMD:C_0402_1005Metric, F.Cu at (78.2, 47.3)
- added D1: WS2812B, LED_SMD:LED_WS2812B_PLCC4_5.0x5.0mm_P3.2mm, B.Cu at (67.7, 41.4)
- added D10: WS2812B, LED_SMD:LED_WS2812B_PLCC4_5.0x5.0mm_P3.2mm, B.Cu at (47.6, 54.3)
- added D11: WS2812B, LED_SMD:LED_WS2812B_PLCC4_5.0x5.0mm_P3.2mm, B.Cu at (55.8, 44.9)
- added D2: WS2812B, LED_SMD:LED_WS2812B_PLCC4_5.0x5.0mm_P3.2mm, B.Cu at (79.5, 44.9)
- added D3: WS2812B, LED_SMD:LED_WS2812B_PLCC4_5.0x5.0mm_P3.2mm, B.Cu at (87.7, 54.3)
- added D4: WS2812B, LED_SMD:LED_WS2812B_PLCC4_5.0x5.0mm_P3.2mm, B.Cu at (89.4, 66.6)
- added D5: WS2812B, LED_SMD:LED_WS2812B_PLCC4_5.0x5.0mm_P3.2mm, B.Cu at (84.3, 77.8)
- added D8: WS2812B, LED_SMD:LED_WS2812B_PLCC4_5.0x5.0mm_P3.2mm, B.Cu at (51.0, 77.8)
- added D9: WS2812B, LED_SMD:LED_WS2812B_PLCC4_5.0x5.0mm_P3.2mm, B.Cu at (45.9, 66.6)
- added J5: DF52-8S-0.8H(21), Connector_Hirose_SD:HIROSE_DF52-8S-0.8H(21), F.Cu at (56.3, 44.8)
- added J6: TC2030-IDC, Connector:Tag-Connect_TC2030-IDC-NL_2x03_P1.27mm_Vertical, F.Cu at (51.6, 49.4)
- added L4: 6.8uh, Inductor_SMD:L_Bourns-SRN6028, F.Cu at (82.7, 62.4)
- added R21: 200k, Resistor_SMD:R_0603_1608Metric_Pad0.98x0.95mm_HandSolder, F.Cu at (77.2, 58.4)
- added R22: 14k, Resistor_SMD:R_0603_1608Metric_Pad0.98x0.95mm_HandSolder, F.Cu at (83.6, 54.7)
- added R23: 52.3k, Resistor_SMD:R_0603_1608Metric_Pad0.98x0.95mm_HandSolder, F.Cu at (82.2, 68.2)
- added R24: 10k, Resistor_SMD:R_0603_1608Metric_Pad0.98x0.95mm_HandSolder, F.Cu at (82.2, 69.5)
- added R25: 36k, Resistor_SMD:R_0402_1005Metric, F.Cu at (85.2, 71.6)
- added R26: 10k, Resistor_SMD:R_0402_1005Metric, F.Cu at (85.2, 70.7)
- added R27: 10k, Resistor_SMD:R_0402_1005Metric, F.Cu at (73.4, 49.5)
- added REF**: 1.28-lcd, Module_Waveshare:1.28-lcd, B.Cu at (67.7, 63.8)
- added TP1: 3V3OUT, TestPoint:TestPoint_Pad_D1.0mm, F.Cu at (79.6, 56.8)
- added TP2: 3V3OUT, TestPoint:TestPoint_Pad_D1.0mm, F.Cu at (79.6, 58.4)
- added TP3: VBAT_SENSE, TestPoint:TestPoint_Pad_D1.0mm, F.Cu at (83.3, 71.1)
- added U4: AP64200Q, Package_SO:SOIC-8-1EP_3.9x4.9mm_P1.27mm_EP2.29x3mm_ThermalVias, F.Cu at (89.4, 62.2)
- added U5: LTC2875-DD, Package_DFN_QFN:DFN-8-1EP_3x3mm_P0.5mm_EP1.66x2.38mm, F.Cu at (75.2, 47.1)
- J3: value DEBUG -> Conn_01x04_Male; footprint Connector:Tag-Connect_TC2030-IDC-FP_2x03_P1.27mm_Vertical -> Connector_JST:JST_GH_BM04B-GHS-TBT_1x04-1MP_P1.25mm_Vertical
- J4: value USB_C_Receptacle_USB2.0 -> USB4120-03-C_REVA; footprint Connector_USB:USB_C_Receptacle_HRO_TYPE-C-31-M-12 -> Connector_GCT_USB:GCT_USB4120-03-C_REVA
- moved C8 63.5 mm to (77.1, 81.8), turned to 180 degrees
- moved AE1 61.7 mm to (72.2, 82.2), turned to 180 degrees
- moved C2 57.7 mm to (59.8, 76.4), turned to -135 degrees
- moved Y1 56.4 mm to (58.3, 75.0), turned to 135 degrees
- moved C6 55.3 mm to (56.9, 73.6), turned to 45 degrees
- moved R18 52.3 mm to (55.2, 70.6), turned to 180 degrees
- moved C5 51.7 mm to (67.1, 73.6), turned to 45 degrees
- moved C15 51.5 mm to (72.0, 73.7), turned to 0 degrees
- moved L2 51.5 mm to (69.1, 73.6), turned to -45 degrees
- moved R17 50.9 mm to (55.3, 69.5), turned to 180 degrees
- moved C4 50.9 mm to (66.1, 72.9), turned to 45 degrees
- moved R7 50.7 mm to (61.6, 71.8), turned to 45 degrees
- moved C14 50.1 mm to (72.0, 72.7), turned to 0 degrees
- moved R6 49.2 mm to (55.3, 68.1), turned to 0 degrees
- moved L1 49.1 mm to (68.0, 71.8), turned to -90 degrees
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Connections:
- J4 pad A1: Net-(J4-PadA1) -> GND
- J4 pad A12: Net-(J4-PadA1) -> GND
- J4 pad A4: Net-(J4-PadA4) -> unconnected-(J4-PadA4)
- J4 pad A5: unconnected-(J4-PadA5) -> /CC1
- J4 pad A9: Net-(J4-PadA4) -> unconnected-(J4-PadA4)
- J4 pad B1: Net-(J4-PadA1) -> GND
- J4 pad B12: Net-(J4-PadA1) -> GND
- J4 pad B4: Net-(J4-PadA4) -> unconnected-(J4-PadB4)
- J4 pad B5: unconnected-(J4-PadB5) -> /CC2
- J4 pad B9: Net-(J4-PadA4) -> unconnected-(J4-PadB4)
- J4 pad S1: unconnected-(J4-PadS1) -> Net-(J4-PadS1)
- R19 pad 1: unconnected-(R19-Pad1) -> /CC2
- R19 pad 2: unconnected-(R19-Pad2) -> GND
- R20 pad 1: unconnected-(R20-Pad1) -> /CC1
- R20 pad 2: unconnected-(R20-Pad2) -> GND
Routing:
- net /SPIWP: track 1.01 -> 32.1 mm, vias 1 -> 4
- net /SPIQ: track 1.09 -> 30.8 mm, vias 1 -> 4
- net /SPICS1: track 4.80 -> 34.0 mm, vias 0 -> 2
- net /SPIHD: track 0.89 -> 26.2 mm, vias 1 -> 4
- net /U0TXD: track 0.00 -> 24.0 mm, vias 0 -> 2
- net /SPID: track 1.26 -> 23.9 mm, vias 1 -> 4
- net /GPIO0_BOOTSTRAP: track 22.1 -> 0.00 mm
- net /SPICLK: track 1.12 -> 23.2 mm, vias 1 -> 4
- net /U0RXD: track 12.2 -> 33.2 mm, vias 0 -> 2
- net /SPICS0: track 6.79 -> 26.9 mm
- net /CAN_N: track 0.00 -> 15.2 mm
- net /CAN_P: track 0.00 -> 10.2 mm
- net /CHIP_PU: track 17.2 -> 7.83 mm, vias 0 -> 1
- net /CAN_DRV_N: track 0.00 -> 8.80 mm
- net /CAN_DRV_P: track 0.00 -> 7.56 mm
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- added copper zone on In2.Cu, net +3V3
- added copper zone on B.Cu, net GND
- added copper zone on In1.Cu, net GND
Other:
- board size 58.5 x 58.5 mm -> 50 x 49.6 mm
- board text added: "DEBUG"
- board text added: "diff pair match"

Commit message: ?remind 2 hours to route the screen next
Parts:
- removed J5: DF52-8S-0.8H(21), Connector_Hirose_SD:HIROSE_DF52-8S-0.8H(21)
- added C31: 1uF, Capacitor_SMD:C_0402_1005Metric, B.Cu at (68.6, 64.2)
- added R28: 10k, Resistor_SMD:R_0402_1005Metric, F.Cu at (76.5, 77.3)
- J3: value Conn_01x04_Male -> PWR_CAN
- moved R24 15.0 mm to (84.6, 54.7), turned to 180 degrees
- moved R23 12.3 mm to (84.6, 56.1), turned to 0 degrees
- moved C28 10.5 mm to (81.1, 68.4), turned to 180 degrees
- moved C25 8.93 mm to (86.7, 66.8), turned to -90 degrees
- moved C27 8.90 mm to (84.2, 58.0), turned to 0 degrees
- moved C24 6.40 mm to (82.2, 51.2), turned to 180 degrees
- moved C29 4.49 mm to (81.1, 66.5), turned to 180 degrees
- moved C26 3.74 mm to (85.5, 50.2), turned to 90 degrees
- moved C21 3.74 mm to (58.4, 77.9), turned to 45 degrees
- moved C23 2.73 mm to (87.7, 70.6)
- moved C22 2.66 mm to (89.6, 70.6)
- moved R22 1.87 mm to (84.7, 53.2), turned to 180 degrees
- moved R26 1.79 mm to (83.5, 70.2)
- moved R25 1.46 mm to (85.5, 70.2)
- moved TP3 1.31 mm to (84.5, 71.6)
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Connections:
- net /GPIO33 renamed /FSPIHD
- C13 pad 2: /VDD3V3 -> +3V3
- J2 pad 2: unconnected-(J2-Pad2) -> /FSPICS0
- J2 pad 3: unconnected-(J2-Pad3) -> /FSPIQ
- J2 pad 4: unconnected-(J2-Pad4) -> +3V3
- J2 pad 5: unconnected-(J2-Pad5) -> /GPIO36
- J2 pad 6: unconnected-(J2-Pad6) -> GND
- J2 pad 7: unconnected-(J2-Pad7) -> /FSPID
- J2 pad P1: Net-(J2-PadP1) -> unconnected-(J2-PadP1)
- J2 pad SWA: unconnected-(J2-PadSWA) -> Net-(J2-PadSWA)
- J2 pad SWB: unconnected-(J2-PadSWB) -> GND
- J4 pad A4: unconnected-(J4-PadA4) -> /USB_VBUS
- J4 pad A9: unconnected-(J4-PadA4) -> /USB_VBUS
- J4 pad B4: unconnected-(J4-PadB4) -> /USB_VBUS
- J4 pad B9: unconnected-(J4-PadB4) -> /USB_VBUS
- L3 pad 1: /VDD3V3 -> +3V3
- U3 pad 2: /VDD3V3 -> +3V3
- U3 pad 3: /VDD3V3 -> +3V3
- U3 pad 39: /GPIO34 -> /FSPICS0
- U3 pad 40: /GPIO35 -> /FSPID
- U3 pad 42: /GPIO37 -> /FSPIQ
Routing:
- net /FSPID: track 0.00 -> 45.9 mm, vias 0 -> 2
- net GND: track 82.2 -> 124.7 mm, vias 18 -> 23
- net /GPIO36: track 7.47 -> 49.7 mm, vias 1 -> 2
- net +3V3: track 38.1 -> 79.9 mm, vias 9 -> 21
- net /FSPIQ: track 0.00 -> 40.4 mm, vias 0 -> 2
- net /VIN: track 0.00 -> 37.7 mm, vias 0 -> 2
- net /FSPICS0: track 0.00 -> 30.2 mm, vias 0 -> 2
- net Net-(R21-Pad1): track 1.39 -> 27.1 mm, vias 1 -> 2
- net /USB_D_P: track 0.00 -> 13.0 mm, vias 0 -> 3
- net /USB_D_N: track 0.00 -> 11.6 mm, vias 0 -> 3
- net Net-(C27-Pad2): track 0.00 -> 11.2 mm, vias 0 -> 2
- net Net-(C26-Pad1): track 0.00 -> 10.1 mm
- net /CC1: track 0.00 -> 9.19 mm
- net /CAN_EN: track 2.53 -> 10.6 mm, vias 0 -> 1
- net /GPIO37: track 8.00 -> 0.00 mm, vias 1 -> 0
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- added copper zone on F.Cu, net +3V3
- added copper zone on F.Cu, net /VBAT_SENSE
- added copper zone on F.Cu, net /VIN
- added copper zone on In2.Cu, net /VIN
- added copper zone on F.Cu, net GND
- added copper zone on In2.Cu, net GND
- added copper zone on F.Cu, net Net-(C25-Pad2)
- added copper zone on In2.Cu, net Net-(C27-Pad2)
Other:
- outline, holes or cut-outs redrawn

Commit message: asdf
Parts:
- added C32: 10uF, Capacitor_SMD:C_0402_1005Metric, B.Cu at (61.0, 44.2)
- added C33: 1uF, Capacitor_SMD:C_0402_1005Metric, B.Cu at (71.3, 41.0)
- added C34: 1uF, Capacitor_SMD:C_0402_1005Metric, B.Cu at (83.4, 47.2)
- added C35: 1uF, Capacitor_SMD:C_0402_1005Metric, B.Cu at (89.1, 58.4)
- added C36: 1uF, Capacitor_SMD:C_0402_1005Metric, B.Cu at (89.2, 70.6)
- added C37: 1uF, Capacitor_SMD:C_0402_1005Metric, B.Cu at (81.8, 81.7)
- added C38: 1uF, Capacitor_SMD:C_0402_1005Metric, B.Cu at (47.0, 75.2)
- added C39: 1uF, Capacitor_SMD:C_0402_1005Metric, B.Cu at (45.2, 62.1)
- added C40: 1uF, Capacitor_SMD:C_0402_1005Metric, B.Cu at (49.2, 50.4)
- added C41: 1uF, Capacitor_SMD:C_0402_1005Metric, B.Cu at (59.5, 42.5)
- added R29: 0, Resistor_SMD:R_0402_1005Metric, B.Cu at (62.4, 43.9)
- U3: footprint Package_DFN_QFN:QFN-56-1EP_7x7mm_P0.4mm_EP5.6x5.6mm -> Package_DFN_QFN:QFN-56-1EP_7x7mm_P0.4mm_EP5.6x5.6mm_ThermalVias
- moved C31 1.96 mm to (67.2, 65.6), turned to 180 degrees
Connections:
- net /GPIO36 renamed /FSPICLK
- D1 pad 1: unconnected-(D1-Pad1) -> Net-(C33-Pad2)
- D1 pad 2: unconnected-(D1-Pad2) -> Net-(D2-Pad4)
- D1 pad 3: unconnected-(D1-Pad3) -> GND
- D1 pad 4: unconnected-(D1-Pad4) -> Net-(D1-Pad4)
- D10 pad 1: unconnected-(D10-Pad1) -> Net-(C40-Pad2)
- D10 pad 2: unconnected-(D10-Pad2) -> Net-(D11-Pad4)
- D10 pad 3: unconnected-(D10-Pad3) -> GND
- D10 pad 4: unconnected-(D10-Pad4) -> Net-(D10-Pad4)
- D11 pad 1: unconnected-(D11-Pad1) -> Net-(C41-Pad2)
- D11 pad 3: unconnected-(D11-Pad3) -> GND
- D11 pad 4: unconnected-(D11-Pad4) -> Net-(D11-Pad4)
- D2 pad 1: unconnected-(D2-Pad1) -> Net-(C34-Pad2)
- D2 pad 2: unconnected-(D2-Pad2) -> Net-(D3-Pad4)
- D2 pad 3: unconnected-(D2-Pad3) -> GND
- D2 pad 4: unconnected-(D2-Pad4) -> Net-(D2-Pad4)
- D3 pad 1: unconnected-(D3-Pad1) -> Net-(C35-Pad2)
- D3 pad 2: unconnected-(D3-Pad2) -> Net-(D3-Pad2)
- D3 pad 3: unconnected-(D3-Pad3) -> GND
- D3 pad 4: unconnected-(D3-Pad4) -> Net-(D3-Pad4)
- D4 pad 1: unconnected-(D4-Pad1) -> Net-(C36-Pad2)
- D4 pad 2: unconnected-(D4-Pad2) -> Net-(D5-Pad4)
- D4 pad 3: unconnected-(D4-Pad3) -> GND
- D4 pad 4: unconnected-(D4-Pad4) -> Net-(D3-Pad2)
- D5 pad 1: unconnected-(D5-Pad1) -> Net-(C37-Pad2)
- D5 pad 2: unconnected-(D5-Pad2) -> Net-(D8-Pad4)
- D5 pad 3: unconnected-(D5-Pad3) -> GND
- D5 pad 4: unconnected-(D5-Pad4) -> Net-(D5-Pad4)
- D8 pad 1: unconnected-(D8-Pad1) -> Net-(D8-Pad1)
- D8 pad 2: unconnected-(D8-Pad2) -> Net-(D9-Pad4)
- D8 pad 3: unconnected-(D8-Pad3) -> GND
- D8 pad 4: unconnected-(D8-Pad4) -> Net-(D8-Pad4)
- D9 pad 1: unconnected-(D9-Pad1) -> Net-(C39-Pad2)
- D9 pad 2: unconnected-(D9-Pad2) -> Net-(D10-Pad4)
- D9 pad 3: unconnected-(D9-Pad3) -> GND
- D9 pad 4: unconnected-(D9-Pad4) -> Net-(D9-Pad4)
- J3 pad 1: unconnected-(J3-Pad1) -> GND
- J3 pad 2: unconnected-(J3-Pad2) -> /VIN
Routing:
- net Net-(D8-Pad4): track 0.00 -> 32.0 mm, vias 0 -> 2
- net +3V3: track 79.9 -> 99.6 mm, vias 21 -> 33
- net Net-(D3-Pad2): track 0.00 -> 11.1 mm, vias 0 -> 2
- net Net-(D9-Pad4): track 0.00 -> 9.73 mm
- net Net-(D3-Pad4): track 0.00 -> 9.40 mm
- net Net-(D10-Pad4): track 0.00 -> 9.07 mm
- net GND: track 124.7 -> 133.6 mm, vias 23 -> 27
- net Net-(D11-Pad4): track 0.00 -> 8.95 mm
- net Net-(D5-Pad4): track 0.00 -> 8.73 mm
- net Net-(D2-Pad4): track 0.00 -> 8.57 mm
- net Net-(D1-Pad4): track 0.00 -> 4.70 mm
- net Net-(C41-Pad2): track 0.00 -> 3.10 mm
- net Net-(C40-Pad2): track 0.00 -> 2.76 mm
- net Net-(C39-Pad2): track 0.00 -> 2.67 mm
- net Net-(C35-Pad2): track 0.00 -> 2.50 mm
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- added copper zone on B.Cu, net +3V3
- added copper zone on In1.Cu, net +3V3
- removed copper zone on In2.Cu, net GND

Commit message: fdsa
Parts:
- added C42: 1uF, Capacitor_SMD:C_0402_1005Metric, F.Cu at (58.9, 78.4)
- added TP10: DC, TestPoint:TestPoint_Pad_D1.0mm, F.Cu at (55.1, 77.6)
- added TP11: RST, TestPoint:TestPoint_Pad_D1.0mm, F.Cu at (56.2, 78.7)
- added TP12: BL, TestPoint:TestPoint_Pad_D1.0mm, F.Cu at (54.0, 76.6)
- added TP13: VDD3V3, TestPoint:TestPoint_Pad_D1.0mm, F.Cu at (57.3, 79.8)
- added TP14: GND, TestPoint:TestPoint_Pad_D1.0mm, F.Cu at (58.3, 80.8)
- added TP4: CHIP_PU, TestPoint:TestPoint_Pad_D1.0mm, F.Cu at (76.6, 71.7)
- added TP5: NEO_OUT, TestPoint:TestPoint_Pad_D1.0mm, B.Cu at (61.2, 46.5)
- added TP6: FSPID, TestPoint:TestPoint_Pad_D1.0mm, F.Cu at (50.8, 73.3)
- added TP7: FSPICS1, TestPoint:TestPoint_Pad_D1.0mm, F.Cu at (52.9, 75.5)
- added TP8: FSPIQ, TestPoint:TestPoint_Pad_D1.0mm, F.Cu at (51.9, 74.4)
- added TP9: FSPICLK, TestPoint:TestPoint_Pad_D1.0mm, F.Cu at (49.7, 72.3)
- moved AE1 1.37 mm to (71.0, 81.5)
Connections:
- J3 pad 3: unconnected-(J3-Pad3) -> /CAN_DRV_N
- J3 pad 4: unconnected-(J3-Pad4) -> /CAN_DRV_P
- R25 pad 2: /VBAT_SENSE -> /GPIO2
- R26 pad 1: /VBAT_SENSE -> /GPIO2
- R27 pad 1: /CAN_EN -> /GPIO21
- R29 pad 1: unconnected-(R29-Pad1) -> /GPIO14
- TP3 pad 1: /VBAT_SENSE -> /GPIO2
- U5 pad 1: /CAN_P -> /GPIO18
- U5 pad 4: /CAN_N -> /GPIO17
- U5 pad 8: /CAN_EN -> /GPIO21
Routing:
- net /GPIO14: track 7.71 -> 35.1 mm
- net /GPIO17: track 7.76 -> 24.1 mm
- net /CAN_N: track 15.4 -> 0.00 mm
- net /GPIO38: track 12.3 -> 0.00 mm, vias 1 -> 0
- net /GPIO21: track 4.45 -> 15.7 mm, vias 1 -> 2
- net /GPIO18: track 7.63 -> 18.3 mm
- net /CAN_EN: track 10.6 -> 0.00 mm, vias 1 -> 0
- net /CAN_P: track 10.2 -> 0.00 mm
- net /GPIO13: track 7.24 -> 0.00 mm, vias 1 -> 0
- net /GPIO12: track 6.81 -> 0.00 mm, vias 1 -> 0
- net /GPIO11: track 6.50 -> 0.00 mm, vias 1 -> 0
- net /GPIO10: track 6.36 -> 0.00 mm, vias 1 -> 0
- net /GPIO2: track 10.5 -> 16.4 mm, vias 1 -> 0
- net +3V3: track 99.6 -> 93.7 mm, vias 33 -> 38
- net /FSPIQ: track 40.4 -> 45.0 mm
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- added copper zone on F.Cu, net /GPIO2
- added copper zone on In2.Cu, net GND
- removed copper zone on In1.Cu, net +3V3
- removed copper zone on F.Cu, net /VBAT_SENSE
Other:
- board text added: "DOUT"

Commit message: route diff pairs or whatever idr
Parts:
- moved C8 9.35 mm to (70.9, 74.8), turned to 135 degrees
- moved R29 2.84 mm to (63.6, 41.3)
- moved C4 2.40 mm to (68.1, 71.5), turned to 0 degrees
- moved L1 1.25 mm to (68.6, 73.0)
- moved L2 0.82 mm to (69.0, 74.4), turned to 0 degrees
- moved C42 0.34 mm to (59.1, 78.6)
- moved C5 0.23 mm to (67.2, 73.8)
Connections:
- net /GPIO17 renamed /CAN_N
- net /GPIO18 renamed /CAN_P
- net /GPIO19 renamed /GPIO_USB_D_N
- net /GPIO20 renamed /GPIO_USB_D_P
- net /GPIO21 renamed /CAN_EN
- net Net-(AE1-Pad1) renamed /RF_ANT
Routing:
- net /FSPICS1: track 0.00 -> 29.5 mm, vias 0 -> 1
- net /BL: track 0.00 -> 28.7 mm, vias 0 -> 1
- net /DC: track 0.00 -> 28.4 mm, vias 0 -> 1
- net /RST: track 0.00 -> 27.8 mm, vias 0 -> 1
- net Net-(C8-Pad2): track 11.5 -> 1.05 mm
- net /CAN_P: track 18.3 -> 23.7 mm
- net +3V3: track 93.7 -> 98.9 mm
- net /GPIO14: track 35.1 -> 38.1 mm
- net Net-(D1-Pad4): track 4.70 -> 2.12 mm
- net /CAN_DRV_P: track 8.71 -> 10.9 mm
- net /RF_ANT: track 11.8 -> 9.66 mm
- net /USB_D_N: track 11.6 -> 13.6 mm
- net Net-(J2-PadSWA): track 3.22 -> 1.73 mm
- net Net-(D3-Pad2): track 11.2 -> 12.5 mm
- net GND: track 130.1 -> 131.0 mm, vias 34 -> 42
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Other:
- board text added: "3V3"
- board text added: "BL"
- board text added: "CLK"
- board text added: "CS"
- board text added: "DC"
- board text added: "DIN"
- board text added: "GND"
- board text added: "JTAG"
- board text added: "RST"
- board text removed: "REMEMBER TO IMPEDIANCE MATCH THIS TRACE DUMMY"
- board text removed: "diff pair match"

Commit message: tune length of spi signal
Parts:
- moved C32 0.64 mm to (61.7, 44.4), turned to -90 degrees
- moved C41 0.42 mm to (59.4, 43.0), turned to 180 degrees
Routing:
- net /SPICLK: track 23.5 -> 30.8 mm
- net /FSPIQ: track 45.0 -> 51.1 mm
- net /FSPID: track 47.7 -> 53.8 mm
- net /SPID: track 21.5 -> 27.0 mm
- net GND: track 131.0 -> 126.9 mm
- net /SPIHD: track 26.4 -> 30.3 mm
- net /SPIWP: track 32.0 -> 33.7 mm
- net Net-(C41-Pad2): track 3.10 -> 1.86 mm
- net +3V3: track 98.9 -> 98.3 mm
Other:
- board text added: "probably want a diode on VIN"

Commit message: Guess it's done
Parts:
- added D6: D_Small, Diode_SMD:D_SOD-123F, F.Cu at (85.8, 69.7)
- added SW1: SW_Push, Connector_CK:PTS810SJG250SMTRLFS, F.Cu at (50.2, 78.3)
- added SW2: SW_Push, Connector_CK:PTS810SJG250SMTRLFS, F.Cu at (55.6, 83.2)
- moved C23 4.31 mm to (87.4, 74.9), turned to 180 degrees
- moved C22 3.24 mm to (87.4, 73.0), turned to 180 degrees
- moved TP3 1.35 mm to (84.6, 72.9)
- moved R25 1.35 mm to (85.6, 71.6)
- moved R26 1.35 mm to (83.6, 71.5)
- moved TP14 1.18 mm to (59.4, 80.3)
- moved TP13 0.78 mm to (57.9, 80.3)
Connections:
- J3 pad 2: /VIN -> /EXT_VIN
- TP11 pad 1: /RST -> /GPIO6
- TP12 pad 1: /BL -> /GPIO8
- TP7 pad 1: /FSPICS1 -> /GPIO9
- U3 pad 12: /GPIO7 -> /DC
Routing:
- net /CHIP_PU: track 9.59 -> 52.4 mm, vias 0 -> 2
- net /EXT_VIN: track 0.00 -> 42.6 mm, vias 0 -> 2
- net /VIN: track 40.5 -> 0.00 mm, vias 3 -> 0
- net /GPIO0_BOOTSTRAP: track 0.00 -> 38.0 mm, vias 0 -> 2
- net /FSPICS1: track 29.5 -> 0.00 mm, vias 1 -> 0
- net /BL: track 28.7 -> 0.00 mm, vias 1 -> 0
- net /RST: track 27.8 -> 0.00 mm, vias 1 -> 0
- net /GPIO6: track 8.72 -> 31.5 mm, vias 1 -> 2
- net /GPIO8: track 7.84 -> 28.0 mm, vias 1 -> 2
- net /GPIO9: track 7.37 -> 26.4 mm, vias 1 -> 2
- net +3V3: track 98.3 -> 114.8 mm, vias 38 -> 36
- net /GPIO3: track 10.1 -> 0.00 mm, vias 1 -> 0
- net /GPIO1: track 9.80 -> 0.00 mm, vias 1 -> 0
- net /GPIO4: track 9.60 -> 0.00 mm, vias 1 -> 0
- net Net-(C21-Pad1): track 0.00 -> 9.27 mm, vias 0 -> 2
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Other:
- board text added: "PU"
- board text removed: "probably want a diode on VIN"
