File: hardware/platform-esp/platform-esp.kicad_pcb (KiCad board)
At the start: 4 copper layers, 50 x 49.6 mm, 115 parts, among them J1 Conn_ARM_JTAG_SWD_10, J2 DM3AT-SF-PEJM5, J3 PWR_CAN, J4 USB4120-03-C_REVA, J6 TC2030-IDC, SW1 SW_Push, SW2 SW_Push, U1 W25Q128JVS, U2 ESP-PSRAM32, U3 ESP32-S3R2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

Commit message: asdf
Routing:
- net /MTDI: track 21.6 -> 22.5 mm
- added copper zone on In1.Cu, net +3V3

Commit message: restart esp gauge
Parts:
- removed C3, C7: C_Small, Capacitor_SMD:C_0402_1005Metric
- removed C31: 1uF, Capacitor_SMD:C_0402_1005Metric
- removed J2: DM3AT-SF-PEJM5, Connector_Hirose_SD:HRS_DM3AT-SF-PEJM5
- removed R2: DNP, Resistor_SMD:R_0402_1005Metric
- removed R28: 10k, Resistor_SMD:R_0402_1005Metric
- removed R8: 0, Resistor_SMD:R_0402_1005Metric
- removed Y2: 32.7k, Crystal:Crystal_SMD_MicroCrystal_CC7V-T1A-2Pin_3.2x1.5mm
- AE1: footprint RF_Antenna:Texas_SWRA117D_2.4GHz_Right -> RF_Antenna:Johanson_2450AT18x100
- C42, TP10, TP11, TP12, TP13, TP14, TP4, TP6, TP7, TP8, TP9: moved to B.Cu
- J1: moved to F.Cu
- SW1, SW2: footprint Connector_CK:PTS810SJG250SMTRLFS -> SW_RS-032G05A3-SMRT:SW_RS-032G05A3-SMRT
- U3: footprint Package_DFN_QFN:QFN-56-1EP_7x7mm_P0.4mm_EP5.6x5.6mm_ThermalVias -> Package_DFN_QFN:QFN-56-1EP_7x7mm_P0.4mm_EP5.6x5.6mm
- moved J6 37.5 mm to (77.1, 76.8), turned to 45 degrees
- moved C22 36.2 mm to (61.7, 47.5), turned to 0 degrees
- moved C23 34.6 mm to (61.7, 51.7), turned to 0 degrees
- moved C35 32.3 mm to (57.1, 62.9), turned to 180 degrees
- moved C36 32.2 mm to (57.7, 64.1), turned to 180 degrees
- moved SW2 31.9 mm to (83.0, 66.8), turned to 90 degrees
- moved SW1 31.1 mm to (79.0, 66.7), turned to 90 degrees
- moved C34 29.6 mm to (57.8, 62.0), turned to 180 degrees
- moved C37 28.8 mm to (57.7, 65.9), turned to 180 degrees
- moved J1 28.6 mm to (81.7, 80.6), turned to 45 degrees
- moved C25 28.0 mm to (61.8, 53.9), turned to 0 degrees
- moved C41 27.5 mm to (56.2, 70.2)
- moved TP4 26.8 mm to (51.1, 63.7), turned to -90 degrees
- moved TP3 26.0 mm to (83.2, 47.0), turned to 90 degrees
- moved R26 25.5 mm to (82.0, 46.0), turned to 90 degrees
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Connections:
- net /GPIO8 renamed /BL
- net /GPIO9 renamed /FSPICS1
- C13 pad 2: +3V3 -> /VDD3V3
- L3 pad 1: +3V3 -> /VDD3V3
- SW1 pad 1: /GPIO0_BOOTSTRAP -> /CHIP_PU
- SW1 pad 2: /GPIO0_BOOTSTRAP -> Net-(C21-Pad1)
- SW2 pad 1: /CHIP_PU -> /GPIO0_BOOTSTRAP
- SW2 pad 2: /CHIP_PU -> GND
- U3 pad 2: +3V3 -> /VDD3V3
- U3 pad 21: /RTC_XTAL_P -> unconnected-(U3-Pad21)
- U3 pad 22: Net-(R8-Pad2) -> unconnected-(U3-Pad22)
- U3 pad 3: +3V3 -> /VDD3V3
Routing:
- net GND: track 119.9 -> 0.00 mm, vias 43 -> 0
- net +3V3: track 114.8 -> 0.00 mm, vias 36 -> 0
- net /FSPID: track 53.8 -> 0.00 mm, vias 2 -> 0
- net /CHIP_PU: track 52.4 -> 0.00 mm, vias 2 -> 0
- net /FSPICLK: track 52.2 -> 0.00 mm, vias 2 -> 0
- net /FSPIQ: track 51.1 -> 0.00 mm, vias 2 -> 0
- net /EXT_VIN: track 42.6 -> 0.00 mm, vias 2 -> 0
- net /GPIO14: track 38.1 -> 0.00 mm, vias 1 -> 0
- net /GPIO0_BOOTSTRAP: track 38.0 -> 0.00 mm, vias 2 -> 0
- net /SPICS1: track 34.0 -> 0.00 mm, vias 2 -> 0
- net /SPIWP: track 33.7 -> 0.00 mm, vias 4 -> 0
- net /U0RXD: track 32.6 -> 0.00 mm, vias 2 -> 0
- net /GPIO6: track 31.5 -> 0.00 mm, vias 2 -> 0
- net /SPIQ: track 31.0 -> 0.00 mm, vias 4 -> 0
- net Net-(D5-Pad2): track 30.9 -> 0.00 mm, vias 2 -> 0
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- removed copper zone on B.Cu, net +3V3
- removed copper zone on F.Cu, net +3V3
- removed copper zone on In1.Cu, net +3V3
- removed copper zone on In2.Cu, net +3V3
- removed copper zone on F.Cu, net /GPIO2
- removed copper zone on F.Cu, net /VIN
- removed copper zone on In2.Cu, net /VIN
- removed copper zone on B.Cu, net GND
- removed copper zone on F.Cu, net GND
- removed copper zone on In1.Cu, net GND
- removed copper zone on In2.Cu, net GND
- removed copper zone on F.Cu, net Net-(C25-Pad2)
- removed copper zone on In2.Cu, net Net-(C27-Pad2)
Other:
- board text removed: "3V3"
- board text removed: "BL"
- board text removed: "CLK"
- board text removed: "CS"
- board text removed: "DC"
- board text removed: "DEBUG"
- board text removed: "DIN"
- board text removed: "DOUT"
- board text removed: "GND"
- board text removed: "JTAG"
- board text removed: "PU"
- board text removed: "RST"
