File: hardware/gauge-controller/neopixels.kicad_sch (KiCad schematic)
At the start: 21 parts

Commit message: asdf
Changed lines of the file:
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@@
     (stroke (width 0) (type default) (color 0 0 0 0))
   )
-  (label "NEO_OUT" (at 24.13 87.63 90)
-    (effects (font (size 1.27 1.27)) (justify left bottom))
+  (hierarchical_label "NEO_OUT" (shape input) (at 24.13 87.63 90)
+    (effects (font (size 1.27 1.27)) (justify left))
   )
   (symbol (lib_id "Device:C_Small") (at 170.815 72.39 0) (unit 1)
