File: hardware/gauge-controller/platform-esp.kicad_pcb (KiCad board)
At the start: 4 copper layers, 50 x 49.6 mm, 107 parts, among them J1 Conn_ARM_JTAG_SWD_10, J3 PWR_CAN, J4 USB4120-03-C_REVA, J6 TC2030-IDC, SW1 SW_Push, SW2 SW_Push, U1 W25Q128JVS, U2 ESP-PSRAM32, U3 ESP32-S3R2, U4 AP64200Q, U5 LTC2875-DD, Y1 40MHZ

Commit message: restart gauge pcb
Parts:
- removed C39, C40, C41, C42: 1uF, Capacitor_SMD:C_0402_1005Metric
- removed D11: WS2812B, LED_SMD:LED_WS2812B_PLCC4_5.0x5.0mm_P3.2mm
- removed J6: TC2030-IDC, Connector:Tag-Connect_TC2030-IDC-NL_2x03_P1.27mm_Vertical
- removed R26, R27: 10k, Resistor_SMD:R_0402_1005Metric
- removed R29: 0, Resistor_SMD:R_0402_1005Metric
- removed REF**: 1.28-lcd, Module_Waveshare:1.28-lcd
- removed TP10: DC, TestPoint:TestPoint_Pad_D1.0mm
- removed TP11: RST, TestPoint:TestPoint_Pad_D1.0mm
- removed TP12: BL, TestPoint:TestPoint_Pad_D1.0mm
- removed TP13: VDD3V3, TestPoint:TestPoint_Pad_D1.0mm
- removed TP14: GND, TestPoint:TestPoint_Pad_D1.0mm
- removed TP6: FSPID, TestPoint:TestPoint_Pad_D1.0mm
- removed TP7: FSPICS1, TestPoint:TestPoint_Pad_D1.0mm
- removed TP8: FSPIQ, TestPoint:TestPoint_Pad_D1.0mm
- removed TP9: FSPICLK, TestPoint:TestPoint_Pad_D1.0mm
- added C3: C_Small, Capacitor_SMD:C_0402_1005Metric, F.Cu at (110.8, 53.7)
- added C31: 1uF, Capacitor_SMD:C_0402_1005Metric, F.Cu at (59.7, 22.9)
- added C7: 1uF, Capacitor_SMD:C_0402_1005Metric, F.Cu at (115.0, 48.7)
- added D7: WS2812B, WS2815B:LED_WS2812B_PLCC4_5.0x5.0mm_P3.2mm, B.Cu at (33.8, 22.9)
- added J2: PWR_CAN, Connector_JST:JST_GH_BM04B-GHS-TBT_1x04-1MP_P1.25mm_Vertical, F.Cu at (102.0, 36.7)
- added J5: USB4120-03-C_REVA, Connector_GCT_USB:GCT_USB4120-03-C_REVA, F.Cu at (90.4, 41.9)
- added R2: 0, Resistor_SMD:R_0402_1005Metric, F.Cu at (125.8, 38.0)
- added R8: 100k, Resistor_SMD:R_0402_1005Metric, F.Cu at (127.5, 31.5)
- C1, C12, C18, C30: value 0.1uF -> 1uF
- C10, C15: value 1uF -> C_Small
- C13, C2: value C_Small -> 10uF
- C14: value 0.1uF -> C_Small
- C16, C19: value 10uF -> 0.1uF
- C17: value 1uF -> 0.1uF
- C20: value 1uF -> 0.1uf; footprint Capacitor_SMD:C_0402_1005Metric -> Capacitor_SMD:C_0805_2012Metric_Pad1.18x1.45mm_HandSolder
- C21: value 1uF -> 10uf; footprint Capacitor_SMD:C_0402_1005Metric -> Capacitor_SMD:C_0805_2012Metric_Pad1.18x1.45mm_HandSolder
- C23: value 10uf -> DNP
- C24: value 5.6nf -> DNP; footprint Capacitor_SMD:C_1206_3216Metric -> Capacitor_SMD:C_0805_2012Metric_Pad1.18x1.45mm_HandSolder
- C25: value 0.1uf -> DNP
- C27: value DNP -> 5.6nf; footprint Capacitor_SMD:C_0805_2012Metric_Pad1.18x1.45mm_HandSolder -> Capacitor_SMD:C_1206_3216Metric
- C28: value DNP -> 1uF; footprint Capacitor_SMD:C_0805_2012Metric_Pad1.18x1.45mm_HandSolder -> Capacitor_SMD:C_0402_1005Metric
- C29: value DNP -> 10uF; footprint Capacitor_SMD:C_0805_2012Metric_Pad1.18x1.45mm_HandSolder -> Capacitor_SMD:C_0402_1005Metric
- C32: value 10uF -> 1uF; moved to F.Cu
- C33, C34, C35, C36, C37, C38, TP5: moved to F.Cu
- C6, C8: value C_Small -> 0.1uF
- D1: value WS2812B -> D_Small; footprint LED_SMD:LED_WS2812B_PLCC4_5.0x5.0mm_P3.2mm -> Diode_SMD:D_SOD-123F; moved to F.Cu
- D10, D2, D3, D4, D5, D8, D9: footprint LED_SMD:LED_WS2812B_PLCC4_5.0x5.0mm_P3.2mm -> WS2815B:LED_WS2812B_PLCC4_5.0x5.0mm_P3.2mm
- D6: value D_Small -> WS2812B; footprint Diode_SMD:D_SOD-123F -> WS2815B:LED_WS2812B_PLCC4_5.0x5.0mm_P3.2mm; moved to B.Cu
- J1: value Conn_ARM_JTAG_SWD_10 -> TC2030-IDC; footprint Connector:Tag-Connect_TC2050-IDC-NL_2x05_P1.27mm_Vertical -> Connector:Tag-Connect_TC2030-IDC-NL_2x03_P1.27mm_Vertical
- J3: value PWR_CAN -> Conn_ARM_JTAG_SWD_10; footprint Connector_JST:JST_GH_BM04B-GHS-TBT_1x04-1MP_P1.25mm_Vertical -> Connector:Tag-Connect_TC2050-IDC-NL_2x05_P1.27mm_Vertical
- J4: value USB4120-03-C_REVA -> Conn_01x09; footprint Connector_GCT_USB:GCT_USB4120-03-C_REVA -> Connector_GC9A01:GC9A01_disp; moved to B.Cu
- R1: value 100k -> 10k
- R12, R13, R15: value 0 -> 10k
- R14: value 0 -> 36k
- R18: value 10k -> 100k
- R19: value 51k -> 52.3k; footprint Resistor_SMD:R_0402_1005Metric -> Resistor_SMD:R_0603_1608Metric_Pad0.98x0.95mm_HandSolder
- R20: value 51k -> 200k; footprint Resistor_SMD:R_0402_1005Metric -> Resistor_SMD:R_0603_1608Metric_Pad0.98x0.95mm_HandSolder
- R21: value 200k -> 14k
- R22: value 14k -> 10k
- R23: value 52.3k -> 51k; footprint Resistor_SMD:R_0603_1608Metric_Pad0.98x0.95mm_HandSolder -> Resistor_SMD:R_0402_1005Metric
- R24: value 10k -> 51k; footprint Resistor_SMD:R_0603_1608Metric_Pad0.98x0.95mm_HandSolder -> Resistor_SMD:R_0402_1005Metric
- R25: value 36k -> 0; moved to B.Cu
- R3: value 100k -> 499
- R4: value 442k -> 0
- R5: value 10k -> 0
- R6: value 499 -> 0
- TP1: value 3V3OUT -> CHIP_PU
- TP2: value 3V3OUT -> VBAT_SENSE
- TP3: value VBAT_SENSE -> 3V3OUT
- TP4: value CHIP_PU -> 3V3OUT; moved to F.Cu
- U1: value W25Q128JVS -> ESP32-S3R2; footprint Package_SO:SOIC-8_5.23x5.23mm_P1.27mm -> Package_DFN_QFN:QFN-56-1EP_7x7mm_P0.4mm_EP5.6x5.6mm
- U2: value ESP-PSRAM32 -> LTC2875-DD; footprint Package_SO:SOIC-8_3.9x4.9mm_P1.27mm -> Package_DFN_QFN:DFN-8-1EP_3x3mm_P0.5mm_EP1.66x2.38mm
- U3: value ESP32-S3R2 -> W25Q128JVS; footprint Package_DFN_QFN:QFN-56-1EP_7x7mm_P0.4mm_EP5.6x5.6mm -> Package_SO:SOIC-8_5.23x5.23mm_P1.27mm
- U4: value AP64200Q -> ESP-PSRAM32; footprint Package_SO:SOIC-8-1EP_3.9x4.9mm_P1.27mm_EP2.29x3mm_ThermalVias -> Package_SO:SOIC-8_3.9x4.9mm_P1.27mm
- U5: value LTC2875-DD -> AP64200Q; footprint Package_DFN_QFN:DFN-8-1EP_3x3mm_P0.5mm_EP1.66x2.38mm -> Package_SO:SOIC-8-1EP_3.9x4.9mm_P1.27mm_EP2.29x3mm_ThermalVias
- moved R10 90.3 mm to (130.4, 31.5)
- moved C10 87.3 mm to (138.0, 26.0), turned to 0 degrees
- moved R1 80.9 mm to (122.7, 34.1)
- moved C5 80.5 mm to (131.4, 33.5)
- moved C18 77.3 mm to (131.6, 35.5), turned to 0 degrees
- moved C13 75.2 mm to (138.0, 28.0), turned to 0 degrees
- moved R22 74.0 mm to (130.9, 29.3)
- moved C9 73.3 mm to (136.1, 31.0), turned to 0 degrees
- moved L1 73.3 mm to (125.8, 36.0), turned to 0 degrees
- moved C2 71.9 mm to (128.7, 37.5), turned to 0 degrees
- moved R5 71.9 mm to (134.5, 29.0), turned to 0 degrees
- moved C11 70.4 mm to (128.7, 35.5), turned to 0 degrees
- moved C19 70.2 mm to (133.3, 31.5), turned to 0 degrees
- moved C4 69.2 mm to (124.3, 40.0)
- moved J1 68.3 mm to (124.7, 27.5), turned to 0 degrees
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Connections:
- C10 pad 1: /SPICLK_P -> GND
- C10 pad 2: GND -> /VDD3V3
- C11 pad 1: /VDDRTC -> +3V3
- C12 pad 1: /VDDCPU -> +3V3
- C13 pad 1: GND -> +3V3
- C13 pad 2: /VDD3V3 -> GND
- C14 pad 1: +3V3 -> /XTAL_P
- C15 pad 1: +3V3 -> /XTAL_N
- C18 pad 1: +3V3 -> Net-(C18-Pad1)
- C2 pad 1: /XTAL_P -> +3V3
- C20 pad 1: +3V3 -> Net-(C20-Pad1)
- C20 pad 2: GND -> Net-(C20-Pad2)
- C21 pad 1: Net-(C21-Pad1) -> GND
- C21 pad 2: GND -> /VIN
- C23 pad 1: GND -> +3V3
- C23 pad 2: /VIN -> Net-(C23-Pad2)
- C24 pad 1: Net-(C24-Pad1) -> +3V3
- C25 pad 1: Net-(C25-Pad1) -> +3V3
- C25 pad 2: Net-(C25-Pad2) -> GND
- C27 pad 1: +3V3 -> Net-(C27-Pad1)
- C27 pad 2: Net-(C27-Pad2) -> GND
- C30 pad 2: GND -> Net-(C30-Pad2)
- C32 pad 2: GND -> Net-(C32-Pad2)
- C4 pad 2: /LNA_IN -> /RF_ANT
- C5 pad 2: /RF_ANT -> Net-(C5-Pad2)
- C6 pad 1: /XTAL_N -> +3V3
- C8 pad 1: GND -> /VDDRTC
- C8 pad 2: Net-(C8-Pad2) -> GND
- C9 pad 1: +3V3 -> /VDDCPU
- D1 pad 1: Net-(C33-Pad2) -> /VIN
- D1 pad 2: Net-(D1-Pad2) -> /EXT_VIN
- D10 pad 1: Net-(C40-Pad2) -> Net-(C37-Pad2)
- D2 pad 1: Net-(C34-Pad2) -> Net-(C30-Pad2)
- D2 pad 4: Net-(D1-Pad2) -> Net-(D2-Pad4)
- D3 pad 1: Net-(C35-Pad2) -> Net-(C31-Pad2)
- D4 pad 1: Net-(C36-Pad2) -> Net-(C32-Pad2)
- D5 pad 1: Net-(C37-Pad2) -> Net-(C33-Pad2)
- D6 pad 1: /VIN -> Net-(C34-Pad2)
- D6 pad 2: /EXT_VIN -> Net-(D6-Pad2)
- D8 pad 1: Net-(C38-Pad2) -> Net-(C35-Pad2)
- D8 pad 4: Net-(D5-Pad2) -> Net-(D6-Pad2)
- D9 pad 1: Net-(C39-Pad2) -> Net-(C36-Pad2)
- J1 pad 2: /MTMS -> unconnected-(J1-Pad2)
- J1 pad 3: GND -> /U0TXD
- J1 pad 4: /MTCK -> /U0RXD
- J1 pad 6: /MTDO -> unconnected-(J1-Pad6)
- J3 pad 1: GND -> unconnected-(J3-Pad1)
- J3 pad 2: /EXT_VIN -> /MTMS
- J3 pad 3: /CAN_DRV_N -> GND
- J3 pad 4: /CAN_DRV_P -> /MTCK
- L2 pad 2: Net-(C8-Pad2) -> Net-(C5-Pad2)
- L4 pad 1: Net-(C25-Pad2) -> Net-(C20-Pad2)
- R1 pad 1: +3V3 -> /CHIP_PU
- R1 pad 2: /SPICS0 -> +3V3
- R10 pad 1: /SPIWP -> /SPIQ
- R11 pad 1: /SPICLK -> /SPID
- R12 pad 1: /SPIQ -> /CAN_EN
- R12 pad 2: Net-(R12-Pad2) -> GND
- R13 pad 1: /SPID -> /GPIO0
- R13 pad 2: Net-(R13-Pad2) -> /GPIO0_BOOTSTRAP
- R14 pad 1: /GPIO_USB_D_N -> /VIN
- R14 pad 2: /USB_D_N -> /GPIO2
- R15 pad 1: /GPIO_USB_D_P -> /GPIO45
- R15 pad 2: /USB_D_P -> GND
- R16 pad 1: /GPIO0 -> /GPIO2
- R16 pad 2: /GPIO0_BOOTSTRAP -> GND
- R17 pad 1: /GPIO45 -> /GPIO46
- R18 pad 1: /GPIO46 -> /SPICS1
- R18 pad 2: GND -> +3V3
- R19 pad 1: /CC2 -> +3V3
- R19 pad 2: GND -> Net-(C23-Pad2)
- R20 pad 1: /CC1 -> Net-(R20-Pad1)
- R21 pad 1: Net-(R21-Pad1) -> Net-(C26-Pad1)
- R21 pad 2: GND -> Net-(C27-Pad1)
- R22 pad 1: Net-(C26-Pad1) -> Net-(C23-Pad2)
- R22 pad 2: Net-(C24-Pad1) -> GND
- R23 pad 1: +3V3 -> /CC1
- R23 pad 2: Net-(C27-Pad2) -> GND
- R24 pad 1: Net-(C27-Pad2) -> /CC2
- R25 pad 1: /VIN -> /neopixels/NEO_OUT
- R25 pad 2: /GPIO2 -> Net-(D2-Pad4)
- R3 pad 1: /SPICS1 -> /U0TXD
- R3 pad 2: +3V3 -> Net-(R3-Pad2)
- R4 pad 1: /SPICLK_P -> /GPIO_USB_D_N
- R4 pad 2: GND -> /USB_D_N
- R5 pad 1: /CHIP_PU -> /GPIO_USB_D_P
- R5 pad 2: +3V3 -> /USB_D_P
- R6 pad 1: /U0TXD -> /SPIHD
- R7 pad 1: /XTAL_N -> /SPIWP
- R9 pad 1: /SPIHD -> /SPICLK
- SW1 pad 2: Net-(C21-Pad1) -> Net-(C18-Pad1)
- TP1 pad 1: GND -> /CHIP_PU
- TP2 pad 1: +3V3 -> /GPIO2
- TP3 pad 1: /GPIO2 -> GND
- TP4 pad 1: /CHIP_PU -> +3V3
- TP5 pad 1: /GPIO14 -> /neopixels/NEO_OUT
- U1 pad 1: /SPICS0 -> /LNA_IN
- U1 pad 2: /SPIQ -> /VDD3V3
- U1 pad 3: /SPIWP -> /VDD3V3
- U1 pad 4: GND -> /CHIP_PU
- U1 pad 5: /SPID -> /GPIO0
- U1 pad 6: /SPICLK -> /GPIO1
- U1 pad 7: /SPIHD -> /GPIO2
- U1 pad 8: +3V3 -> /GPIO3
- U2 pad 1: /SPICS1 -> /CAN_P
- U2 pad 2: /SPID -> GND
- U2 pad 3: /SPIWP -> +3V3
- U2 pad 4: GND -> /CAN_N
- U2 pad 5: /SPIQ -> unconnected-(U2-Pad5)
- U2 pad 6: /SPICLK -> /CAN_DRV_N
- U2 pad 7: /SPIHD -> /CAN_DRV_P
- U2 pad 8: +3V3 -> /CAN_EN
- U3 pad 1: /LNA_IN -> /SPICS0
- U3 pad 2: /VDD3V3 -> /SPIQ
- U3 pad 3: /VDD3V3 -> /SPIWP
- U3 pad 4: /CHIP_PU -> GND
- U3 pad 5: /GPIO0 -> /SPID
- U3 pad 6: /GPIO1 -> /SPICLK
- U3 pad 7: /GPIO2 -> /SPIHD
- U3 pad 8: /GPIO3 -> +3V3
- U4 pad 1: Net-(C25-Pad1) -> /SPICS1
- U4 pad 2: /VIN -> /SPID
- U4 pad 3: /VIN -> /SPIWP
- U4 pad 4: Net-(R21-Pad1) -> GND
- U4 pad 5: Net-(C27-Pad2) -> /SPIQ
- U4 pad 6: Net-(C26-Pad1) -> /SPICLK
- U4 pad 7: GND -> /SPIHD
- U4 pad 8: Net-(C25-Pad2) -> +3V3
- U5 pad 1: /CAN_P -> Net-(C20-Pad1)
- U5 pad 2: GND -> /VIN
- U5 pad 3: +3V3 -> /VIN
- U5 pad 4: /CAN_N -> Net-(R20-Pad1)
- U5 pad 5: unconnected-(U5-Pad5) -> Net-(C23-Pad2)
- U5 pad 6: /CAN_DRV_N -> Net-(C26-Pad1)
- U5 pad 7: /CAN_DRV_P -> GND
- U5 pad 8: /CAN_EN -> Net-(C20-Pad2)
Routing:
- net +3V3: track 0.00 -> 134.7 mm
- net Net-(D6-Pad2): track 0.00 -> 24.0 mm
- net Net-(D3-Pad2): track 0.00 -> 10.7 mm
- net Net-(D2-Pad2): track 0.00 -> 10.7 mm
- net Net-(D4-Pad2): track 0.00 -> 10.7 mm
- net Net-(D5-Pad2): track 0.00 -> 10.4 mm
- net Net-(D9-Pad2): track 0.00 -> 10.4 mm
- net Net-(D8-Pad2): track 0.00 -> 10.3 mm
- net Net-(C37-Pad2): track 0.00 -> 3.74 mm, vias 0 -> 1
- net Net-(C33-Pad2): track 0.00 -> 3.74 mm, vias 0 -> 1
- net Net-(C34-Pad2): track 0.00 -> 3.72 mm, vias 0 -> 1
- net Net-(C36-Pad2): track 0.00 -> 3.72 mm, vias 0 -> 1
- net Net-(C38-Pad2): track 0.00 -> 3.71 mm, vias 0 -> 1
- net Net-(C32-Pad2): track 0.00 -> 3.70 mm, vias 0 -> 1
- net Net-(C35-Pad2): track 0.00 -> 3.68 mm, vias 0 -> 1
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Other:
- board size 50 x 49.6 mm -> 50 x 50 mm

Commit message: asdf
Parts:
- removed C23, C24, C25, C26: DNP, Capacitor_SMD:C_0805_2012Metric_Pad1.18x1.45mm_HandSolder
- removed C27: 5.6nf, Capacitor_SMD:C_1206_3216Metric
- removed J1: TC2030-IDC, Connector:Tag-Connect_TC2030-IDC-NL_2x03_P1.27mm_Vertical
- removed J3: Conn_ARM_JTAG_SWD_10, Connector:Tag-Connect_TC2050-IDC-NL_2x05_P1.27mm_Vertical
- removed L4: 6.8uh, Inductor_SMD:L_Bourns-SRN6028
- removed U4: ESP-PSRAM32, Package_SO:SOIC-8_3.9x4.9mm_P1.27mm
- added D11: D_Small, Diode_SMD:D_SOD-123F, F.Cu at (54.1, 36.9)
- added Q1: Q_NPN_EBC, Package_TO_SOT_SMD:TSOT-23, F.Cu at (44.7, 47.9)
- added R26: 10R, Resistor_SMD:R_0402_1005Metric, F.Cu at (43.7, 48.4)
- added R27: 100k, Resistor_SMD:R_0402_1005Metric, F.Cu at (47.8, 49.7)
- added TP10: 3V3OUT, TestPoint:TestPoint_Pad_D1.0mm, F.Cu at (62.2, 34.2)
- added TP11: 3V3OUT, TestPoint:TestPoint_Pad_D1.0mm, F.Cu at (64.3, 34.1)
- added TP6: MTDO, TestPoint:TestPoint_Pad_D1.0mm, F.Cu at (28.6, 34.5)
- added TP7: MTDI, TestPoint:TestPoint_Pad_D1.0mm, F.Cu at (32.2, 34.6)
- added TP8: TXD, TestPoint:TestPoint_Pad_D1.0mm, F.Cu at (28.7, 37.3)
- added TP9: RXD, TestPoint:TestPoint_Pad_D1.0mm, F.Cu at (28.6, 38.7)
- C10: value C_Small -> 10uF; footprint Capacitor_SMD:C_0402_1005Metric -> Capacitor_SMD:C_0805_2012Metric
- C20: value 0.1uf -> 0.1uF; footprint Capacitor_SMD:C_0805_2012Metric_Pad1.18x1.45mm_HandSolder -> Capacitor_SMD:C_0805_2012Metric
- C21, C22: value 10uf -> 22uF; footprint Capacitor_SMD:C_0805_2012Metric_Pad1.18x1.45mm_HandSolder -> Capacitor_SMD:C_0805_2012Metric
- J4: value Conn_01x09 -> Conn_01x12
- L3: value 0H -> 6.8uh; footprint Inductor_SMD:L_0402_1005Metric -> Inductor_SMD:L_Bourns-SRN6028
- R18: value 100k -> 10k
- R19: value 52.3k -> 100k; footprint Resistor_SMD:R_0603_1608Metric_Pad0.98x0.95mm_HandSolder -> Resistor_SMD:R_0603_1608Metric
- R20: value 200k -> 31k6; footprint Resistor_SMD:R_0603_1608Metric_Pad0.98x0.95mm_HandSolder -> Resistor_SMD:R_0603_1608Metric
- R21: value 14k -> 10k2; footprint Resistor_SMD:R_0603_1608Metric_Pad0.98x0.95mm_HandSolder -> Resistor_SMD:R_0603_1608Metric
- R22: footprint Resistor_SMD:R_0603_1608Metric_Pad0.98x0.95mm_HandSolder -> Resistor_SMD:R_0402_1005Metric
- TP3: value 3V3OUT -> MTCK
- TP4: value 3V3OUT -> MTMS
- U1: footprint Package_DFN_QFN:QFN-56-1EP_7x7mm_P0.4mm_EP5.6x5.6mm -> Package_DFN_QFN:QFN-56-1EP_7x7mm_P0.4mm_EP5.6x5.6mm_ThermalVias
- U3: footprint Package_SO:SOIC-8_5.23x5.23mm_P1.27mm -> Package_SO:SOIC-8W_5.3x5.3mm_P1.27mm
- U5: value AP64200Q -> ADP2303ARDZ-3.3
- Y1: footprint Crystal:Crystal_SMD_2016-4Pin_2.0x1.6mm -> Crystal:Crystal_SMD_3225-4Pin_3.2x2.5mm
- moved C9 102.6 mm to (33.9, 39.7), turned to 135 degrees
- moved TP1 100.0 mm to (40.2, 58.3)
- moved C5 96.9 mm to (36.2, 51.9), turned to 135 degrees
- moved R8 96.4 mm to (31.2, 27.3)
- moved R17 94.8 mm to (31.0, 40.5), turned to 180 degrees
- moved C19 94.1 mm to (40.8, 48.8), turned to 180 degrees
- moved C2 93.8 mm to (35.3, 46.0), turned to 180 degrees
- moved Y1 92.2 mm to (30.4, 43.2), turned to 90 degrees
- moved R2 91.9 mm to (34.1, 43.6)
- moved C13 91.9 mm to (46.6, 36.8)
- moved R22 90.6 mm to (42.7, 49.9), turned to -90 degrees
- moved L1 90.4 mm to (36.3, 48.3), turned to -135 degrees
- moved C4 90.0 mm to (34.8, 49.1), turned to -45 degrees
- moved R10 89.4 mm to (41.0, 34.6), turned to -90 degrees
- moved R5 88.7 mm to (46.6, 40.1)
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Connections:
- net Net-(C18-Pad1) renamed /CHIP_PU_BOOTSTRAP
- net Net-(C20-Pad1) renamed /BST
- net Net-(R10-Pad2) renamed /MCU_SPIQ
- net Net-(R11-Pad2) renamed /MCU_SPID
- net Net-(R2-Pad2) renamed /MCU_XTAL_N
- net Net-(R3-Pad2) renamed /MCU_U0TXD
- net Net-(R6-Pad2) renamed /MCU_SPIHD
- net Net-(R7-Pad2) renamed /MCU_SPIWP
- net Net-(R9-Pad2) renamed /MCU_SPICLK
- C10 pad 2: /VDD3V3 -> /VIN
- C19 pad 1: +3V3 -> /CHIP_PU
- C19 pad 2: GND -> +3V3
- C20 pad 2: Net-(C20-Pad2) -> /SW
- C21 pad 1: GND -> +3V3
- C21 pad 2: /VIN -> GND
- C22 pad 1: GND -> +3V3
- C22 pad 2: /VIN -> GND
- C8 pad 1: /VDDRTC -> +3V3
- C9 pad 1: /VDDCPU -> +3V3
- J2 pad 1: GND -> /CAN_DRV_P
- J2 pad 2: /EXT_VIN -> /CAN_DRV_N
- J2 pad 3: /CAN_DRV_N -> GND
- J2 pad 4: /CAN_DRV_P -> /EXT_VIN
- J4 pad 1: unconnected-(J4-Pad1) -> GND
- J4 pad 10: (no net) -> /FSPIQ
- J4 pad 11: (no net) -> /LCD_RESET
- J4 pad 12: (no net) -> GND
- J4 pad 2: unconnected-(J4-Pad2) -> /LCD_LEDK
- J4 pad 3: unconnected-(J4-Pad3) -> +3V3
- J4 pad 4: unconnected-(J4-Pad4) -> +3V3
- J4 pad 5: unconnected-(J4-Pad5) -> GND
- J4 pad 6: unconnected-(J4-Pad6) -> GND
- J4 pad 7: unconnected-(J4-Pad7) -> /DC
- J4 pad 8: unconnected-(J4-Pad8) -> /LCD_CS
- J4 pad 9: unconnected-(J4-Pad9) -> /FSPICLK
- L3 pad 1: /VDD3V3 -> /SW
- R14 pad 2: /GPIO2 -> /VBAT_SENSE
- R16 pad 1: /GPIO2 -> /VBAT_SENSE
- R18 pad 1: /SPICS1 -> /BL
- R18 pad 2: +3V3 -> /LCD_BL_DIV
- R19 pad 1: +3V3 -> /VIN
- R19 pad 2: Net-(C23-Pad2) -> /PGOOD
- R20 pad 1: Net-(R20-Pad1) -> +3V3
- R20 pad 2: GND -> /FB
- R21 pad 1: Net-(C26-Pad1) -> /FB
- R21 pad 2: Net-(C27-Pad1) -> GND
- R22 pad 1: Net-(C23-Pad2) -> /LCD_BL_DIV
- R22 pad 2: GND -> +3V3
- R25 pad 1: /neopixels/NEO_OUT -> /GPIO34
- TP2 pad 1: /GPIO2 -> /VBAT_SENSE
- TP3 pad 1: GND -> /MTCK
- TP4 pad 1: +3V3 -> /MTMS
- TP5 pad 1: /neopixels/NEO_OUT -> /GPIO34
- U1 pad 14: /FSPICS1 -> /LCD_RESET
- U1 pad 15: /GPIO10 -> /VBAT_SENSE
- U1 pad 16: /GPIO11 -> /LCD_CS
- U1 pad 2: /VDD3V3 -> +3V3
- U1 pad 20: /VDDRTC -> +3V3
- U1 pad 28: /SPICS1 -> unconnected-(U1-Pad28)
- U1 pad 3: /VDD3V3 -> +3V3
- U1 pad 39: /FSPICS0 -> /GPIO34
- U1 pad 46: /VDDCPU -> +3V3
- U5 pad 4: Net-(R20-Pad1) -> /PGOOD
- U5 pad 5: Net-(C23-Pad2) -> /FB
- U5 pad 6: Net-(C26-Pad1) -> unconnected-(U5-Pad6)
- U5 pad 8: Net-(C20-Pad2) -> /SW
Routing:
- net GND: track 0.00 -> 187.8 mm, vias 0 -> 43
- net +3V3: track 134.7 -> 233.5 mm, vias 0 -> 9
- net /FSPIQ: track 0.00 -> 33.9 mm, vias 0 -> 3
- net /FSPICLK: track 0.00 -> 30.0 mm, vias 0 -> 3
- net /USB_D_P: track 0.00 -> 28.6 mm, vias 0 -> 6
- net /GPIO34: track 0.00 -> 28.3 mm, vias 0 -> 2
- net /USB_VBUS: track 0.00 -> 26.8 mm, vias 0 -> 3
- net /USB_D_N: track 0.00 -> 26.3 mm, vias 0 -> 5
- net /VBAT_SENSE: track 0.00 -> 25.1 mm, vias 0 -> 2
- net /SPICS0: track 0.00 -> 21.2 mm, vias 0 -> 2
- net /LCD_CS: track 0.00 -> 19.6 mm, vias 0 -> 4
- net /CAN_N: track 0.00 -> 19.1 mm, vias 0 -> 2
- net /CAN_P: track 0.00 -> 18.2 mm, vias 0 -> 2
- net /MTCK: track 0.00 -> 16.9 mm, vias 0 -> 2
- net /CHIP_PU: track 0.00 -> 16.9 mm
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- added copper zone on B.Cu, net +3V3
- added copper zone on F.Cu, net +3V3
- added copper zone on F.Cu, net /PGOOD
- added copper zone on F.Cu, net /SW
- added copper zone on F.Cu, net /USB_VBUS
- added copper zone on F.Cu, net /VIN
- added copper zone on B.Cu, net GND
- added copper zone on F.Cu, net GND
- added copper zone on In1.Cu, net GND
- added copper zone on In2.Cu, net GND

Commit message: cauge design progress
Parts:
- added G***: LOGO, logos:cone, F.Cu at (55.9, 52.2)
- moved R26 1.47 mm to (43.6, 49.8)
Routing:
- net +3V3: track 233.5 -> 258.8 mm
- net /LCD_LEDK: track 4.69 -> 3.18 mm
- net /Q_LEDK: track 2.08 -> 1.07 mm
- added copper zone on F.Cu, net (none)
Other:
- board text added: "+12V"
- board text added: "3V3"
- board text added: "CAN"
- board text added: "CAN Multi-Gauge"
- board text added: "DOUT"
- board text added: "Designed by Connor Rigby 05 / 22"
- board text added: "GND"
- board text added: "VSENSE"
- board text added: "https://cone.codes"

Commit message: misc cleanup
Parts:
- removed J5: USB4120-03-C_REVA, Connector_GCT_USB:GCT_USB4120-03-C_REVA
- added J1: USB4120-03-C_REVA, ConeCodes:GCT_USB4120-03-C_REVA, F.Cu at (42.0, 24.9)
- J4: footprint Connector_GC9A01:GC9A01_disp -> ConeCodes:GC9A01_disp
- SW1, SW2: footprint SW_RS-032G05A3-SMRT:SW_RS-032G05A3-SMRT -> ConeCodes:SW_RS-032G05A3-SMRT
- U1: footprint Package_DFN_QFN:QFN-56-1EP_7x7mm_P0.4mm_EP5.6x5.6mm_ThermalVias -> ConeCodes:QFN-56
- moved C28 0.14 mm to (45.1, 50.4)
- moved C31 0.13 mm to (59.7, 22.7)
Connections:
- net /LCD_CS renamed /FSPICS0
- net /LCD_RESET renamed /GPIO9
- net /SPICS0 renamed /MCU_SPICS0
- net /VBAT_SENSE renamed /GPIO10
Routing:
- net GND: track 187.8 -> 183.9 mm, vias 43 -> 44
- net +3V3: track 258.8 -> 256.2 mm, vias 9 -> 11
- net /USB_D_P: track 28.6 -> 30.1 mm
- net /CAN_P: track 18.2 -> 19.4 mm
- net /CC1: track 3.64 -> 2.58 mm, vias 1 -> 0
- net /CC2: track 4.39 -> 3.53 mm, vias 1 -> 0
- net /FSPIQ: track 33.9 -> 33.3 mm
- net /USB_D_N: track 26.3 -> 25.7 mm, vias 5 -> 4
- net /XTAL_P: track 6.11 -> 5.58 mm
- net /CAN_EN: vias 1 -> 0
Other:
- board text added: "MTCK"
- board text added: "MTDI"
- board text added: "MTDO"
- board text added: "MTMS"
- board text added: "RXD"
- board text added: "TXD"
