File: hardware/gauge-controller/platform-esp.kicad_sch (KiCad schematic)
At the start: 106 parts, among them J1 Conn_ARM_JTAG_SWD_10, J3 PWR_CAN, J4 USB4120-03-C_REVA, J6 TC2030-IDC, SW1 SW_Push, SW2 SW_Push, U1 W25Q128JVS, U2 ESP-PSRAM32, U3 ESP32-S3R2, U4 AP64200Q, U5 LTC2875-DD, Y1 40MHZ

Commit message: restart gauge pcb
Parts:
- removed C10, C33, C34, C35, C36, C37, C38, C39, C40, C41: 1uF, Capacitor_SMD:C_0402_1005Metric, symbol Device:C_Small
- removed C32: 10uF, Capacitor_SMD:C_0402_1005Metric, symbol Device:C_Small
- removed D1, D10, D11, D2, D3, D4, D5, D8, D9: WS2812B, LED_SMD:LED_WS2812B_PLCC4_5.0x5.0mm_P3.2mm, symbol LED:WS2812B
- removed R29: 0, Resistor_SMD:R_0402_1005Metric, symbol Device:R_Small
- removed R4: 442k, Resistor_SMD:R_0402_1005Metric, symbol Device:R_Small
- removed TP10: DC, TestPoint:TestPoint_Pad_D1.0mm, symbol Connector:TestPoint
- removed TP11: RST, TestPoint:TestPoint_Pad_D1.0mm, symbol Connector:TestPoint
- removed TP12: BL, TestPoint:TestPoint_Pad_D1.0mm, symbol Connector:TestPoint
- removed TP13: VDD3V3, TestPoint:TestPoint_Pad_D1.0mm, symbol Connector:TestPoint
- removed TP14: GND, TestPoint:TestPoint_Pad_D1.0mm, symbol Connector:TestPoint
- removed TP5: NEO_OUT, TestPoint:TestPoint_Pad_D1.0mm, symbol Connector:TestPoint
- removed TP6: FSPID, TestPoint:TestPoint_Pad_D1.0mm, symbol Connector:TestPoint
- removed TP7: FSPICS1, TestPoint:TestPoint_Pad_D1.0mm, symbol Connector:TestPoint
- removed TP8: FSPIQ, TestPoint:TestPoint_Pad_D1.0mm, symbol Connector:TestPoint
- removed TP9: FSPICLK, TestPoint:TestPoint_Pad_D1.0mm, symbol Connector:TestPoint
- added J4: Conn_01x09, Connector_GC9A01:GC9A01_disp, symbol Connector_Generic:Conn_01x09
- renumbered C17 to C1, C13 to C10, C14 to C11, C15 to C12, C16 to C13, C2 to C14, C6 to C15, C30 to C16, C1 to C17, C21 to C18, C9 to C19, C19 to C2, C25 to C20, C22 to C21, C23 to C22, C27 to C23, C28 to C24, C29 to C25, C24 to C27, C42 to C28, C4 to C3, C5 to C4, C8 to C5, C18 to C6, C20 to C7, C11 to C8, C12 to C9, D6 to D1, J6 to J1, J3 to J2, J1 to J3, J4 to J5, R5 to R1, R12 to R10, R13 to R11, R27 to R12, R16 to R13, R25 to R14, R17 to R15, R26 to R16, R18 to R17, R3 to R18, R23 to R19, R7 to R2, R21 to R20, R22 to R21, R24 to R22, R20 to R23, R19 to R24, R6 to R3, R14 to R4, R15 to R5, R9 to R6, R10 to R7, R1 to R8, R11 to R9, TP4 to TP1, TP3 to TP2, TP1 to TP3, TP2 to TP4, U3 to U1, U5 to U2, U1 to U3, U2 to U4, U4 to U5
Connections:
- net SPICLK_N: no longer names the net of U1.36 (SPICLK_N)
- net SPICLK_P: no longer names the net of U1.37 (SPICLK_P)
- no-connect marks 24 -> 26
Other:
- added sheet neopixels (neopixels.kicad_sch)

Commit message: asdf
Parts:
- removed C23, C24, C25, C26: DNP, Capacitor_SMD:C_0805_2012Metric_Pad1.18x1.45mm_HandSolder, symbol Device:C_Small
- removed C27: 5.6nf, Capacitor_SMD:C_1206_3216Metric, symbol Device:C_Small
- removed J1: TC2030-IDC, Connector:Tag-Connect_TC2030-IDC-NL_2x03_P1.27mm_Vertical, symbol Connector_TDC:TC2030-IDC
- removed J3: Conn_ARM_JTAG_SWD_10, Connector:Tag-Connect_TC2050-IDC-NL_2x05_P1.27mm_Vertical, symbol Connector:Conn_ARM_JTAG_SWD_10
- removed L4: 6.8uh, Inductor_SMD:L_Bourns-SRN6028, symbol Device:L_Small
- removed U4: ESP-PSRAM32, Package_SO:SOIC-8_3.9x4.9mm_P1.27mm, symbol Memory_RAM:ESP-PSRAM32
- removed U5: AP64200Q, Package_SO:SOIC-8-1EP_3.9x4.9mm_P1.27mm_EP2.29x3mm_ThermalVias, symbol AP1509-50SG-13:AP64200Q
- added D11: D_Small, Diode_SMD:D_SOD-123F, symbol Device:D_Small
- added Q1: Q_NPN_EBC, Package_TO_SOT_SMD:TSOT-23, symbol Device:Q_NPN_EBC
- added R26: 10R, Resistor_SMD:R_0402_1005Metric, symbol Device:R_Small
- added R27: 100k, Resistor_SMD:R_0402_1005Metric, symbol Device:R_Small
- added TP10, TP11: 3V3OUT, TestPoint:TestPoint_Pad_D1.0mm, symbol Connector:TestPoint
- added TP6: MTDO, TestPoint:TestPoint_Pad_D1.0mm, symbol Connector:TestPoint
- added TP7: MTDI, TestPoint:TestPoint_Pad_D1.0mm, symbol Connector:TestPoint
- added TP8: TXD, TestPoint:TestPoint_Pad_D1.0mm, symbol Connector:TestPoint
- added TP9: RXD, TestPoint:TestPoint_Pad_D1.0mm, symbol Connector:TestPoint
- added U5: ADP2303ARDZ-3.3, Package_SO:SOIC-8-1EP_3.9x4.9mm_P1.27mm_EP2.29x3mm_ThermalVias, symbol Regulator_Switching:ADP2303ARDZ-3.3
- C10: value C_Small -> 10uF; footprint Capacitor_SMD:C_0402_1005Metric -> Capacitor_SMD:C_0805_2012Metric; VOLTAGE (none) -> 25V
- C20: value 0.1uf -> 0.1uF; footprint Capacitor_SMD:C_0805_2012Metric_Pad1.18x1.45mm_HandSolder -> Capacitor_SMD:C_0805_2012Metric; DESCRIPTION CAP CER 0.1UF 16V X7R 0805 -> (none); MPN 0805 (2012 Metric) 0,94mm -> (none)
- C21, C22: value 10uf -> 22uF; footprint Capacitor_SMD:C_0805_2012Metric_Pad1.18x1.45mm_HandSolder -> Capacitor_SMD:C_0805_2012Metric; DESCRIPTION CAP CER 10UF 25V X5R 0805 -> (none); MPN C0805C106M3PAC7800 -> (none)
- J4: value Conn_01x09 -> Conn_01x12; symbol Connector_Generic:Conn_01x09 -> Connector_Generic:Conn_01x12
- L3: value 0H -> 6.8uh; footprint Inductor_SMD:L_0402_1005Metric -> Inductor_SMD:L_Bourns-SRN6028; DESCRIPTION (none) -> FIXED IND 6.8UH 2.2A 63 MOHM SMD; MPN (none) -> SRN6028-6R8M
- R18: value 100k -> 10k
- R19: value 52.3k -> 100k; footprint Resistor_SMD:R_0603_1608Metric_Pad0.98x0.95mm_HandSolder -> Resistor_SMD:R_0603_1608Metric; DESCRIPTION RES 52.3K OHM 1% 1/10W 0603 -> (none); MPN RMCF0603FT52K3 -> (none)
- R20: value 200k -> 31k6; footprint Resistor_SMD:R_0603_1608Metric_Pad0.98x0.95mm_HandSolder -> Resistor_SMD:R_0603_1608Metric; DESCRIPTION RES 200K OHM 5% 1/10W 0603 -> (none); MPN RMCF0603JT200K -> (none)
- R21: value 14k -> 10k2; footprint Resistor_SMD:R_0603_1608Metric_Pad0.98x0.95mm_HandSolder -> Resistor_SMD:R_0603_1608Metric; DESCRIPTION RES 14K OHM 1% 1/10W 0603 -> (none); MPN RMCF0603FT14K0 -> (none)
- R22: footprint Resistor_SMD:R_0603_1608Metric_Pad0.98x0.95mm_HandSolder -> Resistor_SMD:R_0402_1005Metric; DESCRIPTION RES 10K OHM 5% 1/10W 0603 -> (none); MPN RMCF0603JT10K0 -> (none)
- TP3: value 3V3OUT -> MTCK
- TP4: value 3V3OUT -> MTMS
- U1: footprint Package_DFN_QFN:QFN-56-1EP_7x7mm_P0.4mm_EP5.6x5.6mm -> Package_DFN_QFN:QFN-56-1EP_7x7mm_P0.4mm_EP5.6x5.6mm_ThermalVias
- U3: footprint Package_SO:SOIC-8_5.23x5.23mm_P1.27mm -> Package_SO:SOIC-8W_5.3x5.3mm_P1.27mm; JLCPCB (none) -> C97521
- Y1: footprint Crystal:Crystal_SMD_2016-4Pin_2.0x1.6mm -> Crystal:Crystal_SMD_3225-4Pin_3.2x2.5mm; JLCPCB (none) -> C9010; MPN ECS-400-10-37B2-CKY-TR -> (none)
Connections:
- net GPIO11 is gone; now on net FSPICS0: U1.16 (GPIO11)
- net VDDCPU is gone; now on net +3V3: C9.1, U1.46 (VDD3P3_CPU)
- net VDDRTC is gone; now on net +3V3: C8.1, U1.20 (VDD3P3_RTC)
- net +3V3: now also C19.2, C21.1, C22.1, J4.3 (Pin_3), J4.4 (Pin_4), R20.1, R22.2, U1.2 (VDD3P3), U1.3 (VDD3P3), R27.1, TP11.1; no longer C19.1, R18.2, R19.1, TP4.1
- net BL: now also R18.1
- net CAN_DRV_N: now also J2.2 (Pin_2); no longer J2.3 (Pin_3)
- net CAN_DRV_P: now also J2.1 (Pin_1); no longer J2.4 (Pin_4)
- net CHIP_PU: now also C19.1
- net DC: now also J4.7 (Pin_7)
- net EXT_VIN: now also J2.4 (Pin_4); no longer J2.2 (Pin_2)
- net FSPICLK: now also J4.9 (Pin_9)
- net FSPICS0: now also J4.8 (Pin_8), R27.2; no longer U1.39 (GPIO34)
- net FSPIQ: now also J4.10 (Pin_10)
- net GND: now also C21.2, C22.2, J2.3 (Pin_3), J4.1 (Pin_1), J4.12 (Pin_12), J4.5 (Pin_5), J4.6 (Pin_6), R21.2, Q1.1 (E), TP10.1, U5.7 (GND), U5.9 (PADGND); no longer C19.2, C21.1, C22.1, J2.1 (Pin_1), R20.2, R22.2, TP3.1
- net GPIO10: now also R14.2, R16.1, TP2.1
- net GPIO2: no longer R14.2, R16.1, TP2.1
- net MTCK: now also TP3.1
- net MTDI: now also TP7.1
- net MTDO: now also TP6.1
- net MTMS: now also TP4.1
- net U0RXD: now also TP9.1
- net U0TXD: now also TP8.1
- net USB_VBUS: now also D11.2 (A)
- net VIN: now also C10.2, R19.1, D11.1 (K), U5.2 (Vin), U5.3 (EN); no longer C21.2, C22.2
- net MCU_SPIWP: now reaches R7.2, U1.31 (SPIWP)
- net MCU_SPIHD: now reaches R6.2, U1.30 (SPIHD)
- net BST: now reaches C20.1
- net BST: now also U5.1 (BST)
- net LCD_BL_DIV: now reaches R22.1
- net LCD_BL_DIV: now also R18.2, Q1.2 (B); no longer R19.2
- net FB: now reaches R21.1
- net FB: now also R20.2, U5.5 (FB)
- net SW: now reaches C20.2
- net SW: now also L3.1, U5.8 (SW)
- net MCU_SPIQ: now reaches R10.2, U1.34 (SPIQ)
- net MCU_SPICLK: now reaches R9.2, U1.33 (SPICLK)
- net MCU_SPID: now reaches R11.2, U1.35 (SPID)
- net MCU_U0TXD: now reaches R3.2, U1.49 (U0TXD)
- net MCU_XTAL_N: now reaches R2.2, U1.53 (XTAL_N)
- net CHIP_PU_BOOTSTRAP: now reaches C18.1, SW1.2
- net LCD_LEDK: now reaches J4.2 (Pin_2)
- net LCD_LEDK: now also R26.1
- net FSPICS1 renamed GPIO9
- net GPIO9: now also J4.11 (Pin_11)
- net SPICS0 renamed MCU_SPICS0
- net SPICS1: no longer names the net of U1.28 (SPICS1)
- net SPICS1: no longer R18.1
- removed net VDD3V3: C10.2, L3.1, U1.2 (VDD3P3), U1.3 (VDD3P3)
- new net GPIO34: U1.39 (GPIO34)
- new net PGOOD: R19.2, U5.4 (PGOOD)
- new net Q_LEDK: Q1.3 (C), R26.2
- no-connect marks 26 -> 18
Other:
- sheet neopixels ports: added NEO_OUT; removed none
- note removed: "0R resistors should be near chip not cpu"
- note removed: "Pretty sure the resistor network here needs to be recalculated for 3.3V. Consult Datasheet"
- moved on the sheet: AE1, C14, C15, C16, C17, C18, C28, C3, C4, C5, C8, C9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

Commit message: misc cleanup
Parts:
- J1: renamed from J5; footprint Connector_GCT_USB:GCT_USB4120-03-C_REVA -> ConeCodes:GCT_USB4120-03-C_REVA; symbol Connector_GCT_USB:USB4120-03-C_REVA -> ConeCodes:USB4120-03-C_REVA
- J4: footprint Connector_GC9A01:GC9A01_disp -> ConeCodes:GC9A01_disp
- SW1, SW2: footprint SW_RS-032G05A3-SMRT:SW_RS-032G05A3-SMRT -> ConeCodes:SW_RS-032G05A3-SMRT
- U1: footprint Package_DFN_QFN:QFN-56-1EP_7x7mm_P0.4mm_EP5.6x5.6mm_ThermalVias -> ConeCodes:QFN-56; symbol MCU_ESP:ESP32-S3R2 -> ConeCodes:ESP32-S3R2; MP ESP32-S3R2 -> (none); MPN (none) -> ESP32-S3
Changed lines of the file:
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@@
     (pin "1")
   )
-  (symbol (lib_id "MCU_ESP:ESP32-S3R2") (at 154.94 121.92 0) (unit 1)
-    (in_bom yes) (on_board yes) (fields_autoplaced)
-    (property "Reference" "U1" (id 0) (at 154.94 68.58 0))
-    (property "Value" "ESP32-S3R2" (id 1) (at 154.94 71.12 0))
-    (property "Footprint" "Package_DFN_QFN:QFN-56-1EP_7x7mm_P0.4mm_EP5.6x5.6mm_ThermalVias" (id 2) (at 154.94 121.92 0)
+  (symbol (lib_id "ConeCodes:ESP32-S3R2") (at 154.94 121.92 0) (unit 1)
+    (in_bom yes) (on_board yes) (fields_autoplaced)
+    (property "Reference" "U1" (id 0) (at 154.94 66.04 0))
+    (property "Value" "ESP32-S3R2" (id 1) (at 154.94 68.58 0))
+    (property "Footprint" "ConeCodes:QFN-56" (id 2) (at 154.94 121.92 0)
       (effects (font (size 1.27 1.27)) (justify left bottom) hide)
     )
@@
       (effects (font (size 1.27 1.27)) (justify left bottom) hide)
     )
-    (property "Description" "Espressif Systems [ENGINEERING SAMPLES]SMD IC , Dual-Core MCU, Wi-Fi 2.4G & BLE 5.0 combo, 8 MB Octal SPI PSRAM, QFN 56-pin, 7*7 mm" (id 4) (at 193.04 133.35 0)
-      (effects (font (size 1.27 1.27)) (justify left bottom) hide)
-    )
-    (property "MP" "ESP32-S3R2" (id 5) (at 193.04 120.65 0)
-      (effects (font (size 1.27 1.27)) (justify left bottom) hide)
-    )
+    (property "MPN" "ESP32-S3" (id 4) (at 154.94 71.12 0))
     (pin "1")
     (pin "10")
@@
     (property "Reference" "SW1" (id 0) (at 268.605 158.115 0))
     (property "Value" "SW_Push" (id 1) (at 268.605 160.655 0))
-    (property "Footprint" "SW_RS-032G05A3-SMRT:SW_RS-032G05A3-SMRT" (id 2) (at 268.605 161.29 0)
+    (property "Footprint" "ConeCodes:SW_RS-032G05A3-SMRT" (id 2) (at 268.605 161.29 0)
       (effects (font (size 1.27 1.27)) hide)
     )
@@
     (property "Reference" "SW2" (id 0) (at 283.845 170.18 0))
     (property "Value" "SW_Push" (id 1) (at 283.845 172.72 0))
-    (property "Footprint" "SW_RS-032G05A3-SMRT:SW_RS-032G05A3-SMRT" (id 2) (at 283.845 173.355 0)
+    (property "Footprint" "ConeCodes:SW_RS-032G05A3-SMRT" (id 2) (at 283.845 173.355 0)
       (effects (font (size 1.27 1.27)) hide)
     )
@@
       (effects (font (size 1.27 1.27)) (justify left))
     )
-    (property "Footprint" "Connector_GC9A01:GC9A01_disp" (id 2) (at 287.02 259.08 0)
+    (property "Footprint" "ConeCodes:GC9A01_disp" (id 2) (at 287.02 259.08 0)
       (effects (font (size 1.27 1.27)) hide)
     )
@@
     (pin "2")
   )
-  (symbol (lib_id "Connector_GCT_USB:USB4120-03-C_REVA") (at 426.72 278.765 0) (unit 1)
-    (in_bom yes) (on_board yes) (fields_autoplaced)
-    (property "Reference" "J5" (id 0) (at 426.72 255.27 0))
+  (symbol (lib_id "ConeCodes:USB4120-03-C_REVA") (at 426.72 278.765 0) (unit 1)
+    (in_bom yes) (on_board yes) (fields_autoplaced)
+    (property "Reference" "J1" (id 0) (at 426.72 255.27 0))
     (property "Value" "USB4120-03-C_REVA" (id 1) (at 426.72 257.81 0))
-    (property "Footprint" "Connector_GCT_USB:GCT_USB4120-03-C_REVA" (id 2) (at 453.39 282.575 0)
+    (property "Footprint" "ConeCodes:GCT_USB4120-03-C_REVA" (id 2) (at 453.39 282.575 0)
       (effects (font (size 1.27 1.27)) (justify left bottom) hide)
     )
-    (property "Datasheet" "" (id 3) (at 426.72 278.765 0)
+    (property "Datasheet" "https://www.mouser.com/datasheet/2/837/USB4120-2888136.pdf" (id 3) (at 426.72 278.765 0)
       (effects (font (size 1.27 1.27)) (justify left bottom) hide)
     )
@@
       (reference "D11") (unit 1) (value "D_Small") (footprint "Diode_SMD:D_SOD-123F")
     )
+    (path "/cca1fecf-4e0f-4e8c-836b-942398b258c1"
+      (reference "J1") (unit 1) (value "USB4120-03-C_REVA") (footprint "ConeCodes:GCT_USB4120-03-C_REVA")
+    )
     (path "/32d4d42c-48dd-4942-8faa-8acdeacf5d9d"
       (reference "J2") (unit 1) (value "PWR_CAN") (footprint "Connector_JST:JST_GH_BM04B-GHS-TBT_1x04-1MP_P1.25mm_Vertical")
     )
     (path "/c4aca2c6-460e-455d-8b12-0cde9b5f778b"
-      (reference "J4") (unit 1) (value "Conn_01x12") (footprint "Connector_GC9A01:GC9A01_disp")
-    )
-    (path "/cca1fecf-4e0f-4e8c-836b-942398b258c1"
-      (reference "J5") (unit 1) (value "USB4120-03-C_REVA") (footprint "Connector_GCT_USB:GCT_USB4120-03-C_REVA")
+      (reference "J4") (unit 1) (value "Conn_01x12") (footprint "ConeCodes:GC9A01_disp")
     )
     (path "/16394e05-953e-4d85-99a4-e52777725bb0"
@@
     )
     (path "/aec1a0e8-2f0a-40ed-aeb9-24e4d9460012"
-      (reference "SW1") (unit 1) (value "SW_Push") (footprint "SW_RS-032G05A3-SMRT:SW_RS-032G05A3-SMRT")
+      (reference "SW1") (unit 1) (value "SW_Push") (footprint "ConeCodes:SW_RS-032G05A3-SMRT")
     )
     (path "/c25af67b-4b08-42f1-9587-82920da94065"
-      (reference "SW2") (unit 1) (value "SW_Push") (footprint "SW_RS-032G05A3-SMRT:SW_RS-032G05A3-SMRT")
+      (reference "SW2") (unit 1) (value "SW_Push") (footprint "ConeCodes:SW_RS-032G05A3-SMRT")
     )
     (path "/f43ee131-f516-4210-9dfe-a839a99357cc"
@@
     )
     (path "/72f86fac-1de9-4853-b551-bbe9529da2a3"
-      (reference "U1") (unit 1) (value "ESP32-S3R2") (footprint "Package_DFN_QFN:QFN-56-1EP_7x7mm_P0.4mm_EP5.6x5.6mm_ThermalVias")
+      (reference "U1") (unit 1) (value "ESP32-S3R2") (footprint "ConeCodes:QFN-56")
     )
     (path "/db98d1f9-d37d-4661-a306-646143bda473"
