File: hardware/underglow-controller/CONEPROJ.kicad_sch (KiCad schematic)
At the start: 141 parts, among them J2 U.FL-R-SMT-1(10), J3 DM3AT-SF-PEJM5, J4 DTM1312PA12PBR008, J5 Conn_01x10, J6 CONSOLE, J7 U.FL-R-SMT-1(10), J8 JTAG, Q2 Q_Dual_NMOS_S1G1S2G2D2D2D1D1, Q3 Q_Dual_NMOS_S1G1S2G2D2D2D1D1, Q4 Q_Dual_NMOS_S1G1S2G2D2D2D1D1, SW2 SW_Push, SW3 SW_Push, SW4 SW_Push, U10 DRV8844PWP, U11 RP2040, U2 ESP-PSRAM32, U3 SN65HVD230, U4 ESP32-S3R2, U5 W25Q128JVS, U6 WS2815B, U7 W25Q128JVS, U8 ADP2303ARDZ-3.3, U9 RFM69HCW, Y2 40MHZ, Y3 32.7k, Y4 40MHZ

Commit message: asdf
Other:
- note removed: "Pretty sure the resistor network here needs to be recalculated for 3.3V. Consult Datasheet"
Changed lines of the file:
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@@
-    (effects (font (size 1.27 1.27)) (justify left bottom))
-  )
-  (text "Pretty sure the resistor network here\nneeds to be recalculated for\n3.3V. Consult Datasheet"
-    (at 422.275 85.09 0)
     (effects (font (size 1.27 1.27)) (justify left bottom))
   )

Commit message: misc cleanup
Parts:
- J2, J7: footprint U.FL-R-SMT-1_10_:HRS_U.FL-R-SMT-1(10) -> ConeCodes:HRS_U.FL-R-SMT-1(10)
- J3: footprint Connector_Hirose_SD:HRS_DM3AT-SF-PEJM5 -> ConeCodes:HRS_DM3AT-SF-PEJM5; symbol Connector_Hirose_SD:DM3AT-SF-PEJM5 -> ConeCodes:DM3AT-SF-PEJM5
- J4: footprint TE_DTM1312PA12PBR008:TE_DTM1312PA12PBR008 -> TE_DTM1312PA12PBR008; symbol TE_DTM1312PA12PBR008:DTM1312PA12PBR008 -> ConeCodes:DTM1312PA12PBR008; DESCRIPTION CONN HEADER R/A 24POS -> (none); now in the parts list
- SW2, SW3, SW4: footprint SW_RS-032G05A3-SMRT:SW_RS-032G05A3-SMRT -> ConeCodes:SW_RS-032G05A3-SMRT
- U10: footprint DRV8844PWP:IC_TPS61196PWPRQ1 -> Package_SO:HTSSOP-28-1EP_4.4x9.7mm_P0.65mm_EP2.85x5.4mm_ThermalVias; symbol DRV8844PWP:DRV8844PWP -> ConeCodes:DRV8844PWP; DESCRIPTION IC MTR DRV BIPOLR 8-60V 28HTSSOP -> (none)
- U11: footprint RP2040:RP2040-QFN-56 -> ConeCodes:QFN-56; symbol RP2040:RP2040 -> ConeCodes:RP2040
- U4: footprint Package_DFN_QFN:QFN-56-1EP_7x7mm_P0.4mm_EP5.6x5.6mm_ThermalVias -> ConeCodes:QFN-56; symbol MCU_ESP:ESP32-S3R2 -> ConeCodes:ESP32-S3R2; MP ESP32-S3R2 -> (none); MPN (none) -> ESP32-S3
- U6: footprint WS2815B:worldsemi-WS2815B-MFG -> ConeCodes:worldsemi-WS2815B-MFG; symbol WS2815B:WS2815B -> ConeCodes:WS2815B; MPN WS2815B -> (none)
- U9: value RFM69HCW -> COM-13909; footprint XCVR_RFM69HW:XCVR_RFM69HW -> ConeCodes:XCVR_RFM69HW; symbol RFM69HW:COM-13909 -> ConeCodes:COM-13909; DESCRIPTION RX TXRX MODULE ISM < 1GHZ SMD -> (none); MPN COM-13909 -> RFM69HCW; MPN2 (none) -> COM-13909
Connections:
- net GND: no longer U10.30 (GND), U10.31 (GND), U10.32 (GND), U10.33 (GND), U10.34 (GND), U10.35 (GND), U10.36 (GND), U10.37 (GND), U10.38 (GND), U10.39 (GND), U10.40 (GND), U10.41 (GND), U10.42 (GND), U10.43 (GND), U10.44 (GND), U10.45 (GND), U10.46 (GND), U10.47 (GND), U10.48 (GND), U10.49 (GND), U10.50 (GND)
