File: hardware/underglow-controller/CONEPROJ.kicad_sch (KiCad schematic)
At the start: 141 parts, among them J2 U.FL-R-SMT-1(10), J3 DM3AT-SF-PEJM5, J4 DTM1312PA12PBR008, J5 Conn_01x10, J6 Conn_ARM_JTAG_SWD_10, J7 U.FL-R-SMT-1(10), Q2 Q_Dual_NMOS_S1G1S2G2D2D2D1D1, Q3 Q_Dual_NMOS_S1G1S2G2D2D2D1D1, Q4 Q_Dual_NMOS_S1G1S2G2D2D2D1D1, SW2 SW_Push, SW3 SW_Push, SW4 SW_Push, U10 DRV8844PWP, U11 RP2040, U2 ESP-PSRAM32, U3 SN65HVD230, U4 ESP32-S3R2, U5 W25Q128JVS, U6 WS2815B, U7 W25Q128JVS, U8 AP64200Q, U9 RFM69HCW, Y2 40MHZ, Y3 32.7k, Y4 40MHZ

Commit message: Add pullups to sdcard
Parts:
- removed TP?: INT, TestPoint:TestPoint_Pad_D1.0mm, symbol Connector:TestPoint
- added R40, R43, R44, R45: 10k, Resistor_SMD:R_0402_1005Metric, symbol Device:R_Small
Connections:
- net +3V3: now also R40.1, R43.1, R44.1, R45.1
- net FSPID: now also R40.2
- net FSPIQ: now also R43.2
- net SD_D2: now reaches J3.1 (DAT2)
- net SD_D2: now also R45.2
- net SD_D1: now reaches J3.8 (DAT1)
- net SD_D1: now also R44.2
- no-connect marks 30 -> 28

Commit message: Fix antenna impedance
Connections:
- net GPIO0 is gone; now on net CTS: R25.1, U4.5 (GPIO0)
- net RTS is gone; now on net CHIP_PU: TC2.6 (SWO)
- net RF69_RF_ANT_PCB: now reaches AE3.1 (A), R33.2
- net RF_ANT_EXT: now reaches J7.2, R28.1
- net RF69_RF_EXT: now reaches J2.2, R32.2
Other:
- moved on the sheet: AE3, J2, J7, R32, R40, R43, R44, R45

Commit message: add debug headers, change pmic to something in stock
Parts:
- removed C27: 10uf, Capacitor_SMD:C_0805_2012Metric_Pad1.18x1.45mm_HandSolder, symbol Device:C_Small
- removed C30: 5.6nf, Capacitor_SMD:C_1206_3216Metric, symbol Device:C_Small
- removed C34, C36: DNP, Capacitor_SMD:C_0805_2012Metric_Pad1.18x1.45mm_HandSolder, symbol Device:C_Small
- removed J6: Conn_ARM_JTAG_SWD_10, Connector:Tag-Connect_TC2050-IDC-NL_2x05_P1.27mm_Vertical, symbol Connector:Conn_ARM_JTAG_SWD_10
- removed R29: 14k, Resistor_SMD:R_0603_1608Metric_Pad0.98x0.95mm_HandSolder, symbol Device:R_Small
- removed U8: AP64200Q, Package_SO:SOIC-8-1EP_3.9x4.9mm_P1.27mm_EP2.29x3mm_ThermalVias, symbol AP1509-50SG-13:AP64200Q
- added J6: CONSOLE, Connector_PinHeader_1.27mm:PinHeader_1x06_P1.27mm_Vertical, symbol Connector_Generic:Conn_01x06
- added J8: JTAG, Connector_PinHeader_1.27mm:PinHeader_1x06_P1.27mm_Vertical, symbol Connector_Generic:Conn_01x06
- added TC4: TC2030-IDC, Connector:Tag-Connect_TC2030-IDC-NL_2x03_P1.27mm_Vertical, symbol TDC-2030-IDC:TC2030-IDC
- added U8: ADP2303ARDZ-3.3, Package_SO:SOIC-8-1EP_3.9x4.9mm_P1.27mm_EP2.29x3mm, symbol Regulator_Switching:ADP2303ARDZ-3.3
- AE2, AE3, H1, J2, J4, J5, J7, JP2, Q2, Q3, Q4, TC2, U3, U5: now left out of the parts list
- C25: value 10uf -> 10uF; footprint Capacitor_SMD:C_0805_2012Metric_Pad1.18x1.45mm_HandSolder -> Capacitor_SMD:C_0805_2012Metric; DESCRIPTION CAP CER 10UF 25V X5R 0805 -> (none); MPN C0805C106M3PAC7800 -> (none); VOLTAGE (none) -> 25V
- C32, C43: value 0.1uf -> 0.1uF; footprint Capacitor_SMD:C_0805_2012Metric_Pad1.18x1.45mm_HandSolder -> Capacitor_SMD:C_0805_2012Metric; DESCRIPTION CAP CER 0.1UF 16V X7R 0805 -> (none); MPN 0805 (2012 Metric) 0,94mm -> (none)
- C39, C41: value DNP -> 22uF; footprint Capacitor_SMD:C_0805_2012Metric_Pad1.18x1.45mm_HandSolder -> Capacitor_SMD:C_0805_2012Metric
- C42: value 0.47uf -> 0.47uF; footprint Capacitor_SMD:C_0805_2012Metric_Pad1.18x1.45mm_HandSolder -> Capacitor_SMD:C_0805_2012Metric; DESCRIPTION CAP CER 0.47UF 6.3V X7R 0805 -> (none); MPN CGJ4J2X7R0J474K125AA -> (none)
- C44: value 10uf -> 10uF; footprint Capacitor_SMD:C_0805_2012Metric_Pad1.18x1.45mm_HandSolder -> Capacitor_SMD:C_0805_2012Metric; DESCRIPTION CAP CER 10UF 25V X5R 0805 -> (none); MPN C0805C106M3PAC7800 -> (none)
- C45, C5: footprint Capacitor_SMD:C_0805_2012Metric_Pad1.18x1.45mm_HandSolder -> Capacitor_SMD:C_0805_2012Metric; DESCRIPTION CAP CER 10UF 16V X5R 0805 -> (none); MPN CL21A106KOQNNNE -> (none)
- C46: value 0.01uf -> 0.01uF; footprint Capacitor_SMD:C_0805_2012Metric_Pad1.18x1.45mm_HandSolder -> Capacitor_SMD:C_0805_2012Metric; DESCRIPTION CAP CER SMD 0805 .01UF 100V X7R -> (none); MPN C0805C103K1RAC7210 -> (none)
- C47: value 10uf -> 10uF; footprint Capacitor_SMD:CP_Elec_5x5.9 -> Capacitor_SMD:CP_Elec_5x5.3; DESCRIPTION CAP ALUM 10UF 20% 50V SMD -> (none); MPN 50TZV10M5X6.1 -> (none)
- C6: footprint Capacitor_SMD:C_0805_2012Metric_Pad1.18x1.45mm_HandSolder -> Capacitor_SMD:C_0805_2012Metric
- D2, D3, D4: footprint LED_SMD:LED_0603_1608Metric_Pad1.05x0.95mm_HandSolder -> LED_SMD:LED_0603_1608Metric
- R10, R11, R12, R13, R16, R17, R22, R28, R32, R33, R7, R8, R9: value 0 -> 0R
- R18, R19, R20: value 240 -> 240R; footprint Resistor_SMD:R_0603_1608Metric_Pad0.98x0.95mm_HandSolder -> Resistor_SMD:R_0603_1608Metric
- R23: value 200k -> 100k; footprint Resistor_SMD:R_0603_1608Metric_Pad0.98x0.95mm_HandSolder -> Resistor_SMD:R_0603_1608Metric; DESCRIPTION RES 200K OHM 5% 1/10W 0603 -> (none); MPN RMCF0603JT200K -> (none)
- R34: value 52.3k -> 31k6; footprint Resistor_SMD:R_0603_1608Metric_Pad0.98x0.95mm_HandSolder -> Resistor_SMD:R_0603_1608Metric; DESCRIPTION RES 52.3K OHM 1% 1/10W 0603 -> (none); MPN RMCF0603FT52K3 -> (none)
- R35: value 10k -> 10k2; footprint Resistor_SMD:R_0603_1608Metric_Pad0.98x0.95mm_HandSolder -> Resistor_SMD:R_0603_1608Metric; DESCRIPTION RES 10K OHM 5% 1/10W 0603 -> (none); MPN RMCF0603JT10K0 -> (none)
- R39: footprint Resistor_SMD:R_0603_1608Metric_Pad0.98x0.95mm_HandSolder -> Resistor_SMD:R_0603_1608Metric
- R6: value 499 -> 499R
Connections:
- net CHIP_PU: now also J6.6 (Pin_6)
- net CTS: now also J6.5 (Pin_5)
- net GND: now also J6.1 (Pin_1), J8.5 (Pin_5), TC4.5 (GND), U8.7 (GND), U8.9 (PADGND); no longer R23.2
- net MTCK: now also J8.1 (Pin_1), TC4.4 (TCK)
- net MTDI: now also J8.4 (Pin_4), TC4.3 (TDI)
- net MTDO: now also J8.2 (Pin_2), TC4.6 (TDO)
- net MTMS: now also J8.3 (Pin_3), TC4.2 (TMS)
- net RXD: now also J6.2 (Pin_2)
- net TXD: now also J6.3 (Pin_3)
- net VIN: now also R23.1, U8.2 (Vin), U8.3 (EN)
- net BST: now reaches C32.1
- net BST: now also U8.1 (BST)
- net SW: now reaches C32.2, L6.1
- net SW: now also U8.8 (SW)
- net FB: now reaches R34.2, R35.1
- net FB: now also U8.5 (FB)
- new net PGOOD: R23.2, U8.4 (PGOOD)
- no-connect marks 28 -> 30
Other:
- note removed: "PCB Antenna would be nice here for use without an SMA connector"
- moved on the sheet: AE3, C25, C32, C39, C41, L6, R23, R33, R34, R35, TP4, TP7

Commit message: Multi gauge pcb design
Parts:
- J2, J7: footprint U.FL-R-SMT-1_10_:HRS_U.FL-R-SMT-1(10) -> ConeCodes:HRS_U.FL-R-SMT-1(10)
- J3: footprint Connector_Hirose_SD:HRS_DM3AT-SF-PEJM5 -> ConeCodes:HRS_DM3AT-SF-PEJM5; symbol Connector_Hirose_SD:DM3AT-SF-PEJM5 -> ConeCodes:DM3AT-SF-PEJM5
- J4: footprint TE_DTM1312PA12PBR008:TE_DTM1312PA12PBR008 -> TE_DTM1312PA12PBR008; symbol TE_DTM1312PA12PBR008:DTM1312PA12PBR008 -> ConeCodes:DTM1312PA12PBR008; DESCRIPTION CONN HEADER R/A 24POS -> (none); now in the parts list
- SW2, SW3, SW4: footprint SW_RS-032G05A3-SMRT:SW_RS-032G05A3-SMRT -> ConeCodes:SW_RS-032G05A3-SMRT
- U10: footprint DRV8844PWP:IC_TPS61196PWPRQ1 -> Package_SO:HTSSOP-28-1EP_4.4x9.7mm_P0.65mm_EP2.85x5.4mm_ThermalVias; symbol DRV8844PWP:DRV8844PWP -> ConeCodes:DRV8844PWP; DESCRIPTION IC MTR DRV BIPOLR 8-60V 28HTSSOP -> (none)
- U11: footprint RP2040:RP2040-QFN-56 -> ConeCodes:QFN-56; symbol RP2040:RP2040 -> ConeCodes:RP2040
- U4: footprint Package_DFN_QFN:QFN-56-1EP_7x7mm_P0.4mm_EP5.6x5.6mm_ThermalVias -> ConeCodes:QFN-56; symbol MCU_ESP:ESP32-S3R2 -> ConeCodes:ESP32-S3R2; MP ESP32-S3R2 -> (none); MPN (none) -> ESP32-S3
- U6: footprint WS2815B:worldsemi-WS2815B-MFG -> ConeCodes:worldsemi-WS2815B-MFG; symbol WS2815B:WS2815B -> ConeCodes:WS2815B; MPN WS2815B -> (none)
- U9: value RFM69HCW -> COM-13909; footprint XCVR_RFM69HW:XCVR_RFM69HW -> ConeCodes:XCVR_RFM69HW; symbol RFM69HW:COM-13909 -> ConeCodes:COM-13909; DESCRIPTION RX TXRX MODULE ISM < 1GHZ SMD -> (none); MPN COM-13909 -> RFM69HCW; MPN2 (none) -> COM-13909
Connections:
- net GND: no longer U10.30 (GND), U10.31 (GND), U10.32 (GND), U10.33 (GND), U10.34 (GND), U10.35 (GND), U10.36 (GND), U10.37 (GND), U10.38 (GND), U10.39 (GND), U10.40 (GND), U10.41 (GND), U10.42 (GND), U10.43 (GND), U10.44 (GND), U10.45 (GND), U10.46 (GND), U10.47 (GND), U10.48 (GND), U10.49 (GND), U10.50 (GND)
Other:
- note removed: "Pretty sure the resistor network here needs to be recalculated for 3.3V. Consult Datasheet"

Commit message: Update PCBs to share the same components
* 3x flash memory
* CAN transciever
Parts:
- U5, U7: footprint Package_SO:SOIC-8_5.23x5.23mm_P1.27mm -> Package_SO:SOIC-8W_5.3x5.3mm_P1.27mm
Changed lines of the file:
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@@
       (effects (font (size 1.27 1.27)) (justify left))
     )
-    (property "Footprint" "Package_SO:SOIC-8_5.23x5.23mm_P1.27mm" (id 2) (at 408.94 215.9 0)
+    (property "Footprint" "Package_SO:SOIC-8W_5.3x5.3mm_P1.27mm" (id 2) (at 408.94 215.9 0)
       (effects (font (size 1.27 1.27)) hide)
     )
@@
       (effects (font (size 1.27 1.27)) (justify left))
     )
-    (property "Footprint" "Package_SO:SOIC-8_5.23x5.23mm_P1.27mm" (id 2) (at 187.325 284.48 0)
+    (property "Footprint" "Package_SO:SOIC-8W_5.3x5.3mm_P1.27mm" (id 2) (at 187.325 284.48 0)
       (effects (font (size 1.27 1.27)) hide)
     )
@@
     )
     (path "/97d5d817-f71f-49de-beef-e9a1419db36f"
-      (reference "U5") (unit 1) (value "W25Q128JVS") (footprint "Package_SO:SOIC-8_5.23x5.23mm_P1.27mm")
+      (reference "U5") (unit 1) (value "W25Q128JVS") (footprint "Package_SO:SOIC-8W_5.3x5.3mm_P1.27mm")
     )
     (path "/1c2c96c8-998a-414a-b0c9-30634f462a04"
@@
     )
     (path "/5661b0a3-fe72-4ea8-a69d-c3a61f09863a"
-      (reference "U7") (unit 1) (value "W25Q128JVS") (footprint "Package_SO:SOIC-8_5.23x5.23mm_P1.27mm")
+      (reference "U7") (unit 1) (value "W25Q128JVS") (footprint "Package_SO:SOIC-8W_5.3x5.3mm_P1.27mm")
     )
     (path "/955f7cca-9d61-4555-ab43-66adbd5ec258"
