File: hardware/underglow-controller/pico.kicad_sch (KiCad schematic)
At the start: 32 parts, among them J9 Spare IO, SW4 USB BOOT, SW5 SW_Push, U11 RP2040, U7 W25Q128JVS, Y4 12MHZ

Commit message: pcb updates
Parts:
- renumbered D4 to D3, D3 to D4
Connections:
- net USB_DN renamed USB_D_N
- net USB_DP renamed USB_D_P
Other:
- company: (none) -> cone.codes
- title: (none) -> CAN RGB Controller
Changed lines of the file:
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@@
 (kicad_sch (version 20211123) (generator eeschema)
   (paper "A4")
+  (title_block
+    (title "CAN RGB Controller")
+    (date "2022-05-30")
+    (rev "B")
+    (company "cone.codes")
+    (comment 1 "https://github.com/miata-bot/can-link")
+  )
   (junction (at 169.545 44.45) (diameter 0) (color 0 0 0 0)
   )
@@
     (effects (font (size 1.27 1.27)) (justify left))
   )
-  (hierarchical_label "USB_DN" (shape bidirectional) (at 240.665 65.405 0)
+  (hierarchical_label "USB_D_N" (shape bidirectional) (at 240.665 65.405 0)
     (effects (font (size 1.27 1.27)) (justify left))
   )
@@
     (effects (font (size 1.27 1.27)) (justify left))
   )
-  (hierarchical_label "USB_DP" (shape bidirectional) (at 240.665 55.88 0)
+  (hierarchical_label "USB_D_P" (shape bidirectional) (at 240.665 55.88 0)
     (effects (font (size 1.27 1.27)) (justify left))
   )
@@
   (symbol (lib_id "Device:LED") (at 248.92 121.285 0) (mirror x) (unit 1)
     (in_bom yes) (on_board yes)
-    (property "Reference" "D4" (id 0) (at 251.46 117.475 0)
+    (property "Reference" "D3" (id 0) (at 251.46 117.475 0)
       (effects (font (size 1.27 1.27)) (justify right))
     )
@@
   (symbol (lib_id "Device:LED") (at 248.92 113.665 0) (mirror x) (unit 1)
     (in_bom yes) (on_board yes)
-    (property "Reference" "D3" (id 0) (at 251.46 109.855 0)
+    (property "Reference" "D4" (id 0) (at 251.46 109.855 0)
       (effects (font (size 1.27 1.27)) (justify right))
     )

Commit message: i can't believe what they did to my boy
Parts:
- removed D7: CUHS15S30,H3F, Diode_SMD:D_SOD-123F, symbol Device:D_Small
- removed J9: Spare IO, Connector_PinHeader_2.54mm:PinHeader_2x03_P2.54mm_Vertical, symbol Connector_Generic:Conn_02x03_Top_Bottom
- removed TC3: TC2030-IDC, Connector:Tag-Connect_TC2030-IDC-NL_2x03_P1.27mm_Vertical, symbol TDC-2030-IDC:TC2030-IDC
- removed TP12: RP_RUN, TestPoint:TestPoint_Pad_D1.0mm, symbol Connector:TestPoint
Connections:
- net GPIO_GPI1: now also U11.32 (GPIO21); no longer U11.6 (GPIO4)
- net GPIO_GPI2: now also U11.31 (GPIO20); no longer U11.9 (GPIO7)
- net GPIO_GPI3: now also U11.30 (GPIO19); no longer U11.7 (GPIO5)
- net GPIO_GPI4: now also U11.29 (GPIO18); no longer U11.8 (GPIO6)
- net RP_GPIO12: no longer names the net of U11.15 (GPIO12)
- net RP_GPIO13: no longer names the net of U11.16 (GPIO13)
- net RP_GPIO14: no longer names the net of U11.17 (GPIO14)
- net RP_GPIO15: no longer names the net of U11.18 (GPIO15)
- net RP_SWCLK: no longer names the net of U11.24 (SWCLK)
- net RP_SWD: no longer names the net of U11.25 (SWD)
- no-connect marks 12 -> 11
Other:
- moved on the sheet: D3, D4, R19, R20

Commit message: updates nearly complete
Parts:
- C29, C31, C35, C38, C40, C48, C49, C50, C52, C9: MPN C0805C104M3RAC7800 -> 560L104YTT
Changed lines of the file:
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@@
       (effects (font (size 1.27 1.27)) hide)
     )
-    (property "Description" "CAP CER 0.1UF 25V X7R" (id 4) (at 209.55 33.02 0)
-      (effects (font (size 1.27 1.27)) hide)
-    )
-    (property "MPN" "C0805C104M3RAC7800" (id 5) (at 209.55 33.02 0)
+    (property "Description" "CAP CER 0.1UF 16V 0402" (id 4) (at 209.55 33.02 0)
+      (effects (font (size 1.27 1.27)) hide)
+    )
+    (property "MPN" "560L104YTT" (id 5) (at 209.55 33.02 0)
       (effects (font (size 1.27 1.27)) hide)
     )
@@
       (effects (font (size 1.27 1.27)) hide)
     )
-    (property "Description" "CAP CER 0.1UF 25V X7R" (id 4) (at 250.19 33.02 0)
-      (effects (font (size 1.27 1.27)) hide)
-    )
-    (property "MPN" "C0805C104M3RAC7800" (id 5) (at 250.19 33.02 0)
+    (property "Description" "CAP CER 0.1UF 16V 0402" (id 4) (at 250.19 33.02 0)
+      (effects (font (size 1.27 1.27)) hide)
+    )
+    (property "MPN" "560L104YTT" (id 5) (at 250.19 33.02 0)
       (effects (font (size 1.27 1.27)) hide)
     )
@@
       (effects (font (size 1.27 1.27)) hide)
     )
-    (property "Description" "CAP CER 0.1UF 25V X7R" (id 4) (at 189.23 33.02 0)
-      (effects (font (size 1.27 1.27)) hide)
-    )
-    (property "MPN" "C0805C104M3RAC7800" (id 5) (at 189.23 33.02 0)
+    (property "Description" "CAP CER 0.1UF 16V 0402" (id 4) (at 189.23 33.02 0)
+      (effects (font (size 1.27 1.27)) hide)
+    )
+    (property "MPN" "560L104YTT" (id 5) (at 189.23 33.02 0)
       (effects (font (size 1.27 1.27)) hide)
     )
@@
       (effects (font (size 1.27 1.27)) hide)
     )
+    (property "Description" "CRYSTAL 12.0000MHZ 12PF SMD" (id 5) (at 79.375 114.935 0)
+      (effects (font (size 1.27 1.27)) hide)
+    )
     (pin "1")
     (pin "2")
@@
       (effects (font (size 1.27 1.27)) hide)
     )
-    (property "Description" "CAP CER 0.1UF 25V X7R" (id 4) (at 125.095 33.02 0)
-      (effects (font (size 1.27 1.27)) hide)
-    )
-    (property "MPN" "C0805C104M3RAC7800" (id 5) (at 125.095 33.02 0)
+    (property "Description" "CAP CER 0.1UF 16V 0402" (id 4) (at 125.095 33.02 0)
+      (effects (font (size 1.27 1.27)) hide)
+    )
+    (property "MPN" "560L104YTT" (id 5) (at 125.095 33.02 0)
       (effects (font (size 1.27 1.27)) hide)
     )
@@
     )
     (property "LCSC" "C2040" (id 5) (at 165.735 102.87 0)
+      (effects (font (size 1.27 1.27)) hide)
+    )
+    (property "Description" "RP2040TR13" (id 6) (at 165.735 102.87 0)
       (effects (font (size 1.27 1.27)) hide)
     )
@@
       (effects (font (size 1.27 1.27)) hide)
     )
-    (property "Description" "CAP CER 0.1UF 25V X7R" (id 4) (at 53.34 66.04 0)
-      (effects (font (size 1.27 1.27)) hide)
-    )
-    (property "MPN" "C0805C104M3RAC7800" (id 5) (at 53.34 66.04 0)
+    (property "Description" "CAP CER 0.1UF 16V 0402" (id 4) (at 53.34 66.04 0)
+      (effects (font (size 1.27 1.27)) hide)
+    )
+    (property "MPN" "560L104YTT" (id 5) (at 53.34 66.04 0)
       (effects (font (size 1.27 1.27)) hide)
     )
@@
       (effects (font (size 1.27 1.27)) hide)
     )
-    (property "Description" "CAP CER 0.1UF 25V X7R" (id 4) (at 219.71 33.02 0)
-      (effects (font (size 1.27 1.27)) hide)
-    )
-    (property "MPN" "C0805C104M3RAC7800" (id 5) (at 219.71 33.02 0)
+    (property "Description" "CAP CER 0.1UF 16V 0402" (id 4) (at 219.71 33.02 0)
+      (effects (font (size 1.27 1.27)) hide)
+    )
+    (property "MPN" "560L104YTT" (id 5) (at 219.71 33.02 0)
       (effects (font (size 1.27 1.27)) hide)
     )
@@
       (effects (font (size 1.27 1.27)) hide)
     )
-    (property "Description" "CAP CER 0.1UF 25V X7R" (id 4) (at 240.03 33.02 0)
-      (effects (font (size 1.27 1.27)) hide)
-    )
-    (property "MPN" "C0805C104M3RAC7800" (id 5) (at 240.03 33.02 0)
+    (property "Description" "CAP CER 0.1UF 16V 0402" (id 4) (at 240.03 33.02 0)
+      (effects (font (size 1.27 1.27)) hide)
+    )
+    (property "MPN" "560L104YTT" (id 5) (at 240.03 33.02 0)
       (effects (font (size 1.27 1.27)) hide)
     )
@@
       (effects (font (size 1.27 1.27)) hide)
     )
-    (property "Description" "CAP CER 0.1UF 25V X7R" (id 4) (at 198.755 33.02 0)
-      (effects (font (size 1.27 1.27)) hide)
-    )
-    (property "MPN" "C0805C104M3RAC7800" (id 5) (at 198.755 33.02 0)
+    (property "Description" "CAP CER 0.1UF 16V 0402" (id 4) (at 198.755 33.02 0)
+      (effects (font (size 1.27 1.27)) hide)
+    )
+    (property "MPN" "560L104YTT" (id 5) (at 198.755 33.02 0)
       (effects (font (size 1.27 1.27)) hide)
     )
@@
       (effects (font (size 1.27 1.27)) hide)
     )
-    (property "Description" "CAP CER 0.1UF 25V X7R" (id 4) (at 229.87 33.02 0)
-      (effects (font (size 1.27 1.27)) hide)
-    )
-    (property "MPN" "C0805C104M3RAC7800" (id 5) (at 229.87 33.02 0)
+    (property "Description" "CAP CER 0.1UF 16V 0402" (id 4) (at 229.87 33.02 0)
+      (effects (font (size 1.27 1.27)) hide)
+    )
+    (property "MPN" "560L104YTT" (id 5) (at 229.87 33.02 0)
       (effects (font (size 1.27 1.27)) hide)
     )
@@
       (effects (font (size 1.27 1.27)) hide)
     )
-    (property "Description" "CAP CER 0.1UF 25V X7R" (id 4) (at 134.62 33.02 0)
-      (effects (font (size 1.27 1.27)) hide)
-    )
-    (property "MPN" "C0805C104M3RAC7800" (id 5) (at 134.62 33.02 0)
-      (effects (font (size 1.27 1.27)) hide)
-    )
+    (property "Description" "CAP CER 0.1UF 16V 0402" (id 4) (at 134.62 33.02 0)
+      (effects (font (size 1.27 1.27)) hide)
+    )
+    (property "MPN" "560L104YTT" (id 5) (at 134.62 33.02 0)
+      (effects (font (size 1.27 1.27)) hide)
+    )

Commit message: add USB VIN
Parts:
- renumbered C50 to C10, C33 to C11, C51 to C12, C9 to C13, C26 to C14, C24 to C15, C29 to C2, C31 to C3, C35 to C4, C38 to C5, C52 to C6, C40 to C7, C48 to C8, C49 to C9, D4 to D2, R41 to R2, R42 to R3, R37 to R4, R36 to R5, R20 to R6, R19 to R7, R38 to R8, SW4 to SW2, SW5 to SW3, U7 to U2, U11 to U3, Y4 to Y2
