File: hardware/underglow-controller/RGB-controller.kicad_sch (KiCad schematic)
At the start: 136 parts, among them J2 U.FL-R-SMT-1(10), J3 DM3AT-SF-PEJM5, J4 DTM1312PA12PBR008, J5 Conn_01x10, J6 CONSOLE, J7 U.FL-R-SMT-1(10), J8 JTAG, Q2 STS8DNF3LL, Q3 STS8DNF3LL, Q4 STS8DNF3LL, SW2 SW_Push, SW3 SW_Push, SW4 SW_Push, U10 DRV8844PWP, U11 RP2040, U3 SN65HVD230, U4 ESP32-S3R2, U5 W25Q128JVS, U6 WS2815B, U7 W25Q128JVS, U8 ADP2303ARDZ-3.3, U9 COM-13909, Y2 40MHZ, Y3 32.7k, Y4 12MHZ

Commit message: hardware updates: fix SPI bus on pico and flatten radio module
Parts:
- removed AE2: PCB_ANT, RF_Antenna:Texas_SWRA117D_2.4GHz_Right, symbol Device:Antenna_Shield
- removed AE3: PCB_ANT_RFM69, RF_Antenna:Texas_SWRA416_868MHz_915MHz, symbol Device:Antenna
- removed C10, C14, C29, C31, C35, C4, C40, C48, C49, C50, C51, C52, C7, C8, C9: 0.1uF, Capacitor_SMD:C_0402_1005Metric, symbol Device:C_Small
- removed C11, C13, C16, C28, C33, C37, C38: 1uF, Capacitor_SMD:C_0402_1005Metric, symbol Device:C_Small
- removed C12, C15: 10uF, Capacitor_SMD:C_0402_1005Metric, symbol Device:C_Small
- removed C17: 4.6pF, Capacitor_SMD:C_0402_1005Metric, symbol Device:C_Small
- removed C18, C22: 16pF, Capacitor_SMD:C_0402_1005Metric, symbol Device:C_Small
- removed C19, C23: 10pF, Capacitor_SMD:C_0402_1005Metric, symbol Device:C_Small
- removed C20: 4pF, Capacitor_SMD:C_0402_1005Metric, symbol Device:C_Small
- removed C21: 2pF, Capacitor_SMD:C_0402_1005Metric, symbol Device:C_Small
- removed C24, C26: 20pF, Capacitor_SMD:C_0402_1005Metric, symbol Device:C_Small
- removed C25, C44, C45, C5: 10uF, Capacitor_SMD:C_0805_2012Metric, symbol Device:C_Small
- removed C32, C43, C6: 0.1uF, Capacitor_SMD:C_0805_2012Metric, symbol Device:C_Small
- removed C39, C41: 22uF, Capacitor_SMD:C_0805_2012Metric, symbol Device:C_Small
- removed C42: 0.47uF, Capacitor_SMD:C_0805_2012Metric, symbol Device:C_Small
- removed C46: 0.01uF, Capacitor_SMD:C_0805_2012Metric, symbol Device:C_Small
- removed C47: 10uF, Capacitor_SMD:CP_Elec_5x5.3, symbol Device:C_Polarized_Small
- removed D2, D4: GRN, LED_SMD:LED_0603_1608Metric, symbol Device:LED
- removed D3: RED, LED_SMD:LED_0603_1608Metric, symbol Device:LED
- removed D5: D_Small, Diode_SMD:D_SOD-123F, symbol Device:D_Small
- removed H1: MountingHole_Pad, MountingHole:MountingHole_3.2mm_M3_DIN965_Pad, symbol Mechanical:MountingHole_Pad
- removed J2, J7: U.FL-R-SMT-1(10), ConeCodes:HRS_U.FL-R-SMT-1(10), symbol U.FL-R-SMT-1_10_:U.FL-R-SMT-1(10)
- removed J3: DM3AT-SF-PEJM5, ConeCodes:HRS_DM3AT-SF-PEJM5, symbol ConeCodes:DM3AT-SF-PEJM5
- removed J4: DTM1312PA12PBR008, TE_DTM1312PA12PBR008, symbol ConeCodes:DTM1312PA12PBR008
- removed J5: Conn_01x10, Connector_PinHeader_2.54mm:PinHeader_1x10_P2.54mm_Vertical, symbol Connector_Generic:Conn_01x10
- removed J6: CONSOLE, Connector_PinHeader_1.27mm:PinHeader_1x06_P1.27mm_Vertical, symbol Connector_Generic:Conn_01x06
- removed J8: JTAG, Connector_PinHeader_1.27mm:PinHeader_1x06_P1.27mm_Vertical, symbol Connector_Generic:Conn_01x06
- removed JP2: LED Voltage Select, Jumper:SolderJumper-3_P1.3mm_Bridged12_RoundedPad1.0x1.5mm_NumberLabels, symbol Jumper:SolderJumper_3_Bridged12
- removed L3: 2nH, Inductor_SMD:L_0402_1005Metric, symbol Device:L_Small
- removed L4: 2.2nH, Inductor_SMD:L_0402_1005Metric, symbol Device:L_Small
- removed L6: 4.7uH, Inductor_SMD:L_Bourns-SRN6028, symbol Device:L_Small
- removed Q2, Q3, Q4: STS8DNF3LL, Package_SO:SO-8_3.9x4.9mm_P1.27mm, symbol Device:Q_Dual_NMOS_S1G1S2G2D2D2D1D1
- removed R10, R11, R12, R13, R16, R17, R22, R28, R32, R33, R7, R8, R9: 0R, Resistor_SMD:R_0402_1005Metric, symbol Device:R_Small
- removed R14, R36: 1k, Resistor_SMD:R_0402_1005Metric, symbol Device:R_Small
- removed R15, R37: 100k, Resistor_SMD:R_0402_1005Metric, symbol Device:R_Small
- removed R18, R19, R20: 240R, Resistor_SMD:R_0603_1608Metric, symbol Device:R_Small
- removed R21: DNP, Resistor_SMD:R_0402_1005Metric, symbol Device:R_Small
- removed R23: 10k, Resistor_SMD:R_0603_1608Metric, symbol Device:R_Small
- removed R24, R25, R26, R27, R31, R38, R39, R4, R40, R43, R44, R45: 10k, Resistor_SMD:R_0402_1005Metric, symbol Device:R_Small
- removed R3: 120,DNF, Resistor_SMD:R_0805_2012Metric, symbol Device:R_Small
- removed R30: 36k, Resistor_SMD:R_0402_1005Metric, symbol Device:R_Small
- removed R34: 31k6, Resistor_SMD:R_0603_1608Metric, symbol Device:R_Small
- removed R35: 10k2, Resistor_SMD:R_0603_1608Metric, symbol Device:R_Small
- removed R41, R42: 27r4, Resistor_SMD:R_0402_1005Metric, symbol Device:R_Small
- removed R6: 499R, Resistor_SMD:R_0402_1005Metric, symbol Device:R_Small
- removed SW2, SW3, SW4: SW_Push, ConeCodes:SW_RS-032G05A3-SMRT, symbol Switch:SW_Push
- removed TC2, TC3, TC4: TC2030-IDC, Connector:Tag-Connect_TC2030-IDC-NL_2x03_P1.27mm_Vertical, symbol TDC-2030-IDC:TC2030-IDC
- removed TP10: CS1, TestPoint:TestPoint_Pad_D1.0mm, symbol Connector:TestPoint
- removed TP11: CS2, TestPoint:TestPoint_Pad_D1.0mm, symbol Connector:TestPoint
- removed TP12: RP_RUN, TestPoint:TestPoint_Pad_D1.0mm, symbol Connector:TestPoint
- removed TP2: CHIP_PU, TestPoint:TestPoint_Pad_D1.0mm, symbol Connector:TestPoint
- removed TP3: VBAT_SENSE, TestPoint:TestPoint_Pad_D1.0mm, symbol Connector:TestPoint
- removed TP4, TP7: 3V3OUT, TestPoint:TestPoint_Pad_D1.0mm, symbol Connector:TestPoint
- removed TP5: MOSI, TestPoint:TestPoint_Pad_D1.0mm, symbol Connector:TestPoint
- removed TP6: MISO, TestPoint:TestPoint_Pad_D1.0mm, symbol Connector:TestPoint
- removed TP8: SCLK, TestPoint:TestPoint_Pad_D1.0mm, symbol Connector:TestPoint
- removed TP9: CS0, TestPoint:TestPoint_Pad_D1.0mm, symbol Connector:TestPoint
- removed U10: DRV8844PWP, Package_SO:HTSSOP-28-1EP_4.4x9.7mm_P0.65mm_EP2.85x5.4mm_ThermalVias, symbol ConeCodes:DRV8844PWP
- removed U11: RP2040, ConeCodes:QFN-56, symbol ConeCodes:RP2040
- removed U3: SN65HVD230, Package_SO:SOIC-8_3.9x4.9mm_P1.27mm, symbol Interface_CAN_LIN:SN65HVD230
- removed U4: ESP32-S3R2, ConeCodes:QFN-56, symbol ConeCodes:ESP32-S3R2
- removed U5, U7: W25Q128JVS, Package_SO:SOIC-8W_5.3x5.3mm_P1.27mm, symbol Memory_Flash:W25Q128JVS
- removed U6: WS2815B, ConeCodes:worldsemi-WS2815B-MFG, symbol ConeCodes:WS2815B
- removed U8: ADP2303ARDZ-3.3, Package_SO:SOIC-8-1EP_3.9x4.9mm_P1.27mm_EP2.29x3mm, symbol Regulator_Switching:ADP2303ARDZ-3.3
- removed U9: COM-13909, ConeCodes:XCVR_RFM69HW, symbol ConeCodes:COM-13909
- removed Y2: 40MHZ, Crystal:Crystal_SMD_3225-4Pin_3.2x2.5mm, symbol Device:Crystal_GND24_Small
- removed Y3: 32.7k, Crystal:Crystal_SMD_MicroCrystal_CC7V-T1A-2Pin_3.2x1.5mm, symbol Device:Crystal_Small
- removed Y4: 12MHZ, Crystal:Crystal_SMD_3225-4Pin_3.2x2.5mm, symbol Device:Crystal_GND24_Small
Connections:
- no-connect marks 32 -> 0
Other:
- added sheet CAN-Bus (CAN-Bus.kicad_sch)
- added sheet Connectors (Connectors.kicad_sch)
- added sheet ESP32-S3 (ESP32-S3.kicad_sch)
- added sheet External-IO (External-IO.kicad_sch)
- added sheet Motor-Control (Motor-Control.kicad_sch)
- added sheet Pico Remote Proc (pico.kicad_sch)
- added sheet Power (Power.kicad_sch)
- added sheet SX1276 (SX1276.kicad_sch)
- note added: "SPID = MOSI = RPRX SPIQ = MISO = RPTX"
- note removed: "0R resistors should be near chip not cpu"
- note removed: "BUCK CONVERTER"
- note removed: "CAN"
- note removed: "CONNECTORS"
- note removed: "CX1 = CX2 = 2(10pF - 2pF) = 16pF"
- note removed: "CX1 = CX2 = 2(12pF - 2pF) = 20pF"
- note removed: "CX1 = CX2 = 2(7pF - 2pF) = 10pF"
- note removed: "INDIVIDUALLY ADDRESSABLE LED CONTROL"
- note removed: "MOTOR DRIVER"
- note removed: "Main outer connector"
- note removed: "RF69 PACKET RADIO"
- note removed: "RGB PWM LED CONTROL"
- note removed: "SPID = MOSI SPIQ = MISO"
- note removed: "STATUS LEDS"
- note removed: "Unsure if supply voltage should go to VCC or VDD. Datasheet says VDD but that doesn't make a ton of sense to me. If this part doesn't work, bridge the other half"
- note removed: "only r22 or r28 should be installed at a time"
- company: (none) -> cone.codes
- title: (none) -> CAN RGB Controller
