File: hardware/underglow-controller/Motor-Control.kicad_sch (KiCad schematic)
At the start: 7 parts, among them U10 DRV8844PWP

Commit message: i can't believe what they did to my boy
Parts:
- added D6, D9: GRN, LED_SMD:LED_0603_1608Metric, symbol Device:LED
- added R21, R46: 240R, Resistor_SMD:R_0603_1608Metric, symbol Device:R_Small
- R39: footprint Resistor_SMD:R_0402_1005Metric -> Resistor_SMD:R_0603_1608Metric; MPN RMCF0402JT10K0 -> RNCP0603FTD10K0
Connections:
- net +3V3 is gone; now on net V3P3OUT: R39.1
- net GND: now also R21.2
- net NFAULT: now also R46.2
- net V3P3OUT: now also D6.2 (A), D9.2 (A)
- net VIN renamed VOUT
- new net: D6.1 (K), R21.1
- new net: D9.1 (K), R46.1

Commit message: urmom
Connections:
- net V3P3OUT: no longer D6.2 (A), D9.2 (A)
- new net +3V3: D6.2 (A), D9.2 (A)
Changed lines of the file:
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@@
   (junction (at 116.84 53.34) (diameter 0) (color 0 0 0 0)
+  )
+  (junction (at 60.325 26.67) (diameter 0) (color 0 0 0 0)
   )
   (junction (at 113.03 40.64) (diameter 0) (color 0 0 0 0)
@@
     (stroke (width 0) (type default) (color 0 0 0 0))
   )
-  (wire (pts (xy 53.34 31.75) (xy 66.675 31.75))
+  (wire (pts (xy 60.325 24.765) (xy 60.325 26.67))
     (stroke (width 0) (type default) (color 0 0 0 0))
   )
@@
     (stroke (width 0) (type default) (color 0 0 0 0))
   )
-  (wire (pts (xy 21.844 26.924) (xy 35.814 26.924))
+  (wire (pts (xy 21.59 26.67) (xy 35.56 26.67))
     (stroke (width 0) (type default) (color 0 0 0 0))
   )
@@
   (wire (pts (xy 46.355 80.01) (xy 69.215 80.01))
     (stroke (width 0) (type default) (color 255 153 0 1))
+  )
+  (wire (pts (xy 53.34 26.67) (xy 60.325 26.67))
+    (stroke (width 0) (type default) (color 0 0 0 0))
   )
   (wire (pts (xy 113.03 40.64) (xy 129.54 40.64))
@@
     (stroke (width 0) (type default) (color 0 0 0 0))
   )
-  (wire (pts (xy 40.894 26.924) (xy 45.974 26.924))
+  (wire (pts (xy 40.64 26.67) (xy 45.72 26.67))
+    (stroke (width 0) (type default) (color 0 0 0 0))
+  )
+  (wire (pts (xy 60.325 26.67) (xy 60.325 31.75))
     (stroke (width 0) (type default) (color 0 0 0 0))
   )
@@
     (stroke (width 0) (type default) (color 0 0 0 0))
   )
+  (wire (pts (xy 60.325 31.75) (xy 53.34 31.75))
+    (stroke (width 0) (type default) (color 0 0 0 0))
+  )
   (wire (pts (xy 27.305 50.8) (xy 69.215 50.8))
     (stroke (width 0) (type default) (color 128 77 0 1))
@@
     (stroke (width 0) (type default) (color 221 133 0 1))
   )
-  (wire (pts (xy 53.594 26.924) (xy 66.548 26.924))
-    (stroke (width 0) (type default) (color 0 0 0 0))
-  )
   (wire (pts (xy 127.635 74.93) (xy 127.635 78.74))
     (stroke (width 0) (type default) (color 0 0 0 0))
@@
     (effects (font (size 1.27 1.27)) (justify left bottom))
   )
-  (label "LED_DRV_PWR" (at 21.844 26.924 0)
+  (label "LED_DRV_PWR" (at 21.59 26.67 0)
     (effects (font (size 1.27 1.27)) (justify left bottom))
   )
@@
     (effects (font (size 1.27 1.27)) (justify left bottom))
   )
-  (label "V3P3OUT" (at 66.548 26.924 180)
-    (effects (font (size 1.27 1.27)) (justify right bottom))
-  )
   (label "IN3" (at 57.15 77.47 0)
     (effects (font (size 1.27 1.27)) (justify left bottom))
-  )
-  (label "V3P3OUT" (at 66.675 31.75 180)
-    (effects (font (size 1.27 1.27)) (justify right bottom))
   )
   (hierarchical_label "NRESET" (shape output) (at 27.305 45.72 180)
@@
     (pin "2")
   )
-  (symbol (lib_id "Device:LED") (at 49.784 26.924 0) (mirror x) (unit 1)
-    (in_bom yes) (on_board yes) (fields_autoplaced)
-    (property "Reference" "D6" (id 0) (at 48.1965 19.05 0))
-    (property "Value" "GRN" (id 1) (at 48.1965 21.59 0))
-    (property "Footprint" "LED_SMD:LED_0603_1608Metric" (id 2) (at 49.784 26.924 0)
-      (effects (font (size 1.27 1.27)) hide)
-    )
-    (property "Datasheet" "~" (id 3) (at 49.784 26.924 0)
-      (effects (font (size 1.27 1.27)) hide)
-    )
-    (property "MPN" "QBLP601-2IR4" (id 4) (at 49.784 26.924 0)
-      (effects (font (size 1.27 1.27)) hide)
-    )
-    (property "Description" "LED GREEN CLEAR 0603 SMD" (id 6) (at 49.784 26.924 0)
+  (symbol (lib_id "Device:LED") (at 49.53 26.67 0) (mirror x) (unit 1)
+    (in_bom yes) (on_board yes) (fields_autoplaced)
+    (property "Reference" "D6" (id 0) (at 47.9425 18.796 0))
+    (property "Value" "GRN" (id 1) (at 47.9425 21.336 0))
+    (property "Footprint" "LED_SMD:LED_0603_1608Metric" (id 2) (at 49.53 26.67 0)
+      (effects (font (size 1.27 1.27)) hide)
+    )
+    (property "Datasheet" "~" (id 3) (at 49.53 26.67 0)
+      (effects (font (size 1.27 1.27)) hide)
+    )
+    (property "MPN" "QBLP601-2IR4" (id 4) (at 49.53 26.67 0)
+      (effects (font (size 1.27 1.27)) hide)
+    )
+    (property "Description" "LED GREEN CLEAR 0603 SMD" (id 6) (at 49.53 26.67 0)
       (effects (font (size 1.27 1.27)) hide)
     )
@@
     (pin "1")
   )
-  (symbol (lib_id "Device:R_Small") (at 38.354 26.924 270) (unit 1)
+  (symbol (lib_id "Device:R_Small") (at 38.1 26.67 270) (unit 1)
     (in_bom yes) (on_board yes)
-    (property "Reference" "R21" (id 0) (at 39.624 24.384 90)
-      (effects (font (size 1.27 1.27)) (justify left))
-    )
-    (property "Value" "240R" (id 1) (at 34.544 24.384 90)
-      (effects (font (size 1.27 1.27)) (justify left))
-    )
-    (property "Footprint" "Resistor_SMD:R_0603_1608Metric" (id 2) (at 38.354 26.924 0)
-      (effects (font (size 1.27 1.27)) hide)
-    )
-    (property "Datasheet" "~" (id 3) (at 38.354 26.924 0)
-      (effects (font (size 1.27 1.27)) hide)
-    )
-    (property "MPN" "RMCF0402JT240R" (id 4) (at 38.354 26.924 0)
-      (effects (font (size 1.27 1.27)) hide)
-    )
-    (property "Description" "RES 240 OHM 5% 1/16W 0402" (id 5) (at 38.354 26.924 0)
+    (property "Reference" "R21" (id 0) (at 39.37 24.13 90)
+      (effects (font (size 1.27 1.27)) (justify left))
+    )
+    (property "Value" "240R" (id 1) (at 34.29 24.13 90)
+      (effects (font (size 1.27 1.27)) (justify left))
+    )
+    (property "Footprint" "Resistor_SMD:R_0603_1608Metric" (id 2) (at 38.1 26.67 0)
+      (effects (font (size 1.27 1.27)) hide)
+    )
+    (property "Datasheet" "~" (id 3) (at 38.1 26.67 0)
+      (effects (font (size 1.27 1.27)) hide)
+    )
+    (property "MPN" "RMCF0402JT240R" (id 4) (at 38.1 26.67 0)
+      (effects (font (size 1.27 1.27)) hide)
+    )
+    (property "Description" "RES 240 OHM 5% 1/16W 0402" (id 5) (at 38.1 26.67 0)
       (effects (font (size 1.27 1.27)) hide)
     )
@@
     (pin "2")
   )
+  (symbol (lib_id "power:+3V3") (at 60.325 24.765 0) (unit 1)
+    (in_bom yes) (on_board yes) (fields_autoplaced)
+    (property "Reference" "#PWR0123" (id 0) (at 60.325 28.575 0)
+      (effects (font (size 1.27 1.27)) hide)
+    )
+    (property "Value" "+3V3" (id 1) (at 60.325 19.05 0))
+    (property "Footprint" "" (id 2) (at 60.325 24.765 0)
+      (effects (font (size 1.27 1.27)) hide)
+    )
+    (property "Datasheet" "" (id 3) (at 60.325 24.765 0)
+      (effects (font (size 1.27 1.27)) hide)
+    )
+    (pin "1")
+  )
   (symbol (lib_id "power:GND") (at 127.635 83.82 0) (unit 1)
     (in_bom yes) (on_board yes) (fields_autoplaced)
@@
     (pin "2")
   )
-  (symbol (lib_id "power:GND") (at 21.844 26.924 270) (unit 1)
-    (in_bom yes) (on_board yes) (fields_autoplaced)
-    (property "Reference" "#PWR0108" (id 0) (at 15.494 26.924 0)
-      (effects (font (size 1.27 1.27)) hide)
-    )
-    (property "Value" "GND" (id 1) (at 18.034 26.9239 90)
+  (symbol (lib_id "power:GND") (at 21.59 26.67 270) (unit 1)
+    (in_bom yes) (on_board yes) (fields_autoplaced)
+    (property "Reference" "#PWR0108" (id 0) (at 15.24 26.67 0)
+      (effects (font (size 1.27 1.27)) hide)
+    )
+    (property "Value" "GND" (id 1) (at 17.78 26.6699 90)
       (effects (font (size 1.27 1.27)) (justify right))
     )
-    (property "Footprint" "" (id 2) (at 21.844 26.924 0)
-      (effects (font (size 1.27 1.27)) hide)
-    )
-    (property "Datasheet" "" (id 3) (at 21.844 26.924 0)
-      (effects (font (size 1.27 1.27)) hide)
-    )
+    (property "Footprint" "" (id 2) (at 21.59 26.67 0)
+      (effects (font (size 1.27 1.27)) hide)
+    )
+    (property "Datasheet" "" (id 3) (at 21.59 26.67 0)
+      (effects (font (size 1.27 1.27)) hide)
+    )

Commit message: add USB VIN
Parts:
- renumbered C46 to C54, C43 to C55, C44 to C56, C47 to C57, C42 to C58, D6 to D4, D9 to D5, R21 to R37, R46 to R38, U10 to U7
Changed lines of the file:
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@@
   (symbol (lib_id "Device:LED") (at 49.53 26.67 0) (mirror x) (unit 1)
     (in_bom yes) (on_board yes) (fields_autoplaced)
-    (property "Reference" "D6" (id 0) (at 47.9425 18.796 0))
+    (property "Reference" "D4" (id 0) (at 47.9425 18.796 0))
     (property "Value" "GRN" (id 1) (at 47.9425 21.336 0))
     (property "Footprint" "LED_SMD:LED_0603_1608Metric" (id 2) (at 49.53 26.67 0)
@@
   (symbol (lib_id "ConeCodes:DRV8844PWP") (at 86.995 64.77 0) (unit 1)
     (in_bom yes) (on_board yes) (fields_autoplaced)
-    (property "Reference" "U10" (id 0) (at 86.995 26.67 0))
+    (property "Reference" "U7" (id 0) (at 86.995 26.67 0))
     (property "Value" "DRV8844PWP" (id 1) (at 86.995 29.21 0))
     (property "Footprint" "Package_SO:HTSSOP-28-1EP_4.4x9.7mm_P0.65mm_EP2.85x5.4mm_ThermalVias" (id 2) (at 86.995 64.77 0)
@@
   (symbol (lib_id "power:GND") (at 134.62 53.34 0) (unit 1)
     (in_bom yes) (on_board yes) (fields_autoplaced)
-    (property "Reference" "#PWR070" (id 0) (at 134.62 59.69 0)
+    (property "Reference" "#PWR079" (id 0) (at 134.62 59.69 0)
       (effects (font (size 1.27 1.27)) hide)
     )
@@
   (symbol (lib_id "Device:C_Small") (at 116.84 45.72 0) (unit 1)
     (in_bom yes) (on_board yes) (fields_autoplaced)
-    (property "Reference" "C43" (id 0) (at 120.015 44.4562 0)
+    (property "Reference" "C55" (id 0) (at 120.015 44.4562 0)
       (effects (font (size 1.27 1.27)) (justify left))
     )
@@
   (symbol (lib_id "power:GND") (at 108.585 95.25 0) (unit 1)
     (in_bom yes) (on_board yes) (fields_autoplaced)
-    (property "Reference" "#PWR065" (id 0) (at 108.585 101.6 0)
+    (property "Reference" "#PWR081" (id 0) (at 108.585 101.6 0)
       (effects (font (size 1.27 1.27)) hide)
     )
@@
   (symbol (lib_id "Device:R_Small") (at 38.1 26.67 270) (unit 1)
     (in_bom yes) (on_board yes)
-    (property "Reference" "R21" (id 0) (at 39.37 24.13 90)
+    (property "Reference" "R37" (id 0) (at 39.37 24.13 90)
       (effects (font (size 1.27 1.27)) (justify left))
     )
@@
   (symbol (lib_id "Device:LED") (at 49.53 31.75 0) (mirror x) (unit 1)
     (in_bom yes) (on_board yes) (fields_autoplaced)
-    (property "Reference" "D9" (id 0) (at 47.9425 35.56 0))
+    (property "Reference" "D5" (id 0) (at 47.9425 35.56 0))
     (property "Value" "GRN" (id 1) (at 47.9425 38.1 0))
     (property "Footprint" "LED_SMD:LED_0603_1608Metric" (id 2) (at 49.53 31.75 0)
@@
   (symbol (lib_id "power:+3V3") (at 60.325 24.765 0) (unit 1)
     (in_bom yes) (on_board yes) (fields_autoplaced)
-    (property "Reference" "#PWR0123" (id 0) (at 60.325 28.575 0)
+    (property "Reference" "#PWR076" (id 0) (at 60.325 28.575 0)
       (effects (font (size 1.27 1.27)) hide)
     )
@@
   (symbol (lib_id "power:GND") (at 127.635 83.82 0) (unit 1)
     (in_bom yes) (on_board yes) (fields_autoplaced)
-    (property "Reference" "#PWR064" (id 0) (at 127.635 90.17 0)
+    (property "Reference" "#PWR080" (id 0) (at 127.635 90.17 0)
       (effects (font (size 1.27 1.27)) hide)
     )
@@
   (symbol (lib_id "Device:R_Small") (at 38.1 31.75 270) (unit 1)
     (in_bom yes) (on_board yes)
-    (property "Reference" "R46" (id 0) (at 39.37 29.21 90)
+    (property "Reference" "R38" (id 0) (at 39.37 29.21 90)
       (effects (font (size 1.27 1.27)) (justify left))
     )
@@
   (symbol (lib_id "power:GND") (at 21.59 26.67 270) (unit 1)
     (in_bom yes) (on_board yes) (fields_autoplaced)
-    (property "Reference" "#PWR0108" (id 0) (at 15.24 26.67 0)
+    (property "Reference" "#PWR077" (id 0) (at 15.24 26.67 0)
       (effects (font (size 1.27 1.27)) hide)
     )
@@
   (symbol (lib_id "Device:C_Small") (at 127.635 81.28 0) (unit 1)
     (in_bom yes) (on_board yes) (fields_autoplaced)
-    (property "Reference" "C42" (id 0) (at 130.175 80.0162 0)
+    (property "Reference" "C58" (id 0) (at 130.175 80.0162 0)
       (effects (font (size 1.27 1.27)) (justify left))
     )
@@
   (symbol (lib_id "power:GND") (at 129.54 40.64 90) (unit 1)
     (in_bom yes) (on_board yes) (fields_autoplaced)
-    (property "Reference" "#PWR069" (id 0) (at 135.89 40.64 0)
+    (property "Reference" "#PWR078" (id 0) (at 135.89 40.64 0)
       (effects (font (size 1.27 1.27)) hide)
     )
@@
   (symbol (lib_id "Device:C_Small") (at 123.19 35.56 0) (unit 1)
     (in_bom yes) (on_board yes) (fields_autoplaced)
-    (property "Reference" "C46" (id 0) (at 126.365 34.2962 0)
+    (property "Reference" "C54" (id 0) (at 126.365 34.2962 0)
       (effects (font (size 1.27 1.27)) (justify left))
     )
@@
   (symbol (lib_id "Device:C_Polarized_Small") (at 134.62 50.8 0) (unit 1)
     (in_bom yes) (on_board yes) (fields_autoplaced)
-    (property "Reference" "C47" (id 0) (at 137.795 48.9838 0)
+    (property "Reference" "C57" (id 0) (at 137.795 48.9838 0)
       (effects (font (size 1.27 1.27)) (justify left))
     )
@@
   (symbol (lib_id "Device:C_Small") (at 116.84 50.8 0) (unit 1)
     (in_bom yes) (on_board yes) (fields_autoplaced)
-    (property "Reference" "C44" (id 0) (at 120.015 49.5362 0)
-      (effects (font (size 1.27 1.27)) (justify left))
-    )
+    (property "Reference" "C56" (id 0) (at 120.015 49.5362 0)
+      (effects (font (size 1.27 1.27)) (justify left))
+    )

Commit message: god i wish i remembered what this was
Parts:
- removed D4: GRN, LED_SMD:LED_0603_1608Metric, symbol Device:LED
- removed R37: 240R, Resistor_SMD:R_0603_1608Metric, symbol Device:R_Small
Changed lines of the file:
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@@
   (junction (at 116.84 53.34) (diameter 0) (color 0 0 0 0)
-  )
-  (junction (at 60.325 26.67) (diameter 0) (color 0 0 0 0)
   )
   (junction (at 113.03 40.64) (diameter 0) (color 0 0 0 0)
@@
     (stroke (width 0) (type default) (color 0 0 0 0))
   )
-  (wire (pts (xy 60.325 24.765) (xy 60.325 26.67))
+  (wire (pts (xy 60.325 24.765) (xy 60.325 31.75))
     (stroke (width 0) (type default) (color 0 0 0 0))
   )
@@
     (stroke (width 0) (type default) (color 0 0 0 0))
   )
-  (wire (pts (xy 21.59 26.67) (xy 35.56 26.67))
-    (stroke (width 0) (type default) (color 0 0 0 0))
-  )
   (wire (pts (xy 104.775 57.15) (xy 108.585 57.15))
     (stroke (width 0) (type default) (color 0 0 0 0))
@@
   (wire (pts (xy 46.355 80.01) (xy 69.215 80.01))
     (stroke (width 0) (type default) (color 255 153 0 1))
-  )
-  (wire (pts (xy 53.34 26.67) (xy 60.325 26.67))
-    (stroke (width 0) (type default) (color 0 0 0 0))
   )
   (wire (pts (xy 113.03 40.64) (xy 129.54 40.64))
@@
     (stroke (width 0) (type default) (color 0 0 0 0))
   )
-  (wire (pts (xy 40.64 26.67) (xy 45.72 26.67))
-    (stroke (width 0) (type default) (color 0 0 0 0))
-  )
-  (wire (pts (xy 60.325 26.67) (xy 60.325 31.75))
-    (stroke (width 0) (type default) (color 0 0 0 0))
-  )
   (wire (pts (xy 113.03 46.99) (xy 113.03 48.26))
     (stroke (width 0) (type default) (color 0 0 0 0))
@@
     (effects (font (size 1.27 1.27)) (justify left bottom))
   )
-  (label "LED_DRV_PWR" (at 21.59 26.67 0)
-    (effects (font (size 1.27 1.27)) (justify left bottom))
-  )
   (label "VM" (at 139.065 44.45 180)
     (effects (font (size 1.27 1.27)) (justify right bottom))
@@
     )
     (property "Description" "RES 10K OHM 1% 1/8W 0603" (id 6) (at 34.29 43.18 0)
-      (effects (font (size 1.27 1.27)) hide)
-    )
-    (pin "1")
-    (pin "2")
-  )
-  (symbol (lib_id "Device:LED") (at 49.53 26.67 0) (mirror x) (unit 1)
-    (in_bom yes) (on_board yes) (fields_autoplaced)
-    (property "Reference" "D4" (id 0) (at 47.9425 18.796 0))
-    (property "Value" "GRN" (id 1) (at 47.9425 21.336 0))
-    (property "Footprint" "LED_SMD:LED_0603_1608Metric" (id 2) (at 49.53 26.67 0)
-      (effects (font (size 1.27 1.27)) hide)
-    )
-    (property "Datasheet" "~" (id 3) (at 49.53 26.67 0)
-      (effects (font (size 1.27 1.27)) hide)
-    )
-    (property "MPN" "QBLP601-2IR4" (id 4) (at 49.53 26.67 0)
-      (effects (font (size 1.27 1.27)) hide)
-    )
-    (property "Description" "LED GREEN CLEAR 0603 SMD" (id 6) (at 49.53 26.67 0)
       (effects (font (size 1.27 1.27)) hide)
     )
@@
     (pin "1")
   )
-  (symbol (lib_id "Device:R_Small") (at 38.1 26.67 270) (unit 1)
-    (in_bom yes) (on_board yes)
-    (property "Reference" "R37" (id 0) (at 39.37 24.13 90)
-      (effects (font (size 1.27 1.27)) (justify left))
-    )
-    (property "Value" "240R" (id 1) (at 34.29 24.13 90)
-      (effects (font (size 1.27 1.27)) (justify left))
-    )
-    (property "Footprint" "Resistor_SMD:R_0603_1608Metric" (id 2) (at 38.1 26.67 0)
-      (effects (font (size 1.27 1.27)) hide)
-    )
-    (property "Datasheet" "~" (id 3) (at 38.1 26.67 0)
-      (effects (font (size 1.27 1.27)) hide)
-    )
-    (property "MPN" "RMCF0402JT240R" (id 4) (at 38.1 26.67 0)
-      (effects (font (size 1.27 1.27)) hide)
-    )
-    (property "Description" "RES 240 OHM 5% 1/16W 0402" (id 5) (at 38.1 26.67 0)
-      (effects (font (size 1.27 1.27)) hide)
-    )
-    (pin "1")
-    (pin "2")
-  )
   (symbol (lib_id "Device:LED") (at 49.53 31.75 0) (mirror x) (unit 1)
     (in_bom yes) (on_board yes) (fields_autoplaced)
@@
     (pin "2")
   )
-  (symbol (lib_id "power:GND") (at 21.59 26.67 270) (unit 1)
-    (in_bom yes) (on_board yes) (fields_autoplaced)
-    (property "Reference" "#PWR077" (id 0) (at 15.24 26.67 0)
-      (effects (font (size 1.27 1.27)) hide)
-    )
-    (property "Value" "GND" (id 1) (at 17.78 26.6699 90)
-      (effects (font (size 1.27 1.27)) (justify right))
-    )
-    (property "Footprint" "" (id 2) (at 21.59 26.67 0)
-      (effects (font (size 1.27 1.27)) hide)
-    )
-    (property "Datasheet" "" (id 3) (at 21.59 26.67 0)
-      (effects (font (size 1.27 1.27)) hide)
-    )
-    (pin "1")
-  )
   (symbol (lib_id "Device:C_Small") (at 127.635 81.28 0) (unit 1)

Commit message: replace pmic
Parts:
- renumbered D5 to D4, R38 to R37, R39 to R38
Changed lines of the file:
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@@
   (symbol (lib_id "Device:R_Small") (at 34.29 43.18 0) (unit 1)
     (in_bom yes) (on_board yes) (fields_autoplaced)
-    (property "Reference" "R39" (id 0) (at 36.83 41.9099 0)
+    (property "Reference" "R38" (id 0) (at 36.83 41.9099 0)
       (effects (font (size 1.27 1.27)) (justify left))
     )
@@
   (symbol (lib_id "power:GND") (at 134.62 53.34 0) (unit 1)
     (in_bom yes) (on_board yes) (fields_autoplaced)
-    (property "Reference" "#PWR079" (id 0) (at 134.62 59.69 0)
+    (property "Reference" "#PWR078" (id 0) (at 134.62 59.69 0)
       (effects (font (size 1.27 1.27)) hide)
     )
@@
   (symbol (lib_id "power:GND") (at 108.585 95.25 0) (unit 1)
     (in_bom yes) (on_board yes) (fields_autoplaced)
-    (property "Reference" "#PWR081" (id 0) (at 108.585 101.6 0)
+    (property "Reference" "#PWR080" (id 0) (at 108.585 101.6 0)
       (effects (font (size 1.27 1.27)) hide)
     )
@@
   (symbol (lib_id "Device:LED") (at 49.53 31.75 0) (mirror x) (unit 1)
     (in_bom yes) (on_board yes) (fields_autoplaced)
-    (property "Reference" "D5" (id 0) (at 47.9425 35.56 0))
+    (property "Reference" "D4" (id 0) (at 47.9425 35.56 0))
     (property "Value" "GRN" (id 1) (at 47.9425 38.1 0))
     (property "Footprint" "LED_SMD:LED_0603_1608Metric" (id 2) (at 49.53 31.75 0)
@@
   (symbol (lib_id "power:GND") (at 127.635 83.82 0) (unit 1)
     (in_bom yes) (on_board yes) (fields_autoplaced)
-    (property "Reference" "#PWR080" (id 0) (at 127.635 90.17 0)
+    (property "Reference" "#PWR079" (id 0) (at 127.635 90.17 0)
       (effects (font (size 1.27 1.27)) hide)
     )
@@
   (symbol (lib_id "Device:R_Small") (at 38.1 31.75 270) (unit 1)
     (in_bom yes) (on_board yes)
-    (property "Reference" "R38" (id 0) (at 39.37 29.21 90)
+    (property "Reference" "R37" (id 0) (at 39.37 29.21 90)
       (effects (font (size 1.27 1.27)) (justify left))
     )
@@
   (symbol (lib_id "power:GND") (at 129.54 40.64 90) (unit 1)
     (in_bom yes) (on_board yes) (fields_autoplaced)
-    (property "Reference" "#PWR078" (id 0) (at 135.89 40.64 0)
-      (effects (font (size 1.27 1.27)) hide)
-    )
+    (property "Reference" "#PWR077" (id 0) (at 135.89 40.64 0)
+      (effects (font (size 1.27 1.27)) hide)
+    )
