File: hardware/underglow-controller/SX1276.kicad_sch (KiCad schematic)
At the start: 41 parts, among them J10 U.FL-R-SMT-1(10), J2 U.FL-R-SMT-1(10), U2 SX1231HIMLTRT, Y5 32mhz

Commit message: i can't believe what they did to my boy
Parts:
- added AE4: Antenna_Shield, RF_Antenna:Texas_SWRA416_868MHz_915MHz, symbol Device:Antenna
- added R24, R40, R43, R44: 0R, Resistor_SMD:R_0402_1005Metric, symbol Device:R_Small
- AE3: symbol Device:Antenna_Shield -> Device:Antenna
Connections:
- net at C65.1, C67.1, L12.2: now also R24.2, R40.1; no longer J10.2
- net at C64.1, C66.1, L11.2: now also R43.2, R44.1; no longer J2.2
- net at AE3.1 (A): now also R24.1
- new net: J10.2, R40.2
- new net: J2.2, R44.2
- new net: AE4.1 (A), R43.1
Other:
- moved on the sheet: J10, J2

Commit message: updates nearly complete
Parts:
- C2: MPN (none) -> GRT21BC81A106KE01L
- C27, C30, C36, C45: MPN (none) -> 0402B104K250HI
- C3, C34: MPN (none) -> GCM1555C1H160JA16D
- C54: MPN (none) -> C0402C103M5RECAUTO
- C55: MPN (none) -> GRM1555C1H680JA01D
- C56, C59: MPN (none) -> 04025A8R2DAT2A
- C58: MPN (none) -> GRM1555C1H220JA01D
- C62, C63: MPN (none) -> C0402C689D5GAC7867
- C66: MPN (none) -> CC0402CRNPO9BN3R3
- C67: MPN (none) -> CL05C5R6DB5NNNC
- L10, L12: MPN (none) -> LQW15AN6N8J00D
- L11, L9: MPN (none) -> LQW15AN5N6C10D
- L2: MPN (none) -> LQW15AN2N7D00D
- L5: MPN (none) -> LQW15AN3N9C00D
- L7: MPN (none) -> LQW15AN22NG00D
- L8: MPN (none) -> LQW15AN33NJ00D
- R24, R40, R43, R44: MPN (none) -> RC0402JR-070RP
Connections:
- no-connect marks 0 -> 1

Commit message: add USB VIN
Parts:
- renumbered AE4 to AE2, C54 to C16, C60 to C17, C64 to C18, C58 to C19, C62 to C20, C66 to C21, C56 to C22, C53 to C23, C2 to C24, C27 to C25, C30 to C26, C36 to C27, C45 to C28, C55 to C29, C61 to C30, C65 to C31, C59 to C32, C63 to C33, C67 to C34, C57 to C35, C3 to C36, C34 to C37, J10 to J3, L7 to L2, L2 to L3, L9 to L4, L11 to L5, L8 to L6, L5 to L7, L10 to L8, L12 to L9, R44 to R10, R24 to R11, R40 to R12, R43 to R9, TP13 to TP2, TP14 to TP3, TP15 to TP4, TP16 to TP5, TP17 to TP6, TP18 to TP7, U2 to U4, Y5 to Y3

Commit message: iasdf
Parts:
- removed AE2, AE3: Antenna_Shield, RF_Antenna:Texas_SWRA416_868MHz_915MHz, symbol Device:Antenna
- removed J2: U.FL-R-SMT-1(10), ConeCodes:HRS_U.FL-R-SMT-1(10), symbol U.FL-R-SMT-1_10_:U.FL-R-SMT-1(10)
Changed lines of the file:
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@@
     (pin "2")
-  )
-  (symbol (lib_id "U.FL-R-SMT-1_10_:U.FL-R-SMT-1(10)") (at 269.24 51.435 0) (unit 1)
-    (in_bom no) (on_board yes)
-    (property "Reference" "J2" (id 0) (at 270.51 57.785 0))
-    (property "Value" "U.FL-R-SMT-1(10)" (id 1) (at 281.94 54.61 0))
-    (property "Footprint" "ConeCodes:HRS_U.FL-R-SMT-1(10)" (id 2) (at 269.24 51.435 0)
-      (effects (font (size 1.27 1.27)) (justify left bottom) hide)
-    )
-    (property "Datasheet" "" (id 3) (at 269.24 51.435 0)
-      (effects (font (size 1.27 1.27)) (justify left bottom) hide)
-    )
-    (property "MPN" "U.FL-R-SMT-1(10)" (id 11) (at 269.24 51.435 0)
-      (effects (font (size 1.27 1.27)) hide)
-    )
-    (property "Description" "RF Connectors / Coaxial Connectors SMT ML REC AU 50 OHM W/ANTI SLDR WCKNG R" (id 12) (at 269.24 51.435 0)
-      (effects (font (size 1.27 1.27)) hide)
-    )
-    (pin "1")
-    (pin "2")
-    (pin "3")
   )
   (symbol (lib_id "Device:C_Small") (at 228.6 93.98 0) (unit 1)
@@
     (pin "1")
   )
-  (symbol (lib_id "Device:Antenna") (at 269.24 73.66 0) (unit 1)
-    (in_bom yes) (on_board yes) (fields_autoplaced)
-    (property "Reference" "AE3" (id 0) (at 272.415 71.7549 0)
-      (effects (font (size 1.27 1.27)) (justify left))
-    )
-    (property "Value" "Antenna_Shield" (id 1) (at 272.415 74.2949 0)
-      (effects (font (size 1.27 1.27)) (justify left))
-    )
-    (property "Footprint" "RF_Antenna:Texas_SWRA416_868MHz_915MHz" (id 2) (at 269.24 71.12 0)
-      (effects (font (size 1.27 1.27)) hide)
-    )
-    (property "Datasheet" "~" (id 3) (at 269.24 71.12 0)
-      (effects (font (size 1.27 1.27)) hide)
-    )
-    (pin "1")
-  )
   (symbol (lib_id "Device:R_Small") (at 250.19 45.72 0) (unit 1)
     (in_bom yes) (on_board yes) (fields_autoplaced)
@@
     (pin "2")
   )
-  (symbol (lib_id "Device:Antenna") (at 269.24 37.465 0) (unit 1)
-    (in_bom yes) (on_board yes) (fields_autoplaced)
-    (property "Reference" "AE2" (id 0) (at 272.415 35.5599 0)
-      (effects (font (size 1.27 1.27)) (justify left))
-    )
-    (property "Value" "Antenna_Shield" (id 1) (at 272.415 38.0999 0)
-      (effects (font (size 1.27 1.27)) (justify left))
-    )
-    (property "Footprint" "RF_Antenna:Texas_SWRA416_868MHz_915MHz" (id 2) (at 269.24 34.925 0)
-      (effects (font (size 1.27 1.27)) hide)
-    )
-    (property "Datasheet" "~" (id 3) (at 269.24 34.925 0)
-      (effects (font (size 1.27 1.27)) hide)
-    )
-    (pin "1")
-  )
   (symbol (lib_id "Device:C_Small") (at 29.21 67.31 0) (unit 1)

Commit message: schematic rework progress
Parts:
- renumbered C24 to C10, C25 to C11, C26 to C12, C27 to C13, C28 to C14, C29 to C15, C30 to C16, C31 to C17, C32 to C18, C33 to C19, C16 to C2, C34 to C20, C35 to C21, C36 to C22, C37 to C23, C17 to C3, C18 to C4, C19 to C5, C20 to C6, C21 to C7, C22 to C8, C23 to C9, J3 to J2, R9 to R2, R10 to R3, R11 to R4, R12 to R5, U4 to U2, Y3 to Y2
