File: hardware/underglow-controller/RGB-controller.kicad_pcb (KiCad board)
At the start: 4 copper layers, 78.5 x 93 mm, 154 parts, among them J2 U.FL-R-SMT-1(10), J3 CONSOLE, J4 U.FL-R-SMT-1(10), J5 Delphi_Sicma_24, J7 Conn_01x05, Q2 STS8DNF3LL, Q3 STS8DNF3LL, Q4 STS8DNF3LL, Q5 STS8DNF3LL, Q6 STS8DNF3LL, Q7 MBT3904DW1T1G, Q8 MBT3904DW1T1G, SW2 SW_Push, SW3 SW_Push, U2 SX1231HIMLTRT, U3 ESP32-S3R2, U4 W25Q128JVS, U5 TLD55012QVXUMA1, U6 BD33C0AWFP-CE2, U7 SN65HVD230, Y2 32mhz, Y3 40MHZ

Commit message: almost done picking components i think
Parts:
- removed TC2: TC2030-IDC, Connector:Tag-Connect_TC2030-IDC-NL_2x03_P1.27mm_Vertical
- added AE2: SRCW004, ConeCodes:SRCW004, F.Cu at (24.8, 127.8)
- added R11: 0R, Resistor_SMD:R_0402_1005Metric, F.Cu at (24.5, 119.1)
- added R21: RSWCS1, Resistor_SMD:R_0603_1608Metric, F.Cu at (120.8, 78.3)
- added R29: RSWCS2, Resistor_SMD:R_0603_1608Metric, F.Cu at (124.8, 78.3)
- added R41: 0R, Resistor_SMD:R_2512_6332Metric, F.Cu at (117.6, 89.2)
- D5: value D_Small -> RB496EA; footprint Diode_SMD:D_SOD-123F -> Package_TO_SOT_SMD:SOT-23-5
- D6: value D_Small -> D_Schottky_Small; footprint Diode_SMD:D_SOD-123F -> Diode_SMD:D_SMA
- moved D5 41.1 mm to (123.9, 97.6), turned to 0 degrees
- moved D6 40.8 mm to (117.3, 97.6), turned to 0 degrees
- renumbered C4 to C10, C5 to C11, C6 to C12, C7 to C13, C8 to C14, C9 to C2, C10 to C3, C11 to C4, C12 to C5, C58 to C57, C57 to C58, C13 to C6, C14 to C7, C2 to C8, C3 to C9, D8 to D7, D9 to D8, J7 to J6, R11 to R12, R12 to R13, R13 to R14, R14 to R15, R15 to R16, R16 to R17, R17 to R18, R18 to R19, R19 to R20, R21 to R22, R22 to R23, R25 to R24, R26 to R25, R23 to R26, R24 to R27, R31 to R28, R27 to R30, R28 to R31, R29 to R32, R30 to R33, R33 to R34, R34 to R35, R35 to R36, R36 to R37, R37 to R38, R38 to R39, R39 to R40, R44 to R42, R40 to R43, R41 to R44, R42 to R45, R43 to R46, R45 to R47, R46 to R48
Connections:
- net /External-IO/VBAT renamed /External-IO/VBATT
- net /SX1276/DIO1 renamed /SX1231/DIO1
- net /SX1276/DIO2 renamed /SX1231/DIO2
- net /SX1276/DIO3 renamed /SX1231/DIO3
- net /SX1276/DIO4 renamed /SX1231/DIO4
- net /SX1276/DIO5 renamed /SX1231/DIO5
- net /SX1276/PA_BOOST renamed /SX1231/PA_BOOST
- net /SX1276/RADIO_XTAL_N renamed /SX1231/RADIO_XTAL_N
- net /SX1276/RADIO_XTAL_P renamed /SX1231/RADIO_XTAL_P
- net /SX1276/RFIO renamed /SX1231/RFIO
- net /SX1276/VR_ANA renamed /SX1231/VR_ANA
- net /SX1276/VR_DIG renamed /SX1231/VR_DIG
- net /SX1276/VR_PA renamed /SX1231/VR_PA
- C47 pad 1: /External-IO/FBL1 -> /Connectors/RGB1_12V
- C56 pad 1: /External-IO/FBL2 -> /Connectors/RGB2_12V
- C58 pad 2: /VIN -> /Connectors/VBATT
- C60 pad 1: /Connectors/USB_VIN -> /Connectors/USB_VBUS
- C60 pad 2: GND -> /Connectors/USB_VBUS_GND
- D5 pad 1: /Connectors/USB_VIN -> /Connectors/IGNITION
- D6 pad 1: /VIN -> /Connectors/VBATT
- D6 pad 2: /Connectors/IGNITION -> GND
- J3 pad 6: /ESP32-S3/CHIP_PU -> /ESP32-S3/RTS
- J5 pad A1: unconnected-(J5-PadA1) -> /Connectors/IGNITION
- J5 pad A2: unconnected-(J5-PadA2) -> /Connectors/RGB1_R
- J5 pad A3: unconnected-(J5-PadA3) -> /Connectors/RGB1_G
- J5 pad A4: unconnected-(J5-PadA4) -> /Connectors/RGB1_B
- J5 pad A5: unconnected-(J5-PadA5) -> /Connectors/RGB2_R
- J5 pad A6: unconnected-(J5-PadA6) -> /Connectors/RGB2_G
- J5 pad A7: unconnected-(J5-PadA7) -> /Connectors/RGB2_B
- J5 pad A8: unconnected-(J5-PadA8) -> GND
- J5 pad B1: unconnected-(J5-PadB1) -> /Connectors/VBATT
- J5 pad B2: unconnected-(J5-PadB2) -> GND
- J5 pad B3: unconnected-(J5-PadB3) -> /CAN_P
- J5 pad B4: unconnected-(J5-PadB4) -> /CAN_N
- J5 pad B5: unconnected-(J5-PadB5) -> /Connectors/USB_VBUS_GND
- J5 pad B6: unconnected-(J5-PadB6) -> /Connectors/USB_D_P
- J5 pad B7: unconnected-(J5-PadB7) -> /Connectors/USB_D_N
- J5 pad B8: unconnected-(J5-PadB8) -> /Connectors/USB_VBUS
- J5 pad C1: unconnected-(J5-PadC1) -> /Connectors/RGB2_12V
- J5 pad C2: unconnected-(J5-PadC2) -> /Connectors/DI_1
- J5 pad C3: unconnected-(J5-PadC3) -> /Connectors/DI_2
- J5 pad C4: unconnected-(J5-PadC4) -> /Connectors/DI_3
- J5 pad C5: unconnected-(J5-PadC5) -> /Connectors/DI_4
- J5 pad C6: unconnected-(J5-PadC6) -> /Connectors/PIXEL_2
- J5 pad C7: unconnected-(J5-PadC7) -> /Connectors/PIXEL_1
- J5 pad C8: unconnected-(J5-PadC8) -> /Connectors/RGB1_12V
- Q2 pad 2: /GPIO_GPO1 -> /RGB1_R
- Q2 pad 4: /GPIO_GPO2 -> /RGB1_G
- Q2 pad 5: /Connectors/GPO2 -> /Connectors/RGB1_G
- Q2 pad 6: /Connectors/GPO2 -> /Connectors/RGB1_G
- Q2 pad 7: /Connectors/GPO1 -> /Connectors/RGB1_R
- Q2 pad 8: /Connectors/GPO1 -> /Connectors/RGB1_R
- Q3 pad 2: /GPIO_GPO3 -> /RGB1_B
- Q3 pad 4: /GPIO_GPO4 -> /RGB2_R
- Q3 pad 5: /External-IO/GPIO4 -> /Connectors/RGB2_R
- Q3 pad 6: /External-IO/GPIO4 -> /Connectors/RGB2_R
- Q3 pad 7: /Connectors/GPO3 -> /Connectors/RGB1_B
- Q3 pad 8: /Connectors/GPO3 -> /Connectors/RGB1_B
- Q4 pad 2: /External-IO/GPIO_GPO5 -> /RGB2_G
- Q4 pad 4: /External-IO/GPIO_GPO6 -> /RGB2_B
- Q4 pad 5: /External-IO/GPO6 -> /Connectors/RGB2_B
- Q4 pad 6: /External-IO/GPO6 -> /Connectors/RGB2_B
- Q4 pad 7: /External-IO/GPO5 -> /Connectors/RGB2_G
- Q4 pad 8: /External-IO/GPO5 -> /Connectors/RGB2_G
- Q7 pad 3: /GPIO_GPI1 -> /DI_1
- Q7 pad 6: /GPIO_GPI2 -> /DI_2
- Q8 pad 3: /GPIO_GPI3 -> /DI_3
- Q8 pad 6: /GPIO_GPI4 -> /DI_4
- R10 pad 1: unconnected-(R10-Pad1) -> /ESP32-S3/RF_ANT_CHIP
- R14 pad 1: /ESP32-S3/CTS -> /ESP32-S3/GPIO0
- R15 pad 1: /ESP32-S3/GPIO45 -> /DI_2
- R16 pad 1: /ESP32-S3/GPIO46 -> /DI_3
- R17 pad 2: /External-IO/FBL1 -> /Connectors/RGB1_12V
- R24 pad 2: /External-IO/FBL2 -> /Connectors/RGB2_12V
- R26 pad 1: /Connectors/GPI2 -> /Connectors/DI_2
- R27 pad 1: /Connectors/GPI4 -> /Connectors/DI_4
- R34 pad 1: /Connectors/GPI3 -> /Connectors/DI_3
- R35 pad 1: /Connectors/GPI1 -> /Connectors/DI_1
- R40 pad 1: /LEDA -> /RGB1_PIXEL
- R40 pad 2: /Connectors/LEDA -> /Connectors/PIXEL_1
- R43 pad 1: /VIN -> /Connectors/VBATT
- R43 pad 2: /VSENSE -> /DI_1
- R44 pad 1: /VSENSE -> /DI_1
- R7 pad 1: /ESP32-S3/RXD -> /ESP32-S3/U0TXD
- R8 pad 2: /Connectors/USB_D_P -> /Connectors/USB_D_N
- R9 pad 2: /Connectors/USB_D_N -> /Connectors/USB_D_P
- TP8 pad 1: /VSENSE -> /DI_1
- U3 pad 10: /ESP32-S3/GPIO5 -> /RGB1_G
- U3 pad 11: /ESP32-S3/GPIO6 -> /RGB1_B
- U3 pad 12: /ESP32-S3/GPIO7 -> /RGB2_PWM
- U3 pad 13: /ESP32-S3/GPIO8 -> /RGB2_R
- U3 pad 14: unconnected-(U3-Pad14) -> /RGB2_G
- U3 pad 15: /ESP32-S3/GPIO10 -> /RGB2_B
- U3 pad 16: /ESP32-S3/GPIO11 -> /RGB1_PIXEL
- U3 pad 17: /ESP32-S3/GPIO12 -> /RGB2_PIXEL
- U3 pad 18: /VSENSE -> /DI_1
- U3 pad 19: /RP2040_EN -> /LHI
- U3 pad 28: /ESP32-S3/SPICS1 -> unconnected-(U3-Pad28)
- U3 pad 38: /CS2 -> /DI_4
- U3 pad 39: /ESP32-S3/GPIO34 -> /CS0
- U3 pad 43: unconnected-(U3-Pad43) -> /DI_1
- U3 pad 50: /ESP32-S3/TXD -> /ESP32-S3/U0RXD
- U3 pad 51: /ESP32-S3/GPIO45 -> /DI_2
- U3 pad 52: /ESP32-S3/GPIO46 -> /DI_3
- U3 pad 8: /ESP32-S3/GPIO3 -> /RGB1_PWM
- U3 pad 9: /ESP32-S3/GPIO4 -> /RGB1_R
- U5 pad 13: /External-IO/FBL2 -> /Connectors/RGB2_12V
- U5 pad 27: /External-IO/MISO -> /MISO
- U5 pad 28: /External-IO/CSN -> /CS0
- U5 pad 29: /External-IO/SCLK -> /SCLK
- U5 pad 30: /External-IO/MOSI -> /MOSI
- U5 pad 32: /External-IO/PWMI1 -> /RGB1_PWM
- U5 pad 33: /External-IO/PWMI2 -> /RGB2_PWM
- U5 pad 38: /External-IO/LHI -> /LHI
- U5 pad 48: /External-IO/FBL1 -> /Connectors/RGB1_12V
- U6 pad 1: /VIN -> /Connectors/IGNITION
- U6 pad 2: /Power/IGN -> /Connectors/VBATT
Routing:
- net /ESP32-S3/GPIO0: track 0.00 -> 28.6 mm, vias 0 -> 1
- net /ESP32-S3/CTS: track 43.5 -> 14.9 mm, vias 2 -> 1
- net /RGB1_PWM: track 0.00 -> 16.1 mm
- net /ESP32-S3/GPIO3: track 16.1 -> 0.00 mm
- net /DI_4: track 0.00 -> 15.5 mm
- net /CS2: track 15.5 -> 0.00 mm
- net /RGB1_R: track 0.00 -> 14.9 mm
- net /ESP32-S3/GPIO4: track 14.9 -> 0.00 mm
- net /RGB1_G: track 0.00 -> 13.5 mm
- net /ESP32-S3/GPIO5: track 13.5 -> 0.00 mm
- net unconnected-(R10-Pad1): track 13.5 -> 0.00 mm
- net /ESP32-S3/RF_ANT_CHIP: track 0.00 -> 13.5 mm
- net /RGB1_B: track 0.00 -> 12.2 mm
- net /ESP32-S3/GPIO6: track 12.2 -> 0.00 mm
- net /RGB2_PWM: track 0.00 -> 10.8 mm
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