File: hardware/underglow-controller/SX1231.kicad_sch (KiCad schematic)
At the start: 43 parts, among them J2 U.FL-R-SMT-1(10), U2 SX1231HIMLTRT, Y2 32mhz

Commit message: almost done picking components i think
Parts:
- renumbered C4 to C10, C5 to C11, C6 to C12, C7 to C13, C8 to C14, C9 to C2, C10 to C3, C11 to C4, C12 to C5, C13 to C6, C14 to C7, C2 to C8, C3 to C9

Commit message: muh colored schematics
Parts:
- added AE?: Antenna_Chip_MP, ConeCodes:SR4C033-L, symbol ConeCodes:Antenna_Chip_MP
- added J?: U.FL-R-SMT-1(10), ConeCodes:HRS_U.FL-R-SMT-1(10), symbol U.FL-R-SMT-1_10_:U.FL-R-SMT-1(10)
Connections:
- net GND: now also J?.1, J?.3
- net MISO: no longer U2.16 (MISO)
- net MOSI: no longer U2.17 (MOSI)
- net NSS: no longer U2.18 (NSS)
- net PA_BOOST: no longer U2.23 (PA_BOOST)
- net RADIO_XTAL_N: no longer U2.5 (XTB)
- net RADIO_XTAL_P: no longer U2.4 (XTA)
- net SCK: no longer U2.15 (SCK)
- net at R3.2: now also J?.2
Other:
- moved on the sheet: C10, C11, C12, C13, C14, C15, C16, C17, C18, C19, C2, C20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

Commit message: antenna af
Parts:
- removed AE?: Antenna_Chip_MP, ConeCodes:SR4C033-L, symbol ConeCodes:Antenna_Chip_MP
- removed C13: 3.3pF, Capacitor_SMD:C_0402_1005Metric, symbol Device:C_Small
- removed C15: 68pF, Capacitor_SMD:C_0402_1005Metric, symbol Device:C_Small
- removed C16, C17, C21: C_Small, Capacitor_SMD:C_0402_1005Metric, symbol Device:C_Small
- removed C18: 8.2pF, Capacitor_SMD:C_0402_1005Metric, symbol Device:C_Small
- removed C19: 6.8pF, Capacitor_SMD:C_0402_1005Metric, symbol Device:C_Small
- removed C20: 5.6pF, Capacitor_SMD:C_0402_1005Metric, symbol Device:C_Small
- removed L6: 33nH, Inductor_SMD:L_0402_1005Metric, symbol Device:L_Small
- removed L8, L9: 6.8nH, Inductor_SMD:L_0402_1005Metric, symbol Device:L_Small
- removed R5: 0R, Resistor_SMD:R_0402_1005Metric, symbol Device:R_Small
- added C10: 5.6nH, Inductor_SMD:L_0402_1005Metric, symbol Device:L_Small
- added C12, C8: 5.6pF, Capacitor_SMD:C_0402_1005Metric, symbol Device:C_Small
- added C5: 8.2pF, Capacitor_SMD:C_0402_1005Metric, symbol Device:C_Small
- added C9: 100pF, Capacitor_SMD:C_0402_1005Metric, symbol Device:C_Small
- added U2: PE42421SCAA-Z, Package_TO_SOT_SMD:SOT-363_SC-70-6, symbol RF_Switch:AS179-92LF
- C11: value 22pF -> 100pF; MPN GRM1555C1H220JA01D -> (none)
- C3: renamed from C9; value C_Small -> DNF
- C4: renamed from C10; value C_Small -> DNF
- J2: value U.FL-R-SMT-1(10) -> ANT; footprint ConeCodes:HRS_U.FL-R-SMT-1(10) -> (none); MPN U.FL-R-SMT-1(10) -> (none)
- L3: value 2.7nH -> 3.9nH; MPN LQW15AN2N7D00D -> LQW15AN3N9C00D
- L6: renamed from L7; value 3.9nH -> 120nH; MPN LQW15AN3N9C00D -> (none)
- gave numbers to parts that had none: 1
- renumbered C2 to C13, C3 to C14, C4 to C15, C5 to C16, C6 to C17, C7 to C18, C22 to C19, C8 to C2, C23 to C20, C14 to C6, C12 to C7, U2 to U3
Connections:
- net +3V3: now also R4.2, U2.6 (V2)
- net GND: now also L6.2, C12.2, C8.2, U2.2 (GND)
- net MISO: now also U3.16 (MISO)
- net MOSI: now also U3.17 (MOSI)
- net NSS: now also U3.18 (NSS)
- net PA_BOOST: now also U3.23 (PA_BOOST)
- net RADIO_XTAL_N: now also U3.5 (XTB)
- net RADIO_XTAL_P: now also U3.4 (XTA)
- net RFIO: now also C10.1
- net SCK: now also U3.15 (SCK)
- net at C6.1, L2.2, L3.2: now also C5.1; no longer C11.1
- net at C3.2, L4.1: now also C5.2; no longer C11.2
- net at C4.1, L5.2: now also C8.1, C9.1; no longer R2.2, R3.1
- net CER_ANT: now reaches J2.2
- net CER_ANT: now also R2.1
- net EXT_ANT: now reaches J3.2, R3.2
- net RX_TX: now reaches R4.1
- net RX_TX: now also U3.19 (RXTX), U2.4 (V1)
- new net: C10.2, C11.1, C12.1
- new net RF1: C9.2, U2.1 (J3)
- new net RF2: C11.2, U2.3 (J2)
- new net RFC: R2.2, R3.1, U2.5 (J1)
- no-connect marks 1 -> 0
Other:
- note added: "Control Voltages Signal Path Pin 6 (V DD ) = V DD Pin 4 (CTRL) = High RFC to RF2 --------------------- Pin 6 (V DD ) = V DD Pin 4 (CTRL) = Low RFC to RF1"
- note added: "High Power settings MUST be turned off when using PA0, and in Receive mode"
- note added: "REF says 33nH"
- note added: "THEORY: this is a CMOS chip that requires a higher voltage than the ESP or SX1231 can supply. By defaulting V1 to HIGH thru a pull up resistor, it will set the switch thru PA_BOOST by default, but when RXTX goes low (which happens for RXing), it should select RFIO"
- moved on the sheet: C2, C3, C4, C6, C7, J3, L2, L4, L5, L6, R2, R3

Commit message: pizz
Parts:
- removed J2: ANT, symbol U.FL-R-SMT-1_10_:U.FL-R-SMT-1(10)
- removed J3: U.FL-R-SMT-1(10), ConeCodes:HRS_U.FL-R-SMT-1(10), symbol U.FL-R-SMT-1_10_:U.FL-R-SMT-1(10)
- removed R2, R3: 0R, Resistor_SMD:R_0402_1005Metric, symbol Device:R_Small
- added AE2: 7488910915, ConeCodes:7488910915, symbol ConeCodes:7488910915
- added C10: 1.2pF, Capacitor_SMD:C_0402_1005Metric, symbol Device:C_Small
- added C11: DNF, Capacitor_SMD:C_0402_1005Metric, symbol Device:C_Small
- added C9: 0.5pF, Capacitor_SMD:C_0402_1005Metric, symbol Device:C_Small
- renumbered C9 to C12, C10 to C13, C11 to C14, C12 to C15, C13 to C16, C14 to C17, C15 to C18, C16 to C19, C17 to C20, C18 to C21, C19 to C22, C20 to C23
Connections:
- net CER_ANT: now also AE2.3 (FEED), C11.2, C9.2
- net GND: now also AE2.1 (PCB_Trace), AE2.2 (PCB_Trace), C10.1, C11.1
- net RFC: now also C10.2, C9.1
Other:
- moved on the sheet: R4

Commit message: im a piece of garbage
Parts:
- removed TP2: DIO0, TestPoint:TestPoint_Pad_D1.0mm, symbol Connector:TestPoint
- removed TP3: DIO1, TestPoint:TestPoint_Pad_D1.0mm, symbol Connector:TestPoint
- removed TP4: DIO2, TestPoint:TestPoint_Pad_D1.0mm, symbol Connector:TestPoint
- removed TP5: DIO3, TestPoint:TestPoint_Pad_D1.0mm, symbol Connector:TestPoint
- removed TP6: DIO4, TestPoint:TestPoint_Pad_D1.0mm, symbol Connector:TestPoint
- removed TP7: DIO5, TestPoint:TestPoint_Pad_D1.0mm, symbol Connector:TestPoint
Changed lines of the file:
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@@
   (junction (at 267.97 69.215) (diameter 0) (color 0 0 0 0)
   )
-  (wire (pts (xy 118.11 175.26) (xy 125.73 175.26))
-    (stroke (width 0) (type default) (color 0 0 0 0))
-  )
   (wire (pts (xy 59.69 117.475) (xy 83.82 117.475))
     (stroke (width 0) (type default) (color 0 0 0 0))
@@
     (stroke (width 0) (type default) (color 0 0 0 0))
   )
-  (wire (pts (xy 118.11 187.96) (xy 125.73 187.96))
-    (stroke (width 0) (type default) (color 0 0 0 0))
-  )
   (wire (pts (xy 166.37 42.545) (xy 166.37 43.815))
     (stroke (width 0) (type default) (color 0 0 0 0))
@@
     (stroke (width 0) (type default) (color 0 0 0 0))
   )
-  (wire (pts (xy 118.11 182.88) (xy 125.73 182.88))
-    (stroke (width 0) (type default) (color 0 0 0 0))
-  )
   (wire (pts (xy 246.38 64.135) (xy 254.635 64.135))
     (stroke (width 0) (type default) (color 0 0 0 0))
@@
     (stroke (width 0) (type default) (color 0 0 0 0))
   )
-  (wire (pts (xy 118.11 180.34) (xy 125.73 180.34))
-    (stroke (width 0) (type default) (color 0 0 0 0))
-  )
   (wire (pts (xy 166.37 19.685) (xy 160.02 19.685))
     (stroke (width 0) (type default) (color 0 0 0 0))
@@
     (stroke (width 0) (type default) (color 0 0 0 0))
   )
-  (wire (pts (xy 118.11 185.42) (xy 125.73 185.42))
-    (stroke (width 0) (type default) (color 0 0 0 0))
-  )
   (wire (pts (xy 128.27 138.43) (xy 128.27 134.62))
     (stroke (width 0) (type default) (color 0 0 0 0))
@@
   )
   (wire (pts (xy 196.85 42.545) (xy 196.85 43.815))
-    (stroke (width 0) (type default) (color 0 0 0 0))
-  )
-  (wire (pts (xy 118.11 177.8) (xy 125.73 177.8))
     (stroke (width 0) (type default) (color 0 0 0 0))
   )
@@
     (effects (font (size 1.27 1.27) italic) (justify left bottom))
   )
-  (label "DIO2" (at 125.73 180.34 180)
-    (effects (font (size 1.27 1.27)) (justify right bottom))
-  )
   (label "DIO3" (at 132.08 121.92 180)
     (effects (font (size 1.27 1.27)) (justify right bottom))
@@
     (effects (font (size 1.27 1.27)) (justify right bottom))
   )
-  (label "DIO1" (at 125.73 177.8 180)
-    (effects (font (size 1.27 1.27)) (justify right bottom))
-  )
   (label "RX_TX" (at 247.015 69.215 0)
     (effects (font (size 1.27 1.27) italic) (justify left bottom))
@@
     (effects (font (size 1.27 1.27)) (justify right bottom))
   )
-  (label "DIO4" (at 125.73 185.42 180)
-    (effects (font (size 1.27 1.27)) (justify right bottom))
-  )
-  (label "DIO5" (at 125.73 187.96 180)
-    (effects (font (size 1.27 1.27)) (justify right bottom))
-  )
   (label "RFIO" (at 135.89 102.87 180)
     (effects (font (size 1.27 1.27)) (justify right bottom))
@@
     (effects (font (size 1.27 1.27)) (justify left bottom))
   )
-  (label "DIO0" (at 125.73 175.26 180)
-    (effects (font (size 1.27 1.27)) (justify right bottom))
-  )
   (label "MOSI" (at 78.74 132.715 180)
     (effects (font (size 1.27 1.27)) (justify right bottom))
@@
   (label "RF1" (at 222.885 61.595 0)
     (effects (font (size 1.27 1.27)) (justify left bottom))
-  )
-  (label "DIO3" (at 125.73 182.88 180)
-    (effects (font (size 1.27 1.27)) (justify right bottom))
   )
   (label "VBAT1" (at 46.99 88.9 0)
@@
     (pin "2")
   )
-  (symbol (lib_id "Connector:TestPoint") (at 118.11 180.34 90) (unit 1)
-    (in_bom yes) (on_board yes)
-    (property "Reference" "TP4" (id 0) (at 111.76 180.34 90))
-    (property "Value" "DIO2" (id 1) (at 106.68 180.34 90))
-    (property "Footprint" "TestPoint:TestPoint_Pad_D1.0mm" (id 2) (at 118.11 175.26 0)
-      (effects (font (size 1.27 1.27)) hide)
-    )
-    (property "Datasheet" "~" (id 3) (at 118.11 175.26 0)
-      (effects (font (size 1.27 1.27)) hide)
-    )
-    (pin "1")
-  )
   (symbol (lib_id "Device:C_Small") (at 166.37 46.355 0) (unit 1)
     (in_bom yes) (on_board yes) (fields_autoplaced)
@@
     (pin "1")
   )
-  (symbol (lib_id "Connector:TestPoint") (at 118.11 185.42 90) (unit 1)
-    (in_bom yes) (on_board yes)
-    (property "Reference" "TP6" (id 0) (at 111.76 185.42 90))
-    (property "Value" "DIO4" (id 1) (at 106.68 185.42 90))
-    (property "Footprint" "TestPoint:TestPoint_Pad_D1.0mm" (id 2) (at 118.11 180.34 0)
-      (effects (font (size 1.27 1.27)) hide)
-    )
-    (property "Datasheet" "~" (id 3) (at 118.11 180.34 0)
-      (effects (font (size 1.27 1.27)) hide)
-    )
-    (pin "1")
-  )
-  (symbol (lib_id "Connector:TestPoint") (at 118.11 187.96 90) (unit 1)
-    (in_bom yes) (on_board yes)
-    (property "Reference" "TP7" (id 0) (at 111.76 187.96 90))
-    (property "Value" "DIO5" (id 1) (at 106.68 187.96 90))
-    (property "Footprint" "TestPoint:TestPoint_Pad_D1.0mm" (id 2) (at 118.11 182.88 0)
-      (effects (font (size 1.27 1.27)) hide)
-    )
-    (property "Datasheet" "~" (id 3) (at 118.11 182.88 0)
-      (effects (font (size 1.27 1.27)) hide)
-    )
-    (pin "1")
-  )
   (symbol (lib_id "power:GND") (at 153.67 29.845 0) (unit 1)
     (in_bom yes) (on_board yes) (fields_autoplaced)
@@
     (pin "1")
     (pin "2")
-  )
-  (symbol (lib_id "Connector:TestPoint") (at 118.11 177.8 90) (unit 1)
-    (in_bom yes) (on_board yes)
-    (property "Reference" "TP3" (id 0) (at 111.76 177.8 90))
-    (property "Value" "DIO1" (id 1) (at 106.68 177.8 90))
-    (property "Footprint" "TestPoint:TestPoint_Pad_D1.0mm" (id 2) (at 118.11 172.72 0)
-      (effects (font (size 1.27 1.27)) hide)
-    )
-    (property "Datasheet" "~" (id 3) (at 118.11 172.72 0)
-      (effects (font (size 1.27 1.27)) hide)
-    )
-    (pin "1")
-  )
-  (symbol (lib_id "Connector:TestPoint") (at 118.11 175.26 90) (unit 1)
-    (in_bom yes) (on_board yes)
-    (property "Reference" "TP2" (id 0) (at 111.76 175.26 90))
-    (property "Value" "DIO0" (id 1) (at 106.68 175.26 90))
-    (property "Footprint" "TestPoint:TestPoint_Pad_D1.0mm" (id 2) (at 118.11 170.18 0)
-      (effects (font (size 1.27 1.27)) hide)
-    )
-    (property "Datasheet" "~" (id 3) (at 118.11 170.18 0)
-      (effects (font (size 1.27 1.27)) hide)
-    )
-    (pin "1")
   )
   (symbol (lib_id "RF_Switch:AS179-92LF") (at 236.22 66.675 0) (mirror y) (unit 1)
@@
     (pin "9")
   )
-  (symbol (lib_id "Connector:TestPoint") (at 118.11 182.88 90) (unit 1)
-    (in_bom yes) (on_board yes)
-    (property "Reference" "TP5" (id 0) (at 111.76 182.88 90))
-    (property "Value" "DIO3" (id 1) (at 106.68 182.88 90))
-    (property "Footprint" "TestPoint:TestPoint_Pad_D1.0mm" (id 2) (at 118.11 177.8 0)
-      (effects (font (size 1.27 1.27)) hide)
-    )
-    (property "Datasheet" "~" (id 3) (at 118.11 177.8 0)
-      (effects (font (size 1.27 1.27)) hide)
-    )
-    (pin "1")
-  )
   (symbol (lib_id "Device:C_Small") (at 220.345 61.595 90) (unit 1)

Commit message: aaaaa
Parts:
- renumbered R4 to R2
Changed lines of the file:
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@@
   (symbol (lib_id "power:+3V3") (at 46.99 83.82 0) (unit 1)
     (in_bom yes) (on_board yes) (fields_autoplaced)
-    (property "Reference" "#PWR015" (id 0) (at 46.99 87.63 0)
+    (property "Reference" "#PWR014" (id 0) (at 46.99 87.63 0)
       (effects (font (size 1.27 1.27)) hide)
     )
@@
   (symbol (lib_id "power:GND") (at 24.13 128.27 0) (unit 1)
     (in_bom yes) (on_board yes) (fields_autoplaced)
-    (property "Reference" "#PWR023" (id 0) (at 24.13 134.62 0)
+    (property "Reference" "#PWR022" (id 0) (at 24.13 134.62 0)
       (effects (font (size 1.27 1.27)) hide)
     )
@@
   (symbol (lib_id "power:GND") (at 204.47 73.025 0) (unit 1)
     (in_bom yes) (on_board yes) (fields_autoplaced)
-    (property "Reference" "#PWR011" (id 0) (at 204.47 79.375 0)
+    (property "Reference" "#PWR010" (id 0) (at 204.47 79.375 0)
       (effects (font (size 1.27 1.27)) hide)
     )
@@
   (symbol (lib_id "power:GND") (at 43.18 128.27 0) (unit 1)
     (in_bom yes) (on_board yes) (fields_autoplaced)
-    (property "Reference" "#PWR025" (id 0) (at 43.18 134.62 0)
+    (property "Reference" "#PWR024" (id 0) (at 43.18 134.62 0)
       (effects (font (size 1.27 1.27)) hide)
     )
@@
   (symbol (lib_id "power:GND") (at 26.67 104.14 0) (unit 1)
     (in_bom yes) (on_board yes) (fields_autoplaced)
-    (property "Reference" "#PWR016" (id 0) (at 26.67 110.49 0)
+    (property "Reference" "#PWR015" (id 0) (at 26.67 110.49 0)
       (effects (font (size 1.27 1.27)) hide)
     )
@@
   (symbol (lib_id "power:GND") (at 46.99 104.14 0) (unit 1)
     (in_bom yes) (on_board yes) (fields_autoplaced)
-    (property "Reference" "#PWR018" (id 0) (at 46.99 110.49 0)
+    (property "Reference" "#PWR017" (id 0) (at 46.99 110.49 0)
       (effects (font (size 1.27 1.27)) hide)
     )
@@
   (symbol (lib_id "power:GND") (at 36.83 104.14 0) (unit 1)
     (in_bom yes) (on_board yes) (fields_autoplaced)
-    (property "Reference" "#PWR017" (id 0) (at 36.83 110.49 0)
+    (property "Reference" "#PWR016" (id 0) (at 36.83 110.49 0)
       (effects (font (size 1.27 1.27)) hide)
     )
@@
   (symbol (lib_id "power:+3V3") (at 36.83 83.82 0) (unit 1)
     (in_bom yes) (on_board yes) (fields_autoplaced)
-    (property "Reference" "#PWR014" (id 0) (at 36.83 87.63 0)
+    (property "Reference" "#PWR013" (id 0) (at 36.83 87.63 0)
       (effects (font (size 1.27 1.27)) hide)
     )
@@
   (symbol (lib_id "power:GND") (at 34.29 118.11 180) (unit 1)
     (in_bom yes) (on_board yes) (fields_autoplaced)
-    (property "Reference" "#PWR022" (id 0) (at 34.29 111.76 0)
+    (property "Reference" "#PWR021" (id 0) (at 34.29 111.76 0)
       (effects (font (size 1.27 1.27)) hide)
     )
@@
   (symbol (lib_id "power:+3V3") (at 26.67 83.82 0) (unit 1)
     (in_bom yes) (on_board yes) (fields_autoplaced)
-    (property "Reference" "#PWR013" (id 0) (at 26.67 87.63 0)
+    (property "Reference" "#PWR012" (id 0) (at 26.67 87.63 0)
       (effects (font (size 1.27 1.27)) hide)
     )
@@
   (symbol (lib_id "power:GND") (at 128.27 138.43 0) (unit 1)
     (in_bom yes) (on_board yes) (fields_autoplaced)
-    (property "Reference" "#PWR026" (id 0) (at 128.27 144.78 0)
+    (property "Reference" "#PWR025" (id 0) (at 128.27 144.78 0)
       (effects (font (size 1.27 1.27)) hide)
     )
@@
   (symbol (lib_id "power:GND") (at 233.68 76.835 0) (unit 1)
     (in_bom yes) (on_board yes) (fields_autoplaced)
-    (property "Reference" "#PWR012" (id 0) (at 233.68 83.185 0)
+    (property "Reference" "#PWR011" (id 0) (at 233.68 83.185 0)
       (effects (font (size 1.27 1.27)) hide)
     )
@@
   (symbol (lib_id "Device:R_Small") (at 260.985 69.215 90) (unit 1)
     (in_bom yes) (on_board yes)
-    (property "Reference" "R4" (id 0) (at 259.715 67.31 90))
+    (property "Reference" "R2" (id 0) (at 259.715 67.31 90))
     (property "Value" "0R" (id 1) (at 262.255 67.31 90))
     (property "Footprint" "Resistor_SMD:R_0402_1005Metric" (id 2) (at 260.985 69.215 0)
@@
   (symbol (lib_id "power:GND") (at 189.23 73.025 0) (unit 1)
     (in_bom yes) (on_board yes) (fields_autoplaced)
-    (property "Reference" "#PWR010" (id 0) (at 189.23 79.375 0)
+    (property "Reference" "#PWR09" (id 0) (at 189.23 79.375 0)
       (effects (font (size 1.27 1.27)) hide)
     )
@@
   (symbol (lib_id "power:GND") (at 148.59 104.14 90) (unit 1)
     (in_bom yes) (on_board yes) (fields_autoplaced)
-    (property "Reference" "#PWR021" (id 0) (at 154.94 104.14 0)
+    (property "Reference" "#PWR020" (id 0) (at 154.94 104.14 0)
       (effects (font (size 1.27 1.27)) hide)
     )
@@
   (symbol (lib_id "power:GND") (at 68.58 104.14 0) (unit 1)
     (in_bom yes) (on_board yes) (fields_autoplaced)
-    (property "Reference" "#PWR020" (id 0) (at 68.58 110.49 0)
+    (property "Reference" "#PWR019" (id 0) (at 68.58 110.49 0)
       (effects (font (size 1.27 1.27)) hide)
     )
@@
   (symbol (lib_id "power:GND") (at 34.29 128.27 0) (unit 1)
     (in_bom yes) (on_board yes) (fields_autoplaced)
-    (property "Reference" "#PWR024" (id 0) (at 34.29 134.62 0)
+    (property "Reference" "#PWR023" (id 0) (at 34.29 134.62 0)
       (effects (font (size 1.27 1.27)) hide)
     )
@@
   (symbol (lib_id "power:GND") (at 58.42 104.14 0) (unit 1)
     (in_bom yes) (on_board yes) (fields_autoplaced)
-    (property "Reference" "#PWR019" (id 0) (at 58.42 110.49 0)
-      (effects (font (size 1.27 1.27)) hide)
-    )
+    (property "Reference" "#PWR018" (id 0) (at 58.42 110.49 0)
+      (effects (font (size 1.27 1.27)) hide)
+    )
