File: hardware/underglow-controller/Connectors.kicad_sch (KiCad schematic)
At the start: 6 parts, among them J5 Delphi_Sicma_24, J7 Conn_01x05

Commit message: almost done picking components i think
Parts:
- renumbered D8 to D7, D9 to D8, J7 to J6
Changed lines of the file:
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@@
   (symbol (lib_id "power:GND") (at 22.86 67.31 0) (unit 1)
     (in_bom yes) (on_board yes) (fields_autoplaced)
-    (property "Reference" "#PWR?" (id 0) (at 22.86 73.66 0)
+    (property "Reference" "#PWR084" (id 0) (at 22.86 73.66 0)
       (effects (font (size 1.27 1.27)) hide)
     )
@@
   (symbol (lib_id "Device:D_TVS_Dual_AAC") (at 48.26 149.225 0) (unit 1)
     (in_bom yes) (on_board yes) (fields_autoplaced)
-    (property "Reference" "D9" (id 0) (at 48.26 142.24 0))
+    (property "Reference" "D8" (id 0) (at 48.26 142.24 0))
     (property "Value" "PESD2CANFD24V-T" (id 1) (at 48.26 144.78 0))
     (property "Footprint" "Package_TO_SOT_SMD:SOT-23" (id 2) (at 44.45 149.225 0)
@@
   (symbol (lib_id "power:GND") (at 48.26 137.16 0) (unit 1)
     (in_bom yes) (on_board yes) (fields_autoplaced)
-    (property "Reference" "#PWR086" (id 0) (at 48.26 143.51 0)
+    (property "Reference" "#PWR085" (id 0) (at 48.26 143.51 0)
       (effects (font (size 1.27 1.27)) hide)
     )
@@
   (symbol (lib_id "power:GND") (at 48.26 153.035 0) (unit 1)
     (in_bom yes) (on_board yes) (fields_autoplaced)
-    (property "Reference" "#PWR089" (id 0) (at 48.26 159.385 0)
+    (property "Reference" "#PWR086" (id 0) (at 48.26 159.385 0)
       (effects (font (size 1.27 1.27)) hide)
     )
@@
   (symbol (lib_id "power:GND") (at 19.05 38.1 0) (unit 1)
     (in_bom yes) (on_board yes) (fields_autoplaced)
-    (property "Reference" "#PWR?" (id 0) (at 19.05 44.45 0)
+    (property "Reference" "#PWR083" (id 0) (at 19.05 44.45 0)
       (effects (font (size 1.27 1.27)) hide)
     )
@@
   (symbol (lib_id "Device:D_TVS_Dual_AAC") (at 48.26 133.35 0) (unit 1)
     (in_bom yes) (on_board yes) (fields_autoplaced)
-    (property "Reference" "D8" (id 0) (at 48.26 126.365 0))
+    (property "Reference" "D7" (id 0) (at 48.26 126.365 0))
     (property "Value" "PESD2CANFD24V-T" (id 1) (at 48.26 128.905 0))
     (property "Footprint" "Package_TO_SOT_SMD:SOT-23" (id 2) (at 44.45 133.35 0)
@@
   (symbol (lib_id "Connector_Generic:Conn_01x05") (at 132.08 184.785 0) (unit 1)
     (in_bom yes) (on_board yes) (fields_autoplaced)
-    (property "Reference" "J7" (id 0) (at 135.255 183.5149 0)
-      (effects (font (size 1.27 1.27)) (justify left))
-    )
+    (property "Reference" "J6" (id 0) (at 135.255 183.5149 0)
+      (effects (font (size 1.27 1.27)) (justify left))
+    )

Commit message: muh colored schematics
Parts:
- removed D7: PESD2CANFD24V-T, Package_TO_SOT_SMD:SOT-23, symbol Device:D_TVS_Dual_AAC
- added D7: PESD2USB3UV-T, Package_TO_SOT_SMD:SOT-23, symbol Device:D_Zener_Dual_CommonAnode_KKA_Parallel
- added H? (x2): MountingHole_Pad, symbol Mechanical:MountingHole_Pad
Connections:
- net USB_GND is gone; now on net GND: C60.2, J5.B5
- net GND: now also D7.3 (A), H?.1, H?.1
- net USB_D_N: now also D7.1 (K)
- net USB_D_P: now also D7.2 (K)
Other:
- note added: "DEBUG"
- note added: "ESD"
- moved on the sheet: C60, C61, D8, J5, J6

Commit message: antenna af
Parts:
- gave numbers to parts that had none: 2
- renumbered C60 to C57, C61 to C58, J5 to J6, J6 to J7
Changed lines of the file:
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@@
   (symbol (lib_id "power:GND") (at 22.86 67.31 270) (unit 1)
     (in_bom yes) (on_board yes) (fields_autoplaced)
-    (property "Reference" "#PWR084" (id 0) (at 16.51 67.31 0)
+    (property "Reference" "#PWR085" (id 0) (at 16.51 67.31 0)
       (effects (font (size 1.27 1.27)) hide)
     )
@@
   (symbol (lib_id "power:GND") (at 160.02 53.34 0) (unit 1)
     (in_bom yes) (on_board yes) (fields_autoplaced)
-    (property "Reference" "#PWR085" (id 0) (at 160.02 59.69 0)
+    (property "Reference" "#PWR084" (id 0) (at 160.02 59.69 0)
       (effects (font (size 1.27 1.27)) hide)
     )
@@
   (symbol (lib_id "Mechanical:MountingHole_Pad") (at 107.95 92.71 0) (unit 1)
     (in_bom yes) (on_board yes) (fields_autoplaced)
-    (property "Reference" "H?" (id 0) (at 110.49 90.1699 0)
+    (property "Reference" "H3" (id 0) (at 110.49 90.1699 0)
       (effects (font (size 1.27 1.27)) (justify left))
     )
@@
   (symbol (lib_id "power:GND") (at 160.02 74.93 0) (unit 1)
     (in_bom yes) (on_board yes) (fields_autoplaced)
-    (property "Reference" "#PWR086" (id 0) (at 160.02 81.28 0)
+    (property "Reference" "#PWR087" (id 0) (at 160.02 81.28 0)
       (effects (font (size 1.27 1.27)) hide)
     )
@@
   (symbol (lib_id "Device:C_Small") (at 34.29 109.22 90) (unit 1)
     (in_bom yes) (on_board yes) (fields_autoplaced)
-    (property "Reference" "C61" (id 0) (at 34.2963 102.235 90))
+    (property "Reference" "C58" (id 0) (at 34.2963 102.235 90))
     (property "Value" "10uF" (id 1) (at 34.2963 104.775 90))
     (property "Footprint" "Capacitor_SMD:C_0805_2012Metric" (id 2) (at 34.29 109.22 0)
@@
   (symbol (lib_id "Device:C_Small") (at 106.68 68.58 0) (unit 1)
     (in_bom yes) (on_board yes)
-    (property "Reference" "C60" (id 0) (at 108.585 67.3162 0)
+    (property "Reference" "C57" (id 0) (at 108.585 67.3162 0)
       (effects (font (size 1.27 1.27)) (justify left))
     )
@@
   (symbol (lib_id "power:GND") (at 26.67 111.76 270) (unit 1)
     (in_bom yes) (on_board yes)
-    (property "Reference" "#PWR088" (id 0) (at 20.32 111.76 0)
+    (property "Reference" "#PWR091" (id 0) (at 20.32 111.76 0)
       (effects (font (size 1.27 1.27)) hide)
     )
@@
   (symbol (lib_id "power:GND") (at 107.95 95.25 0) (unit 1)
     (in_bom yes) (on_board yes) (fields_autoplaced)
-    (property "Reference" "#PWR?" (id 0) (at 107.95 101.6 0)
+    (property "Reference" "#PWR089" (id 0) (at 107.95 101.6 0)
       (effects (font (size 1.27 1.27)) hide)
     )
@@
   (symbol (lib_id "Mechanical:MountingHole_Pad") (at 97.79 92.71 0) (unit 1)
     (in_bom yes) (on_board yes) (fields_autoplaced)
-    (property "Reference" "H?" (id 0) (at 100.33 90.1699 0)
+    (property "Reference" "H2" (id 0) (at 100.33 90.1699 0)
       (effects (font (size 1.27 1.27)) (justify left))
     )
@@
   (symbol (lib_id "power:GND") (at 97.79 95.25 0) (unit 1)
     (in_bom yes) (on_board yes) (fields_autoplaced)
-    (property "Reference" "#PWR?" (id 0) (at 97.79 101.6 0)
+    (property "Reference" "#PWR088" (id 0) (at 97.79 101.6 0)
       (effects (font (size 1.27 1.27)) hide)
     )
@@
   (symbol (lib_id "ConeCodes:Delphi_Sicma_24") (at 58.42 44.45 0) (unit 1)
     (in_bom yes) (on_board yes) (fields_autoplaced)
-    (property "Reference" "J5" (id 0) (at 58.42 26.67 0))
+    (property "Reference" "J6" (id 0) (at 58.42 26.67 0))
     (property "Value" "Delphi_Sicma_24" (id 1) (at 58.42 29.21 0))
     (property "Footprint" "ConeCodes:Delphi_Sicma_24_Black" (id 2) (at 58.42 27.94 0)
@@
   (symbol (lib_id "power:+3V3") (at 40.64 106.68 0) (unit 1)
     (in_bom yes) (on_board yes) (fields_autoplaced)
-    (property "Reference" "#PWR087" (id 0) (at 40.64 110.49 0)
+    (property "Reference" "#PWR090" (id 0) (at 40.64 110.49 0)
       (effects (font (size 1.27 1.27)) hide)
     )
@@
   (symbol (lib_id "Connector_Generic:Conn_01x05") (at 57.15 116.84 0) (unit 1)
     (in_bom yes) (on_board yes) (fields_autoplaced)
-    (property "Reference" "J6" (id 0) (at 60.325 115.5699 0)
+    (property "Reference" "J7" (id 0) (at 60.325 115.5699 0)
       (effects (font (size 1.27 1.27)) (justify left))
     )
@@
   (symbol (lib_id "power:GND") (at 106.68 73.66 0) (unit 1)
     (in_bom yes) (on_board yes) (fields_autoplaced)
-    (property "Reference" "#PWR?" (id 0) (at 106.68 80.01 0)
-      (effects (font (size 1.27 1.27)) hide)
-    )
+    (property "Reference" "#PWR086" (id 0) (at 106.68 80.01 0)
+      (effects (font (size 1.27 1.27)) hide)
+    )

Commit message: pizz
Parts:
- renumbered C57 to C60, C58 to C61, J6 to J5, J7 to J6
Connections:
- net USB_D_N: now also D7.2 (K); no longer D7.1 (K)
- net USB_D_P: now also D7.1 (K); no longer D7.2 (K)
Changed lines of the file:
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@@
     (effects (font (size 1.27 1.27)) (justify left bottom))
   )
-  (label "USB_D_N" (at 181.61 43.18 180)
+  (label "USB_D_P" (at 181.61 43.18 180)
     (effects (font (size 1.27 1.27)) (justify right bottom))
   )
@@
     (effects (font (size 1.27 1.27)) (justify right bottom))
   )
-  (label "USB_D_P" (at 140.97 43.18 0)
+  (label "USB_D_N" (at 140.97 43.18 0)
     (effects (font (size 1.27 1.27)) (justify left bottom))
   )
@@
   (symbol (lib_id "power:GND") (at 22.86 67.31 270) (unit 1)
     (in_bom yes) (on_board yes) (fields_autoplaced)
-    (property "Reference" "#PWR085" (id 0) (at 16.51 67.31 0)
+    (property "Reference" "#PWR086" (id 0) (at 16.51 67.31 0)
       (effects (font (size 1.27 1.27)) hide)
     )
@@
   (symbol (lib_id "power:GND") (at 160.02 53.34 0) (unit 1)
     (in_bom yes) (on_board yes) (fields_autoplaced)
-    (property "Reference" "#PWR084" (id 0) (at 160.02 59.69 0)
+    (property "Reference" "#PWR085" (id 0) (at 160.02 59.69 0)
       (effects (font (size 1.27 1.27)) hide)
     )
@@
   (symbol (lib_id "power:GND") (at 160.02 74.93 0) (unit 1)
     (in_bom yes) (on_board yes) (fields_autoplaced)
-    (property "Reference" "#PWR087" (id 0) (at 160.02 81.28 0)
+    (property "Reference" "#PWR088" (id 0) (at 160.02 81.28 0)
       (effects (font (size 1.27 1.27)) hide)
     )
@@
   (symbol (lib_id "Device:C_Small") (at 34.29 109.22 90) (unit 1)
     (in_bom yes) (on_board yes) (fields_autoplaced)
-    (property "Reference" "C58" (id 0) (at 34.2963 102.235 90))
+    (property "Reference" "C61" (id 0) (at 34.2963 102.235 90))
     (property "Value" "10uF" (id 1) (at 34.2963 104.775 90))
     (property "Footprint" "Capacitor_SMD:C_0805_2012Metric" (id 2) (at 34.29 109.22 0)
@@
   (symbol (lib_id "Device:C_Small") (at 106.68 68.58 0) (unit 1)
     (in_bom yes) (on_board yes)
-    (property "Reference" "C57" (id 0) (at 108.585 67.3162 0)
+    (property "Reference" "C60" (id 0) (at 108.585 67.3162 0)
       (effects (font (size 1.27 1.27)) (justify left))
     )
@@
   (symbol (lib_id "power:GND") (at 22.86 36.83 270) (unit 1)
     (in_bom yes) (on_board yes) (fields_autoplaced)
-    (property "Reference" "#PWR083" (id 0) (at 16.51 36.83 0)
+    (property "Reference" "#PWR084" (id 0) (at 16.51 36.83 0)
       (effects (font (size 1.27 1.27)) hide)
     )
@@
   (symbol (lib_id "power:GND") (at 26.67 111.76 270) (unit 1)
     (in_bom yes) (on_board yes)
-    (property "Reference" "#PWR091" (id 0) (at 20.32 111.76 0)
+    (property "Reference" "#PWR092" (id 0) (at 20.32 111.76 0)
       (effects (font (size 1.27 1.27)) hide)
     )
@@
   (symbol (lib_id "power:GND") (at 107.95 95.25 0) (unit 1)
     (in_bom yes) (on_board yes) (fields_autoplaced)
-    (property "Reference" "#PWR089" (id 0) (at 107.95 101.6 0)
+    (property "Reference" "#PWR090" (id 0) (at 107.95 101.6 0)
       (effects (font (size 1.27 1.27)) hide)
     )
@@
   (symbol (lib_id "power:GND") (at 97.79 95.25 0) (unit 1)
     (in_bom yes) (on_board yes) (fields_autoplaced)
-    (property "Reference" "#PWR088" (id 0) (at 97.79 101.6 0)
+    (property "Reference" "#PWR089" (id 0) (at 97.79 101.6 0)
       (effects (font (size 1.27 1.27)) hide)
     )
@@
   (symbol (lib_id "ConeCodes:Delphi_Sicma_24") (at 58.42 44.45 0) (unit 1)
     (in_bom yes) (on_board yes) (fields_autoplaced)
-    (property "Reference" "J6" (id 0) (at 58.42 26.67 0))
+    (property "Reference" "J5" (id 0) (at 58.42 26.67 0))
     (property "Value" "Delphi_Sicma_24" (id 1) (at 58.42 29.21 0))
     (property "Footprint" "ConeCodes:Delphi_Sicma_24_Black" (id 2) (at 58.42 27.94 0)
@@
   (symbol (lib_id "power:+3V3") (at 40.64 106.68 0) (unit 1)
     (in_bom yes) (on_board yes) (fields_autoplaced)
-    (property "Reference" "#PWR090" (id 0) (at 40.64 110.49 0)
+    (property "Reference" "#PWR091" (id 0) (at 40.64 110.49 0)
       (effects (font (size 1.27 1.27)) hide)
     )
@@
   (symbol (lib_id "Connector_Generic:Conn_01x05") (at 57.15 116.84 0) (unit 1)
     (in_bom yes) (on_board yes) (fields_autoplaced)
-    (property "Reference" "J7" (id 0) (at 60.325 115.5699 0)
+    (property "Reference" "J6" (id 0) (at 60.325 115.5699 0)
       (effects (font (size 1.27 1.27)) (justify left))
     )
@@
   (symbol (lib_id "power:GND") (at 106.68 73.66 0) (unit 1)
     (in_bom yes) (on_board yes) (fields_autoplaced)
-    (property "Reference" "#PWR086" (id 0) (at 106.68 80.01 0)
-      (effects (font (size 1.27 1.27)) hide)
-    )
+    (property "Reference" "#PWR087" (id 0) (at 106.68 80.01 0)
+      (effects (font (size 1.27 1.27)) hide)
+    )

Commit message: im a piece of garbage
Parts:
- removed C60: 10uF, Capacitor_SMD:C_0805_2012Metric, symbol Device:C_Small
- H2, H3: footprint (none) -> MountingHole:MountingHole_6.4mm_M6_Pad_Via
Changed lines of the file:
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@@
     (comment 1 "https://github.com/miata-bot/can-link")
-  )
-  (junction (at 106.68 73.66) (diameter 0) (color 0 0 0 1)
   )
   (junction (at 40.64 109.22) (diameter 0) (color 0 0 0 0)
@@
     (stroke (width 0) (type default) (color 0 194 194 1))
   )
-  (wire (pts (xy 106.68 73.66) (xy 106.68 71.12))
-    (stroke (width 0) (type default) (color 0 0 0 1))
-  )
   (wire (pts (xy 87.63 67.31) (xy 64.77 67.31))
     (stroke (width 0) (type default) (color 255 255 255 1))
@@
   (wire (pts (xy 31.75 46.99) (xy 48.26 46.99))
     (stroke (width 0) (type default) (color 0 0 255 1))
-  )
-  (wire (pts (xy 106.68 63.5) (xy 106.68 66.04))
-    (stroke (width 0) (type default) (color 72 0 0 1))
   )
   (text "DEBUG" (at 16.51 91.44 0)
@@
       (effects (font (size 1.27 1.27)) (justify left) hide)
     )
-    (property "Footprint" "" (id 2) (at 107.95 92.71 0)
+    (property "Footprint" "MountingHole:MountingHole_6.4mm_M6_Pad_Via" (id 2) (at 107.95 92.71 0)
       (effects (font (size 1.27 1.27)) hide)
     )
@@
     (pin "2")
   )
-  (symbol (lib_id "Device:C_Small") (at 106.68 68.58 0) (unit 1)
-    (in_bom yes) (on_board yes)
-    (property "Reference" "C60" (id 0) (at 108.585 67.3162 0)
-      (effects (font (size 1.27 1.27)) (justify left))
-    )
-    (property "Value" "10uF" (id 1) (at 108.585 69.8562 0)
-      (effects (font (size 1.27 1.27)) (justify left))
-    )
-    (property "Footprint" "Capacitor_SMD:C_0805_2012Metric" (id 2) (at 106.68 68.58 0)
-      (effects (font (size 1.27 1.27)) hide)
-    )
-    (property "Datasheet" "~" (id 3) (at 106.68 68.58 0)
-      (effects (font (size 1.27 1.27)) hide)
-    )
-    (property "Description" "CAP CER 10UF 10V 0805" (id 6) (at 106.68 68.58 0)
-      (effects (font (size 1.27 1.27)) hide)
-    )
-    (property "MPN" "GRT21BC81A106KE01L" (id 7) (at 106.68 68.58 0)
-      (effects (font (size 1.27 1.27)) hide)
-    )
-    (pin "1")
-    (pin "2")
-  )
   (symbol (lib_id "power:GND") (at 22.86 36.83 270) (unit 1)
     (in_bom yes) (on_board yes) (fields_autoplaced)
@@
       (effects (font (size 1.27 1.27)) (justify left) hide)
     )
-    (property "Footprint" "" (id 2) (at 97.79 92.71 0)
-      (effects (font (size 1.27 1.27)) hide)
-    )
+    (property "Footprint" "MountingHole:MountingHole_6.4mm_M6_Pad_Via" (id 2) (at 97.79 92.71 0)
+      (effects (font (size 1.27 1.27)) hide)
+    )

Commit message: aaaaa
Parts:
- renumbered C61 to C45, D7 to D5, D8 to D6, J5 to J3, J6 to J4
Changed lines of the file:
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@@
   (symbol (lib_id "power:GND") (at 22.86 67.31 270) (unit 1)
     (in_bom yes) (on_board yes) (fields_autoplaced)
-    (property "Reference" "#PWR086" (id 0) (at 16.51 67.31 0)
+    (property "Reference" "#PWR072" (id 0) (at 16.51 67.31 0)
       (effects (font (size 1.27 1.27)) hide)
     )
@@
   (symbol (lib_id "Device:D_TVS_Dual_AAC") (at 160.02 71.12 0) (unit 1)
     (in_bom yes) (on_board yes) (fields_autoplaced)
-    (property "Reference" "D8" (id 0) (at 160.02 64.135 0))
+    (property "Reference" "D6" (id 0) (at 160.02 64.135 0))
     (property "Value" "PESD2CANFD24V-T" (id 1) (at 160.02 66.675 0))
     (property "Footprint" "Package_TO_SOT_SMD:SOT-23" (id 2) (at 156.21 71.12 0)
@@
   (symbol (lib_id "power:GND") (at 160.02 53.34 0) (unit 1)
     (in_bom yes) (on_board yes) (fields_autoplaced)
-    (property "Reference" "#PWR085" (id 0) (at 160.02 59.69 0)
+    (property "Reference" "#PWR071" (id 0) (at 160.02 59.69 0)
       (effects (font (size 1.27 1.27)) hide)
     )
@@
   (symbol (lib_id "power:GND") (at 160.02 74.93 0) (unit 1)
     (in_bom yes) (on_board yes) (fields_autoplaced)
-    (property "Reference" "#PWR088" (id 0) (at 160.02 81.28 0)
+    (property "Reference" "#PWR074" (id 0) (at 160.02 81.28 0)
       (effects (font (size 1.27 1.27)) hide)
     )
@@
   (symbol (lib_id "Device:C_Small") (at 34.29 109.22 90) (unit 1)
     (in_bom yes) (on_board yes) (fields_autoplaced)
-    (property "Reference" "C61" (id 0) (at 34.2963 102.235 90))
+    (property "Reference" "C45" (id 0) (at 34.2963 102.235 90))
     (property "Value" "10uF" (id 1) (at 34.2963 104.775 90))
     (property "Footprint" "Capacitor_SMD:C_0805_2012Metric" (id 2) (at 34.29 109.22 0)
@@
   (symbol (lib_id "power:GND") (at 22.86 36.83 270) (unit 1)
     (in_bom yes) (on_board yes) (fields_autoplaced)
-    (property "Reference" "#PWR084" (id 0) (at 16.51 36.83 0)
+    (property "Reference" "#PWR070" (id 0) (at 16.51 36.83 0)
       (effects (font (size 1.27 1.27)) hide)
     )
@@
   (symbol (lib_id "power:GND") (at 26.67 111.76 270) (unit 1)
     (in_bom yes) (on_board yes)
-    (property "Reference" "#PWR092" (id 0) (at 20.32 111.76 0)
+    (property "Reference" "#PWR078" (id 0) (at 20.32 111.76 0)
       (effects (font (size 1.27 1.27)) hide)
     )
@@
   (symbol (lib_id "power:GND") (at 107.95 95.25 0) (unit 1)
     (in_bom yes) (on_board yes) (fields_autoplaced)
-    (property "Reference" "#PWR090" (id 0) (at 107.95 101.6 0)
+    (property "Reference" "#PWR076" (id 0) (at 107.95 101.6 0)
       (effects (font (size 1.27 1.27)) hide)
     )
@@
   (symbol (lib_id "power:GND") (at 97.79 95.25 0) (unit 1)
     (in_bom yes) (on_board yes) (fields_autoplaced)
-    (property "Reference" "#PWR089" (id 0) (at 97.79 101.6 0)
+    (property "Reference" "#PWR075" (id 0) (at 97.79 101.6 0)
       (effects (font (size 1.27 1.27)) hide)
     )
@@
   (symbol (lib_id "ConeCodes:Delphi_Sicma_24") (at 58.42 44.45 0) (unit 1)
     (in_bom yes) (on_board yes) (fields_autoplaced)
-    (property "Reference" "J5" (id 0) (at 58.42 26.67 0))
+    (property "Reference" "J3" (id 0) (at 58.42 26.67 0))
     (property "Value" "Delphi_Sicma_24" (id 1) (at 58.42 29.21 0))
     (property "Footprint" "ConeCodes:Delphi_Sicma_24_Black" (id 2) (at 58.42 27.94 0)
@@
   (symbol (lib_id "Device:D_Zener_Dual_CommonAnode_KKA_Parallel") (at 160.02 48.26 270) (mirror x) (unit 1)
     (in_bom yes) (on_board yes) (fields_autoplaced)
-    (property "Reference" "D7" (id 0) (at 165.1 46.9264 90)
+    (property "Reference" "D5" (id 0) (at 165.1 46.9264 90)
       (effects (font (size 1.27 1.27)) (justify left))
     )
@@
   (symbol (lib_id "power:+3V3") (at 40.64 106.68 0) (unit 1)
     (in_bom yes) (on_board yes) (fields_autoplaced)
-    (property "Reference" "#PWR091" (id 0) (at 40.64 110.49 0)
+    (property "Reference" "#PWR077" (id 0) (at 40.64 110.49 0)
       (effects (font (size 1.27 1.27)) hide)
     )
@@
   (symbol (lib_id "Connector_Generic:Conn_01x05") (at 57.15 116.84 0) (unit 1)
     (in_bom yes) (on_board yes) (fields_autoplaced)
-    (property "Reference" "J6" (id 0) (at 60.325 115.5699 0)
+    (property "Reference" "J4" (id 0) (at 60.325 115.5699 0)
       (effects (font (size 1.27 1.27)) (justify left))
     )
@@
   (symbol (lib_id "power:GND") (at 106.68 73.66 0) (unit 1)
     (in_bom yes) (on_board yes) (fields_autoplaced)
-    (property "Reference" "#PWR087" (id 0) (at 106.68 80.01 0)
-      (effects (font (size 1.27 1.27)) hide)
-    )
+    (property "Reference" "#PWR073" (id 0) (at 106.68 80.01 0)
+      (effects (font (size 1.27 1.27)) hide)
+    )

Commit message: urmom
Connections:
- net RGB1_12V: now also J3.C1; no longer J3.C8
- net RGB2_12V: now also J3.B1; no longer J3.C1
- net VBATT: now also J3.C8; no longer J3.B1
Changed lines of the file:
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@@
+    (stroke (width 0) (type default) (color 0 0 0 0))
+  )
+  (wire (pts (xy 45.72 63.5) (xy 49.53 63.5))
     (stroke (width 0) (type default) (color 0 0 0 0))
   )
@@
     (stroke (width 0) (type default) (color 72 0 0 1))
   )
+  (wire (pts (xy 49.53 63.5) (xy 49.53 59.69))
+    (stroke (width 0) (type default) (color 0 0 0 0))
+  )
   (wire (pts (xy 31.75 52.07) (xy 45.72 52.07))
     (stroke (width 0) (type default) (color 255 0 0 1))
@@
     (stroke (width 0) (type default) (color 255 153 0 1))
   )
-  (wire (pts (xy 63.5 36.83) (xy 87.63 36.83))
+  (wire (pts (xy 45.72 63.5) (xy 21.59 63.5))
     (stroke (width 0) (type default) (color 255 255 0 1))
-  )
-  (wire (pts (xy 49.53 63.5) (xy 49.53 59.69))
-    (stroke (width 0) (type default) (color 132 0 0 1))
   )
   (wire (pts (xy 62.23 69.85) (xy 62.23 59.69))
@@
     (stroke (width 0) (type default) (color 0 0 0 1))
   )
-  (wire (pts (xy 31.75 63.5) (xy 49.53 63.5))
+  (wire (pts (xy 87.63 36.83) (xy 63.5 36.83))
     (stroke (width 0) (type default) (color 132 0 0 1))
   )
@@
     (effects (font (size 1.27 1.27)) (justify left bottom))
   )
-  (label "RGB2_12V" (at 87.63 54.61 180)
+  (label "RGB1_12V" (at 87.63 54.61 180)
     (effects (font (size 1.27 1.27)) (justify right bottom))
   )
@@
     (effects (font (size 1.27 1.27)) (justify left bottom))
   )
-  (label "VBATT" (at 31.75 63.5 0)
-    (effects (font (size 1.27 1.27)) (justify left bottom))
+  (label "VBATT" (at 87.63 36.83 180)
+    (effects (font (size 1.27 1.27)) (justify right bottom))
   )
   (label "USB_D_P" (at 87.63 69.85 180)
     (effects (font (size 1.27 1.27)) (justify right bottom))
   )
-  (label "RGB1_12V" (at 87.63 36.83 180)
-    (effects (font (size 1.27 1.27)) (justify right bottom))
+  (label "RGB2_12V" (at 21.59 63.5 0)
+    (effects (font (size 1.27 1.27)) (justify left bottom))
   )
   (label "RGB1_R" (at 31.75 52.07 0)
@@
     (effects (font (size 1.27 1.27)) (justify left))
   )
-  (hierarchical_label "RGB1_12V" (shape input) (at 87.63 36.83 0)
-    (effects (font (size 1.27 1.27)) (justify left))
+  (hierarchical_label "RGB2_12V" (shape input) (at 21.59 63.5 180)
+    (effects (font (size 1.27 1.27)) (justify right))
   )
   (hierarchical_label "MOSI" (shape input) (at 22.86 121.92 180)
     (effects (font (size 1.27 1.27)) (justify right))
   )
-  (hierarchical_label "VBATT" (shape input) (at 31.75 63.5 180)
-    (effects (font (size 1.27 1.27)) (justify right))
+  (hierarchical_label "VBATT" (shape input) (at 87.63 36.83 0)
+    (effects (font (size 1.27 1.27)) (justify left))
   )
   (hierarchical_label "CAN_H" (shape bidirectional) (at 31.75 71.12 180)
@@
     (effects (font (size 1.27 1.27)) (justify right))
   )
-  (hierarchical_label "RGB2_12V" (shape input) (at 87.63 54.61 0)
-    (effects (font (size 1.27 1.27)) (justify left))
-  )
+  (hierarchical_label "RGB1_12V" (shape input) (at 87.63 54.61 0)
+    (effects (font (size 1.27 1.27)) (justify left))
+  )
