File: hardware/underglow-controller/Connectors.kicad_sch (KiCad schematic)
At the start: 7 parts, among them J3 Delphi_Sicma_24, J4 Conn_01x05

Commit message: routing nearly done.
Connections:
- net USB_D_N: now also D5.1 (K), J3.B6; no longer D5.2 (K), J3.B7
- net USB_D_P: now also D5.2 (K), J3.B7; no longer D5.1 (K), J3.B6
Changed lines of the file:
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@@
     (effects (font (size 1.27 1.27)) (justify left bottom))
   )
-  (label "USB_D_P" (at 181.61 43.18 180)
-    (effects (font (size 1.27 1.27)) (justify right bottom))
+  (label "USB_D_P" (at 140.97 43.18 0)
+    (effects (font (size 1.27 1.27)) (justify left bottom))
   )
   (label "CAN_L" (at 31.75 73.66 0)
@@
     (effects (font (size 1.27 1.27)) (justify right bottom))
   )
-  (label "USB_D_P" (at 87.63 69.85 180)
+  (label "USB_D_P" (at 87.63 67.31 180)
     (effects (font (size 1.27 1.27)) (justify right bottom))
   )
@@
     (effects (font (size 1.27 1.27)) (justify left bottom))
   )
-  (label "USB_D_N" (at 87.63 67.31 180)
+  (label "USB_D_N" (at 87.63 69.85 180)
     (effects (font (size 1.27 1.27)) (justify right bottom))
   )
@@
     (effects (font (size 1.27 1.27)) (justify right bottom))
   )
-  (label "USB_D_N" (at 140.97 43.18 0)
-    (effects (font (size 1.27 1.27)) (justify left bottom))
+  (label "USB_D_N" (at 181.61 43.18 180)
+    (effects (font (size 1.27 1.27)) (justify right bottom))
   )
   (label "FSPICLK" (at 27.94 116.84 0)
@@
     (effects (font (size 1.27 1.27)) (justify right))
   )
-  (hierarchical_label "USB_D_N" (shape bidirectional) (at 87.63 67.31 0)
+  (hierarchical_label "USB_D_N" (shape bidirectional) (at 87.63 69.85 0)
     (effects (font (size 1.27 1.27)) (justify left))
   )
@@
     (effects (font (size 1.27 1.27)) (justify left))
   )
-  (hierarchical_label "USB_D_P" (shape bidirectional) (at 87.63 69.85 0)
+  (hierarchical_label "USB_D_P" (shape bidirectional) (at 87.63 67.31 0)
     (effects (font (size 1.27 1.27)) (justify left))
   )
