File: hardware/underglow-controller/External-IO.kicad_sch (KiCad schematic)
At the start: 20 parts, among them Q2 STS8DNF3LL, Q3 STS8DNF3LL, Q4 STS8DNF3LL, Q5 MBT3904DW1T1G, Q6 MBT3904DW1T1G, U6 WS2815B

Commit message: i can't believe what they did to my boy
Parts:
- removed C6: 0.1uF, Capacitor_SMD:C_0805_2012Metric, symbol Device:C_Small
- removed JP2: LED Voltage Select, Jumper:SolderJumper-3_P1.3mm_Bridged12_RoundedPad1.0x1.5mm_NumberLabels, symbol Jumper:SolderJumper_3_Bridged12
- removed Q4: STS8DNF3LL, Package_SO:SO-8_3.9x4.9mm_P1.27mm, symbol Device:Q_Dual_NMOS_S1G1S2G2D2D2D1D1
- removed U6: WS2815B, ConeCodes:worldsemi-WS2815B-MFG, symbol ConeCodes:WS2815B
- added R45: 0R, Resistor_SMD:R_2512_6332Metric, symbol Device:R_Small
Connections:
- net LEDA_IN: now also R45.1
- net LEDA_OUT: now also R45.2
Other:
- note added: "from mcu"
- note added: "to LED"
- note removed: "Unsure if supply voltage should go to VCC or VDD. Datasheet says VDD but that doesn't make a ton of sense to me. If this part doesn't work, bridge the other half"

Commit message: urmom
Parts:
- added R47: 10k, Resistor_SMD:R_0603_1608Metric, symbol Device:R_Small
Connections:
- net GND: now also R47.2
- net GPIO_GP04: now also R47.1
- net GP04 renamed VOUT_EN
Other:
- moved on the sheet: R8
Changed lines of the file:
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@@
   (junction (at 87.63 34.29) (diameter 0) (color 0 0 0 0)
   )
+  (junction (at 93.345 129.54) (diameter 0) (color 0 0 0 0)
+  )
+  (junction (at 102.87 187.325) (diameter 0) (color 0 0 0 0)
+  )
+  (junction (at 105.41 144.145) (diameter 0) (color 0 0 0 0)
+  )
+  (junction (at 90.805 172.72) (diameter 0) (color 0 0 0 0)
+  )
+  (junction (at 151.13 45.72) (diameter 0) (color 0 0 0 0)
+  )
+  (junction (at 127 34.29) (diameter 0) (color 0 0 0 0)
+  )
+  (junction (at 49.53 187.325) (diameter 0) (color 0 0 0 0)
+  )
+  (junction (at 163.195 34.29) (diameter 0) (color 0 0 0 0)
+  )
+  (junction (at 163.195 57.15) (diameter 0) (color 0 0 0 0)
+  )
+  (junction (at 49.53 144.145) (diameter 0) (color 0 0 0 0)
+  )
+  (junction (at 37.465 129.54) (diameter 0) (color 0 0 0 0)
+  )
   (junction (at 37.465 172.72) (diameter 0) (color 0 0 0 0)
   )
-  (junction (at 93.345 129.54) (diameter 0) (color 0 0 0 0)
-  )
-  (junction (at 102.87 187.325) (diameter 0) (color 0 0 0 0)
-  )
-  (junction (at 105.41 144.145) (diameter 0) (color 0 0 0 0)
-  )
-  (junction (at 90.805 172.72) (diameter 0) (color 0 0 0 0)
-  )
-  (junction (at 127 34.29) (diameter 0) (color 0 0 0 0)
-  )
-  (junction (at 49.53 187.325) (diameter 0) (color 0 0 0 0)
-  )
-  (junction (at 163.195 34.29) (diameter 0) (color 0 0 0 0)
-  )
-  (junction (at 49.53 144.145) (diameter 0) (color 0 0 0 0)
-  )
-  (junction (at 37.465 129.54) (diameter 0) (color 0 0 0 0)
-  )
   (wire (pts (xy 51.435 34.29) (xy 48.895 34.29))
     (stroke (width 0) (type default) (color 0 0 0 0))
@@
     (stroke (width 0) (type default) (color 0 0 0 0))
   )
+  (wire (pts (xy 37.465 160.655) (xy 37.465 166.37))
+    (stroke (width 0) (type default) (color 0 0 0 0))
+  )
   (wire (pts (xy 87.63 34.29) (xy 87.63 40.64))
     (stroke (width 0) (type default) (color 0 0 0 0))
@@
     (stroke (width 0) (type default) (color 0 0 0 0))
   )
-  (wire (pts (xy 163.195 50.8) (xy 163.195 62.23))
+  (wire (pts (xy 163.195 50.8) (xy 163.195 57.15))
     (stroke (width 0) (type default) (color 0 0 0 0))
   )
@@
     (stroke (width 0) (type default) (color 0 0 0 0))
   )
+  (wire (pts (xy 151.13 45.72) (xy 155.575 45.72))
+    (stroke (width 0) (type default) (color 0 0 0 0))
+  )
   (wire (pts (xy 105.41 118.745) (xy 105.41 124.46))
     (stroke (width 0) (type default) (color 0 0 0 0))
@@
     (stroke (width 0) (type default) (color 0 0 0 0))
   )
+  (wire (pts (xy 151.13 54.61) (xy 151.13 57.15))
+    (stroke (width 0) (type default) (color 0 0 0 0))
+  )
+  (wire (pts (xy 163.195 57.15) (xy 163.195 62.23))
+    (stroke (width 0) (type default) (color 0 0 0 0))
+  )
   (wire (pts (xy 90.805 187.325) (xy 102.87 187.325))
     (stroke (width 0) (type default) (color 0 0 0 0))
@@
     (stroke (width 0) (type default) (color 0 0 0 0))
   )
-  (wire (pts (xy 37.465 160.655) (xy 37.465 165.1))
-    (stroke (width 0) (type default) (color 0 0 0 0))
-  )
   (wire (pts (xy 102.87 177.8) (xy 102.87 187.325))
     (stroke (width 0) (type default) (color 0 0 0 0))
@@
     (stroke (width 0) (type default) (color 0 0 0 0))
   )
-  (wire (pts (xy 37.465 170.18) (xy 37.465 172.72))
-    (stroke (width 0) (type default) (color 0 0 0 0))
-  )
   (wire (pts (xy 105.41 144.145) (xy 105.41 147.32))
     (stroke (width 0) (type default) (color 0 0 0 0))
@@
     (stroke (width 0) (type default) (color 0 0 0 0))
   )
+  (wire (pts (xy 37.465 171.45) (xy 37.465 172.72))
+    (stroke (width 0) (type default) (color 0 0 0 0))
+  )
   (wire (pts (xy 93.345 142.24) (xy 93.345 144.145))
     (stroke (width 0) (type default) (color 0 0 0 0))
@@
     (stroke (width 0) (type default) (color 0 0 0 0))
   )
-  (wire (pts (xy 143.51 45.72) (xy 155.575 45.72))
+  (wire (pts (xy 143.51 45.72) (xy 151.13 45.72))
     (stroke (width 0) (type default) (color 0 0 0 0))
   )
@@
     (stroke (width 0) (type default) (color 0 0 0 0))
   )
+  (wire (pts (xy 151.13 57.15) (xy 163.195 57.15))
+    (stroke (width 0) (type default) (color 0 0 0 0))
+  )
   (wire (pts (xy 129.54 34.29) (xy 129.54 40.64))
     (stroke (width 0) (type default) (color 0 0 0 0))
@@
   )
   (wire (pts (xy 127 50.8) (xy 127 62.23))
+    (stroke (width 0) (type default) (color 0 0 0 0))
+  )
+  (wire (pts (xy 151.13 49.53) (xy 151.13 45.72))
     (stroke (width 0) (type default) (color 0 0 0 0))
   )
@@
     (effects (font (size 1.27 1.27)) (justify left bottom))
   )
-  (label "GPO4" (at 146.05 34.29 0)
+  (label "VOUT_EN" (at 146.05 34.29 0)
     (effects (font (size 1.27 1.27)) (justify left bottom))
   )
@@
     (effects (font (size 1.27 1.27)) (justify left))
   )
-  (hierarchical_label "GP04" (shape output) (at 143.51 34.29 180)
+  (hierarchical_label "VOUT_EN" (shape output) (at 143.51 34.29 180)
     (effects (font (size 1.27 1.27)) (justify right))
   )
@@
     (pin "2")
   )
-  (symbol (lib_id "Device:R_Small") (at 37.465 167.64 0) (unit 1)
-    (in_bom yes) (on_board yes) (fields_autoplaced)
-    (property "Reference" "R8" (id 0) (at 35.56 166.3699 0)
+  (symbol (lib_id "Device:R_Small") (at 37.465 168.91 0) (unit 1)
+    (in_bom yes) (on_board yes) (fields_autoplaced)
+    (property "Reference" "R8" (id 0) (at 35.56 167.6399 0)
       (effects (font (size 1.27 1.27)) (justify right))
     )
-    (property "Value" "10k" (id 1) (at 35.56 168.9099 0)
+    (property "Value" "10k" (id 1) (at 35.56 170.1799 0)
       (effects (font (size 1.27 1.27)) (justify right))
     )
-    (property "Footprint" "Resistor_SMD:R_0402_1005Metric" (id 2) (at 37.465 167.64 0)
-      (effects (font (size 1.27 1.27)) hide)
-    )
-    (property "Datasheet" "~" (id 3) (at 37.465 167.64 0)
-      (effects (font (size 1.27 1.27)) hide)
-    )
-    (property "Description" "RES 10K OHM 5% 1/16W 0402" (id 4) (at 37.465 167.64 0)
-      (effects (font (size 1.27 1.27)) hide)
-    )
-    (property "MPN" "RMCF0402JT10K0" (id 5) (at 37.465 167.64 0)
+    (property "Footprint" "Resistor_SMD:R_0402_1005Metric" (id 2) (at 37.465 168.91 0)
+      (effects (font (size 1.27 1.27)) hide)
+    )
+    (property "Datasheet" "~" (id 3) (at 37.465 168.91 0)
+      (effects (font (size 1.27 1.27)) hide)
+    )
+    (property "Description" "RES 10K OHM 5% 1/16W 0402" (id 4) (at 37.465 168.91 0)
+      (effects (font (size 1.27 1.27)) hide)
+    )
+    (property "MPN" "RMCF0402JT10K0" (id 5) (at 37.465 168.91 0)
       (effects (font (size 1.27 1.27)) hide)
     )
@@
     (pin "8")
   )
+  (symbol (lib_id "Device:R_Small") (at 151.13 52.07 0) (mirror y) (unit 1)
+    (in_bom yes) (on_board yes) (fields_autoplaced)
+    (property "Reference" "R47" (id 0) (at 153.67 50.7999 0)
+      (effects (font (size 1.27 1.27)) (justify right))
+    )
+    (property "Value" "10k" (id 1) (at 153.67 53.3399 0)
+      (effects (font (size 1.27 1.27)) (justify right))
+    )
+    (property "Footprint" "Resistor_SMD:R_0603_1608Metric" (id 2) (at 151.13 52.07 0)
+      (effects (font (size 1.27 1.27)) hide)
+    )
+    (property "Datasheet" "~" (id 3) (at 151.13 52.07 0)
+      (effects (font (size 1.27 1.27)) hide)
+    )
+    (property "MPN" "RNCP0603FTD10K0" (id 5) (at 151.13 52.07 0)
+      (effects (font (size 1.27 1.27)) hide)
+    )
+    (property "Description" "RES 10K OHM 1% 1/8W 0603" (id 6) (at 151.13 52.07 0)
+      (effects (font (size 1.27 1.27)) hide)
+    )
+    (pin "1")
+    (pin "2")
+  )
   (symbol (lib_id "Device:R_Small") (at 93.345 134.62 0) (unit 1)

Commit message: updates nearly complete
Parts:
- Q5, Q6: MPN (none) -> MBT3904DW1T1G
- R45: MPN (none) -> RMCF2512ZT0R00
Changed lines of the file:
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@@
+      (effects (font (size 1.27 1.27)) hide)
+    )
+    (property "MPN" "RMCF2512ZT0R00" (id 4) (at 201.93 119.38 0)
+      (effects (font (size 1.27 1.27)) hide)
+    )
+    (property "Description" "RMCF2512ZT0R00" (id 5) (at 201.93 119.38 0)
       (effects (font (size 1.27 1.27)) hide)
     )
@@
     )
     (property "Datasheet" "~" (id 3) (at 46.99 172.72 0)
+      (effects (font (size 1.27 1.27)) hide)
+    )
+    (property "MPN" "MBT3904DW1T1G" (id 4) (at 46.99 172.72 0)
+      (effects (font (size 1.27 1.27)) hide)
+    )
+    (property "Description" "TRANS 2NPN 40V 0.2A SC88/SC70-6" (id 5) (at 46.99 172.72 0)
       (effects (font (size 1.27 1.27)) hide)
     )
@@
       (effects (font (size 1.27 1.27)) hide)
     )
+    (property "Description" "TRANS 2NPN 40V 0.2A SC88/SC70-6" (id 5) (at 46.99 129.54 0)
+      (effects (font (size 1.27 1.27)) hide)
+    )
     (pin "1")
     (pin "2")
@@
     )
     (property "Datasheet" "~" (id 3) (at 100.33 172.72 0)
+      (effects (font (size 1.27 1.27)) hide)
+    )
+    (property "MPN" "MBT3904DW1T1G" (id 4) (at 100.33 172.72 0)
+      (effects (font (size 1.27 1.27)) hide)
+    )
+    (property "Description" "TRANS 2NPN 40V 0.2A SC88/SC70-6" (id 5) (at 100.33 172.72 0)
       (effects (font (size 1.27 1.27)) hide)
     )
@@
       (effects (font (size 1.27 1.27)) hide)
     )
+    (property "Description" "TRANS 2NPN 40V 0.2A SC88/SC70-6" (id 5) (at 102.87 129.54 0)
+      (effects (font (size 1.27 1.27)) hide)
+    )
