File: hardware/underglow-controller/External-IO.kicad_sch (KiCad schematic)
At the start: 31 parts, among them Q601 STS8DNF3LL, Q602 STS8DNF3LL, Q603 STS8DNF3LL, Q604 SBC847CDW1T1G, Q605 SBC847CDW1T1G, Q606 AUIRF7316QTR, Q607 STS8DNF3LL

Commit message: Layout updates
Connections:
- net +3V3: now also R601.1, R603.1
- net VBATT: no longer R601.1, R603.1
Other:
- moved on the sheet: R601, R603
Changed lines of the file:
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@@
   (junction (at 184.15 255.27) (diameter 0) (color 0 0 0 0)
   )
-  (junction (at 81.28 39.37) (diameter 0) (color 0 0 0 0)
-  )
   (junction (at 149.86 242.57) (diameter 0) (color 0 0 0 0)
   )
   (junction (at 81.28 77.47) (diameter 0) (color 0 0 0 0)
-  )
-  (junction (at 81.28 114.3) (diameter 0) (color 0 0 0 0)
   )
   (junction (at 355.6 48.26) (diameter 0) (color 0 0 255 1)
@@
     (stroke (width 0) (type default) (color 255 0 0 1))
   )
-  (wire (pts (xy 87.63 50.8) (xy 81.28 50.8))
+  (wire (pts (xy 76.2 50.8) (xy 87.63 50.8))
     (stroke (width 0) (type default) (color 0 0 0 0))
   )
@@
     (stroke (width 0) (type default) (color 0 0 0 0))
   )
-  (wire (pts (xy 81.28 50.8) (xy 81.28 48.26))
-    (stroke (width 0) (type default) (color 0 0 0 0))
-  )
-  (wire (pts (xy 63.5 39.37) (xy 81.28 39.37))
+  (wire (pts (xy 63.5 39.37) (xy 95.25 39.37))
     (stroke (width 0) (type default) (color 0 0 0 0))
   )
@@
     (stroke (width 0) (type default) (color 0 0 0 0))
   )
-  (wire (pts (xy 81.28 114.3) (xy 95.25 114.3))
+  (wire (pts (xy 63.5 114.3) (xy 95.25 114.3))
     (stroke (width 0) (type default) (color 0 0 0 0))
   )
@@
     (stroke (width 0) (type default) (color 0 0 255 1))
   )
+  (wire (pts (xy 63.5 50.8) (xy 71.12 50.8))
+    (stroke (width 0) (type default) (color 0 0 0 0))
+  )
   (wire (pts (xy 97.79 143.51) (xy 95.25 143.51))
     (stroke (width 0) (type default) (color 0 0 0 0))
@@
     (stroke (width 0) (type default) (color 255 0 0 1))
   )
-  (wire (pts (xy 87.63 125.73) (xy 81.28 125.73))
-    (stroke (width 0) (type default) (color 0 0 0 0))
-  )
   (wire (pts (xy 128.27 242.57) (xy 137.16 242.57))
     (stroke (width 0) (type default) (color 0 0 0 0))
@@
     (stroke (width 0) (type default) (color 0 0 0 0))
   )
-  (wire (pts (xy 81.28 39.37) (xy 95.25 39.37))
-    (stroke (width 0) (type default) (color 0 0 0 0))
-  )
   (wire (pts (xy 149.86 260.35) (xy 149.86 269.24))
     (stroke (width 0) (type default) (color 0 0 0 0))
   )
   (wire (pts (xy 81.28 152.4) (xy 81.28 153.67))
-    (stroke (width 0) (type default) (color 0 0 0 0))
-  )
-  (wire (pts (xy 81.28 125.73) (xy 81.28 123.19))
     (stroke (width 0) (type default) (color 0 0 0 0))
   )
@@
     (stroke (width 0) (type default) (color 0 255 0 1))
   )
-  (wire (pts (xy 81.28 114.3) (xy 81.28 118.11))
-    (stroke (width 0) (type default) (color 0 0 0 0))
-  )
   (wire (pts (xy 95.25 137.16) (xy 95.25 130.81))
+    (stroke (width 0) (type default) (color 0 0 0 0))
+  )
+  (wire (pts (xy 76.2 125.73) (xy 87.63 125.73))
     (stroke (width 0) (type default) (color 0 0 0 0))
   )
@@
     (stroke (width 0) (type default) (color 0 255 0 1))
   )
-  (wire (pts (xy 63.5 114.3) (xy 81.28 114.3))
-    (stroke (width 0) (type default) (color 0 0 0 0))
-  )
   (wire (pts (xy 257.81 64.77) (xy 257.81 77.47))
     (stroke (width 0) (type default) (color 0 0 0 1))
@@
     (stroke (width 0) (type default) (color 0 0 0 0))
   )
+  (wire (pts (xy 63.5 125.73) (xy 71.12 125.73))
+    (stroke (width 0) (type default) (color 0 0 0 0))
+  )
   (wire (pts (xy 307.34 77.47) (xy 355.6 77.47))
     (stroke (width 0) (type default) (color 0 0 0 1))
@@
   )
   (wire (pts (xy 149.86 242.57) (xy 149.86 250.19))
-    (stroke (width 0) (type default) (color 0 0 0 0))
-  )
-  (wire (pts (xy 81.28 39.37) (xy 81.28 43.18))
     (stroke (width 0) (type default) (color 0 0 0 0))
   )
@@
     (pin "1")
   )
-  (symbol (lib_id "Device:R_Small") (at 81.28 45.72 0) (unit 1)
-    (in_bom yes) (on_board yes) (fields_autoplaced)
-    (property "Reference" "R601" (id 0) (at 78.74 44.4499 0)
-      (effects (font (size 1.27 1.27)) (justify right))
-    )
-    (property "Value" "10k" (id 1) (at 78.74 46.9899 0)
-      (effects (font (size 1.27 1.27)) (justify right))
-    )
-    (property "Footprint" "Resistor_SMD:R_0805_2012Metric" (id 2) (at 81.28 45.72 0)
-      (effects (font (size 1.27 1.27)) hide)
-    )
-    (property "Datasheet" "~" (id 3) (at 81.28 45.72 0)
-      (effects (font (size 1.27 1.27)) hide)
-    )
-    (property "Description" "RES 10K OHM 1% 1/4W 0805" (id 4) (at 81.28 45.72 0)
-      (effects (font (size 1.27 1.27)) hide)
-    )
-    (property "MPN" "RNCP0805FTD10K0" (id 5) (at 81.28 45.72 0)
+  (symbol (lib_id "Device:R_Small") (at 73.66 50.8 90) (unit 1)
+    (in_bom yes) (on_board yes) (fields_autoplaced)
+    (property "Reference" "R601" (id 0) (at 73.66 44.45 90))
+    (property "Value" "10k" (id 1) (at 73.66 46.99 90))
+    (property "Footprint" "Resistor_SMD:R_0805_2012Metric" (id 2) (at 73.66 50.8 0)
+      (effects (font (size 1.27 1.27)) hide)
+    )
+    (property "Datasheet" "~" (id 3) (at 73.66 50.8 0)
+      (effects (font (size 1.27 1.27)) hide)
+    )
+    (property "Description" "RES 10K OHM 1% 1/4W 0805" (id 4) (at 73.66 50.8 0)
+      (effects (font (size 1.27 1.27)) hide)
+    )
+    (property "MPN" "RNCP0805FTD10K0" (id 5) (at 73.66 50.8 0)
       (effects (font (size 1.27 1.27)) hide)
     )
@@
     (pin "1")
     (pin "2")
+  )
+  (symbol (lib_id "power:+3V3") (at 63.5 50.8 90) (unit 1)
+    (in_bom yes) (on_board yes) (fields_autoplaced)
+    (property "Reference" "#PWR?" (id 0) (at 67.31 50.8 0)
+      (effects (font (size 1.27 1.27)) hide)
+    )
+    (property "Value" "+3V3" (id 1) (at 62.23 46.99 90))
+    (property "Footprint" "" (id 2) (at 63.5 50.8 0)
+      (effects (font (size 1.27 1.27)) hide)
+    )
+    (property "Datasheet" "" (id 3) (at 63.5 50.8 0)
+      (effects (font (size 1.27 1.27)) hide)
+    )
+    (pin "1")
   )
   (symbol (lib_id "Device:R_Small") (at 36.83 228.6 0) (unit 1)
@@
     (pin "6")
   )
-  (symbol (lib_id "Device:R_Small") (at 81.28 120.65 0) (unit 1)
-    (in_bom yes) (on_board yes) (fields_autoplaced)
-    (property "Reference" "R603" (id 0) (at 78.74 119.3799 0)
-      (effects (font (size 1.27 1.27)) (justify right))
-    )
-    (property "Value" "10k" (id 1) (at 78.74 121.9199 0)
-      (effects (font (size 1.27 1.27)) (justify right))
-    )
-    (property "Footprint" "Resistor_SMD:R_0805_2012Metric" (id 2) (at 81.28 120.65 0)
-      (effects (font (size 1.27 1.27)) hide)
-    )
-    (property "Datasheet" "~" (id 3) (at 81.28 120.65 0)
-      (effects (font (size 1.27 1.27)) hide)
-    )
-    (property "Description" "RES 10K OHM 1% 1/4W 0805" (id 4) (at 81.28 120.65 0)
-      (effects (font (size 1.27 1.27)) hide)
-    )
-    (property "MPN" "RNCP0805FTD10K0" (id 5) (at 81.28 120.65 0)
+  (symbol (lib_id "Device:R_Small") (at 73.66 125.73 90) (unit 1)
+    (in_bom yes) (on_board yes) (fields_autoplaced)
+    (property "Reference" "R603" (id 0) (at 73.66 119.38 90))
+    (property "Value" "10k" (id 1) (at 73.66 121.92 90))
+    (property "Footprint" "Resistor_SMD:R_0805_2012Metric" (id 2) (at 73.66 125.73 0)
+      (effects (font (size 1.27 1.27)) hide)
+    )
+    (property "Datasheet" "~" (id 3) (at 73.66 125.73 0)
+      (effects (font (size 1.27 1.27)) hide)
+    )
+    (property "Description" "RES 10K OHM 1% 1/4W 0805" (id 4) (at 73.66 125.73 0)
+      (effects (font (size 1.27 1.27)) hide)
+    )
+    (property "MPN" "RNCP0805FTD10K0" (id 5) (at 73.66 125.73 0)
       (effects (font (size 1.27 1.27)) hide)
     )
@@
     (pin "6")
   )
+  (symbol (lib_id "power:+3V3") (at 63.5 125.73 90) (unit 1)
+    (in_bom yes) (on_board yes) (fields_autoplaced)
+    (property "Reference" "#PWR?" (id 0) (at 67.31 125.73 0)
+      (effects (font (size 1.27 1.27)) hide)
+    )
+    (property "Value" "+3V3" (id 1) (at 62.23 121.92 90))
+    (property "Footprint" "" (id 2) (at 63.5 125.73 0)
+      (effects (font (size 1.27 1.27)) hide)
+    )
+    (property "Datasheet" "" (id 3) (at 63.5 125.73 0)
+      (effects (font (size 1.27 1.27)) hide)
+    )
+    (pin "1")
+  )
   (symbol (lib_id "power:+3V3") (at 196.85 233.68 0) (unit 1)

Commit message: V5 Rev B Hardware release
Parts:
- added C601: 0.1uF, Capacitor_SMD:C_0402_1005Metric, symbol Device:C_Small
- added C602: 10uF, Capacitor_SMD:CP_Elec_5x5.9, symbol Device:C_Polarized_Small
- added R621, R622: 0R, Resistor_SMD:R_2512_6332Metric, symbol Device:R_Small
- added TP601: CUR_3, TestPoint:TestPoint_Pad_D1.0mm, symbol Connector:TestPoint
- added TP602: CUR_2, TestPoint:TestPoint_Pad_D1.0mm, symbol Connector:TestPoint
- added U601: INA2181A1IDGST, Package_SO:VSSOP-10_3x3mm_P0.5mm, symbol ConeCodes:INA2181A1IDGST
Connections:
- net +3V3: now also C601.1, U601.10 (VS)
- net GND: now also C601.2, C602.2, U601.4 (GND)
- net RGB1_12V: now also R621.1, U601.2 (IN-1); no longer Q606.7 (D), Q606.8 (G)
- net RGB1_GND: now also U601.5 (REF1)
- net RGB2_12V: now also R622.1, U601.8 (IN-2); no longer Q606.5 (D), Q606.6 (G)
- net RGB2_GND: now also U601.6 (REF2)
- net VBATT: now also C602.1
- net at R601.2: now also Q606.4 (G); no longer Q606.2 (G)
- net at R603.2: now also Q606.2 (G); no longer Q606.4 (G)
- new net CUR_SENSE_1: TP601.1, U601.1 (OUT1)
- new net CUR_SENSE_2: TP602.1, U601.9 (OUT2)
- new net RGB1_FET_OUTPUT: Q606.5 (D), Q606.6 (G), R621.2, U601.3 (IN+1)
- new net RGB2_FET_OUTPUT: Q606.7 (D), Q606.8 (G), R622.2, U601.7 (IN+2)
Other:
- note added: "CURRENT SENSE"
- moved on the sheet: ALED601, ALED602, Q604A, Q604B, Q605A, Q605B, Q606A, Q606B, R23, R24, R605, R606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

Commit message: Add FET drivers
Parts:
- added R623, R624, R625, R626, R627, R628, R641, R642: 1k, Resistor_SMD:R_0402_1005Metric, symbol Device:R_Small
- added R629, R630, R631, R632, R633, R634, R635, R636, R637, R638, R639, R640, R643, R644, R645, R646: 0R, Resistor_SMD:R_0805_2012Metric, symbol Device:R_Small
- added U602, U603, U604, U605, U606, U607, U608, U609: ZXGD3009E6, Package_TO_SOT_SMD:SOT-23-6, symbol Driver_FET:ZXGD3009E6
Connections:
- net GND: now also U608.3 (VEE), U609.3 (VEE)
- net PWMI1: now also R641.1; no longer Q607.2 (G), R602.1
- net PWMI2: now also R642.1; no longer Q607.4 (G), R604.1
- net RGB1_FET_OUTPUT: now also U602.1 (VCC), U603.1 (VCC), U604.1 (VCC)
- net RGB1_GND: now also U602.3 (VEE), U603.3 (VEE), U604.3 (VEE)
- net RGB2_FET_OUTPUT: now also U605.1 (VCC), U606.1 (VCC), U607.1 (VCC)
- net RGB2_GND: now also U605.3 (VEE), U606.3 (VEE), U607.3 (VEE)
- net TTL_RGB1_B: now also R625.1; no longer Q602.2 (G)
- net TTL_RGB1_G: now also R624.1; no longer Q601.4 (G)
- net TTL_RGB1_R: now also R623.1; no longer Q601.2 (G)
- net TTL_RGB2_B: now also R628.1; no longer Q603.4 (G)
- net TTL_RGB2_G: now also R627.1; no longer Q603.2 (G)
- net TTL_RGB2_R: now also R626.1; no longer Q602.4 (G)
- net VBATT: now also U608.1 (VCC), U609.1 (VCC)
- new net: R626.2, U605.2 (IN)
- new net: R624.2, U603.2 (IN)
- new net: R627.2, U606.2 (IN)
- new net: Q607.4 (G), R604.1, R645.2, R646.2
- new net: Q607.2 (G), R602.1, R643.2, R644.2
- new net: R625.2, U604.2 (IN)
- new net: R628.2, U607.2 (IN)
- new net: R623.2, U602.2 (IN)
- new net: R642.2, U609.2 (IN)
- new net: R641.2, U608.2 (IN)
- new net RGB1_B_GATE: Q602.2 (G), R633.2, R634.2
- new net RGB1_B_SINK: R634.1, U604.4 (SINK)
- new net RGB1_B_SOURCE: R633.1, U604.6 (SOURCE)
- new net RGB1_G_GATE: Q601.4 (G), R631.2, R632.2
- new net RGB1_G_SINK: R632.1, U603.4 (SINK)
- new net RGB1_G_SOURCE: R631.1, U603.6 (SOURCE)
- new net RGB1_R_GATE: Q601.2 (G), R629.2, R630.2
- new net RGB1_R_SINK: R630.1, U602.4 (SINK)
- new net RGB1_R_SOURCE: R629.1, U602.6 (SOURCE)
- new net RGB1_SINK: R644.1, U608.4 (SINK)
- new net RGB1_SOURCE: R643.1, U608.6 (SOURCE)
- new net RGB2_B_GATE: Q603.4 (G), R639.2, R640.2
- new net RGB2_B_SINK: R640.1, U607.4 (SINK)
- new net RGB2_B_SOURCE: R639.1, U607.6 (SOURCE)
- new net RGB2_G_GATE: Q603.2 (G), R637.2, R638.2
- new net RGB2_G_SINK: R638.1, U606.4 (SINK)
- new net RGB2_G_SOURCE: R637.1, U606.6 (SOURCE)
- new net RGB2_R_GATE: Q602.4 (G), R635.2, R636.2
- new net RGB2_R_SINK: R636.1, U605.4 (SINK)
- new net RGB2_R_SOURCE: R635.1, U605.6 (SOURCE)
- new net RGB2_SINK: R646.1, U609.4 (SINK)
- new net RGB2_SOURCE: R645.1, U609.6 (SOURCE)
Other:
- moved on the sheet: Q601A, Q601B, Q602A, Q602B, Q603A, Q603B

Commit message: hw updates based on latest boards
Parts:
- added R647, R649, R650, R652: 0R, Resistor_SMD:R_0805_2012Metric, symbol Device:R_Small
- added R648, R651: 1k, Resistor_SMD:R_0402_1005Metric, symbol Device:R_Small
- added U610, U611: ZXGD3009E6, Package_TO_SOT_SMD:SOT-23-6, symbol Driver_FET:ZXGD3009E6
Connections:
- net +3V3: no longer R601.1, R603.1
- net GND: now also R601.1, R603.1, U610.3 (VEE), U611.3 (VEE)
- net PWMI1: now also R648.1
- net PWMI2: now also R651.1
- net VBATT: now also U610.1 (VCC), U611.1 (VCC)
- net RGB1_GATE: now reaches Q606.4 (G), R601.2
- net RGB1_GATE: now also R647.2, R649.2
- net RGB2_GATE: now reaches Q606.2 (G), R603.2
- net RGB2_GATE: now also R650.2, R652.2
- new net: R649.1, U610.4 (SINK)
- new net: R650.1, U611.6 (SOURCE)
- new net: R648.2, U610.2 (IN)
- new net: R647.1, U610.6 (SOURCE)
- new net: R651.2, U611.2 (IN)
- new net: R652.1, U611.4 (SINK)
Other:
- moved on the sheet: C602, Q606A, Q606B, Q607A, Q607B, R601, R602, R603, R604, R642, R643, R644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

Commit message: https://www.youtube.com/watch?v=FZUcpVmEHuk&ab_channel=billwurtz
Parts:
- R629, R630, R631, R632, R633, R634, R635, R636, R637, R638, R639, R640, R643, R644, R645, R646, R647, R649, R650, R652: MPN (none) -> RES SMD 0 OHM JUMPER 1/8W 0805
- U602, U603, U604, U605, U606, U607, U608, U609, U610, U611: MPN (none) -> ZXGD3009E6

Commit message: hardware updates
Parts:
- removed R647, R650: 0R, Resistor_SMD:R_0805_2012Metric, symbol Device:R_Small
- removed U610, U611: ZXGD3009E6, Package_TO_SOT_SMD:SOT-23-6, symbol Driver_FET:ZXGD3009E6
- added D601, D602: 3v3, Diode_SMD:D_SOD-123F, symbol Device:D_Zener
- added U610, U611: TC4431VOA713, ConeCodes:SOIC127P600X175-8N, symbol ConeCodes:TC4431VOA713
- R23, R24: value 0R -> 100R; MPN RMCF2512ZT0R00 -> (none)
- U601: MPN (none) -> INA2181A1IDGSR
Connections:
- net GND: now also D601.2 (A), D602.2 (A), U610.4 (GND), U610.5 (GND), U611.4 (GND), U611.5 (GND)
- net PIXEL1_IN: now also D601.1 (K)
- net PIXEL2_IN: now also D602.1 (K)
- net VBATT: now also U610.1 (VDD), U610.8 (VDD), U611.1 (VDD), U611.8 (VDD)
- net at R649.1: now also U610.6 (~{OUT}), U610.7 (~{OUT})
- net at R648.2: now also U610.2 (IN)
- net at R651.2: now also U611.2 (IN)
- net at R652.1: now also U611.6 (~{OUT}), U611.7 (~{OUT})
- no-connect marks 4 -> 6
Other:
- note added: "The lockout pin enables/disables the undervoltage lockout feature of the device. If undervoltage lockout is desired (output is not enabled until the bias voltage reaches 8.4V (typical) on the rising edge and is disabled when the bias voltage reaches 7.7V (typical) on the falling edge), the lockout pin should be left float- ing. If operation below 7V is desired, the lockout pin should be tied to g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"
- moved on the sheet: C602, Q606A, Q606B, Q607B, R24, R601, R603, R604, R642, R645, R646, R648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

Commit message: ughughughugh
Parts:
- added TP603: TP_DI_2, TestPoint:TestPoint_Pad_D1.0mm, symbol Connector:TestPoint
- added TP604: TP_DI_1, TestPoint:TestPoint_Pad_D1.0mm, symbol Connector:TestPoint
- added TP605: TP_DI_4, TestPoint:TestPoint_Pad_D1.0mm, symbol Connector:TestPoint
- added TP606: TP_DI_3, TestPoint:TestPoint_Pad_D1.0mm, symbol Connector:TestPoint
Connections:
- net TTL_DI_1: now also TP604.1
- net TTL_DI_2: now also TP603.1
- net TTL_DI_3: now also TP606.1
- net TTL_DI_4: now also TP605.1
Changed lines of the file:
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@@
     (stroke (width 0) (type default) (color 0 255 0 1))
   )
+  (wire (pts (xy 49.53 196.85) (xy 49.53 201.93))
+    (stroke (width 0) (type default) (color 0 0 0 0))
+  )
   (wire (pts (xy 208.28 53.34) (xy 208.28 54.61))
     (stroke (width 0) (type default) (color 0 0 0 0))
@@
     (stroke (width 0) (type default) (color 0 0 0 0))
   )
+  (wire (pts (xy 72.39 241.3) (xy 72.39 246.38))
+    (stroke (width 0) (type default) (color 0 0 0 0))
+  )
   (wire (pts (xy 113.03 119.38) (xy 113.03 107.95))
     (stroke (width 0) (type default) (color 0 0 0 0))
@@
     (stroke (width 0) (type default) (color 0 0 0 0))
   )
+  (wire (pts (xy 120.65 241.3) (xy 118.11 241.3))
+    (stroke (width 0) (type default) (color 0 0 0 0))
+  )
   (wire (pts (xy 208.28 132.08) (xy 208.28 133.35))
     (stroke (width 0) (type default) (color 0 0 0 0))
@@
     (stroke (width 0) (type default) (color 0 0 0 0))
   )
+  (wire (pts (xy 74.93 241.3) (xy 72.39 241.3))
+    (stroke (width 0) (type default) (color 0 0 0 0))
+  )
   (wire (pts (xy 63.5 40.64) (xy 80.01 40.64))
     (stroke (width 0) (type default) (color 0 0 0 0))
   )
+  (wire (pts (xy 118.11 241.3) (xy 118.11 246.38))
+    (stroke (width 0) (type default) (color 0 0 0 0))
+  )
   (wire (pts (xy 106.68 68.58) (xy 106.68 72.39))
     (stroke (width 0) (type default) (color 0 0 0 0))
@@
     (stroke (width 0) (type default) (color 132 0 0 1))
   )
+  (wire (pts (xy 49.53 196.85) (xy 52.07 196.85))
+    (stroke (width 0) (type default) (color 0 0 0 0))
+  )
   (wire (pts (xy 234.95 140.97) (xy 257.81 140.97))
     (stroke (width 0) (type default) (color 0 72 0 1))
@@
     (stroke (width 0) (type default) (color 0 0 0 1))
   )
+  (wire (pts (xy 100.33 196.85) (xy 99.06 196.85))
+    (stroke (width 0) (type default) (color 0 0 0 0))
+  )
   (wire (pts (xy 158.75 31.75) (xy 208.28 31.75))
     (stroke (width 0) (type default) (color 0 0 0 0))
@@
     (stroke (width 0) (type default) (color 0 0 0 0))
   )
+  (wire (pts (xy 99.06 196.85) (xy 99.06 201.93))
+    (stroke (width 0) (type default) (color 0 0 0 0))
+  )
   (wire (pts (xy 31.75 134.62) (xy 31.75 124.46))
     (stroke (width 0) (type default) (color 0 0 0 0))
@@
     (pin "2")
   )
+  (symbol (lib_id "Connector:TestPoint") (at 74.93 241.3 270) (unit 1)
+    (in_bom no) (on_board yes) (fields_autoplaced)
+    (property "Reference" "TP604" (id 0) (at 80.01 240.0299 90)
+      (effects (font (size 1.27 1.27)) (justify left))
+    )
+    (property "Value" "TP_DI_1" (id 1) (at 80.01 242.5699 90)
+      (effects (font (size 1.27 1.27)) (justify left))
+    )
+    (property "Footprint" "TestPoint:TestPoint_Pad_D1.0mm" (id 2) (at 74.93 246.38 0)
+      (effects (font (size 1.27 1.27)) hide)
+    )
+    (property "Datasheet" "~" (id 3) (at 74.93 246.38 0)
+      (effects (font (size 1.27 1.27)) hide)
+    )
+    (pin "1")
+  )
   (symbol (lib_id "Driver_FET:ZXGD3009E6") (at 208.28 119.38 0) (unit 1)
     (in_bom yes) (on_board yes) (fields_autoplaced)
@@
       (effects (font (size 1.27 1.27)) hide)
     )
-    (pin "1")
-    (pin "2")
-    (pin "6")
     (pin "3")
     (pin "4")
@@
     (pin "7")
     (pin "8")
-    (pin "3")
-    (pin "4")
-    (pin "5")
-    (pin "6")
   )
   (symbol (lib_id "Device:R_Small") (at 109.22 240.03 0) (unit 1)
@@
     (pin "2")
     (pin "6")
-    (pin "3")
-    (pin "4")
-    (pin "5")
   )
   (symbol (lib_id "Driver_FET:ZXGD3009E6") (at 208.28 62.23 0) (unit 1)
@@
     (pin "1")
   )
+  (symbol (lib_id "Connector:TestPoint") (at 120.65 241.3 270) (unit 1)
+    (in_bom no) (on_board yes) (fields_autoplaced)
+    (property "Reference" "TP606" (id 0) (at 125.73 240.0299 90)
+      (effects (font (size 1.27 1.27)) (justify left))
+    )
+    (property "Value" "TP_DI_3" (id 1) (at 125.73 242.5699 90)
+      (effects (font (size 1.27 1.27)) (justify left))
+    )
+    (property "Footprint" "TestPoint:TestPoint_Pad_D1.0mm" (id 2) (at 120.65 246.38 0)
+      (effects (font (size 1.27 1.27)) hide)
+    )
+    (property "Datasheet" "~" (id 3) (at 120.65 246.38 0)
+      (effects (font (size 1.27 1.27)) hide)
+    )
+    (pin "1")
+  )
   (symbol (lib_id "Device:R_Small") (at 186.69 119.38 90) (mirror x) (unit 1)
     (in_bom yes) (on_board yes) (fields_autoplaced)
@@
     (pin "2")
   )
+  (symbol (lib_id "Connector:TestPoint") (at 52.07 196.85 270) (unit 1)
+    (in_bom no) (on_board yes) (fields_autoplaced)
+    (property "Reference" "TP603" (id 0) (at 57.15 195.5799 90)
+      (effects (font (size 1.27 1.27)) (justify left))
+    )
+    (property "Value" "TP_DI_2" (id 1) (at 57.15 198.1199 90)
+      (effects (font (size 1.27 1.27)) (justify left))
+    )
+    (property "Footprint" "TestPoint:TestPoint_Pad_D1.0mm" (id 2) (at 52.07 201.93 0)
+      (effects (font (size 1.27 1.27)) hide)
+    )
+    (property "Datasheet" "~" (id 3) (at 52.07 201.93 0)
+      (effects (font (size 1.27 1.27)) hide)
+    )
+    (pin "1")
+  )
   (symbol (lib_id "Device:R_Small") (at 232.41 59.69 90) (unit 1)
     (in_bom yes) (on_board yes)
@@
       (effects (font (size 1.27 1.27)) hide)
     )
-    (pin "1")
-    (pin "2")
-    (pin "6")
     (pin "3")
     (pin "4")
@@
       (effects (font (size 1.27 1.27)) hide)
     )
-    (pin "1")
-    (pin "2")
-    (pin "7")
-    (pin "8")
     (pin "3")
     (pin "4")
@@
     (pin "2")
     (pin "6")
-    (pin "3")
-    (pin "4")
-    (pin "5")
   )
   (symbol (lib_id "Device:R_Small") (at 99.06 127 180) (unit 1)
@@
       (effects (font (size 1.27 1.27)) hide)
     )
-    (pin "1")
-    (pin "2")
-    (pin "7")
-    (pin "8")
     (pin "3")
     (pin "4")
@@
       (effects (font (size 1.27 1.27)) hide)
     )
-    (pin "1")
-    (pin "2")
-    (pin "7")
-    (pin "8")
     (pin "3")
     (pin "4")
@@
       (effects (font (size 1.27 1.27)) hide)
     )
-    (pin "1")
-    (pin "2")
-    (pin "7")
-    (pin "8")
     (pin "3")
     (pin "4")
@@
     (pin "7")
     (pin "8")
-    (pin "3")
-    (pin "4")
-    (pin "5")
-    (pin "6")
   )
   (symbol (lib_id "Device:R_Small") (at 25.4 134.62 90) (mirror x) (unit 1)
@@
     (pin "7")
     (pin "8")
-    (pin "3")
-    (pin "4")
-    (pin "5")
-    (pin "6")
   )
   (symbol (lib_id "Device:R_Small") (at 80.01 66.04 90) (unit 1)
@@
     (pin "7")
     (pin "8")
-    (pin "3")
-    (pin "4")
-    (pin "5")
-    (pin "6")
   )
   (symbol (lib_id "Device:R_Small") (at 77.47 208.28 0) (unit 1)
@@
     (pin "7")
     (pin "8")
-    (pin "3")
-    (pin "4")
-    (pin "5")
-    (pin "6")
   )
   (symbol (lib_id "Device:Q_Dual_NMOS_S1G1S2G2D2D2D1D1") (at 101.6 156.21 0) (unit 2)
@@
       (effects (font (size 1.27 1.27)) hide)
     )
-    (pin "1")
-    (pin "2")
-    (pin "7")
-    (pin "8")
     (pin "3")
     (pin "4")
@@
       (effects (font (size 1.27 1.27)) hide)
     )
+    (pin "1")
+  )
+  (symbol (lib_id "Connector:TestPoint") (at 100.33 196.85 270) (unit 1)
+    (in_bom no) (on_board yes) (fields_autoplaced)
+    (property "Reference" "TP605" (id 0) (at 105.41 195.5799 90)
+      (effects (font (size 1.27 1.27)) (justify left))
+    )
+    (property "Value" "TP_DI_4" (id 1) (at 105.41 198.1199 90)
+      (effects (font (size 1.27 1.27)) (justify left))
+    )
+    (property "Footprint" "TestPoint:TestPoint_Pad_D1.0mm" (id 2) (at 100.33 201.93 0)
+      (effects (font (size 1.27 1.27)) hide)
+    )
+    (property "Datasheet" "~" (id 3) (at 100.33 201.93 0)
+      (effects (font (size 1.27 1.27)) hide)
+    )
