File: hardware/underglow-controller/Power.kicad_sch (KiCad schematic)
At the start: 17 parts, among them U8 ADP2303ARDZ-3.3

Commit message: i can't believe what they did to my boy
Parts:
- removed D5: D_Small, Diode_SMD:D_SOD-123F, symbol Device:D_Small
- added Q7: Q_PMOS_GDS, Package_TO_SOT_SMD:TO-252-2, symbol Device:Q_PMOS_GDS
- added R47, R48: 10k, Resistor_SMD:R_0603_1608Metric, symbol Device:R_Small
Connections:
- net VBAT: now also Q7.3 (S), R48.2
- new net VOUT: Q7.2 (D)
- new net VOUT_EN: Q7.1 (G), R48.1
Changed lines of the file:
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@@
   (junction (at 111.125 92.71) (diameter 0) (color 0 0 0 0)
   )
+  (junction (at 70.485 139.065) (diameter 0) (color 0 0 0 0)
+  )
   (junction (at 29.21 92.71) (diameter 0) (color 0 0 0 0)
   )
@@
   (junction (at 111.125 81.28) (diameter 0) (color 0 0 0 0)
   )
+  (junction (at 83.185 148.59) (diameter 0) (color 0 0 0 0)
+  )
   (junction (at 133.985 72.39) (diameter 0) (color 0 0 0 0)
   )
@@
     (stroke (width 0) (type default) (color 0 0 0 0))
   )
+  (wire (pts (xy 87.63 148.59) (xy 83.185 148.59))
+    (stroke (width 0) (type default) (color 0 0 0 0))
+  )
   (wire (pts (xy 125.095 74.93) (xy 125.095 80.01))
     (stroke (width 0) (type default) (color 0 0 0 0))
   )
+  (wire (pts (xy 83.185 148.59) (xy 83.185 144.145))
+    (stroke (width 0) (type default) (color 0 0 0 0))
+  )
   (wire (pts (xy 82.55 76.2) (xy 82.55 74.93))
     (stroke (width 0) (type default) (color 0 0 0 0))
   )
+  (wire (pts (xy 70.485 139.065) (xy 70.485 142.875))
+    (stroke (width 0) (type default) (color 0 0 0 0))
+  )
+  (wire (pts (xy 65.405 139.065) (xy 70.485 139.065))
+    (stroke (width 0) (type default) (color 0 0 0 0))
+  )
   (wire (pts (xy 72.39 45.085) (xy 86.995 45.085))
     (stroke (width 0) (type default) (color 0 0 0 0))
@@
     (stroke (width 0) (type default) (color 0 0 0 0))
   )
+  (wire (pts (xy 70.485 139.065) (xy 75.565 139.065))
+    (stroke (width 0) (type default) (color 0 0 0 0))
+  )
   (wire (pts (xy 76.2 35.56) (xy 72.39 35.56))
     (stroke (width 0) (type default) (color 0 0 0 0))
@@
     (stroke (width 0) (type default) (color 0 0 0 0))
   )
+  (wire (pts (xy 83.185 128.905) (xy 83.185 133.985))
+    (stroke (width 0) (type default) (color 0 0 0 0))
+  )
   (wire (pts (xy 111.125 64.77) (xy 111.125 67.31))
     (stroke (width 0) (type default) (color 0 0 0 0))
@@
     (stroke (width 0) (type default) (color 0 0 0 0))
   )
+  (wire (pts (xy 70.485 148.59) (xy 70.485 147.955))
+    (stroke (width 0) (type default) (color 0 0 0 0))
+  )
+  (wire (pts (xy 83.185 148.59) (xy 70.485 148.59))
+    (stroke (width 0) (type default) (color 0 0 0 0))
+  )
   (wire (pts (xy 69.215 86.36) (xy 69.215 92.71))
     (stroke (width 0) (type default) (color 0 0 0 0))
   )
+  (wire (pts (xy 86.995 128.905) (xy 83.185 128.905))
+    (stroke (width 0) (type default) (color 0 0 0 0))
+  )
   (wire (pts (xy 43.18 71.12) (xy 53.975 71.12))
     (stroke (width 0) (type default) (color 0 0 0 0))
@@
   )
   (wire (pts (xy 29.21 88.9) (xy 29.21 92.71))
-    (stroke (width 0) (type default) (color 0 0 0 0))
-  )
-  (wire (pts (xy 41.275 45.085) (xy 48.895 45.085))
-    (stroke (width 0) (type default) (color 0 0 0 0))
-  )
-  (wire (pts (xy 29.21 45.085) (xy 36.195 45.085))
     (stroke (width 0) (type default) (color 0 0 0 0))
   )
@@
     (effects (font (size 1.27 1.27)) (justify left bottom))
   )
-  (label "VBAT" (at 31.115 45.085 0)
-    (effects (font (size 1.27 1.27)) (justify left bottom))
-  )
   (label "PGOOD" (at 44.45 81.28 0)
     (effects (font (size 1.27 1.27)) (justify left bottom))
   )
-  (label "VIN" (at 46.355 45.085 180)
-    (effects (font (size 1.27 1.27)) (justify right bottom))
-  )
   (label "3.3V" (at 118.745 74.93 180)
     (effects (font (size 1.27 1.27)) (justify right bottom))
@@
     (effects (font (size 1.27 1.27)) (justify left))
   )
-  (hierarchical_label "VBAT" (shape input) (at 29.21 45.085 180)
+  (hierarchical_label "VBAT" (shape input) (at 87.63 148.59 0)
+    (effects (font (size 1.27 1.27)) (justify left))
+  )
+  (hierarchical_label "VIN" (shape input) (at 25.4 71.12 180)
     (effects (font (size 1.27 1.27)) (justify right))
   )
-  (hierarchical_label "VIN" (shape output) (at 48.895 45.085 0)
+  (hierarchical_label "VOUT_EN" (shape input) (at 65.405 139.065 180)
+    (effects (font (size 1.27 1.27)) (justify right))
+  )
+  (hierarchical_label "VOUT" (shape output) (at 86.995 128.905 0)
     (effects (font (size 1.27 1.27)) (justify left))
   )
@@
     (pin "2")
   )
-  (symbol (lib_id "Device:D_Small") (at 38.735 45.085 180) (unit 1)
+  (symbol (lib_id "Device:C_Small") (at 133.985 82.55 0) (unit 1)
+    (in_bom yes) (on_board yes)
+    (property "Reference" "C41" (id 0) (at 135.89 81.2862 0)
+      (effects (font (size 1.27 1.27)) (justify left))
+    )
+    (property "Value" "22uF" (id 1) (at 135.89 83.8262 0)
+      (effects (font (size 1.27 1.27)) (justify left))
+    )
+    (property "Footprint" "Capacitor_SMD:C_0805_2012Metric" (id 2) (at 133.985 82.55 0)
+      (effects (font (size 1.27 1.27)) hide)
+    )
+    (property "Datasheet" "~" (id 3) (at 133.985 82.55 0)
+      (effects (font (size 1.27 1.27)) hide)
+    )
+    (property "MPN" "CL21A226MOQNNNE" (id 5) (at 133.985 82.55 0)
+      (effects (font (size 1.27 1.27)) hide)
+    )
+    (property "Description" "CAP CER 22UF 16V X5R 0805" (id 6) (at 133.985 82.55 0)
+      (effects (font (size 1.27 1.27)) hide)
+    )
+    (pin "1")
+    (pin "2")
+  )
+  (symbol (lib_id "Device:R_Small") (at 57.785 128.27 0) (unit 1)
     (in_bom yes) (on_board yes) (fields_autoplaced)
-    (property "Reference" "D5" (id 0) (at 38.735 41.275 0))
-    (property "Value" "D_Small" (id 1) (at 40.0049 42.545 90)
-      (effects (font (size 1.27 1.27)) (justify right) hide)
-    )
-    (property "Footprint" "Diode_SMD:D_SOD-123F" (id 2) (at 38.735 45.085 90)
-      (effects (font (size 1.27 1.27)) hide)
-    )
-    (property "Datasheet" "~" (id 3) (at 38.735 45.085 90)
-      (effects (font (size 1.27 1.27)) hide)
-    )
-    (property "MPN" "CUHS15S30,H3F" (id 4) (at 38.735 45.085 0)
-      (effects (font (size 1.27 1.27)) hide)
-    )
-    (property "Description" "SBD SINGLE 30V, 1.5A, IN 2 PIN U" (id 6) (at 38.735 45.085 0)
-      (effects (font (size 1.27 1.27)) hide)
-    )
-    (pin "1")
-    (pin "2")
-  )
-  (symbol (lib_id "Device:C_Small") (at 133.985 82.55 0) (unit 1)
-    (in_bom yes) (on_board yes)
-    (property "Reference" "C41" (id 0) (at 135.89 81.2862 0)
-      (effects (font (size 1.27 1.27)) (justify left))
-    )
-    (property "Value" "22uF" (id 1) (at 135.89 83.8262 0)
-      (effects (font (size 1.27 1.27)) (justify left))
-    )
-    (property "Footprint" "Capacitor_SMD:C_0805_2012Metric" (id 2) (at 133.985 82.55 0)
-      (effects (font (size 1.27 1.27)) hide)
-    )
-    (property "Datasheet" "~" (id 3) (at 133.985 82.55 0)
-      (effects (font (size 1.27 1.27)) hide)
-    )
-    (property "MPN" "CL21A226MOQNNNE" (id 5) (at 133.985 82.55 0)
-      (effects (font (size 1.27 1.27)) hide)
-    )
-    (property "Description" "CAP CER 22UF 16V X5R 0805" (id 6) (at 133.985 82.55 0)
+    (property "Reference" "R47" (id 0) (at 60.325 126.9999 0)
+      (effects (font (size 1.27 1.27)) (justify left))
+    )
+    (property "Value" "10k" (id 1) (at 60.325 129.5399 0)
+      (effects (font (size 1.27 1.27)) (justify left))
+    )
+    (property "Footprint" "Resistor_SMD:R_0603_1608Metric" (id 2) (at 57.785 128.27 0)
+      (effects (font (size 1.27 1.27)) hide)
+    )
+    (property "Datasheet" "~" (id 3) (at 57.785 128.27 0)
+      (effects (font (size 1.27 1.27)) hide)
+    )
+    (property "MPN" "RNCP0603FTD10K0" (id 5) (at 57.785 128.27 0)
+      (effects (font (size 1.27 1.27)) hide)
+    )
+    (property "Description" "RES 10K OHM 1% 1/8W 0603" (id 6) (at 57.785 128.27 0)
       (effects (font (size 1.27 1.27)) hide)
     )
@@
       (effects (font (size 1.27 1.27)) hide)
     )
+    (pin "1")
+    (pin "2")
+  )
+  (symbol (lib_id "Device:Q_PMOS_GDS") (at 80.645 139.065 0) (unit 1)
+    (in_bom yes) (on_board yes) (fields_autoplaced)
+    (property "Reference" "Q7" (id 0) (at 86.36 137.7949 0)
+      (effects (font (size 1.27 1.27)) (justify left))
+    )
+    (property "Value" "Q_PMOS_GDS" (id 1) (at 86.36 140.3349 0)
+      (effects (font (size 1.27 1.27)) (justify left))
+    )
+    (property "Footprint" "Package_TO_SOT_SMD:TO-252-2" (id 2) (at 85.725 136.525 0)
+      (effects (font (size 1.27 1.27)) hide)
+    )
+    (property "Datasheet" "~" (id 3) (at 80.645 139.065 0)
+      (effects (font (size 1.27 1.27)) hide)
+    )
+    (property "MPN" "STD15P6F6AG" (id 4) (at 80.645 139.065 0)
+      (effects (font (size 1.27 1.27)) hide)
+    )
+    (pin "1")
+    (pin "2")
+    (pin "3")
+  )
+  (symbol (lib_id "Device:R_Small") (at 70.485 145.415 0) (unit 1)
+    (in_bom yes) (on_board yes) (fields_autoplaced)
+    (property "Reference" "R48" (id 0) (at 73.025 144.1449 0)
+      (effects (font (size 1.27 1.27)) (justify left))
+    )
+    (property "Value" "10k" (id 1) (at 73.025 146.6849 0)
+      (effects (font (size 1.27 1.27)) (justify left))
+    )
+    (property "Footprint" "Resistor_SMD:R_0603_1608Metric" (id 2) (at 70.485 145.415 0)
+      (effects (font (size 1.27 1.27)) hide)
+    )
+    (property "Datasheet" "~" (id 3) (at 70.485 145.415 0)
+      (effects (font (size 1.27 1.27)) hide)
+    )
+    (property "MPN" "RNCP0603FTD10K0" (id 5) (at 70.485 145.415 0)
+      (effects (font (size 1.27 1.27)) hide)
+    )
+    (property "Description" "RES 10K OHM 1% 1/8W 0603" (id 6) (at 70.485 145.415 0)
+      (effects (font (size 1.27 1.27)) hide)
+    )

Commit message: urmom
Parts:
- removed R47: 10k, Resistor_SMD:R_0603_1608Metric, symbol Device:R_Small
- removed TP4: 3V3OUT, TestPoint:TestPoint_Pad_D1.0mm, symbol Connector:TestPoint
Changed lines of the file:
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@@
-    (stroke (width 0) (type default) (color 0 0 0 0))
-  )
-  (wire (pts (xy 111.125 64.77) (xy 111.125 67.31))
     (stroke (width 0) (type default) (color 0 0 0 0))
   )
@@
     (pin "2")
   )
-  (symbol (lib_id "power:GND") (at 111.125 67.31 0) (unit 1)
-    (in_bom yes) (on_board yes) (fields_autoplaced)
-    (property "Reference" "#PWR051" (id 0) (at 111.125 73.66 0)
-      (effects (font (size 1.27 1.27)) hide)
-    )
-    (property "Value" "GND" (id 1) (at 113.03 68.5799 0)
-      (effects (font (size 1.27 1.27)) (justify left))
-    )
-    (property "Footprint" "" (id 2) (at 111.125 67.31 0)
-      (effects (font (size 1.27 1.27)) hide)
-    )
-    (property "Datasheet" "" (id 3) (at 111.125 67.31 0)
-      (effects (font (size 1.27 1.27)) hide)
-    )
-    (pin "1")
-  )
   (symbol (lib_id "Device:R_Small") (at 111.125 85.09 0) (mirror y) (unit 1)
     (in_bom yes) (on_board yes)
@@
     )
     (property "Description" "CAP CER 22UF 16V X5R 0805" (id 6) (at 133.985 82.55 0)
-      (effects (font (size 1.27 1.27)) hide)
-    )
-    (pin "1")
-    (pin "2")
-  )
-  (symbol (lib_id "Device:R_Small") (at 57.785 128.27 0) (unit 1)
-    (in_bom yes) (on_board yes) (fields_autoplaced)
-    (property "Reference" "R47" (id 0) (at 60.325 126.9999 0)
-      (effects (font (size 1.27 1.27)) (justify left))
-    )
-    (property "Value" "10k" (id 1) (at 60.325 129.5399 0)
-      (effects (font (size 1.27 1.27)) (justify left))
-    )
-    (property "Footprint" "Resistor_SMD:R_0603_1608Metric" (id 2) (at 57.785 128.27 0)
-      (effects (font (size 1.27 1.27)) hide)
-    )
-    (property "Datasheet" "~" (id 3) (at 57.785 128.27 0)
-      (effects (font (size 1.27 1.27)) hide)
-    )
-    (property "MPN" "RNCP0603FTD10K0" (id 5) (at 57.785 128.27 0)
-      (effects (font (size 1.27 1.27)) hide)
-    )
-    (property "Description" "RES 10K OHM 1% 1/8W 0603" (id 6) (at 57.785 128.27 0)
       (effects (font (size 1.27 1.27)) hide)
     )
@@
     (pin "2")
   )
-  (symbol (lib_id "Connector:TestPoint") (at 111.125 64.77 270) (unit 1)
-    (in_bom yes) (on_board yes)
-    (property "Reference" "TP4" (id 0) (at 117.475 62.865 90))
-    (property "Value" "3V3OUT" (id 1) (at 119.38 64.77 90))
-    (property "Footprint" "TestPoint:TestPoint_Pad_D1.0mm" (id 2) (at 111.125 69.85 0)
-      (effects (font (size 1.27 1.27)) hide)
-    )
-    (property "Datasheet" "~" (id 3) (at 111.125 69.85 0)
-      (effects (font (size 1.27 1.27)) hide)
-    )
-    (pin "1")
-  )
   (symbol (lib_id "Regulator_Switching:ADP2303ARDZ-3.3") (at 66.675 76.2 0) (unit 1)
