File: hardware/underglow-controller/CAN-Bus.kicad_sch (KiCad schematic)
At the start: 4 parts, among them U401 SN65HVD230

Commit message: hardware: prepare for production run
Signed-off-by: Connor Rigby <connorr@hey.com>
Parts:
- U401: LCSC C12084 -> (none); now in the parts list
Changed lines of the file:
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@@
   )
   (symbol (lib_id "Interface_CAN_LIN:SN65HVD230") (at 86.36 66.04 0) (mirror y) (unit 1)
-    (in_bom no) (on_board yes) (fields_autoplaced)
+    (in_bom yes) (on_board yes) (fields_autoplaced)
     (property "Reference" "U401" (id 0) (at 86.8806 55.88 0)
       (effects (font (size 1.27 1.27)) (justify right))
@@
       (effects (font (size 1.27 1.27)) hide)
     )
-    (property "LCSC" "C12084" (id 7) (at 86.36 66.04 0)
-      (effects (font (size 1.27 1.27)) hide)
-    )

Commit message: hardware: select some JLCPCB components
Signed-off-by: Connor Rigby <connorr@hey.com>
Parts:
- C401: Digikey (none) -> CGA2B1X7T0G105M050BC; MPN CGA2B1X7T0G105M050BC -> (none)
- R401: Digikey (none) -> RMCF0805JT120R; MPN RMCF0805JT120R -> (none)
- R402: Digikey (none) -> RMCF0402FT1K00; MPN RMCF0402FT1K00 -> (none)
- U401: Digikey (none) -> SN65HVD230D; MPN SN65HVD230D -> (none)
Changed lines of the file:
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@@
       (effects (font (size 1.27 1.27)) hide)
     )
-    (property "MPN" "CGA2B1X7T0G105M050BC" (id 5) (at 113.03 52.07 0)
+    (property "Digikey" "CGA2B1X7T0G105M050BC" (id 5) (at 113.03 52.07 0)
       (effects (font (size 1.27 1.27)) hide)
     )
@@
       (effects (font (size 1.27 1.27)) hide)
     )
-    (property "MPN" "RMCF0805JT120R" (id 4) (at 68.58 67.31 0)
+    (property "Digikey" "RMCF0805JT120R" (id 4) (at 68.58 67.31 0)
       (effects (font (size 1.27 1.27)) hide)
     )
@@
       (effects (font (size 1.27 1.27)) hide)
     )
-    (property "MPN" "RMCF0402FT1K00" (id 4) (at 105.41 74.93 0)
+    (property "Digikey" "RMCF0402FT1K00" (id 4) (at 105.41 74.93 0)
       (effects (font (size 1.27 1.27)) hide)
     )
@@
       (effects (font (size 1.27 1.27)) hide)
     )
-    (property "MPN" "SN65HVD230D" (id 4) (at 86.36 66.04 0)
+    (property "Digikey" "SN65HVD230D" (id 4) (at 86.36 66.04 0)
       (effects (font (size 1.27 1.27)) hide)
     )
