File: hardware/underglow-controller/Microphone.kicad_sch (KiCad schematic)
At the start: 3 parts

Commit message: Bom fillout + wiring
Parts:
- R801: MPN (none) -> RMCF0402JT10K0
Changed lines of the file:
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@@
       (effects (font (size 1.27 1.27)) (justify left bottom) hide)
+    )
+    (property "Description" "MICROPHONE MEMS DIGITAL I2S OMNI" (id 5) (at 105.41 69.85 0)
+      (effects (font (size 1.27 1.27)) hide)
     )
     (pin "1")
@@
       (effects (font (size 1.27 1.27)) hide)
     )
-    (property "Description" "" (id 4) (at 83.82 60.96 0)
+    (property "Description" "RES 10K OHM 5% 1/16W 0402" (id 4) (at 83.82 60.96 0)
       (effects (font (size 1.27 1.27)) hide)
     )
-    (property "MPN" "" (id 5) (at 83.82 60.96 0)
+    (property "MPN" "RMCF0402JT10K0" (id 5) (at 83.82 60.96 0)
       (effects (font (size 1.27 1.27)) hide)
     )

Commit message: hw updates based on prototype issues
* Removes unused hardware and firmware projectes
* Adds some documentation and bom
* cleanup READMEs
Other:
- company: (none) -> Connor Rigby
- title: (none) -> ${Title}
Changed lines of the file:
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@@
 (kicad_sch (version 20211123) (generator eeschema)
   (paper "A5")
+  (title_block
+    (title "${Title}")
+    (date "2022-06-24")
+    (rev "${Revision}")
+    (company "Connor Rigby")
+    (comment 1 "https://github.com/miata-bot/can-link")
+    (comment 2 "https://cone.codes")
+  )
   (junction (at 124.46 80.01) (diameter 0) (color 0 0 0 0)
   )

Commit message: hardware: select some JLCPCB components
Signed-off-by: Connor Rigby <connorr@hey.com>
Parts:
- C801: Digikey (none) -> 0402B104K250HI; MPN 0402B104K250HI -> (none)
- MK801: Digikey (none) -> ICS-43434; MPN ICS-43434 -> (none)
- R801: Digikey (none) -> RMCF0402JT10K0; MPN RMCF0402JT10K0 -> (none)
Changed lines of the file:
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@@
       (effects (font (size 1.27 1.27)) hide)
     )
-    (property "MPN" "0402B104K250HI" (id 5) (at 124.46 71.12 0)
+    (property "Digikey" "0402B104K250HI" (id 5) (at 124.46 71.12 0)
       (effects (font (size 1.27 1.27)) hide)
     )
@@
       (effects (font (size 1.27 1.27)) (justify left bottom) hide)
     )
-    (property "MPN" "ICS-43434" (id 4) (at 115.57 67.31 0)
+    (property "Digikey" "ICS-43434" (id 4) (at 115.57 67.31 0)
       (effects (font (size 1.27 1.27)) (justify left bottom) hide)
     )
@@
       (effects (font (size 1.27 1.27)) hide)
     )
-    (property "MPN" "RMCF0402JT10K0" (id 5) (at 83.82 60.96 0)
+    (property "Digikey" "RMCF0402JT10K0" (id 5) (at 83.82 60.96 0)
       (effects (font (size 1.27 1.27)) hide)
     )
