File: hardware/motor-controller/motor-controller.kicad_sch (KiCad schematic)
At the start: 136 parts, among them J2 U.FL-R-SMT-1(10), J3 DM3AT-SF-PEJM5, J4 DTM1312PA12PBR008, J5 Conn_01x10, J6 CONSOLE, J7 U.FL-R-SMT-1(10), J8 JTAG, Q2 STS8DNF3LL, Q3 STS8DNF3LL, Q4 STS8DNF3LL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

Commit message: Radio hardware and software design
Parts:
- removed AE3: PCB_ANT_RFM69, RF_Antenna:Texas_SWRA416_868MHz_915MHz, symbol Device:Antenna
- removed C24, C26: 20pF, Capacitor_SMD:C_0402_1005Metric, symbol Device:C_Small
- removed C28, C33, C38: 1uF, Capacitor_SMD:C_0402_1005Metric, symbol Device:C_Small
- removed C29, C31, C35, C40, C48, C49, C50, C51, C52, C9: 0.1uF, Capacitor_SMD:C_0402_1005Metric, symbol Device:C_Small
- removed C45: 10uF, Capacitor_SMD:C_0805_2012Metric, symbol Device:C_Small
- removed C6: 0.1uF, Capacitor_SMD:C_0805_2012Metric, symbol Device:C_Small
- removed D4: GRN, LED_SMD:LED_0603_1608Metric, symbol Device:LED
- removed H1: MountingHole_Pad, MountingHole:MountingHole_3.2mm_M3_DIN965_Pad, symbol Mechanical:MountingHole_Pad
- removed J2: U.FL-R-SMT-1(10), ConeCodes:HRS_U.FL-R-SMT-1(10), symbol U.FL-R-SMT-1_10_:U.FL-R-SMT-1(10)
- removed J3: DM3AT-SF-PEJM5, ConeCodes:HRS_DM3AT-SF-PEJM5, symbol ConeCodes:DM3AT-SF-PEJM5
- removed J4: DTM1312PA12PBR008, TE_DTM1312PA12PBR008, symbol ConeCodes:DTM1312PA12PBR008
- removed J5: Conn_01x10, Connector_PinHeader_2.54mm:PinHeader_1x10_P2.54mm_Vertical, symbol Connector_Generic:Conn_01x10
- removed JP2: LED Voltage Select, Jumper:SolderJumper-3_P1.3mm_Bridged12_RoundedPad1.0x1.5mm_NumberLabels, symbol Jumper:SolderJumper_3_Bridged12
- removed Q2, Q3, Q4: STS8DNF3LL, Package_SO:SO-8_3.9x4.9mm_P1.27mm, symbol Device:Q_Dual_NMOS_S1G1S2G2D2D2D1D1
- removed R20: 240R, Resistor_SMD:R_0603_1608Metric, symbol Device:R_Small
- removed R40, R43, R44, R45: 10k, Resistor_SMD:R_0402_1005Metric, symbol Device:R_Small
- removed R41: 27r4, Resistor_SMD:R_0402_1005Metric, symbol Device:R_Small
- removed SW4: SW_Push, ConeCodes:SW_RS-032G05A3-SMRT, symbol Switch:SW_Push
- removed TC3: TC2030-IDC, Connector:Tag-Connect_TC2030-IDC-NL_2x03_P1.27mm_Vertical, symbol TDC-2030-IDC:TC2030-IDC
- removed TP10: CS1, TestPoint:TestPoint_Pad_D1.0mm, symbol Connector:TestPoint
- removed TP11: CS2, TestPoint:TestPoint_Pad_D1.0mm, symbol Connector:TestPoint
- removed TP12: RP_RUN, TestPoint:TestPoint_Pad_D1.0mm, symbol Connector:TestPoint
- removed TP5: MOSI, TestPoint:TestPoint_Pad_D1.0mm, symbol Connector:TestPoint
- removed TP6: MISO, TestPoint:TestPoint_Pad_D1.0mm, symbol Connector:TestPoint
- removed TP8: SCLK, TestPoint:TestPoint_Pad_D1.0mm, symbol Connector:TestPoint
- removed TP9: CS0, TestPoint:TestPoint_Pad_D1.0mm, symbol Connector:TestPoint
- removed U11: RP2040, ConeCodes:QFN-56, symbol ConeCodes:RP2040
- removed U6: WS2815B, ConeCodes:worldsemi-WS2815B-MFG, symbol ConeCodes:WS2815B
- removed U7: W25Q128JVS, Package_SO:SOIC-8W_5.3x5.3mm_P1.27mm, symbol Memory_Flash:W25Q128JVS
- removed U9: COM-13909, ConeCodes:XCVR_RFM69HW, symbol ConeCodes:COM-13909
- removed Y4: 12MHZ, Crystal:Crystal_SMD_3225-4Pin_3.2x2.5mm, symbol Device:Crystal_GND24_Small
- added J4: DTM13-12PA-R008, ConeCodes:TE_DTM13-12PA-R008, symbol ConeCodes:DTM13-12PA-R008
- added R2, R29, R5: R_Small, Resistor_SMD:R_0805_2012Metric, symbol Device:R_Small
- R24, R38: value 10k -> R_Small; footprint Resistor_SMD:R_0402_1005Metric -> Resistor_SMD:R_0805_2012Metric; MPN RMCF0402JT10K0 -> (none)
- R32, R33: value 0R -> R_Small; footprint Resistor_SMD:R_0402_1005Metric -> Resistor_SMD:R_0805_2012Metric
- R36: value 1k -> R_Small; footprint Resistor_SMD:R_0402_1005Metric -> Resistor_SMD:R_0805_2012Metric; MPN RMCF0402FT1K00 -> (none)
- R37: value 100k -> R_Small; footprint Resistor_SMD:R_0402_1005Metric -> Resistor_SMD:R_0805_2012Metric; MPN RNCF0402DTE100K -> (none)
- R42: value 27r4 -> R_Small; footprint Resistor_SMD:R_0402_1005Metric -> Resistor_SMD:R_0805_2012Metric; MPN RMCF0402FT27R4 -> (none)
Connections:
- net FSPICLK is gone; now on net GPIO36: U4.41 (GPIO36)
- net FSPIHD is gone; now on net GPIO33: U4.38 (GPIO33)
- net LED_RED is gone; now on net GPIO37: R19.2
- net RF69_RF_ANT_PCB is gone; now on net GND: R33.2
- net RF69_RF_EXT is gone; now on net GPIO34: R32.2
- net RP_USB_D_M is gone; now on net GND: R42.2
- net USB_BOOT is gone; now on net GND: R36.2
- net +3V3: no longer R24.1, R37.1, R38.1
- net CAN_N: now also J4.5
- net CAN_P: now also J4.6
- net GND: now also R37.2, J4.12, R2.1, R5.1; no longer U10.6 (SRC12), U10.9 (SRC34)
- net GPIO14: no longer R38.2
- net MOTOR1_OUT1: now also J4.7
- net MOTOR1_OUT2: now also J4.8
- net MOTOR2_OUT1: now also J4.9
- net MOTOR2_OUT2: now also J4.10
- net VBAT: now also J4.11
- net GPIO36: now reaches R24.2
- net GPIO36: now also R33.1
- net CONN_RP_USB_D_N renamed GPIO33
- net GPIO33: now also R38.2
- net FSPICS0 renamed GPIO34
- net GPIO34: now also R37.1
- net FSPICS1 renamed GPIO9
- net FSPICS2 renamed GPIO13
- net FSPID renamed GPIO35
- net GPIO35: now also R36.1, R29.2
- net FSPIQ renamed GPIO37
- net RF69_RF_ANT renamed GPI3
- net GPI3: now also J4.3; no longer R33.1
- removed net RP_SS: R36.1, R37.2
- new net GPI1: J4.1, R24.1
- new net GPI2: J4.2, R29.1
- new net GPI4: J4.4, R38.1
- new net SRC12: R2.2, U10.6 (SRC12)
- new net SRC34: R5.2, U10.9 (SRC34)
- no-connect marks 32 -> 10
Other:
- note removed: "CX1 = CX2 = 2(12pF - 2pF) = 20pF"
- note removed: "INDIVIDUALLY ADDRESSABLE LED CONTROL"
- note removed: "RF69 PACKET RADIO"
- note removed: "RGB PWM LED CONTROL"
- note removed: "SPID = MOSI SPIQ = MISO"
- note removed: "Unsure if supply voltage should go to VCC or VDD. Datasheet says VDD but that doesn't make a ton of sense to me. If this part doesn't work, bridge the other half"
