File: hardware/usb-stick/usb-stick.kicad_sch (KiCad schematic)
At the start: 136 parts, among them J2 U.FL-R-SMT-1(10), J3 DM3AT-SF-PEJM5, J4 DTM1312PA12PBR008, J5 Conn_01x10, J6 CONSOLE, J7 U.FL-R-SMT-1(10), J8 JTAG, Q2 STS8DNF3LL, Q3 STS8DNF3LL, Q4 STS8DNF3LL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

Commit message: Radio hardware and software design
Parts:
- removed C24, C26: 20pF, Capacitor_SMD:C_0402_1005Metric, symbol Device:C_Small
- removed C29, C31, C35, C40, C48, C49, C50, C51, C52, C9: 0.1uF, Capacitor_SMD:C_0402_1005Metric, symbol Device:C_Small
- removed C33, C38: 1uF, Capacitor_SMD:C_0402_1005Metric, symbol Device:C_Small
- removed C42: 0.47uF, Capacitor_SMD:C_0805_2012Metric, symbol Device:C_Small
- removed C43, C6: 0.1uF, Capacitor_SMD:C_0805_2012Metric, symbol Device:C_Small
- removed C44, C5: 10uF, Capacitor_SMD:C_0805_2012Metric, symbol Device:C_Small
- removed C46: 0.01uF, Capacitor_SMD:C_0805_2012Metric, symbol Device:C_Small
- removed C47: 10uF, Capacitor_SMD:CP_Elec_5x5.3, symbol Device:C_Polarized_Small
- removed H1: MountingHole_Pad, MountingHole:MountingHole_3.2mm_M3_DIN965_Pad, symbol Mechanical:MountingHole_Pad
- removed J4: DTM1312PA12PBR008, TE_DTM1312PA12PBR008, symbol ConeCodes:DTM1312PA12PBR008
- removed J5: Conn_01x10, Connector_PinHeader_2.54mm:PinHeader_1x10_P2.54mm_Vertical, symbol Connector_Generic:Conn_01x10
- removed JP2: LED Voltage Select, Jumper:SolderJumper-3_P1.3mm_Bridged12_RoundedPad1.0x1.5mm_NumberLabels, symbol Jumper:SolderJumper_3_Bridged12
- removed Q2, Q3, Q4: STS8DNF3LL, Package_SO:SO-8_3.9x4.9mm_P1.27mm, symbol Device:Q_Dual_NMOS_S1G1S2G2D2D2D1D1
- removed R14, R36: 1k, Resistor_SMD:R_0402_1005Metric, symbol Device:R_Small
- removed R37: 100k, Resistor_SMD:R_0402_1005Metric, symbol Device:R_Small
- removed R38, R39: 10k, Resistor_SMD:R_0402_1005Metric, symbol Device:R_Small
- removed R41, R42: 27r4, Resistor_SMD:R_0402_1005Metric, symbol Device:R_Small
- removed SW4: SW_Push, ConeCodes:SW_RS-032G05A3-SMRT, symbol Switch:SW_Push
- removed TC3: TC2030-IDC, Connector:Tag-Connect_TC2030-IDC-NL_2x03_P1.27mm_Vertical, symbol TDC-2030-IDC:TC2030-IDC
- removed TP12: RP_RUN, TestPoint:TestPoint_Pad_D1.0mm, symbol Connector:TestPoint
- removed U10: DRV8844PWP, Package_SO:HTSSOP-28-1EP_4.4x9.7mm_P0.65mm_EP2.85x5.4mm_ThermalVias, symbol ConeCodes:DRV8844PWP
- removed U11: RP2040, ConeCodes:QFN-56, symbol ConeCodes:RP2040
- removed U3: SN65HVD230, Package_SO:SOIC-8_3.9x4.9mm_P1.27mm, symbol Interface_CAN_LIN:SN65HVD230
- removed U6: WS2815B, ConeCodes:worldsemi-WS2815B-MFG, symbol ConeCodes:WS2815B
- removed U7: W25Q128JVS, Package_SO:SOIC-8W_5.3x5.3mm_P1.27mm, symbol Memory_Flash:W25Q128JVS
- removed Y4: 12MHZ, Crystal:Crystal_SMD_3225-4Pin_3.2x2.5mm, symbol Device:Crystal_GND24_Small
- added P2: USB_C_Plug, Connector_USB:USB_C_Plug_Molex_105444, symbol Connector:USB_C_Plug
- added R2: R_Small, Resistor_SMD:R_0402_1005Metric, symbol Device:R_Small
- R3: value 120,DNF -> R_Small; footprint Resistor_SMD:R_0805_2012Metric -> Resistor_SMD:R_0402_1005Metric; MPN RMCF0805JT120R -> (none)
Connections:
- net FSPICS2: no longer U4.18 (GPIO13)
- net CAN_N: no longer names the net of R3.1
- net CAN_P: no longer names the net of R3.2
- net DRV_SLEEP renamed GPIO12
- net EN1 renamed GPIO4
- net EN2 renamed GPIO6
- net EN3 renamed GPIO8
- net EN4 renamed GPIO11
- new net: P2.A1 (GND), P2.A12 (GND), P2.B1 (GND), P2.B12 (GND)
- new net: P2.A4 (VBUS), P2.A9 (VBUS), P2.B4 (VBUS), P2.B9 (VBUS)
- new net GPIO13: U4.18 (GPIO13)
- no-connect marks 32 -> 11
Other:
- note removed: "CAN"
- note removed: "CONNECTORS"
- note removed: "CX1 = CX2 = 2(12pF - 2pF) = 20pF"
- note removed: "INDIVIDUALLY ADDRESSABLE LED CONTROL"
- note removed: "MOTOR DRIVER"
- note removed: "Main outer connector"
- note removed: "RGB PWM LED CONTROL"
- note removed: "Unsure if supply voltage should go to VCC or VDD. Datasheet says VDD but that doesn't make a ton of sense to me. If this part doesn't work, bridge the other half"
