File: hardware/daxproj/daxproj.kicad_sch (KiCad schematic)
At the start: 78 parts, among them J1 Conn_01x04, J2 6437288-1, J3 JTAG, Q1 Q_PMOS_GDS, Q2 MBT3904DW1T1G, Q3 MBT3904DW1T1G, Q4 MBT3904DW1T1G, SW1 SW_Push, U1 TPS5430DDA, U2 SN65HVD230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

Commit message: Finish routing motor controller board
Parts:
- removed J2: 6437288-1, ConeCodes:6437288-1, symbol ConeCodes:6437288-1
- added J2: Conn_02x08_Top_Bottom, ConeCodes:953371, symbol Connector_Generic:Conn_02x08_Top_Bottom
Connections:
- net CAN_N is gone; now on net CANH: D7.2 (A2)
- net CAN_P is gone; now on net CANL: D7.1 (A1)
- net +12V: now also J2.1 (Pin_1)
- net CANH: now also J2.16 (Pin_16)
- net CANL: now also J2.8 (Pin_8)
- net GPI1: now also J2.12 (Pin_12)
- net MOTOR1_OUT1: now also J2.4 (Pin_4)
- net MOTOR1_OUT2: now also J2.5 (Pin_5)
- net MOTOR2_OUT1: now also J2.6 (Pin_6)
- net MOTOR2_OUT2: now also J2.7 (Pin_7)
- net VBAT_IN: now also J2.2 (Pin_2), J2.3 (Pin_3)
Other:
- moved on the sheet: D7
