File: hardware/input-expander/input-expander.kicad_pcb (KiCad board)
At the start: 4 copper layers, 78.5 x 93 mm, 71 parts, among them J2 Delphi_Sicma_24, J6 CONSOLE, J8 JTAG, Q2 MBT3904DW1T1G, Q3 MBT3904DW1T1G, Q4 MBT3904DW1T1G, U2 TLS850B0TEV33ATMA1, U3 SN65HVD230, U4 TLS850F2TAV50ATMA1, U5 STM32G491CEU6

Commit message: idk
Parts:
- added R7: >= 5.1k, Resistor_SMD:R_0805_2012Metric, F.Cu at (40.1, 57.8)
- moved U3 46.8 mm to (91.7, 52.0), turned to -90 degrees
- moved D5 42.2 mm to (81.6, 52.0), turned to -90 degrees
- moved C3 35.1 mm to (86.7, 48.1), turned to -90 degrees
- moved U4 30.3 mm to (72.6, 54.6), turned to -90 degrees
- moved C6 29.2 mm to (67.2, 47.8), turned to -90 degrees
- moved C5 26.0 mm to (79.7, 73.3)
- moved C4 26.0 mm to (75.3, 73.3)
- moved U2 20.7 mm to (62.3, 64.4)
- moved R6 20.7 mm to (58.9, 63.8)
- moved R4 15.6 mm to (60.7, 44.9)
- moved D7 12.2 mm to (60.7, 48.3)
- moved C10 10.4 mm to (80.6, 91.0)
- moved C11 10.4 mm to (80.6, 93.1)
- moved C2 10.4 mm to (77.7, 103.5)
- moved C7 10.4 mm to (51.4, 78.4)
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- renumbered C5 to C2, C4 to C3, C2 to C4, C3 to C5, C8 to C6, C6 to C7, C7 to C8, D8 to D3, D3 to D4, D7 to D5, D5 to D6, D6 to D7, D4 to D8, H3 to H2, H2 to H3, J8 to J2, J6 to J3, J2 to J4, R5 to R10, R9 to R11, R21 to R12, R27 to R13, R33 to R14, R22 to R15, R28 to R16, R34 to R17, R17 to R18, R20 to R19, R18 to R2, R25 to R20, R26 to R21, R31 to R22, R32 to R23, R10 to R24, R6 to R25, R7 to R26, R8 to R27, R12 to R28, R23 to R29, R11 to R3, R35 to R30, R15 to R31, R29 to R32, R37 to R33, R13 to R34, R24 to R35, R16 to R37, R30 to R38, R38 to R39, R3 to R4, R19 to R5, R14 to R6, R2 to R8, R4 to R9, U3 to U2, U2 to U3
Connections:
- net Net-(U4-Pad1) renamed /VIN
- net Net-(U4-Pad5) renamed /5V_DIV
- J4 pad A4: VBUS -> +5VA
- J4 pad A6: +5VA -> /IGNITION
- J4 pad A7: /IGNITION -> VBUS
- J4 pad B2: /CAN_H -> /CAN_L
- R4 pad 1: /CAN_N -> /CAN_L
- R4 pad 2: /CAN_P -> /CAN_H
- U2 pad 6: /CAN_N -> /CAN_L
- U2 pad 7: /CAN_P -> /CAN_H
- U4 pad 3: unconnected-(U4-Pad3) -> /5V_WO
- U4 pad 6: unconnected-(U4-Pad6) -> /5V_WI
Routing:
- net /CAN_L: track 0.00 -> 14.1 mm
- net /CAN_H: track 0.00 -> 14.0 mm
- net GND1: track 0.00 -> 13.9 mm, vias 0 -> 1
- net +5VA: track 0.00 -> 9.31 mm
- net /USB_D+: track 0.00 -> 7.22 mm
- net /USB_D-: track 0.00 -> 7.18 mm
- net /5V_WI: track 0.00 -> 2.61 mm, vias 0 -> 1
- net /5V_DIV: track 0.00 -> 2.60 mm, vias 0 -> 1
- net GND: track 0.00 -> 1.20 mm, vias 0 -> 1
- added copper zone on F.Cu, net +12V
- added copper zone on F.Cu, net +5VA
- added copper zone on F.Cu, net /IGNITION
- added copper zone on F.Cu, net GND
- added copper zone on F.Cu, net VBUS

Commit message: u like resistors
Parts:
- removed D6: BAT54AW,115, Package_TO_SOT_SMD:SOT-323_SC-70
- added R10: R_Small, Resistor_SMD:R_0805_2012Metric, F.Cu at (83.6, 60.8)
- added R9: R_Small, Resistor_SMD:R_0805_2012Metric, F.Cu at (83.6, 62.8)
- moved R36 62.5 mm to (48.8, 50.4), turned to 0 degrees
- moved R21 62.4 mm to (93.0, 67.0)
- moved R20 61.4 mm to (93.0, 65.2)
- moved R22 61.1 mm to (93.0, 72.3)
- moved R14 61.0 mm to (93.0, 63.4)
- moved R17 60.9 mm to (93.0, 68.7)
- moved R23 60.9 mm to (93.0, 74.1)
- moved R15 59.6 mm to (93.0, 70.5)
- moved R24 57.8 mm to (93.0, 79.4)
- moved R18 56.8 mm to (93.0, 75.8)
- moved R16 55.4 mm to (93.0, 77.6)
- moved R25 55.0 mm to (93.0, 81.2)
- moved R30 54.9 mm to (48.8, 48.5)
- moved R19 54.5 mm to (93.0, 83.0)
- moved R34 54.0 mm to (48.8, 61.5)
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- renumbered R9 to R11, R10 to R12, R11 to R13, R12 to R14, R13 to R15, R14 to R16, R15 to R17, R16 to R18, R17 to R19, R18 to R20, R19 to R21, R20 to R22, R21 to R23, R22 to R24, R23 to R25, R24 to R26, R25 to R27, R26 to R28, R27 to R29, R28 to R30, R29 to R31, R30 to R32, R31 to R33, R32 to R34, R33 to R35, R34 to R36, R35 to R37, R36 to R38, R37 to R39, R38 to R40, R39 to R41
Connections:
- D10 pad 1: /ADC_IN3 -> /ADC2_IN5
- D10 pad 2: /ADC_IN4 -> /ADC1_IN15
- D11 pad 1: /ADC_IN5 -> /ADC1_IN12
- D11 pad 2: /ADC_IN6 -> /ADC2_IN12
- D9 pad 1: /ADC_IN1 -> /ADC2_IN13
- D9 pad 2: /ADC_IN2 -> /ADC2_IN4
- J4 pad B3: /DIN1 -> /DIN6
- J4 pad B4: /DIN2 -> /DIN5
- J4 pad B5: /DIN3 -> /AIN3
- J4 pad B6: /DIN4 -> /AIN2
- J4 pad B7: /DIN5 -> GNDS
- J4 pad B8: /DIN6 -> /AIN1
- J4 pad C1: GNDPWR -> /DIN2
- J4 pad C2: GNDS -> /DIN1
- J4 pad C3: /AIN6 -> /DIN3
- J4 pad C4: /AIN5 -> /DIN4
- J4 pad C5: /AIN4 -> GNDPWR
- J4 pad C6: /AIN3 -> /AIN4
- J4 pad C7: /AIN2 -> /AIN5
- J4 pad C8: /AIN1 -> /AIN6
- R14 pad 1: /ADC_IN1 -> /ADC2_IN13
- R15 pad 1: /ADC_IN3 -> /ADC2_IN5
- R16 pad 1: /ADC_IN5 -> /ADC1_IN12
- R17 pad 1: /ADC_IN2 -> /ADC2_IN4
- R18 pad 1: /ADC_IN4 -> /ADC1_IN15
- R19 pad 1: /ADC_IN6 -> /ADC2_IN12
- R20 pad 2: /ADC_IN1 -> /ADC2_IN13
- R21 pad 2: /ADC_IN2 -> /ADC2_IN4
- R22 pad 2: /ADC_IN3 -> /ADC2_IN5
- R23 pad 2: /ADC_IN4 -> /ADC1_IN15
- R24 pad 2: /ADC_IN5 -> /ADC1_IN12
- R25 pad 2: /ADC_IN6 -> /ADC2_IN12
- R27 pad 1: GND -> GNDS
- R28 pad 1: GND -> GNDS
- U2 pad 1: /GPIO_CAN_P -> /FDCAN2_TX
- U2 pad 4: /GPIO_CAN_N -> /FDCAN2_RX
- U5 pad 11: unconnected-(U5-Pad11) -> /ADC1_IN4
- U5 pad 12: unconnected-(U5-Pad12) -> /ADC2_IN17
- U5 pad 13: unconnected-(U5-Pad13) -> /ADC2_IN13
- U5 pad 14: unconnected-(U5-Pad14) -> /ADC2_IN3
- U5 pad 15: unconnected-(U5-Pad15) -> /ADC2_IN4
- U5 pad 16: unconnected-(U5-Pad16) -> /ADC2_IN5
- U5 pad 17: unconnected-(U5-Pad17) -> /ADC1_IN15
- U5 pad 18: unconnected-(U5-Pad18) -> /ADC1_IN12
- U5 pad 19: unconnected-(U5-Pad19) -> /ADC2_IN12
- U5 pad 33: unconnected-(U5-Pad33) -> /USB_D-
- U5 pad 34: unconnected-(U5-Pad34) -> /USB_D+
- U5 pad 36: unconnected-(U5-Pad36) -> /SWDIO-JTMS
- U5 pad 37: unconnected-(U5-Pad37) -> /SWCLK-JTCK
- U5 pad 38: unconnected-(U5-Pad38) -> /JTDI
- U5 pad 40: unconnected-(U5-Pad40) -> /JTDO
- U5 pad 42: unconnected-(U5-Pad42) -> /FDCAN2_TX
- U5 pad 43: unconnected-(U5-Pad43) -> /FDCAN2_RX
- U5 pad 5: unconnected-(U5-Pad5) -> /ADC1_IN10
- U5 pad 6: unconnected-(U5-Pad6) -> /ADC2_IN10
- U5 pad 8: unconnected-(U5-Pad8) -> /ADC12_IN1
- U5 pad 9: unconnected-(U5-Pad9) -> /ADC12_IN2
Routing:
- net /AIN6: track 0.00 -> 65.6 mm
- net /AIN4: track 0.00 -> 65.4 mm
- net /AIN5: track 0.00 -> 64.6 mm
- net /AIN3: track 0.00 -> 61.5 mm
- net /AIN2: track 0.00 -> 55.3 mm
- net unconnected-(Q2-Pad3): track 0.00 -> 48.9 mm
- net /DIN6: track 0.00 -> 48.7 mm
- net /DIN5: track 0.00 -> 46.9 mm
- net /DIN4: track 0.00 -> 45.7 mm
- net unconnected-(Q2-Pad6): track 0.00 -> 42.4 mm
- net unconnected-(Q3-Pad3): track 0.00 -> 39.7 mm
- net /AIN1: track 0.00 -> 39.6 mm
- net GND: track 1.20 -> 40.3 mm, vias 1 -> 39
- net /DIN3: track 0.00 -> 37.5 mm
- net /ADC2_IN13: track 0.00 -> 35.6 mm, vias 0 -> 2
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- added copper zone on F.Cu, net +3V3
- added copper zone on F.Cu, net /VDDA
- added copper zone on F.Cu, net /VIN
- added copper zone on B.Cu, net GNDS
- added copper zone on F.Cu, net GNDS
- added copper zone on In1.Cu, net GNDS
- added copper zone on In2.Cu, net GNDS

Commit message: finished i guess
Parts:
- removed J3: CONSOLE, Connector_PinHeader_1.27mm:PinHeader_1x06_P1.27mm_Vertical
- added C12: tbd, Capacitor_SMD:C_0402_1005Metric, F.Cu at (66.7, 70.1)
- added C13: tbd, Capacitor_SMD:C_0402_1005Metric, F.Cu at (66.7, 72.3)
- added C14: 0.1uF, Capacitor_SMD:C_0402_1005Metric, F.Cu at (64.5, 74.5)
- added R42: 0R, Resistor_SMD:R_2512_6332Metric, F.Cu at (83.4, 83.4)
- added SW2: SW_Push, ConeCodes:SW_RS-032G05A3-SMRT, F.Cu at (65.0, 81.9)
- added TP2: RX, TestPoint:TestPoint_Pad_D1.0mm, F.Cu at (84.8, 71.7)
- added TP3: TX, TestPoint:TestPoint_Pad_D1.0mm, F.Cu at (83.4, 73.2)
- added Y2: Crystal_GND24_Small, Crystal:Crystal_SMD_3225-4Pin_3.2x2.5mm, F.Cu at (64.4, 70.6)
- moved R2 51.2 mm to (96.2, 54.8), turned to -90 degrees
- moved D2 50.4 mm to (96.2, 51.5), turned to 90 degrees
- moved G*** 45.7 mm to (43.2, 88.2)
- moved D3 24.4 mm to (66.1, 57.8), turned to 90 degrees
- moved J2 24.0 mm to (82.6, 67.2), turned to -90 degrees
- moved R3 23.2 mm to (66.1, 61.0), turned to -90 degrees
- moved R5 15.9 mm to (68.3, 80.0), turned to 90 degrees
- moved D4 12.0 mm to (68.3, 83.3), turned to -90 degrees
- moved R26 0.64 mm to (80.7, 70.7)
- moved R12 0.40 mm to (68.8, 70.2)
Connections:
- D3 pad 2: +3V3 -> +5VA
- D8 pad 1: /USB_D+ -> /USB_D-
- D8 pad 2: /USB_D- -> /USB_D+
- D9 pad 1: /ADC2_IN13 -> /ADC_IN1
- J2 pad 1: /MTCK -> /MTMS
- J2 pad 2: /MTDO -> GND
- J2 pad 3: /MTMS -> /MTCK
- J2 pad 4: /MTDI -> /JTDI
- J2 pad 6: unconnected-(J2-Pad6) -> /JTDO
- J4 pad A2: /USB_D- -> /USB_D+
- J4 pad A3: /USB_D+ -> /USB_D-
- Q2 pad 3: unconnected-(Q2-Pad3) -> /GPIO_DIN2
- Q2 pad 6: unconnected-(Q2-Pad6) -> /GPIO_DIN1
- Q3 pad 3: unconnected-(Q3-Pad3) -> /GPIO_DIN4
- Q3 pad 6: unconnected-(Q3-Pad6) -> /GPIO_DIN3
- Q4 pad 3: unconnected-(Q4-Pad3) -> /GPIO_DIN6
- Q4 pad 6: unconnected-(Q4-Pad6) -> /GPIO_DIN5
- R14 pad 1: /ADC2_IN13 -> /ADC_IN1
- R20 pad 2: /ADC2_IN13 -> /ADC_IN1
- R5 pad 2: /LED_RED -> /LED_STATUS
- U5 pad 13: /ADC2_IN13 -> /VSENSE
- U5 pad 14: /ADC2_IN3 -> /ADC_IN1
- U5 pad 2: unconnected-(U5-Pad2) -> /GPIO_CAN_EN
- U5 pad 25: unconnected-(U5-Pad25) -> /GPIO_DIN2
- U5 pad 26: unconnected-(U5-Pad26) -> /GPIO_DIN1
- U5 pad 27: unconnected-(U5-Pad27) -> /GPIO_DIN4
- U5 pad 28: unconnected-(U5-Pad28) -> /GPIO_DIN3
- U5 pad 29: unconnected-(U5-Pad29) -> /GPIO_DIN6
- U5 pad 30: unconnected-(U5-Pad30) -> /GPIO_DIN5
- U5 pad 31: unconnected-(U5-Pad31) -> /USART1_TX
- U5 pad 32: unconnected-(U5-Pad32) -> /USART1_RX
- U5 pad 36: /SWDIO-JTMS -> /MTMS
- U5 pad 37: /SWCLK-JTCK -> /MTCK
- U5 pad 46: unconnected-(U5-Pad46) -> /BOOT0
- U5 pad 5: /ADC1_IN10 -> /OSC_IN
- U5 pad 6: /ADC2_IN10 -> /OSC_OUT
- U5 pad 7: unconnected-(U5-Pad7) -> /NRST
- U5 pad 8: /ADC12_IN1 -> unconnected-(U5-Pad8)
- U5 pad 9: /ADC12_IN2 -> /LED_STATUS
Routing:
- net /GPIO_DIN2: track 0.00 -> 73.5 mm, vias 0 -> 2
- net /GPIO_DIN1: track 0.00 -> 68.0 mm, vias 0 -> 2
- net /GPIO_DIN4: track 0.00 -> 65.5 mm, vias 0 -> 2
- net /GPIO_DIN3: track 0.00 -> 60.2 mm, vias 0 -> 2
- net /GPIO_DIN6: track 0.00 -> 58.4 mm, vias 0 -> 2
- net /GPIO_DIN5: track 0.00 -> 53.1 mm, vias 0 -> 2
- net unconnected-(Q2-Pad3): track 48.9 -> 0.00 mm
- net unconnected-(Q2-Pad6): track 42.4 -> 0.00 mm
- net unconnected-(Q3-Pad3): track 39.7 -> 0.00 mm
- net /ADC_IN1: track 0.00 -> 36.9 mm, vias 0 -> 2
- net /ADC2_IN13: track 35.6 -> 0.00 mm, vias 2 -> 0
- net unconnected-(Q3-Pad6): track 33.7 -> 0.00 mm
- net /VSENSE: track 2.02 -> 33.5 mm, vias 0 -> 2
- net /GPIO_CAN_EN: track 2.42 -> 33.8 mm, vias 0 -> 2
- net unconnected-(Q4-Pad3): track 31.0 -> 0.00 mm
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- added copper zone on In2.Cu, net +3V3
- added copper zone on B.Cu, net GND
- removed copper zone on In2.Cu, net GND
Other:
- board text added: "CLK"
- board text added: "ConeCAN Input Expander"
- board text added: "DI"
- board text added: "DO"
- board text added: "GND"
- board text added: "REV A Designed by Connor Rigby 06/22"
- board text added: "TMS"

Commit message: panelize i guess idk
Parts:
- added C10: 1uf, Capacitor_SMD:C_0805_2012Metric, F.Cu at (155.2, 82.6)
- added C11: 1uf, Capacitor_SMD:C_0805_2012Metric, F.Cu at (157.3, 82.6)
- added C12: tbd, Capacitor_SMD:C_0402_1005Metric, F.Cu at (147.4, 70.0)
- added C13: tbd, Capacitor_SMD:C_0402_1005Metric, F.Cu at (147.4, 72.2)
- added C14: 0.1uF, Capacitor_SMD:C_0402_1005Metric, F.Cu at (145.2, 74.5)
- added C2: 10uF, Capacitor_SMD:C_0805_2012Metric, F.Cu at (141.4, 59.5)
- added C3: 1uf, Capacitor_SMD:C_0805_2012Metric, F.Cu at (167.4, 48.0)
- added C4: 47uf, Capacitor_SMD:C_0805_2012Metric, F.Cu at (168.9, 58.8)
- added C5: 100nf, Capacitor_SMD:C_0805_2012Metric, F.Cu at (168.9, 61.0)
- added C6: 1uf, Capacitor_SMD:C_0805_2012Metric, F.Cu at (147.8, 47.7)
- added C7: 47uf, Capacitor_SMD:C_0805_2012Metric, F.Cu at (160.4, 58.6)
- added C8: 100nf, Capacitor_SMD:C_0805_2012Metric, F.Cu at (160.4, 60.7)
- added C9: 10uf, Capacitor_SMD:C_0805_2012Metric, F.Cu at (162.2, 79.8)
- added D10: PESD2USB3UV-T, Package_TO_SOT_SMD:SOT-23, F.Cu at (170.2, 73.1)
- added D11: PESD2USB3UV-T, Package_TO_SOT_SMD:SOT-23, F.Cu at (170.2, 80.0)
- added D2: GRN, LED_SMD:LED_0603_1608Metric, F.Cu at (176.9, 51.4)
- added D3: GRN, LED_SMD:LED_0603_1608Metric, F.Cu at (146.8, 57.7)
- added D4: RED, LED_SMD:LED_0603_1608Metric, F.Cu at (149.0, 83.2)
- added D5: MBRD20200CT, Package_TO_SOT_SMD:TO-252-2, F.Cu at (162.3, 51.9)
- added D7: PESD2CANFD24V-T, Package_TO_SOT_SMD:SOT-23, F.Cu at (141.4, 48.2)
- added D8: PESD2USB3UV-T, Package_TO_SOT_SMD:SOT-23, F.Cu at (145.2, 48.2)
- added D9: PESD2USB3UV-T, Package_TO_SOT_SMD:SOT-23, F.Cu at (170.2, 66.1)
- added FB2: FerriteBead_Small, Inductor_SMD:L_0805_2012Metric, F.Cu at (159.3, 80.6)
- added G***: LOGO, logos:cone, F.Cu at (123.9, 88.1)
- added H2: MountingHole_Pad, MountingHole:MountingHole_6.4mm_M6_Pad_Via, F.Cu at (182.9, 110.0)
- added H3: MountingHole_Pad, MountingHole:MountingHole_6.4mm_M6_Pad_Via, F.Cu at (121.0, 110.0)
- added J2: JTAG, Connector_PinHeader_1.27mm:PinHeader_1x06_P1.27mm_Vertical, F.Cu at (163.3, 67.1)
- added J4: Delphi_Sicma_24, ConeCodes:Delphi_Sicma_24_Black, F.Cu at (151.9, 24.4)
- added Q2: MBT3904DW1T1G, Package_TO_SOT_SMD:SOT-363_SC-70-6, F.Cu at (125.5, 51.3)
- added Q3: MBT3904DW1T1G, Package_TO_SOT_SMD:SOT-363_SC-70-6, F.Cu at (125.5, 57.9)
- added Q4: MBT3904DW1T1G, Package_TO_SOT_SMD:SOT-363_SC-70-6, F.Cu at (125.5, 64.5)
- added R10: R_Small, Resistor_SMD:R_0805_2012Metric, F.Cu at (164.3, 60.7)
- added R11: R_Small, Resistor_SMD:R_0805_2012Metric, F.Cu at (153.8, 43.8)
- added R12: 100nf, Resistor_SMD:R_0402_1005Metric, F.Cu at (149.4, 70.2)
- added R13: 100nf, Resistor_SMD:R_0402_1005Metric, F.Cu at (152.6, 67.0)
- added R14: R_Small, Resistor_SMD:R_0603_1608Metric, F.Cu at (173.8, 63.3)
- added R15: R_Small, Resistor_SMD:R_0603_1608Metric, F.Cu at (173.8, 70.4)
- added R16: R_Small, Resistor_SMD:R_0603_1608Metric, F.Cu at (173.8, 77.5)
- added R17: R_Small, Resistor_SMD:R_0603_1608Metric, F.Cu at (173.8, 68.6)
- added R18: R_Small, Resistor_SMD:R_0603_1608Metric, F.Cu at (173.8, 75.7)
- added R19: R_Small, Resistor_SMD:R_0603_1608Metric, F.Cu at (173.8, 82.8)
- added R2: 240R, Resistor_SMD:R_0603_1608Metric, F.Cu at (176.9, 54.7)
- added R20: R_Small, Resistor_SMD:R_0603_1608Metric, F.Cu at (173.8, 65.1)
- added R21: R_Small, Resistor_SMD:R_0603_1608Metric, F.Cu at (173.8, 66.9)
- added R22: R_Small, Resistor_SMD:R_0603_1608Metric, F.Cu at (173.8, 72.2)
- added R23: R_Small, Resistor_SMD:R_0603_1608Metric, F.Cu at (173.8, 74.0)
- added R24: R_Small, Resistor_SMD:R_0603_1608Metric, F.Cu at (173.8, 79.3)
- added R25: R_Small, Resistor_SMD:R_0603_1608Metric, F.Cu at (173.8, 81.1)
- added R26: 100nf, Resistor_SMD:R_0402_1005Metric, F.Cu at (161.4, 70.5)
- added R27: 100nf, Resistor_SMD:R_0402_1005Metric, F.Cu at (159.3, 83.4)
- added R28: 100nf, Resistor_SMD:R_0402_1005Metric, F.Cu at (153.7, 82.2)
- added R29: 100nf, Resistor_SMD:R_0402_1005Metric, F.Cu at (160.7, 79.8)
- added R3: 240R, Resistor_SMD:R_0603_1608Metric, F.Cu at (146.8, 60.9)
- added R30: 10k, Resistor_SMD:R_0603_1608Metric, F.Cu at (129.5, 48.4)
- added R31: 10k, Resistor_SMD:R_0603_1608Metric, F.Cu at (129.5, 55.9)
- added R32: 10k, Resistor_SMD:R_0603_1608Metric, F.Cu at (129.5, 63.3)
- added R33: 10k, Resistor_SMD:R_0603_1608Metric, F.Cu at (129.5, 54.0)
- added R34: 10k, Resistor_SMD:R_0603_1608Metric, F.Cu at (129.5, 61.4)
- added R35: 10k, Resistor_SMD:R_0603_1608Metric, F.Cu at (129.5, 68.9)
- added R36: 1k5, Resistor_SMD:R_0603_1608Metric, F.Cu at (129.5, 50.3)
- added R37: 1k5, Resistor_SMD:R_0603_1608Metric, F.Cu at (129.5, 57.7)
- added R38: 1k5, Resistor_SMD:R_0603_1608Metric, F.Cu at (129.5, 65.2)
- added R39: 1k5, Resistor_SMD:R_0603_1608Metric, F.Cu at (129.5, 52.1)
- added R4: 120,DNF, Resistor_SMD:R_0805_2012Metric, F.Cu at (141.4, 44.8)
- added R40: 1k5, Resistor_SMD:R_0603_1608Metric, F.Cu at (129.5, 59.6)
- added R41: 1k5, Resistor_SMD:R_0603_1608Metric, F.Cu at (129.5, 67.0)
- added R42: 0R, Resistor_SMD:R_2512_6332Metric, F.Cu at (164.1, 83.3)
- added R5: 240R, Resistor_SMD:R_0603_1608Metric, F.Cu at (149.0, 79.9)
- added R6: 1k, Resistor_SMD:R_0402_1005Metric, F.Cu at (138.9, 49.2)
- added R7: >= 5.1k, Resistor_SMD:R_0805_2012Metric, F.Cu at (146.8, 53.3)
- added R8: R_Small, Resistor_SMD:R_0805_2012Metric, F.Cu at (150.4, 43.8)
- added R9: R_Small, Resistor_SMD:R_0805_2012Metric, F.Cu at (164.3, 62.7)
- added SW2: SW_Push, ConeCodes:SW_RS-032G05A3-SMRT, F.Cu at (145.7, 81.8)
- added TP2: RX, TestPoint:TestPoint_Pad_D1.0mm, F.Cu at (165.5, 71.5)
- added TP3: TX, TestPoint:TestPoint_Pad_D1.0mm, F.Cu at (164.1, 73.0)
- added U2: SN65HVD230, Package_SO:SOIC-8_3.9x4.9mm_P1.27mm, F.Cu at (141.4, 54.4)
- added U3: TLS850B0TEV33ATMA1, ConeCodes:TO-252-5_TabPin3, F.Cu at (172.4, 51.9)
- added U4: TLS850F2TAV50ATMA1, ConeCodes:DPAK127P1500X440-8N, F.Cu at (153.3, 54.5)
- added U5: STM32G491CEU6, ConeCodes:STM32G491CEU6, F.Cu at (155.3, 73.3)
- added Y2: Crystal_GND24_Small, Crystal:Crystal_SMD_3225-4Pin_3.2x2.5mm, F.Cu at (145.1, 70.5)
- added mouse-bite-2mm-slot: VAL**, ConeCodes:mouse-bite-2mm-slot, F.Cu at (111.6, 66.7)
- added mouse-bite-2mm-slot: VAL**, ConeCodes:mouse-bite-2mm-slot, F.Cu at (111.6, 106.6)
- added mouse-bite-2mm-slot: VAL**, ConeCodes:mouse-bite-2mm-slot, F.Cu at (111.6, 48.6)
- added mouse-bite-2mm-slot: VAL**, ConeCodes:mouse-bite-2mm-slot, F.Cu at (111.6, 30.4)
- added mouse-bite-2mm-slot: VAL**, ConeCodes:mouse-bite-2mm-slot, F.Cu at (111.6, 84.7)
Routing:
- net /GPIO_DIN2: track 73.5 -> 147.0 mm, vias 2 -> 4
- net /GPIO_DIN1: track 68.0 -> 136.0 mm, vias 2 -> 4
- net /GPIO_DIN4: track 65.5 -> 130.9 mm, vias 2 -> 4
- net /AIN6: track 65.1 -> 130.2 mm
- net /AIN4: track 64.9 -> 129.7 mm
- net /AIN5: track 64.0 -> 128.1 mm
- net GND: track 62.9 -> 125.7 mm, vias 59 -> 118
- net /AIN3: track 61.0 -> 122.0 mm
- net /GPIO_DIN3: track 60.2 -> 120.4 mm, vias 2 -> 4
- net /GPIO_DIN6: track 58.4 -> 116.8 mm, vias 2 -> 4
- net /AIN2: track 54.7 -> 109.4 mm
- net /USB_D-: track 54.7 -> 109.3 mm
- net /USB_D+: track 54.0 -> 108.0 mm
- net /GPIO_DIN5: track 53.1 -> 106.2 mm, vias 2 -> 4
- net /DIN6: track 48.7 -> 97.4 mm
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Other:
- board size 78.5 x 93 mm -> 159.2 x 93.1 mm
