File: hardware/input-expander/input-expander.kicad_sch (KiCad schematic)
At the start: 70 parts, among them J2 Delphi_Sicma_24, J6 CONSOLE, J8 JTAG, Q2 MBT3904DW1T1G, Q3 MBT3904DW1T1G, Q4 MBT3904DW1T1G, U2 TLS850B0TEV33ATMA1, U3 SN65HVD230, U4 TLS850F2TAV50ATMA1, U5 STM32G491CEU6

Commit message: idk
Parts:
- added R7: >= 5.1k, Resistor_SMD:R_0805_2012Metric, symbol Device:R_Small
- renumbered C5 to C2, C4 to C3, C2 to C4, C3 to C5, C8 to C6, C6 to C7, C7 to C8, D8 to D3, D3 to D4, D7 to D5, D5 to D6, D6 to D7, D4 to D8, H3 to H2, H2 to H3, J8 to J2, J6 to J3, J2 to J4, R5 to R10, R9 to R11, R21 to R12, R27 to R13, R33 to R14, R22 to R15, R28 to R16, R34 to R17, R17 to R18, R20 to R19, R18 to R2, R25 to R20, R26 to R21, R31 to R22, R32 to R23, R10 to R24, R6 to R25, R7 to R26, R8 to R27, R12 to R28, R23 to R29, R11 to R3, R35 to R30, R15 to R31, R29 to R32, R37 to R33, R13 to R34, R24 to R35, R16 to R37, R30 to R38, R38 to R39, R3 to R4, R19 to R5, R14 to R6, R2 to R8, R4 to R9, U3 to U2, U2 to U3
Connections:
- net CAN_N is gone; now on net CAN_L: R4.1, U2.6 (CANL)
- net CAN_P is gone; now on net CAN_H: R4.2, U2.7 (CANH)
- net +5VA: now also J4.A4, R7.1; no longer J4.A6
- net CAN_H: no longer J4.B2
- net CAN_L: now also J4.B2
- net IGNITION: now also J4.A6; no longer J4.A7
- net VBUS: now also J4.A7; no longer J4.A4
- net VIN: now reaches C4.1, C5.1, C7.1, C8.1, D5.2 (K), D6.1 (K), D6.2 (K), U3.1 (I), U4.1 (I)
- net 5V_WO: now reaches U4.3 (RO/WO)
- net 5V_WO: now also R7.2
- net 5V_DIV: now reaches R8.2, R9.1, U4.5 (RADJ)
- net 5V_WI: now reaches U4.6 (WI)
Other:
- moved on the sheet: D5

Commit message: u like resistors
Parts:
- removed D6: BAT54AW,115, Package_TO_SOT_SMD:SOT-323_SC-70, symbol Device:D_Schottky_Dual_CommonAnode_KKA
- added R10, R9: R_Small, Resistor_SMD:R_0805_2012Metric, symbol Device:R_Small
- renumbered R9 to R11, R10 to R12, R11 to R13, R12 to R14, R13 to R15, R14 to R16, R15 to R17, R16 to R18, R17 to R19, R18 to R20, R19 to R21, R20 to R22, R21 to R23, R22 to R24, R23 to R25, R24 to R26, R25 to R27, R26 to R28, R27 to R29, R28 to R30, R29 to R31, R30 to R32, R31 to R33, R32 to R34, R33 to R35, R34 to R36, R35 to R37, R36 to R38, R37 to R39, R38 to R40, R39 to R41
Connections:
- net ADC_IN1 is gone; now on net ADC2_IN13: D9.1 (K), R14.1, R20.2
- net ADC_IN2 is gone; now on net ADC2_IN4: D9.2 (K), R17.1, R21.2
- net ADC_IN3 is gone; now on net ADC2_IN5: D10.1 (K), R15.1, R22.2
- net ADC_IN4 is gone; now on net ADC1_IN15: D10.2 (K), R18.1, R23.2
- net ADC_IN5 is gone; now on net ADC1_IN12: D11.1 (K), R16.1, R24.2
- net ADC_IN6 is gone; now on net ADC2_IN12: D11.2 (K), R19.1, R25.2
- net GPIO_CAN_N is gone; now on net FDCAN2_RX: U2.4 (R)
- net GPIO_CAN_P is gone; now on net FDCAN2_TX: U2.1 (D)
- net AIN1: now also J4.B8; no longer J4.C8
- net AIN2: now also J4.B6; no longer J4.C7
- net AIN3: now also J4.B5; no longer J4.C6
- net AIN4: now also J4.C6; no longer J4.C5
- net AIN5: now also J4.C7; no longer J4.C4
- net AIN6: now also J4.C8; no longer J4.C3
- net DIN1: now also J4.C2; no longer J4.B3
- net DIN2: now also J4.C1; no longer J4.B4
- net DIN3: now also J4.C3; no longer J4.B5
- net DIN4: now also J4.C4; no longer J4.B6
- net DIN5: now also J4.B4; no longer J4.B7
- net DIN6: now also J4.B3; no longer J4.B8
- net GND: no longer R27.1, R28.1
- net GNDPWR: now also J4.C5; no longer J4.C1
- net GNDS: now also J4.B7, R27.1, R28.1, R9.2; no longer J4.C2
- net USB_D+: now also U5.34 (PA12)
- net USB_D-: now also U5.33 (PA11)
- net VIN: now also R10.1
- net ADC1_IN4: now reaches U5.11 (PA3)
- net ADC2_IN17: now reaches U5.12 (PA4)
- net ADC2_IN13: now reaches U5.13 (PA5)
- net ADC2_IN3: now reaches U5.14 (PA6)
- net ADC2_IN4: now reaches U5.15 (PA7)
- net ADC2_IN5: now reaches U5.16 (PC4)
- net ADC1_IN15: now reaches U5.17 (PB0)
- net ADC1_IN12: now reaches U5.18 (PB1)
- net ADC2_IN12: now reaches U5.19 (PB2)
- net SWDIO-JTMS: now reaches U5.36 (PA13)
- net SWCLK-JTCK: now reaches U5.37 (PA14)
- net JTDI: now reaches U5.38 (PA15)
- net JTDO: now reaches U5.40 (PC11)
- net FDCAN2_TX: now reaches U5.42 (PB4)
- net FDCAN2_RX: now reaches U5.43 (PB5)
- net ADC1_IN10: now reaches U5.5 (PF0-OSC_IN)
- net ADC2_IN10: now reaches U5.6 (PF1-OSC_OUT)
- net ADC12_IN1: now reaches U5.8 (PA0)
- net ADC12_IN2: now reaches U5.9 (PA1)
- new net VSENSE: R10.2, R9.1
Other:
- moved on the sheet: R26

Commit message: finished i guess
Parts:
- removed J3: CONSOLE, Connector_PinHeader_1.27mm:PinHeader_1x06_P1.27mm_Vertical, symbol Connector_Generic:Conn_01x06
- added C12, C13: tbd, Capacitor_SMD:C_0402_1005Metric, symbol Device:C_Small
- added C14: 0.1uF, Capacitor_SMD:C_0402_1005Metric, symbol Device:C_Small
- added R42: 0R, Resistor_SMD:R_2512_6332Metric, symbol Device:R_Small
- added SW2: SW_Push, ConeCodes:SW_RS-032G05A3-SMRT, symbol Switch:SW_Push
- added TP2: RX, TestPoint:TestPoint_Pad_D1.0mm, symbol Connector:TestPoint
- added TP3: TX, TestPoint:TestPoint_Pad_D1.0mm, symbol Connector:TestPoint
- added Y2: Crystal_GND24_Small, Crystal:Crystal_SMD_3225-4Pin_3.2x2.5mm, symbol Device:Crystal_GND24_Small
Connections:
- net LED_RED is gone; now on net LED_STATUS: R5.2
- net MTDI is gone; now on net JTDI: J2.4 (Pin_4)
- net MTDO is gone; now on net GND: J2.2 (Pin_2)
- net SWCLK-JTCK is gone; now on net MTCK: U5.37 (PA14)
- net SWDIO-JTMS is gone; now on net MTMS: U5.36 (PA13)
- net VSENSE is gone; now on net ADC2_IN13: R10.2, R9.1
- net +3V3: no longer D3.2 (A)
- net +5VA: now also D3.2 (A)
- net ADC2_IN13: no longer D9.1 (K), R14.1, R20.2
- net ADC2_IN3: now also D9.1 (K), R14.1, R20.2
- net GND: now also C12.2, C13.2, C14.1, R42.1, SW2.1, Y2.2, Y2.4
- net GNDS: now also R42.2
- net GPIO_CAN_EN: now also U5.2 (PC13)
- net JTDO: now also J2.6 (Pin_6)
- net MTCK: now also J2.3 (Pin_3); no longer J2.1 (Pin_1)
- net MTMS: now also J2.1 (Pin_1); no longer J2.3 (Pin_3)
- net USB_D+: now also D8.2 (K), J4.A2; no longer D8.1 (K), J4.A3
- net USB_D-: now also D8.1 (K), J4.A3; no longer D8.2 (K), J4.A2
- net GPIO_DIN4: now reaches Q3.3 (C2)
- net GPIO_DIN4: now also U5.27 (PB14)
- net GPIO_DIN6: now reaches Q4.3 (C2)
- net GPIO_DIN6: now also U5.29 (PC6)
- net GPIO_DIN2: now reaches Q2.3 (C2)
- net GPIO_DIN2: now also U5.25 (PB12)
- net GPIO_DIN1: now reaches U5.26 (PB13)
- net GPIO_DIN1: now also Q2.6 (C1)
- net GPIO_DIN3: now reaches U5.28 (PB15)
- net GPIO_DIN3: now also Q3.6 (C1)
- net GPIO_DIN5: now reaches U5.30 (PA8)
- net GPIO_DIN5: now also Q4.6 (C1)
- net USART1_TX: now reaches U5.31 (PA9)
- net USART1_TX: now also TP3.1
- net USART1_RX: now reaches U5.32 (PA10)
- net USART1_RX: now also TP2.1
- net BOOT0: now reaches U5.46 (PB8-BOOT0)
- net NRST: now reaches U5.7 (PG10-NRST)
- net NRST: now also C14.2, SW2.2
- net ADC12_IN1: no longer names the net of U5.8 (PA0)
- net ADC12_IN2 renamed LED_STATUS
- net ADC1_IN10 renamed OSC_IN
- net OSC_IN: now also C12.1, Y2.1
- net ADC2_IN10 renamed OSC_OUT
- net OSC_OUT: now also C13.1, Y2.3
- no-connect marks 3 -> 12
Other:
- moved on the sheet: J2

Commit message: Hardware updates
* fix messed up +12v pin
* add a ground output for neopixels on both channels
* add a i2c microphone
* clean up schematic
* calculate component values for the LED drivers
Changed lines of the file:
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@@
     (effects (font (size 1.27 1.27)) (justify left bottom))
+  )
+  (label "BOOT0" (at 71.755 192.405 180)
+    (effects (font (size 1.27 1.27)) (justify right bottom))
   )
   (label "AIN3" (at 388.62 236.22 180)
