File: hardware/davecu2/AnalogInput.kicad_sch (KiCad schematic)
At the start: 16 parts

Commit message: schematic cleanup
Parts:
- added R?: 10k, Resistor_SMD:R_0402_1005Metric, symbol Device:R_Small
- added R?: 36k, Resistor_SMD:R_0402_1005Metric, symbol Device:R_Small
- added TP?: VSENSE, TestPoint:TestPoint_Pad_D1.0mm, symbol Connector:TestPoint
Connections:
- net GND: now also R?.2
- new net VBATT: R?.1
- new net VSENSE_OUT: R?.1, R?.2, TP?.1
Changed lines of the file:
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@@
   (junction (at 97.79 33.02) (diameter 0) (color 0 0 0 0)
   )
+  (junction (at 63.5 126.365) (diameter 0) (color 0 0 0 0)
+  )
   (junction (at 97.79 58.42) (diameter 0) (color 0 0 0 0)
   )
+  (wire (pts (xy 63.5 126.365) (xy 63.5 123.825))
+    (stroke (width 0) (type default) (color 0 0 0 0))
+  )
   (wire (pts (xy 97.79 25.4) (xy 97.79 26.67))
     (stroke (width 0) (type default) (color 0 0 0 0))
@@
     (stroke (width 0) (type default) (color 0 0 0 0))
   )
+  (wire (pts (xy 63.5 116.84) (xy 63.5 118.745))
+    (stroke (width 0) (type default) (color 0 0 0 0))
+  )
+  (wire (pts (xy 63.5 126.365) (xy 78.105 126.365))
+    (stroke (width 0) (type default) (color 0 0 0 0))
+  )
   (wire (pts (xy 64.77 33.02) (xy 64.77 34.29))
     (stroke (width 0) (type default) (color 0 0 0 0))
@@
     (stroke (width 0) (type default) (color 0 0 0 0))
   )
+  (wire (pts (xy 63.5 128.27) (xy 63.5 126.365))
+    (stroke (width 0) (type default) (color 0 0 0 0))
+  )
   (wire (pts (xy 114.3 58.42) (xy 115.57 58.42))
     (stroke (width 0) (type default) (color 0 0 0 0))
@@
     (stroke (width 0) (type default) (color 0 0 0 0))
   )
+  (wire (pts (xy 63.5 116.84) (xy 78.74 116.84))
+    (stroke (width 0) (type default) (color 0 0 0 0))
+  )
   (wire (pts (xy 97.79 58.42) (xy 106.68 58.42))
     (stroke (width 0) (type default) (color 0 0 0 0))
   )
-  (hierarchical_label "CLT_LEVEL" (shape output) (at 187.96 69.85 180)
-    (effects (font (size 1.27 1.27)) (justify right))
+  (label "VSENSE" (at 75.565 126.365 180)
+    (effects (font (size 1.27 1.27)) (justify right bottom))
+  )
+  (label "VBATT" (at 78.105 116.84 180)
+    (effects (font (size 1.27 1.27)) (justify right bottom))
+  )
+  (hierarchical_label "CLT_LEVEL_OUT" (shape output) (at 187.96 69.85 180)
+    (effects (font (size 1.27 1.27)) (justify right))
+  )
+  (hierarchical_label "IAT_IN" (shape input) (at 195.58 33.02 0)
+    (effects (font (size 1.27 1.27)) (justify left))
   )
   (hierarchical_label "TPS1_OUT" (shape output) (at 66.04 33.02 0)
     (effects (font (size 1.27 1.27)) (justify left))
   )
+  (hierarchical_label "APV_ANGLE_IN" (shape input) (at 186.69 43.18 180)
+    (effects (font (size 1.27 1.27)) (justify right))
+  )
   (hierarchical_label "APP1_OUT" (shape output) (at 115.57 33.02 0)
     (effects (font (size 1.27 1.27)) (justify left))
   )
-  (hierarchical_label "MAF" (shape output) (at 196.85 59.69 0)
-    (effects (font (size 1.27 1.27)) (justify left))
-  )
-  (hierarchical_label "IAT" (shape output) (at 196.85 57.15 0)
+  (hierarchical_label "KNOCK_IN" (shape input) (at 195.58 40.64 0)
+    (effects (font (size 1.27 1.27)) (justify left))
+  )
+  (hierarchical_label "CLT_LEVEL_IN" (shape input) (at 186.69 45.72 180)
+    (effects (font (size 1.27 1.27)) (justify right))
+  )
+  (hierarchical_label "MAF_OUT" (shape output) (at 196.85 59.69 0)
+    (effects (font (size 1.27 1.27)) (justify left))
+  )
+  (hierarchical_label "IAT_OUT" (shape output) (at 196.85 57.15 0)
     (effects (font (size 1.27 1.27)) (justify left))
   )
@@
     (effects (font (size 1.27 1.27)) (justify right))
   )
+  (hierarchical_label "BARO_IN" (shape input) (at 195.58 38.1 0)
+    (effects (font (size 1.27 1.27)) (justify left))
+  )
+  (hierarchical_label "MAF_IN" (shape input) (at 195.58 35.56 0)
+    (effects (font (size 1.27 1.27)) (justify left))
+  )
+  (hierarchical_label "VSENSE_OUT" (shape output) (at 78.105 126.365 0)
+    (effects (font (size 1.27 1.27)) (justify left))
+  )
   (hierarchical_label "APP2_OUT" (shape output) (at 115.57 58.42 0)
     (effects (font (size 1.27 1.27)) (justify left))
   )
-  (hierarchical_label "APV_ANGLE" (shape output) (at 187.96 67.31 180)
+  (hierarchical_label "ECT_IN" (shape input) (at 186.69 38.1 180)
+    (effects (font (size 1.27 1.27)) (justify right))
+  )
+  (hierarchical_label "VBATT" (shape input) (at 78.74 116.84 0)
+    (effects (font (size 1.27 1.27)) (justify left))
+  )
+  (hierarchical_label "APV_ANGLE_OUT" (shape output) (at 187.96 67.31 180)
     (effects (font (size 1.27 1.27)) (justify right))
   )
@@
     (effects (font (size 1.27 1.27)) (justify left))
   )
-  (hierarchical_label "KNOCK" (shape output) (at 196.85 64.77 0)
+  (hierarchical_label "KNOCK_OUT" (shape output) (at 196.85 64.77 0)
     (effects (font (size 1.27 1.27)) (justify left))
   )
@@
     (effects (font (size 1.27 1.27)) (justify right))
   )
-  (hierarchical_label "ECT" (shape output) (at 187.96 62.23 180)
+  (hierarchical_label "ECT_OUT" (shape output) (at 187.96 62.23 180)
     (effects (font (size 1.27 1.27)) (justify right))
   )
@@
     (effects (font (size 1.27 1.27)) (justify right))
   )
-  (hierarchical_label "BARO" (shape output) (at 196.85 62.23 0)
-    (effects (font (size 1.27 1.27)) (justify left))
+  (hierarchical_label "BARO_OUT" (shape output) (at 196.85 62.23 0)
+    (effects (font (size 1.27 1.27)) (justify left))
+  )
+  (symbol (lib_id "Device:R_Small") (at 63.5 130.81 0) (unit 1)
+    (in_bom yes) (on_board yes)
+    (property "Reference" "R?" (id 0) (at 65.405 130.175 0)
+      (effects (font (size 1.27 1.27)) (justify left))
+    )
+    (property "Value" "10k" (id 1) (at 65.405 132.08 0)
+      (effects (font (size 1.27 1.27)) (justify left))
+    )
+    (property "Footprint" "Resistor_SMD:R_0402_1005Metric" (id 2) (at 63.5 130.81 0)
+      (effects (font (size 1.27 1.27)) hide)
+    )
+    (property "Datasheet" "~" (id 3) (at 63.5 130.81 0)
+      (effects (font (size 1.27 1.27)) hide)
+    )
+    (property "MPN" "RMCF0402JT10K0" (id 4) (at 63.5 130.81 0)
+      (effects (font (size 1.27 1.27)) hide)
+    )
+    (property "Description" "RES 10K OHM 5% 1/16W 0402" (id 6) (at 63.5 130.81 0)
+      (effects (font (size 1.27 1.27)) hide)
+    )
+    (pin "1")
+    (pin "2")
   )
   (symbol (lib_id "power:GND") (at 97.79 39.37 0) (unit 1)
@@
     (pin "2")
   )
+  (symbol (lib_id "Connector:TestPoint") (at 63.5 126.365 90) (unit 1)
+    (in_bom yes) (on_board yes)
+    (property "Reference" "TP?" (id 0) (at 53.34 124.46 90))
+    (property "Value" "VSENSE" (id 1) (at 55.245 126.365 90))
+    (property "Footprint" "TestPoint:TestPoint_Pad_D1.0mm" (id 2) (at 63.5 121.285 0)
+      (effects (font (size 1.27 1.27)) hide)
+    )
+    (property "Datasheet" "~" (id 3) (at 63.5 121.285 0)
+      (effects (font (size 1.27 1.27)) hide)
+    )
+    (pin "1")
+  )
   (symbol (lib_id "Device:D_Schottky_Small") (at 57.15 36.83 270) (unit 1)
     (in_bom yes) (on_board yes) (fields_autoplaced)
@@
     (pin "2")
   )
+  (symbol (lib_id "power:GND") (at 63.5 133.35 0) (unit 1)
+    (in_bom yes) (on_board yes)
+    (property "Reference" "#PWR?" (id 0) (at 63.5 139.7 0)
+      (effects (font (size 1.27 1.27)) hide)
+    )
+    (property "Value" "GND" (id 1) (at 66.675 136.525 0))
+    (property "Footprint" "" (id 2) (at 63.5 133.35 0)
+      (effects (font (size 1.27 1.27)) hide)
+    )
+    (property "Datasheet" "" (id 3) (at 63.5 133.35 0)
+      (effects (font (size 1.27 1.27)) hide)
+    )
+    (pin "1")
+  )
   (symbol (lib_id "power:GND") (at 48.26 39.37 0) (unit 1)
     (in_bom yes) (on_board yes) (fields_autoplaced)
@@
     (pin "1")
   )
+  (symbol (lib_id "Device:R_Small") (at 63.5 121.285 0) (unit 1)
+    (in_bom yes) (on_board yes)
+    (property "Reference" "R?" (id 0) (at 64.77 120.015 0)
+      (effects (font (size 1.27 1.27)) (justify left))
+    )
+    (property "Value" "36k" (id 1) (at 64.77 121.92 0)
+      (effects (font (size 1.27 1.27)) (justify left))
+    )
+    (property "Footprint" "Resistor_SMD:R_0402_1005Metric" (id 2) (at 63.5 121.285 0)
+      (effects (font (size 1.27 1.27)) hide)
+    )
+    (property "Datasheet" "~" (id 3) (at 63.5 121.285 0)
+      (effects (font (size 1.27 1.27)) hide)
+    )
+    (property "MPN" "RC0402FR-0736KL" (id 4) (at 63.5 121.285 0)
+      (effects (font (size 1.27 1.27)) hide)
+    )
+    (property "Description" "RES 36K OHM 5% 1/16W 0402" (id 6) (at 63.5 121.285 0)
+      (effects (font (size 1.27 1.27)) hide)
+    )
+    (pin "1")
+    (pin "2")
+  )
   (symbol (lib_id "Device:R_Small") (at 48.26 29.21 0) (unit 1)
