File: hardware/davecu2/CAN-Bus.kicad_sch (KiCad schematic)
At the start: 4 parts, among them U9 SN65HVD230

Commit message: schematic cleanup
Connections:
- net +3V3 renamed VDD
- net EN renamed CAN_EN
- net GPIO_CAN_N renamed CAN_RX
- net GPIO_CAN_P renamed CAN_TX
Other:
- moved on the sheet: C44, R30, R31, U9
