File: hardware/davecu2/Power.kicad_sch (KiCad schematic)
At the start: 15 parts, among them U8 BD33C0AWFP-CE2

Commit message: schematic cleanup
Parts:
- removed R28: 36k, Resistor_SMD:R_0402_1005Metric, symbol Device:R_Small
- removed R29: 10k, Resistor_SMD:R_0402_1005Metric, symbol Device:R_Small
- removed TP3: VSENSE, TestPoint:TestPoint_Pad_D1.0mm, symbol Connector:TestPoint
Changed lines of the file:
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@@
   (junction (at 106.045 78.74) (diameter 0) (color 0 0 0 0)
   )
-  (junction (at 151.13 81.28) (diameter 0) (color 0 0 0 0)
+  (junction (at 125.73 78.74) (diameter 0) (color 0 0 0 0)
   )
   (junction (at 44.45 77.47) (diameter 0) (color 0 0 0 0)
@@
     (stroke (width 0) (type default) (color 0 0 0 0))
   )
-  (wire (pts (xy 151.13 81.28) (xy 165.735 81.28))
-    (stroke (width 0) (type default) (color 0 0 0 0))
-  )
-  (wire (pts (xy 151.13 71.755) (xy 151.13 73.66))
-    (stroke (width 0) (type default) (color 0 0 0 0))
-  )
   (wire (pts (xy 63.5 54.61) (xy 63.5 77.47))
     (stroke (width 0) (type default) (color 0 0 0 0))
@@
     (stroke (width 0) (type default) (color 0 0 0 0))
   )
-  (wire (pts (xy 165.735 71.755) (xy 151.13 71.755))
-    (stroke (width 0) (type default) (color 0 0 0 0))
-  )
   (wire (pts (xy 127 42.545) (xy 140.97 42.545))
     (stroke (width 0) (type default) (color 0 0 0 0))
@@
     (stroke (width 0) (type default) (color 0 0 0 0))
   )
+  (wire (pts (xy 125.73 78.74) (xy 130.81 78.74))
+    (stroke (width 0) (type default) (color 0 0 0 0))
+  )
   (wire (pts (xy 25.4 82.55) (xy 26.67 82.55))
     (stroke (width 0) (type default) (color 0 0 0 0))
@@
     (stroke (width 0) (type default) (color 0 0 0 0))
   )
-  (wire (pts (xy 151.13 83.185) (xy 151.13 81.28))
-    (stroke (width 0) (type default) (color 0 0 0 0))
-  )
   (wire (pts (xy 93.345 60.96) (xy 96.52 60.96))
     (stroke (width 0) (type default) (color 0 0 0 0))
@@
     (stroke (width 0) (type default) (color 0 0 0 0))
   )
-  (wire (pts (xy 106.045 78.74) (xy 114.3 78.74))
+  (wire (pts (xy 106.045 78.74) (xy 125.73 78.74))
     (stroke (width 0) (type default) (color 0 0 0 0))
   )
@@
   )
   (wire (pts (xy 158.75 42.545) (xy 179.07 42.545))
-    (stroke (width 0) (type default) (color 0 0 0 0))
-  )
-  (wire (pts (xy 151.13 81.28) (xy 151.13 78.74))
     (stroke (width 0) (type default) (color 0 0 0 0))
   )
@@
     (effects (font (size 1.27 1.27)) (justify left bottom))
   )
-  (label "VSENSE" (at 163.195 81.28 180)
-    (effects (font (size 1.27 1.27)) (justify right bottom))
-  )
   (label "IGNITION" (at 46.355 72.39 0)
     (effects (font (size 1.27 1.27)) (justify left bottom))
   )
-  (label "VBATT" (at 165.735 71.755 180)
-    (effects (font (size 1.27 1.27)) (justify right bottom))
-  )
   (label "LED_PWR" (at 127 42.545 0)
     (effects (font (size 1.27 1.27)) (justify left bottom))
@@
     (effects (font (size 1.27 1.27)) (justify right))
   )
-  (hierarchical_label "VSENSE" (shape output) (at 165.735 81.28 0)
-    (effects (font (size 1.27 1.27)) (justify left))
-  )
   (hierarchical_label "USB_VBUS" (shape input) (at 25.4 82.55 180)
     (effects (font (size 1.27 1.27)) (justify right))
   )
+  (hierarchical_label "VDD" (shape output) (at 130.81 78.74 0)
+    (effects (font (size 1.27 1.27)) (justify left))
+  )
   (hierarchical_label "VBATT" (shape input) (at 21.59 77.47 180)
     (effects (font (size 1.27 1.27)) (justify right))
@@
     (pin "1")
   )
-  (symbol (lib_id "power:+3V3") (at 114.3 78.74 0) (unit 1)
-    (in_bom yes) (on_board yes) (fields_autoplaced)
-    (property "Reference" "#PWR062" (id 0) (at 114.3 82.55 0)
-      (effects (font (size 1.27 1.27)) hide)
-    )
-    (property "Value" "+3V3" (id 1) (at 114.3 73.66 0))
-    (property "Footprint" "" (id 2) (at 114.3 78.74 0)
-      (effects (font (size 1.27 1.27)) hide)
-    )
-    (property "Datasheet" "" (id 3) (at 114.3 78.74 0)
+  (symbol (lib_id "power:+3V3") (at 125.73 78.74 0) (unit 1)
+    (in_bom yes) (on_board yes) (fields_autoplaced)
+    (property "Reference" "#PWR062" (id 0) (at 125.73 82.55 0)
+      (effects (font (size 1.27 1.27)) hide)
+    )
+    (property "Value" "+3V3" (id 1) (at 125.73 73.66 0))
+    (property "Footprint" "" (id 2) (at 125.73 78.74 0)
+      (effects (font (size 1.27 1.27)) hide)
+    )
+    (property "Datasheet" "" (id 3) (at 125.73 78.74 0)
       (effects (font (size 1.27 1.27)) hide)
     )
@@
     )
     (pin "1")
-  )
-  (symbol (lib_id "Device:R_Small") (at 151.13 76.2 0) (unit 1)
-    (in_bom yes) (on_board yes)
-    (property "Reference" "R28" (id 0) (at 152.4 74.93 0)
-      (effects (font (size 1.27 1.27)) (justify left))
-    )
-    (property "Value" "36k" (id 1) (at 152.4 76.835 0)
-      (effects (font (size 1.27 1.27)) (justify left))
-    )
-    (property "Footprint" "Resistor_SMD:R_0402_1005Metric" (id 2) (at 151.13 76.2 0)
-      (effects (font (size 1.27 1.27)) hide)
-    )
-    (property "Datasheet" "~" (id 3) (at 151.13 76.2 0)
-      (effects (font (size 1.27 1.27)) hide)
-    )
-    (property "MPN" "RC0402FR-0736KL" (id 4) (at 151.13 76.2 0)
-      (effects (font (size 1.27 1.27)) hide)
-    )
-    (property "Description" "RES 36K OHM 5% 1/16W 0402" (id 6) (at 151.13 76.2 0)
-      (effects (font (size 1.27 1.27)) hide)
-    )
-    (pin "1")
-    (pin "2")
   )
   (symbol (lib_id "Device:C_Small") (at 63.5 80.01 180) (unit 1)
@@
     (pin "2")
   )
-  (symbol (lib_id "Device:R_Small") (at 151.13 85.725 0) (unit 1)
-    (in_bom yes) (on_board yes)
-    (property "Reference" "R29" (id 0) (at 153.035 85.09 0)
-      (effects (font (size 1.27 1.27)) (justify left))
-    )
-    (property "Value" "10k" (id 1) (at 153.035 86.995 0)
-      (effects (font (size 1.27 1.27)) (justify left))
-    )
-    (property "Footprint" "Resistor_SMD:R_0402_1005Metric" (id 2) (at 151.13 85.725 0)
-      (effects (font (size 1.27 1.27)) hide)
-    )
-    (property "Datasheet" "~" (id 3) (at 151.13 85.725 0)
-      (effects (font (size 1.27 1.27)) hide)
-    )
-    (property "MPN" "RMCF0402JT10K0" (id 4) (at 151.13 85.725 0)
-      (effects (font (size 1.27 1.27)) hide)
-    )
-    (property "Description" "RES 10K OHM 5% 1/16W 0402" (id 6) (at 151.13 85.725 0)
-      (effects (font (size 1.27 1.27)) hide)
-    )
-    (pin "1")
-    (pin "2")
-  )
   (symbol (lib_id "Device:D_Schottky_Small") (at 56.515 80.01 270) (unit 1)
     (in_bom yes) (on_board yes) (fields_autoplaced)
@@
     (pin "2")
   )
-  (symbol (lib_id "power:GND") (at 151.13 88.265 0) (unit 1)
-    (in_bom yes) (on_board yes)
-    (property "Reference" "#PWR066" (id 0) (at 151.13 94.615 0)
-      (effects (font (size 1.27 1.27)) hide)
-    )
-    (property "Value" "GND" (id 1) (at 154.305 91.44 0))
-    (property "Footprint" "" (id 2) (at 151.13 88.265 0)
-      (effects (font (size 1.27 1.27)) hide)
-    )
-    (property "Datasheet" "" (id 3) (at 151.13 88.265 0)
-      (effects (font (size 1.27 1.27)) hide)
-    )
-    (pin "1")
-  )
   (symbol (lib_id "power:+3V3") (at 179.07 42.545 0) (unit 1)
     (in_bom yes) (on_board yes) (fields_autoplaced)
@@
       (effects (font (size 1.27 1.27)) hide)
     )
-    (pin "1")
-  )
-  (symbol (lib_id "Connector:TestPoint") (at 151.13 81.28 90) (unit 1)
-    (in_bom yes) (on_board yes)
-    (property "Reference" "TP3" (id 0) (at 140.97 79.375 90))
-    (property "Value" "VSENSE" (id 1) (at 142.875 81.28 90))
-    (property "Footprint" "TestPoint:TestPoint_Pad_D1.0mm" (id 2) (at 151.13 76.2 0)
-      (effects (font (size 1.27 1.27)) hide)
-    )
-    (property "Datasheet" "~" (id 3) (at 151.13 76.2 0)
-      (effects (font (size 1.27 1.27)) hide)
-    )
