File: hardware/davecu2/STM32F723ZET6.kicad_sch (KiCad schematic)
At the start: 36 parts

Commit message: schematic cleanup
Connections:
- net SPI1_NSS renamed SPI1_NSS1
Changed lines of the file:
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@@
     (effects (font (size 1.27 1.27)) (justify left bottom))
   )
-  (label "SPI1_NSS" (at 110.49 90.17 0)
+  (label "SPI1_NSS1" (at 110.49 90.17 0)
     (effects (font (size 1.27 1.27)) (justify left bottom))
   )
@@
     (effects (font (size 1.27 1.27)) (justify left))
   )
+  (hierarchical_label "SPI1_MOSI" (shape output) (at 106.68 107.95 180)
+    (effects (font (size 1.27 1.27)) (justify right))
+  )
   (hierarchical_label "MAF" (shape input) (at 205.74 54.61 0)
     (effects (font (size 1.27 1.27)) (justify left))
@@
     (effects (font (size 1.27 1.27)) (justify left))
   )
+  (hierarchical_label "SPI1_MISO" (shape output) (at 106.68 105.41 180)
+    (effects (font (size 1.27 1.27)) (justify right))
+  )
+  (hierarchical_label "SPI1_NSS2" (shape output) (at 82.55 105.41 180)
+    (effects (font (size 1.27 1.27)) (justify right))
+  )
   (hierarchical_label "DBW_MOTOR_+" (shape output) (at 27.94 54.61 0)
     (effects (font (size 1.27 1.27)) (justify left))
@@
     (effects (font (size 1.27 1.27)) (justify left))
   )
-  (hierarchical_label "SPI1_NSS" (shape output) (at 106.68 90.17 180)
-    (effects (font (size 1.27 1.27)) (justify right))
-  )
+  (hierarchical_label "SPI1_NSS1" (shape output) (at 106.68 90.17 180)
+    (effects (font (size 1.27 1.27)) (justify right))
+  )
